File: AMC_connector.sch (KiCad schematic (older format))
At the start: 2 parts, among them P3 CMP-0001-00058-2

Commit message: FPGA power finished, significant progress on PCB
Parts:
- D1: symbol AMC_FMC_Carrier-PcbDoc-rescue:SS16-Diodes -> AMC_FMC_Carrier-PcbDoc-rescue:SS16-Diodes-AMC_FMC_Carrier-PcbDoc-rescue-AMC_FMC_Carrier-PcbDoc-rescue
- P3: symbol AMC_FMC_Carrier-PcbDoc-rescue:CMP-0001-00058-2-AMC-AMC_FMC_Carrier-PcbDoc-rescue -> AMC_FMC_Carrier-PcbDoc-rescue:CMP-0001-00058-2-AMC-AMC_FMC_Carrier-PcbDoc-rescue-AMC_FMC_Carrier-PcbDoc-rescue-AMC_FMC_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
Changed lines of the file:
@@
 $EndDescr
 $Comp
-L AMC_FMC_Carrier-PcbDoc-rescue:CMP-0001-00058-2-AMC-AMC_FMC_Carrier-PcbDoc-rescue P?
+L AMC_FMC_Carrier-PcbDoc-rescue:CMP-0001-00058-2-AMC-AMC_FMC_Carrier-PcbDoc-rescue-AMC_FMC_Carrier-PcbDoc-rescue-AMC_FMC_Carrier-PcbDoc-rescue P?
 U 1 1 5BD3210B
 P 1550 7900
@@
 Tx_7_P
 $Comp
-L AMC_FMC_Carrier-PcbDoc-rescue:+12V_AMC-powerMG-AMC_FMC_Carrier-PcbDoc-rescue #PWR029
+L AMC_FMC_Carrier-PcbDoc-rescue:+12V_AMC-powerMG-AMC_FMC_Carrier-PcbDoc-rescue-AMC_FMC_Carrier-PcbDoc-rescue-AMC_FMC_Carrier-PcbDoc-rescue #PWR029
 U 1 1 5DEC6F0B
 P 1750 6500
+AR Path="/5DEC6F0B" Ref="#PWR029"  Part="1"
+AR Path="/5BD320D5/5DEC6F0B" Ref="#PWR029"  Part="1"
 F 0 "#PWR029" H 1750 6350 50  0001 C CNN
 F 1 "+12V_AMC" H 1765 6673 50  0000 C CNN
@@
 	1750 6500 1750 7700
 $Comp
-L AMC_FMC_Carrier-PcbDoc-rescue:+12V_AMC-powerMG-AMC_FMC_Carrier-PcbDoc-rescue #PWR031
+L AMC_FMC_Carrier-PcbDoc-rescue:+12V_AMC-powerMG-AMC_FMC_Carrier-PcbDoc-rescue-AMC_FMC_Carrier-PcbDoc-rescue-AMC_FMC_Carrier-PcbDoc-rescue #PWR031
 U 1 1 5DF1FECB
 P 2450 6500
+AR Path="/5DF1FECB" Ref="#PWR031"  Part="1"
+AR Path="/5BD320D5/5DF1FECB" Ref="#PWR031"  Part="1"
 F 0 "#PWR031" H 2450 6350 50  0001 C CNN
 F 1 "+12V_AMC" H 2465 6673 50  0000 C CNN
@@
 $EndComp
 $Comp
-L AMC_FMC_Carrier-PcbDoc-rescue:+12V_AMC-powerMG-AMC_FMC_Carrier-PcbDoc-rescue #PWR032
+L AMC_FMC_Carrier-PcbDoc-rescue:+12V_AMC-powerMG-AMC_FMC_Carrier-PcbDoc-rescue-AMC_FMC_Carrier-PcbDoc-rescue-AMC_FMC_Carrier-PcbDoc-rescue #PWR032
 U 1 1 5DF4CACF
 P 3350 6500
+AR Path="/5DF4CACF" Ref="#PWR032"  Part="1"
+AR Path="/5BD320D5/5DF4CACF" Ref="#PWR032"  Part="1"
 F 0 "#PWR032" H 3350 6350 50  0001 C CNN
 F 1 "+12V_AMC" H 3365 6673 50  0000 C CNN
@@
 $EndComp
 $Comp
-L AMC_FMC_Carrier-PcbDoc-rescue:+12V_AMC-powerMG-AMC_FMC_Carrier-PcbDoc-rescue #PWR033
+L AMC_FMC_Carrier-PcbDoc-rescue:+12V_AMC-powerMG-AMC_FMC_Carrier-PcbDoc-rescue-AMC_FMC_Carrier-PcbDoc-rescue-AMC_FMC_Carrier-PcbDoc-rescue #PWR033
 U 1 1 5DFD25BA
 P 4250 6500
+AR Path="/5DFD25BA" Ref="#PWR033"  Part="1"
+AR Path="/5BD320D5/5DFD25BA" Ref="#PWR033"  Part="1"
 F 0 "#PWR033" H 4250 6350 50  0001 C CNN
 F 1 "+12V_AMC" H 4265 6673 50  0000 C CNN
@@
 $EndComp
 $Comp
-L AMC_FMC_Carrier-PcbDoc-rescue:+12V_AMC-powerMG-AMC_FMC_Carrier-PcbDoc-rescue #PWR034
+L AMC_FMC_Carrier-PcbDoc-rescue:+12V_AMC-powerMG-AMC_FMC_Carrier-PcbDoc-rescue-AMC_FMC_Carrier-PcbDoc-rescue-AMC_FMC_Carrier-PcbDoc-rescue #PWR034
 U 1 1 5DFFEFC3
 P 5750 6500
+AR Path="/5DFFEFC3" Ref="#PWR034"  Part="1"
+AR Path="/5BD320D5/5DFFEFC3" Ref="#PWR034"  Part="1"
 F 0 "#PWR034" H 5750 6350 50  0001 C CNN
 F 1 "+12V_AMC" H 5765 6673 50  0000 C CNN
@@
 $EndComp
 $Comp
-L AMC_FMC_Carrier-PcbDoc-rescue:+12V_AMC-powerMG-AMC_FMC_Carrier-PcbDoc-rescue #PWR035
+L AMC_FMC_Carrier-PcbDoc-rescue:+12V_AMC-powerMG-AMC_FMC_Carrier-PcbDoc-rescue-AMC_FMC_Carrier-PcbDoc-rescue-AMC_FMC_Carrier-PcbDoc-rescue #PWR035
 U 1 1 5E02B9CC
 P 7250 6500
+AR Path="/5E02B9CC" Ref="#PWR035"  Part="1"
+AR Path="/5BD320D5/5E02B9CC" Ref="#PWR035"  Part="1"
 F 0 "#PWR035" H 7250 6350 50  0001 C CNN
 F 1 "+12V_AMC" H 7265 6673 50  0000 C CNN
@@
 $EndComp
 $Comp
-L AMC_FMC_Carrier-PcbDoc-rescue:+12V_AMC-powerMG-AMC_FMC_Carrier-PcbDoc-rescue #PWR036
+L AMC_FMC_Carrier-PcbDoc-rescue:+12V_AMC-powerMG-AMC_FMC_Carrier-PcbDoc-rescue-AMC_FMC_Carrier-PcbDoc-rescue-AMC_FMC_Carrier-PcbDoc-rescue #PWR036
 U 1 1 5E0583D5
 P 8750 6500
+AR Path="/5E0583D5" Ref="#PWR036"  Part="1"
+AR Path="/5BD320D5/5E0583D5" Ref="#PWR036"  Part="1"
 F 0 "#PWR036" H 8750 6350 50  0001 C CNN
 F 1 "+12V_AMC" H 8765 6673 50  0000 C CNN
@@
 $EndComp
 $Comp
-L AMC_FMC_Carrier-PcbDoc-rescue:+12V_AMC-powerMG-AMC_FMC_Carrier-PcbDoc-rescue #PWR037
+L AMC_FMC_Carrier-PcbDoc-rescue:+12V_AMC-powerMG-AMC_FMC_Carrier-PcbDoc-rescue-AMC_FMC_Carrier-PcbDoc-rescue-AMC_FMC_Carrier-PcbDoc-rescue #PWR037
 U 1 1 5E084DDE
 P 9950 6500
+AR Path="/5E084DDE" Ref="#PWR037"  Part="1"
+AR Path="/5BD320D5/5E084DDE" Ref="#PWR037"  Part="1"
 F 0 "#PWR037" H 9950 6350 50  0001 C CNN
 F 1 "+12V_AMC" H 9965 6673 50  0000 C CNN
@@
 	3350 7700 3350 6500
 $Comp
-L AMC_FMC_Carrier-PcbDoc-rescue:SS16-Diodes D1
+L AMC_FMC_Carrier-PcbDoc-rescue:SS16-Diodes-AMC_FMC_Carrier-PcbDoc-rescue-AMC_FMC_Carrier-PcbDoc-rescue D1
 U 1 1 5CAB1052
 P 12000 5400

Commit message: new board outline, rearranging banks connections, SODIMM memory
Parts:
- D1: symbol AMC_FMC_Carrier-PcbDoc-rescue:SS16-Diodes-AMC_FMC_Carrier-PcbDoc-rescue-AMC_FMC_Carrier-PcbDoc-rescue -> AMC_FMC_Carrier-PcbDoc-rescue:SS16-Diodes-AMC_FMC_Carrier-PcbDoc-rescue
- P3: symbol AMC_FMC_Carrier-PcbDoc-rescue:CMP-0001-00058-2-AMC-AMC_FMC_Carrier-PcbDoc-rescue-AMC_FMC_Carrier-PcbDoc-rescue-AMC_FMC_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 -> AMC_FMC_Carrier-PcbDoc-rescue:CMP-0001-00058-2-AMC-AMC_FMC_Carrier-PcbDoc-rescue-AMC_FMC_Carrier-PcbDoc-rescue
Changed lines of the file:
@@
 EESchema Schematic File Version 4
-LIBS:AMC_FMC_Carrier-PcbDoc-cache
 EELAYER 30 0
 EELAYER END
 $Descr A3 16535 11693
 encoding utf-8
-Sheet 4 25
+Sheet 4 26
 Title "Marble"
 Date "2019-01-16"
@@
 $EndDescr
 $Comp
-L AMC_FMC_Carrier-PcbDoc-rescue:CMP-0001-00058-2-AMC-AMC_FMC_Carrier-PcbDoc-rescue-AMC_FMC_Carrier-PcbDoc-rescue-AMC_FMC_Carrier-PcbDoc-rescue P?
+L AMC_FMC_Carrier-PcbDoc-rescue:CMP-0001-00058-2-AMC-AMC_FMC_Carrier-PcbDoc-rescue-AMC_FMC_Carrier-PcbDoc-rescue P?
 U 1 1 5BD3210B
 P 1550 7900
@@
 Tx_7_P
 $Comp
-L AMC_FMC_Carrier-PcbDoc-rescue:+12V_AMC-powerMG-AMC_FMC_Carrier-PcbDoc-rescue-AMC_FMC_Carrier-PcbDoc-rescue-AMC_FMC_Carrier-PcbDoc-rescue #PWR029
+L AMC_FMC_Carrier-PcbDoc-rescue:+12V_AMC-powerMG-AMC_FMC_Carrier-PcbDoc-rescue-AMC_FMC_Carrier-PcbDoc-rescue #PWR029
 U 1 1 5DEC6F0B
 P 1750 6500
@@
 	1750 6500 1750 7700
 $Comp
-L AMC_FMC_Carrier-PcbDoc-rescue:+12V_AMC-powerMG-AMC_FMC_Carrier-PcbDoc-rescue-AMC_FMC_Carrier-PcbDoc-rescue-AMC_FMC_Carrier-PcbDoc-rescue #PWR031
+L AMC_FMC_Carrier-PcbDoc-rescue:+12V_AMC-powerMG-AMC_FMC_Carrier-PcbDoc-rescue-AMC_FMC_Carrier-PcbDoc-rescue #PWR031
 U 1 1 5DF1FECB
 P 2450 6500
@@
 $EndComp
 $Comp
-L AMC_FMC_Carrier-PcbDoc-rescue:+12V_AMC-powerMG-AMC_FMC_Carrier-PcbDoc-rescue-AMC_FMC_Carrier-PcbDoc-rescue-AMC_FMC_Carrier-PcbDoc-rescue #PWR032
+L AMC_FMC_Carrier-PcbDoc-rescue:+12V_AMC-powerMG-AMC_FMC_Carrier-PcbDoc-rescue-AMC_FMC_Carrier-PcbDoc-rescue #PWR032
 U 1 1 5DF4CACF
 P 3350 6500
@@
 $EndComp
 $Comp
-L AMC_FMC_Carrier-PcbDoc-rescue:+12V_AMC-powerMG-AMC_FMC_Carrier-PcbDoc-rescue-AMC_FMC_Carrier-PcbDoc-rescue-AMC_FMC_Carrier-PcbDoc-rescue #PWR033
+L AMC_FMC_Carrier-PcbDoc-rescue:+12V_AMC-powerMG-AMC_FMC_Carrier-PcbDoc-rescue-AMC_FMC_Carrier-PcbDoc-rescue #PWR033
 U 1 1 5DFD25BA
 P 4250 6500
@@
 $EndComp
 $Comp
-L AMC_FMC_Carrier-PcbDoc-rescue:+12V_AMC-powerMG-AMC_FMC_Carrier-PcbDoc-rescue-AMC_FMC_Carrier-PcbDoc-rescue-AMC_FMC_Carrier-PcbDoc-rescue #PWR034
+L AMC_FMC_Carrier-PcbDoc-rescue:+12V_AMC-powerMG-AMC_FMC_Carrier-PcbDoc-rescue-AMC_FMC_Carrier-PcbDoc-rescue #PWR034
 U 1 1 5DFFEFC3
 P 5750 6500
@@
 $EndComp
 $Comp
-L AMC_FMC_Carrier-PcbDoc-rescue:+12V_AMC-powerMG-AMC_FMC_Carrier-PcbDoc-rescue-AMC_FMC_Carrier-PcbDoc-rescue-AMC_FMC_Carrier-PcbDoc-rescue #PWR035
+L AMC_FMC_Carrier-PcbDoc-rescue:+12V_AMC-powerMG-AMC_FMC_Carrier-PcbDoc-rescue-AMC_FMC_Carrier-PcbDoc-rescue #PWR035
 U 1 1 5E02B9CC
 P 7250 6500
@@
 $EndComp
 $Comp
-L AMC_FMC_Carrier-PcbDoc-rescue:+12V_AMC-powerMG-AMC_FMC_Carrier-PcbDoc-rescue-AMC_FMC_Carrier-PcbDoc-rescue-AMC_FMC_Carrier-PcbDoc-rescue #PWR036
+L AMC_FMC_Carrier-PcbDoc-rescue:+12V_AMC-powerMG-AMC_FMC_Carrier-PcbDoc-rescue-AMC_FMC_Carrier-PcbDoc-rescue #PWR036
 U 1 1 5E0583D5
 P 8750 6500
@@
 $EndComp
 $Comp
-L AMC_FMC_Carrier-PcbDoc-rescue:+12V_AMC-powerMG-AMC_FMC_Carrier-PcbDoc-rescue-AMC_FMC_Carrier-PcbDoc-rescue-AMC_FMC_Carrier-PcbDoc-rescue #PWR037
+L AMC_FMC_Carrier-PcbDoc-rescue:+12V_AMC-powerMG-AMC_FMC_Carrier-PcbDoc-rescue-AMC_FMC_Carrier-PcbDoc-rescue #PWR037
 U 1 1 5E084DDE
 P 9950 6500
@@
 	3350 7700 3350 6500
 $Comp
-L AMC_FMC_Carrier-PcbDoc-rescue:SS16-Diodes-AMC_FMC_Carrier-PcbDoc-rescue-AMC_FMC_Carrier-PcbDoc-rescue D1
+L AMC_FMC_Carrier-PcbDoc-rescue:SS16-Diodes-AMC_FMC_Carrier-PcbDoc-rescue D1
 U 1 1 5CAB1052
 P 12000 5400
