File: FMC_2.sch (KiCad schematic (older format))
At the start: 16 parts, among them P2 SAMTEC_ASP-134486-01, U55 MIC2090-1YM5TR

Commit message: testpoints added, LEDs on the right site and other minor changes
Parts:
- C5: value CC0402_100NF_16V_10%_X5R -> CC0402_100NF_25V_10%_X7R_YUDEN_TMK105B7104KVHF; footprint CAPC1005X55N -> Capacitors SMD:CAPC1005X55N; symbol Capacitors_SMD:CC0402_100NF_16V_10%_X5R -> Capacitors_SMD:CC0402_100NF_25V_10%_X7R_YUDEN_TMK105B7104KVHF; Comment =Value -> 100nF; ComponentHeight ~~ -> 0.55mm; CreateDate 12/10/13 00:00:00 -> 05/10/17 00:00:00; Database Table Name (none) -> Capacitors SMD; Footprint Library (none) -> Capacitors SMD; LatestRevisionDate 12/10/13 00:00:00 -> 05/10/17 00:00:00; Library Name Capacitors SMD -> Capacitors.DbLib; Manufacturer GENERIC -> TAIYO YUDEN; Manufacturer Part Number CC0402_100NF_16V_10%_X5R -> TMK105B7104KVHF; Manufacturer1 ComponentHeight 0.55mm -> (none); Manufacturer1 Example MURATA -> (none); Manufacturer1 Part Number GRM155R61C104KA88D -> (none); PackageDescription ~~ -> (none); Part Description SMD Multilayer Chip Ceramic Capacitor -> SMD Multilayer Chip Ceramic Capacitor (High Dielectric Type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; Part Number CC0402_100NF_16V_10%_X5R -> CC0402_100NF_25V_10%_X7R_YUDEN_TMK105B7104KVHF; Pin Count 2.0000000000000000e+00 -> 2; PressFit ~~ -> (none); Sense Comment ~~ -> (none); Status None -> Not Recommended; Status Comment ~~ -> (none); TC X5R -> X7R; Voltage 16V -> 25V
Changed lines of the file:
@@
 	1750 4650 2250 4650
 $Comp
-L Capacitors_SMD:CC0402_100NF_16V_10%_X5R C?
+L Capacitors_SMD:CC0402_100NF_25V_10%_X7R_YUDEN_TMK105B7104KVHF C?
 U 1 1 5C8FFE06
 P 1750 4650
@@
 AR Path="/5BD31F9F/5C8FFE06" Ref="C5"  Part="1"
 F 0 "C5" V 1800 4650 50  0000 L CNN
-F 1 "CC0402_100NF_16V_10%_X5R" H 1750 4390 60  0001 L CNN
-F 2 "CAPC1005X55N" H 1750 3580 60  0001 L CNN
+F 1 "CC0402_100NF_25V_10%_X7R_YUDEN_TMK105B7104KVHF" H 1750 4390 60  0001 L CNN
+F 2 "Capacitors SMD:CAPC1005X55N" H 1750 3580 60  0001 L CNN
 F 3 "\\\\cern.ch\\dfs\\Applications\\Altium\\Datasheets\\CC0402_X5R_MURATA_GRM.pdf" H 1750 4210 60  0001 L CNN
 F 4 "100nF" V 2000 4650 50  0000 L CNN "~"
-F 5 "CC0402_100NF_16V_10%_X5R" H 1750 4120 60  0001 L CNN "Part Number"
+F 5 "CC0402_100NF_25V_10%_X7R_YUDEN_TMK105B7104KVHF" H 1750 4120 60  0001 L CNN "Part Number"
 F 6 "Capacitor - non polarized" H 1750 4030 60  0001 L CNN "Library Ref"
 F 7 "SchLib\\Capacitors.SchLib" H 1750 3940 60  0001 L CNN "Library Path"
-F 8 "=Value" H 1750 3850 60  0001 L CNN "Comment"
+F 8 "100nF" H 1750 3850 60  0001 L CNN "Comment"
 F 9 "Standard" H 1750 3760 60  0001 L CNN "Component Kind"
 F 10 "Standard" H 1750 3670 60  0001 L CNN "Component Type"
-F 11 "2.0000000000000000e+00" H 1750 3490 60  0001 L CNN "Pin Count"
+F 11 "2" H 1750 3490 60  0001 L CNN "Pin Count"
 F 12 "PcbLib\\Capacitors SMD.PcbLib" H 1750 3400 60  0001 L CNN "Footprint Path"
 F 13 "CAPC1005X55N" H 1750 3310 60  0001 L CNN "Footprint Ref"
-F 14 "~~" H 1750 3220 60  0001 L CNN "PackageDescription"
+F 14 " " H 1750 3220 60  0001 L CNN "PackageDescription"
 F 15 "100nF" H 1750 3130 60  0001 L CNN "Val"
-F 16 "None" H 1750 3040 60  0001 L CNN "Status"
-F 17 "~~" H 1750 2950 60  0001 L CNN "Status Comment"
-F 18 "16V" H 1750 2860 60  0001 L CNN "Voltage"
-F 19 "X5R" H 1750 2770 60  0001 L CNN "TC"
+F 16 "Not Recommended" H 1750 3040 60  0001 L CNN "Status"
+F 17 " " H 1750 2950 60  0001 L CNN "Status Comment"
+F 18 "25V" H 1750 2860 60  0001 L CNN "Voltage"
+F 19 "X7R" H 1750 2770 60  0001 L CNN "TC"
 F 20 "±10%" H 1750 2680 60  0001 L CNN "Tolerance"
-F 21 "SMD Multilayer Chip Ceramic Capacitor" H 1750 2590 60  0001 L CNN "Part Description"
-F 22 "GENERIC" H 1750 2500 60  0001 L CNN "Manufacturer"
-F 23 "CC0402_100NF_16V_10%_X5R" H 1750 2410 60  0001 L CNN "Manufacturer Part Number"
+F 21 "SMD Multilayer Chip Ceramic Capacitor (High Dielectric Type) for Automotive / Industrial Applications" H 1750 2590 60  0001 L CNN "Part Description"
+F 22 "TAIYO YUDEN" H 1750 2500 60  0001 L CNN "Manufacturer"
+F 23 "TMK105B7104KVHF" H 1750 2410 60  0001 L CNN "Manufacturer Part Number"
 F 24 "0402" H 1750 2320 60  0001 L CNN "Case"
 F 25 "Yes" H 1750 2230 60  0001 L CNN "Mounted"
 F 26 "No" H 1750 2140 60  0001 L CNN "Socket"
 F 27 "Yes" H 1750 2050 60  0001 L CNN "SMD"
-F 28 "~~" H 1750 1960 60  0001 L CNN "PressFit"
+F 28 " " H 1750 1960 60  0001 L CNN "PressFit"
 F 29 "No" H 1750 1870 60  0001 L CNN "Sense"
-F 30 "~~" H 1750 1780 60  0001 L CNN "Sense Comment"
-F 31 "~~" H 1750 1690 60  0001 L CNN "ComponentHeight"
-F 32 "MURATA" H 1750 1600 60  0001 L CNN "Manufacturer1 Example"
-F 33 "GRM155R61C104KA88D" H 1750 1510 60  0001 L CNN "Manufacturer1 Part Number"
-F 34 "0.55mm" H 1750 1420 60  0001 L CNN "Manufacturer1 ComponentHeight"
+F 30 " " H 1750 1780 60  0001 L CNN "Sense Comment"
+F 31 "0.55mm" H 1750 1690 60  0001 L CNN "ComponentHeight"
+F 32 " " H 1750 1600 60  0001 L CNN "Manufacturer1 Example"
+F 33 " " H 1750 1510 60  0001 L CNN "Manufacturer1 Part Number"
+F 34 " " H 1750 1420 60  0001 L CNN "Manufacturer1 ComponentHeight"
 F 35 "\\\\cern.ch\\dfs\\Applications\\Altium\\Datasheets\\CC0402_X5R_MURATA_GRM.pdf" H 1750 1330 60  0001 L CNN "HelpURL"
 F 36 "CERN DEM JLC" H 1750 1240 60  0001 L CNN "Author"
-F 37 "12/10/13 00:00:00" H 1750 1150 60  0001 L CNN "CreateDate"
-F 38 "12/10/13 00:00:00" H 1750 1060 60  0001 L CNN "LatestRevisionDate"
-F 39 "Capacitors SMD" H 1750 970 60  0001 L CNN "Library Name"
+F 37 "05/10/17 00:00:00" H 1750 1150 60  0001 L CNN "CreateDate"
+F 38 "05/10/17 00:00:00" H 1750 1060 60  0001 L CNN "LatestRevisionDate"
+F 39 "Capacitors.DbLib" H 1750 970 60  0001 L CNN "Library Name"
 F 40 "This work is licensed under the Creative Commons CC-BY-SA 4.0 License. To the extent that circuit schematics that use Licensed Material can be considered to be ‘Adapted Material’, then the copyright holder waives article 3.b of the license with respect to these schematics." H 1750 880 60  0001 L CNN "License"
+F 41 "Capacitors SMD" H 1750 4650 50  0001 C CNN "Database Table Name"
+F 42 "Capacitors SMD" H 1750 4650 50  0001 C CNN "Footprint Library"
 	1    1750 4650
 	0    1    1    0
