File: WhiteRabbit.sch (KiCad schematic (older format))
At the start: 57 parts, among them U13 LP5951MF-3.0/NOPB, U14 LM336M-2.5, U16 AD5662BRMZ-1, U19 AD5662BRMZ-1, U20 CDCM61004RHBT, Y1 OSC_25MHZ_RAKON_IVT3205CR, Y2 VM53S3-25.000-2.5/-30+75, Y3 OSC_20MHZ_IQD_LFVCXO026156, Y6 OSC_10-280MHZ_SILICON-LAB_Si5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

Commit message: PN updated for some components, README_fab.txt updated
Parts:
- Y1: Manufacturer Part Number IVT3205CR 25.0 MHz -> IVT3205CR 25.0 MHz or TXEAADSANF-25.000000; Part Number OSC_25MHZ_RAKON_IVT3205CR -> OSC_25MHZ_RAKON_IVT3205CR or TXEAADSANF-25.000000
- Y3: Manufacturer Part Number LFVCXO026156 -> LFVCXO026156 or KV7050B20.0000C3GD00; Part Number OSC_20MHZ_IQD_LFVCXO026156 -> OSC_20MHZ_IQD_LFVCXO026156 or KV7050B20.0000C3GD00
Changed lines of the file:
@@
 F 3 "" H 7850 3780 60  0001 L CNN
 F 4 "20MHz" H 8250 4624 50  0000 C CNN "~"
-F 5 "OSC_20MHZ_IQD_LFVCXO026156" H 7850 3690 60  0001 L CNN "Part Number"
+F 5 "OSC_20MHZ_IQD_LFVCXO026156 or KV7050B20.0000C3GD00" H 7850 3690 60  0001 L CNN "Part Number"
 F 6 "Oscillator IQD_CFPV-45" H 7850 3600 60  0001 L CNN "Library Ref"
 F 7 "SchLib\\Crystals & Oscillators.SchLib" H 7850 3510 60  0001 L CNN "Library Path"
@@
 F 15 "3.3V, ±100ppm, 15pF, 0..70°C, HCMOS Tri-State Surface Mount, VCXO Voltage Controlled Oscillator (CFPV-45 Series)" H 7850 2700 60  0001 L CNN "Part Description"
 F 16 "IQD FREQUENCY PRODUCTS" H 7850 2610 60  0001 L CNN "Manufacturer"
-F 17 "LFVCXO026156" H 7850 2520 60  0001 L CNN "Manufacturer Part Number"
+F 17 "LFVCXO026156 or KV7050B20.0000C3GD00" H 7850 2520 60  0001 L CNN "Manufacturer Part Number"
 F 18 "6" H 7850 2430 60  0001 L CNN "Pin Count"
 F 19 "~~" H 7850 2340 60  0001 L CNN "Case"
@@
 F 3 "" H 4050 380 60  0001 L CNN
 F 4 "25MHz" H 4350 1224 50  0000 C CNN "~"
-F 5 "OSC_25MHZ_RAKON_IVT3205CR" H 4050 290 60  0001 L CNN "Part Number"
+F 5 "OSC_25MHZ_RAKON_IVT3205CR or TXEAADSANF-25.000000" H 4050 290 60  0001 L CNN "Part Number"
 F 6 "Oscillator 1VCO 3GND 4OUT 6VCC" H 4050 200 60  0001 L CNN "Library Ref"
 F 7 "SchLib\\Crystals & Oscillators.SchLib" H 4050 110 60  0001 L CNN "Library Path"
@@
 F 15 "11pF 3.3V ±1ppm Surface Mount TCXO Voltage Controlled Oscillator (IT3200C Series)" H 4050 -700 60  0001 L CNN "Part Description"
 F 16 "RAKON" H 4050 -790 60  0001 L CNN "Manufacturer"
-F 17 "IVT3205CR 25.0 MHz" H 4050 -880 60  0001 L CNN "Manufacturer Part Number"
+F 17 "IVT3205CR 25.0 MHz or TXEAADSANF-25.000000" H 4050 -880 60  0001 L CNN "Manufacturer Part Number"
 F 18 "4" H 4050 -970 60  0001 L CNN "Pin Count"
 F 19 "~~" H 4050 -1060 60  0001 L CNN "Case"

Commit message: new PN for LEDs
Parts:
- U13: symbol AMC_FMC_Carrier-PcbDoc-rescue:LP5951-clocks-SchDoc-cache-AMC_FMC_Carrier-PcbDoc-rescue-AMC_FMC_Carrier-PcbDoc-rescue -> AMC_FMC_Carrier-PcbDoc-rescue:LP5951-clocks-SchDoc-cache-AMC_FMC_Carrier-PcbDoc-rescue-AMC_FMC_Carrier-PcbDoc-rescue-AM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
- U14: symbol AMC_FMC_Carrier-PcbDoc-rescue:LM336M-2.5-clocks-SchDoc-cache-AMC_FMC_Carrier-PcbDoc-rescue-AMC_FMC_Carrier-PcbDoc-rescue -> AMC_FMC_Carrier-PcbDoc-rescue:LM336M-2.5-clocks-SchDoc-cache-AMC_FMC_Carrier-PcbDoc-rescue-AMC_FMC_Carrier-PcbDoc-rescu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
- Y2: symbol AMC_FMC_Carrier-PcbDoc-rescue:Oscillator_1VC_2GND_3OUT_4+Vs-clocks-SchDoc-cache-AMC_FMC_Carrier-PcbDoc-rescue-AMC_FMC_Carrier-PcbDoc-rescue -> AMC_FMC_Carrier-PcbDoc-rescue:Oscillator_1VC_2GND_3OUT_4+Vs-clocks-SchDoc-cache-AMC_FMC_Carrier-PcbDoc-rescue-AMC_FMC_Carrier-PcbDoc-rescue-AMC_FMC_Carrier-PcbDoc-rescue
Changed lines of the file:
@@
 	3750 4450 3750 5450
 $Comp
-L AMC_FMC_Carrier-PcbDoc-rescue:LM336M-2.5-clocks-SchDoc-cache-AMC_FMC_Carrier-PcbDoc-rescue-AMC_FMC_Carrier-PcbDoc-rescue U14
+L AMC_FMC_Carrier-PcbDoc-rescue:LM336M-2.5-clocks-SchDoc-cache-AMC_FMC_Carrier-PcbDoc-rescue-AMC_FMC_Carrier-PcbDoc-rescue-AMC_FMC_Carrier-PcbDoc-rescue U14
 U 1 1 5C21F363
 P 2200 6900
@@
 	8850 4850 8850 4950
 $Comp
-L AMC_FMC_Carrier-PcbDoc-rescue:+3V3_CLEAN-powerMG-AMC_FMC_Carrier-PcbDoc-rescue-AMC_FMC_Carrier-PcbDoc-rescue #PWR0175
+L AMC_FMC_Carrier-PcbDoc-rescue:+3V3_CLEAN-powerMG-AMC_FMC_Carrier-PcbDoc-rescue-AMC_FMC_Carrier-PcbDoc-rescue-AMC_FMC_Carrier-PcbDoc-rescue #PWR0175
 U 1 1 5C2DA97A
 P 2300 6100
@@
 $EndComp
 $Comp
-L AMC_FMC_Carrier-PcbDoc-rescue:+3V3_CLEAN-powerMG-AMC_FMC_Carrier-PcbDoc-rescue-AMC_FMC_Carrier-PcbDoc-rescue #PWR0174
+L AMC_FMC_Carrier-PcbDoc-rescue:+3V3_CLEAN-powerMG-AMC_FMC_Carrier-PcbDoc-rescue-AMC_FMC_Carrier-PcbDoc-rescue-AMC_FMC_Carrier-PcbDoc-rescue #PWR0174
 U 1 1 5C2DA9DF
 P 2250 5650
@@
 $EndComp
 $Comp
-L AMC_FMC_Carrier-PcbDoc-rescue:+3V3_CLEAN-powerMG-AMC_FMC_Carrier-PcbDoc-rescue-AMC_FMC_Carrier-PcbDoc-rescue #PWR0209
+L AMC_FMC_Carrier-PcbDoc-rescue:+3V3_CLEAN-powerMG-AMC_FMC_Carrier-PcbDoc-rescue-AMC_FMC_Carrier-PcbDoc-rescue-AMC_FMC_Carrier-PcbDoc-rescue #PWR0209
 U 1 1 5C2DD28D
 P 7450 4850
@@
 $EndComp
 $Comp
-L AMC_FMC_Carrier-PcbDoc-rescue:+3V3_CLEAN-powerMG-AMC_FMC_Carrier-PcbDoc-rescue-AMC_FMC_Carrier-PcbDoc-rescue #PWR0173
+L AMC_FMC_Carrier-PcbDoc-rescue:+3V3_CLEAN-powerMG-AMC_FMC_Carrier-PcbDoc-rescue-AMC_FMC_Carrier-PcbDoc-rescue-AMC_FMC_Carrier-PcbDoc-rescue #PWR0173
 U 1 1 5C2DDAC4
 P 2250 4650
@@
 CLK20_VCXO
 $Comp
-L AMC_FMC_Carrier-PcbDoc-rescue:LP5951-clocks-SchDoc-cache-AMC_FMC_Carrier-PcbDoc-rescue-AMC_FMC_Carrier-PcbDoc-rescue U13
+L AMC_FMC_Carrier-PcbDoc-rescue:LP5951-clocks-SchDoc-cache-AMC_FMC_Carrier-PcbDoc-rescue-AMC_FMC_Carrier-PcbDoc-rescue-AMC_FMC_Carrier-PcbDoc-rescue U13
 U 1 1 5C2E75E7
 P 1700 2500
@@
 $EndComp
 $Comp
-L AMC_FMC_Carrier-PcbDoc-rescue:+3V3_CLEAN-powerMG-AMC_FMC_Carrier-PcbDoc-rescue-AMC_FMC_Carrier-PcbDoc-rescue #PWR0169
+L AMC_FMC_Carrier-PcbDoc-rescue:+3V3_CLEAN-powerMG-AMC_FMC_Carrier-PcbDoc-rescue-AMC_FMC_Carrier-PcbDoc-rescue-AMC_FMC_Carrier-PcbDoc-rescue #PWR0169
 U 1 1 5C2EF25E
 P 700 2500
@@
 $EndComp
 $Comp
-L AMC_FMC_Carrier-PcbDoc-rescue:Oscillator_1VC_2GND_3OUT_4+Vs-clocks-SchDoc-cache-AMC_FMC_Carrier-PcbDoc-rescue-AMC_FMC_Carrier-PcbDoc-rescue Y2
+L AMC_FMC_Carrier-PcbDoc-rescue:Oscillator_1VC_2GND_3OUT_4+Vs-clocks-SchDoc-cache-AMC_FMC_Carrier-PcbDoc-rescue-AMC_FMC_Carrier-PcbDoc-rescue-AMC_FMC_Carrier-PcbDoc-rescue Y2
 U 1 1 5C2F3070
 P 4050 1950
@@
 $EndComp
 $Comp
-L AMC_FMC_Carrier-PcbDoc-rescue:+3V3_CLEAN-powerMG-AMC_FMC_Carrier-PcbDoc-rescue-AMC_FMC_Carrier-PcbDoc-rescue #PWR0206
+L AMC_FMC_Carrier-PcbDoc-rescue:+3V3_CLEAN-powerMG-AMC_FMC_Carrier-PcbDoc-rescue-AMC_FMC_Carrier-PcbDoc-rescue-AMC_FMC_Carrier-PcbDoc-rescue #PWR0206
 U 1 1 5C33B37A
 P 6550 6900
@@
 	6300 6250 6300 6300
 $Comp
-L AMC_FMC_Carrier-PcbDoc-rescue:+3V3_CLEAN-powerMG-AMC_FMC_Carrier-PcbDoc-rescue-AMC_FMC_Carrier-PcbDoc-rescue #PWR0189
+L AMC_FMC_Carrier-PcbDoc-rescue:+3V3_CLEAN-powerMG-AMC_FMC_Carrier-PcbDoc-rescue-AMC_FMC_Carrier-PcbDoc-rescue-AMC_FMC_Carrier-PcbDoc-rescue #PWR0189
 U 1 1 5C3A12D5
 P 5300 5900
@@
 	5300 5900 5300 5950
 $Comp
-L AMC_FMC_Carrier-PcbDoc-rescue:+3V3_CLEAN-powerMG-AMC_FMC_Carrier-PcbDoc-rescue-AMC_FMC_Carrier-PcbDoc-rescue #PWR0211
+L AMC_FMC_Carrier-PcbDoc-rescue:+3V3_CLEAN-powerMG-AMC_FMC_Carrier-PcbDoc-rescue-AMC_FMC_Carrier-PcbDoc-rescue-AMC_FMC_Carrier-PcbDoc-rescue #PWR0211
 U 1 1 5C8A0C88
 P 6500 1450
@@
 	10150 3050 10150 3100
 $Comp
-L AMC_FMC_Carrier-PcbDoc-rescue:+3V3_CLEAN-powerMG-AMC_FMC_Carrier-PcbDoc-rescue-AMC_FMC_Carrier-PcbDoc-rescue #PWR0399
+L AMC_FMC_Carrier-PcbDoc-rescue:+3V3_CLEAN-powerMG-AMC_FMC_Carrier-PcbDoc-rescue-AMC_FMC_Carrier-PcbDoc-rescue-AMC_FMC_Carrier-PcbDoc-rescue #PWR0399
 U 1 1 5D15AFE0
 P 10450 3400
@@
 NoConn ~ 2500 2800
 $Comp
-L AMC_FMC_Carrier-PcbDoc-rescue:+3V3_CLEAN-powerMG-AMC_FMC_Carrier-PcbDoc-rescue-AMC_FMC_Carrier-PcbDoc-rescue #PWR0401
+L AMC_FMC_Carrier-PcbDoc-rescue:+3V3_CLEAN-powerMG-AMC_FMC_Carrier-PcbDoc-rescue-AMC_FMC_Carrier-PcbDoc-rescue-AMC_FMC_Carrier-PcbDoc-rescue #PWR0401
 U 1 1 5D19EDBE
 P 10850 2700

Commit message: fixed bugs
Parts:
- U13: symbol AMC_FMC_Carrier-PcbDoc-rescue:LP5951-clocks-SchDoc-cache-AMC_FMC_Carrier-PcbDoc-rescue-AMC_FMC_Carrier-PcbDoc-rescue-AMC_FMC_Carrier-PcbDoc-rescue -> AMC_FMC_Carrier-PcbDoc-rescue:LP5951-clocks-SchDoc-cache-AMC_FMC_Carrier-PcbDoc-rescue-AMC_FMC_Carrier-PcbDoc-rescue-AMC_FMC_Carrier-PcbDoc-rescue-AMC_FMC_Carrier-PcbDoc-rescue
- U14: symbol AMC_FMC_Carrier-PcbDoc-rescue:LM336M-2.5-clocks-SchDoc-cache-AMC_FMC_Carrier-PcbDoc-rescue-AMC_FMC_Carrier-PcbDoc-rescue-AMC_FMC_Carrier-PcbDoc-rescue -> AMC_FMC_Carrier-PcbDoc-rescue:LM336M-2.5-clocks-SchDoc-cache-AMC_FMC_Carrier-PcbDoc-rescue-AMC_FMC_Carrier-PcbDoc-rescue-AMC_FMC_Carrier-PcbDoc-rescue-AMC_FMC_Carrier-PcbDoc-rescue
- Y2: symbol AMC_FMC_Carrier-PcbDoc-rescue:Oscillator_1VC_2GND_3OUT_4+Vs-clocks-SchDoc-cache-AMC_FMC_Carrier-PcbDoc-rescue-AMC_FMC_Carrier-PcbDoc-rescue-AMC_FMC_Carrier-PcbDoc-rescue -> AMC_FMC_Carrier-PcbDoc-rescue:Oscillator_1VC_2GND_3OUT_4+Vs-clocks-SchDoc-cache-AMC_FMC_Carrier-PcbDoc-rescue-AMC_FMC_Carrier-PcbDoc-rescue-AMC_FMC_Carrier-PcbDoc-rescue-AMC_FMC_Carrier-PcbDoc-rescue
Changed lines of the file:
@@
 	3750 4450 3750 5450
 $Comp
-L AMC_FMC_Carrier-PcbDoc-rescue:LM336M-2.5-clocks-SchDoc-cache-AMC_FMC_Carrier-PcbDoc-rescue-AMC_FMC_Carrier-PcbDoc-rescue-AMC_FMC_Carrier-PcbDoc-rescue U14
+L AMC_FMC_Carrier-PcbDoc-rescue:LM336M-2.5-clocks-SchDoc-cache-AMC_FMC_Carrier-PcbDoc-rescue-AMC_FMC_Carrier-PcbDoc-rescue-AMC_FMC_Carrier-PcbDoc-rescue-AMC_FMC_Carrier-PcbDoc-rescue U14
 U 1 1 5C21F363
 P 2200 6900
@@
 	8850 4850 8850 4950
 $Comp
-L AMC_FMC_Carrier-PcbDoc-rescue:+3V3_CLEAN-powerMG-AMC_FMC_Carrier-PcbDoc-rescue-AMC_FMC_Carrier-PcbDoc-rescue-AMC_FMC_Carrier-PcbDoc-rescue #PWR0175
+L AMC_FMC_Carrier-PcbDoc-rescue:+3V3_CLEAN-powerMG-AMC_FMC_Carrier-PcbDoc-rescue-AMC_FMC_Carrier-PcbDoc-rescue-AMC_FMC_Carrier-PcbDoc-rescue-AMC_FMC_Carrier-PcbDoc-rescue #PWR0175
 U 1 1 5C2DA97A
 P 2300 6100
@@
 $EndComp
 $Comp
-L AMC_FMC_Carrier-PcbDoc-rescue:+3V3_CLEAN-powerMG-AMC_FMC_Carrier-PcbDoc-rescue-AMC_FMC_Carrier-PcbDoc-rescue-AMC_FMC_Carrier-PcbDoc-rescue #PWR0174
+L AMC_FMC_Carrier-PcbDoc-rescue:+3V3_CLEAN-powerMG-AMC_FMC_Carrier-PcbDoc-rescue-AMC_FMC_Carrier-PcbDoc-rescue-AMC_FMC_Carrier-PcbDoc-rescue-AMC_FMC_Carrier-PcbDoc-rescue #PWR0174
 U 1 1 5C2DA9DF
 P 2250 5650
@@
 $EndComp
 $Comp
-L AMC_FMC_Carrier-PcbDoc-rescue:+3V3_CLEAN-powerMG-AMC_FMC_Carrier-PcbDoc-rescue-AMC_FMC_Carrier-PcbDoc-rescue-AMC_FMC_Carrier-PcbDoc-rescue #PWR0209
+L AMC_FMC_Carrier-PcbDoc-rescue:+3V3_CLEAN-powerMG-AMC_FMC_Carrier-PcbDoc-rescue-AMC_FMC_Carrier-PcbDoc-rescue-AMC_FMC_Carrier-PcbDoc-rescue-AMC_FMC_Carrier-PcbDoc-rescue #PWR0209
 U 1 1 5C2DD28D
 P 7450 4850
@@
 $EndComp
 $Comp
-L AMC_FMC_Carrier-PcbDoc-rescue:+3V3_CLEAN-powerMG-AMC_FMC_Carrier-PcbDoc-rescue-AMC_FMC_Carrier-PcbDoc-rescue-AMC_FMC_Carrier-PcbDoc-rescue #PWR0173
+L AMC_FMC_Carrier-PcbDoc-rescue:+3V3_CLEAN-powerMG-AMC_FMC_Carrier-PcbDoc-rescue-AMC_FMC_Carrier-PcbDoc-rescue-AMC_FMC_Carrier-PcbDoc-rescue-AMC_FMC_Carrier-PcbDoc-rescue #PWR0173
 U 1 1 5C2DDAC4
 P 2250 4650
@@
 CLK20_VCXO
 $Comp
-L AMC_FMC_Carrier-PcbDoc-rescue:LP5951-clocks-SchDoc-cache-AMC_FMC_Carrier-PcbDoc-rescue-AMC_FMC_Carrier-PcbDoc-rescue-AMC_FMC_Carrier-PcbDoc-rescue U13
+L AMC_FMC_Carrier-PcbDoc-rescue:LP5951-clocks-SchDoc-cache-AMC_FMC_Carrier-PcbDoc-rescue-AMC_FMC_Carrier-PcbDoc-rescue-AMC_FMC_Carrier-PcbDoc-rescue-AMC_FMC_Carrier-PcbDoc-rescue U13
 U 1 1 5C2E75E7
 P 1700 2500
@@
 $EndComp
 $Comp
-L AMC_FMC_Carrier-PcbDoc-rescue:+3V3_CLEAN-powerMG-AMC_FMC_Carrier-PcbDoc-rescue-AMC_FMC_Carrier-PcbDoc-rescue-AMC_FMC_Carrier-PcbDoc-rescue #PWR0169
+L AMC_FMC_Carrier-PcbDoc-rescue:+3V3_CLEAN-powerMG-AMC_FMC_Carrier-PcbDoc-rescue-AMC_FMC_Carrier-PcbDoc-rescue-AMC_FMC_Carrier-PcbDoc-rescue-AMC_FMC_Carrier-PcbDoc-rescue #PWR0169
 U 1 1 5C2EF25E
 P 700 2500
@@
 $EndComp
 $Comp
-L AMC_FMC_Carrier-PcbDoc-rescue:Oscillator_1VC_2GND_3OUT_4+Vs-clocks-SchDoc-cache-AMC_FMC_Carrier-PcbDoc-rescue-AMC_FMC_Carrier-PcbDoc-rescue-AMC_FMC_Carrier-PcbDoc-rescue Y2
+L AMC_FMC_Carrier-PcbDoc-rescue:Oscillator_1VC_2GND_3OUT_4+Vs-clocks-SchDoc-cache-AMC_FMC_Carrier-PcbDoc-rescue-AMC_FMC_Carrier-PcbDoc-rescue-AMC_FMC_Carrier-PcbDoc-rescue-AMC_FMC_Carrier-PcbDoc-rescue Y2
 U 1 1 5C2F3070
 P 4050 1950
@@
 $EndComp
 $Comp
-L AMC_FMC_Carrier-PcbDoc-rescue:+3V3_CLEAN-powerMG-AMC_FMC_Carrier-PcbDoc-rescue-AMC_FMC_Carrier-PcbDoc-rescue-AMC_FMC_Carrier-PcbDoc-rescue #PWR0206
+L AMC_FMC_Carrier-PcbDoc-rescue:+3V3_CLEAN-powerMG-AMC_FMC_Carrier-PcbDoc-rescue-AMC_FMC_Carrier-PcbDoc-rescue-AMC_FMC_Carrier-PcbDoc-rescue-AMC_FMC_Carrier-PcbDoc-rescue #PWR0206
 U 1 1 5C33B37A
 P 6550 6900
@@
 	6300 6250 6300 6300
 $Comp
-L AMC_FMC_Carrier-PcbDoc-rescue:+3V3_CLEAN-powerMG-AMC_FMC_Carrier-PcbDoc-rescue-AMC_FMC_Carrier-PcbDoc-rescue-AMC_FMC_Carrier-PcbDoc-rescue #PWR0189
+L AMC_FMC_Carrier-PcbDoc-rescue:+3V3_CLEAN-powerMG-AMC_FMC_Carrier-PcbDoc-rescue-AMC_FMC_Carrier-PcbDoc-rescue-AMC_FMC_Carrier-PcbDoc-rescue-AMC_FMC_Carrier-PcbDoc-rescue #PWR0189
 U 1 1 5C3A12D5
 P 5300 5900
@@
 	5300 5900 5300 5950
 $Comp
-L AMC_FMC_Carrier-PcbDoc-rescue:+3V3_CLEAN-powerMG-AMC_FMC_Carrier-PcbDoc-rescue-AMC_FMC_Carrier-PcbDoc-rescue-AMC_FMC_Carrier-PcbDoc-rescue #PWR0211
+L AMC_FMC_Carrier-PcbDoc-rescue:+3V3_CLEAN-powerMG-AMC_FMC_Carrier-PcbDoc-rescue-AMC_FMC_Carrier-PcbDoc-rescue-AMC_FMC_Carrier-PcbDoc-rescue-AMC_FMC_Carrier-PcbDoc-rescue #PWR0211
 U 1 1 5C8A0C88
 P 6500 1450
@@
 	10150 3050 10150 3100
 $Comp
-L AMC_FMC_Carrier-PcbDoc-rescue:+3V3_CLEAN-powerMG-AMC_FMC_Carrier-PcbDoc-rescue-AMC_FMC_Carrier-PcbDoc-rescue-AMC_FMC_Carrier-PcbDoc-rescue #PWR0399
+L AMC_FMC_Carrier-PcbDoc-rescue:+3V3_CLEAN-powerMG-AMC_FMC_Carrier-PcbDoc-rescue-AMC_FMC_Carrier-PcbDoc-rescue-AMC_FMC_Carrier-PcbDoc-rescue-AMC_FMC_Carrier-PcbDoc-rescue #PWR0399
 U 1 1 5D15AFE0
 P 10450 3400
@@
 NoConn ~ 2500 2800
 $Comp
-L AMC_FMC_Carrier-PcbDoc-rescue:+3V3_CLEAN-powerMG-AMC_FMC_Carrier-PcbDoc-rescue-AMC_FMC_Carrier-PcbDoc-rescue-AMC_FMC_Carrier-PcbDoc-rescue #PWR0401
+L AMC_FMC_Carrier-PcbDoc-rescue:+3V3_CLEAN-powerMG-AMC_FMC_Carrier-PcbDoc-rescue-AMC_FMC_Carrier-PcbDoc-rescue-AMC_FMC_Carrier-PcbDoc-rescue-AMC_FMC_Carrier-PcbDoc-rescue #PWR0401
 U 1 1 5D19EDBE
 P 10850 2700

Commit message: Automated edit to move cache / rescue symbols to actual eeschem library
Results of running dissect_lib3.py, not posted here
Parts:
- U13: symbol AMC_FMC_Carrier-PcbDoc-rescue:LP5951-clocks-SchDoc-cache-AMC_FMC_Carrier-PcbDoc-rescue-AMC_FMC_Carrier-PcbDoc-rescue-AM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 -> marble_misc:LP5951-clocks-SchDoc-cache
- U14: symbol AMC_FMC_Carrier-PcbDoc-rescue:LM336M-2.5-clocks-SchDoc-cache-AMC_FMC_Carrier-PcbDoc-rescue-AMC_FMC_Carrier-PcbDoc-rescu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 -> marble_misc:LM336M-2.5-clocks-SchDoc-cache
- Y2: symbol AMC_FMC_Carrier-PcbDoc-rescue:Oscillator_1VC_2GND_3OUT_4+Vs-clocks-SchDoc-cache-AMC_FMC_Carrier-PcbDoc-rescue-AMC_FMC_C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 -> marble_misc:Oscillator_1VC_2GND_3OUT_4+Vs-clocks-SchDoc-cache
Changed lines of the file:
@@
 	3750 4450 3750 5450
 $Comp
-L AMC_FMC_Carrier-PcbDoc-rescue:LM336M-2.5-clocks-SchDoc-cache-AMC_FMC_Carrier-PcbDoc-rescue-AMC_FMC_Carrier-PcbDoc-rescue-AMC_FMC_Carrier-PcbDoc-rescue-AMC_FMC_Carrier-PcbDoc-rescue U14
+L marble_misc:LM336M-2.5-clocks-SchDoc-cache U14
 U 1 1 5C21F363
 P 2200 6900
@@
 	8850 4850 8850 4950
 $Comp
-L AMC_FMC_Carrier-PcbDoc-rescue:+3V3_CLEAN-powerMG-AMC_FMC_Carrier-PcbDoc-rescue-AMC_FMC_Carrier-PcbDoc-rescue-AMC_FMC_Carrier-PcbDoc-rescue-AMC_FMC_Carrier-PcbDoc-rescue #PWR0175
+L marble_misc:+3V3_CLEAN #PWR0175
 U 1 1 5C2DA97A
 P 2300 6100
@@
 $EndComp
 $Comp
-L AMC_FMC_Carrier-PcbDoc-rescue:+3V3_CLEAN-powerMG-AMC_FMC_Carrier-PcbDoc-rescue-AMC_FMC_Carrier-PcbDoc-rescue-AMC_FMC_Carrier-PcbDoc-rescue-AMC_FMC_Carrier-PcbDoc-rescue #PWR0174
+L marble_misc:+3V3_CLEAN #PWR0174
 U 1 1 5C2DA9DF
 P 2250 5650
@@
 $EndComp
 $Comp
-L AMC_FMC_Carrier-PcbDoc-rescue:+3V3_CLEAN-powerMG-AMC_FMC_Carrier-PcbDoc-rescue-AMC_FMC_Carrier-PcbDoc-rescue-AMC_FMC_Carrier-PcbDoc-rescue-AMC_FMC_Carrier-PcbDoc-rescue #PWR0209
+L marble_misc:+3V3_CLEAN #PWR0209
 U 1 1 5C2DD28D
 P 7450 4850
@@
 $EndComp
 $Comp
-L AMC_FMC_Carrier-PcbDoc-rescue:+3V3_CLEAN-powerMG-AMC_FMC_Carrier-PcbDoc-rescue-AMC_FMC_Carrier-PcbDoc-rescue-AMC_FMC_Carrier-PcbDoc-rescue-AMC_FMC_Carrier-PcbDoc-rescue #PWR0173
+L marble_misc:+3V3_CLEAN #PWR0173
 U 1 1 5C2DDAC4
 P 2250 4650
@@
 CLK20_VCXO
 $Comp
-L AMC_FMC_Carrier-PcbDoc-rescue:LP5951-clocks-SchDoc-cache-AMC_FMC_Carrier-PcbDoc-rescue-AMC_FMC_Carrier-PcbDoc-rescue-AMC_FMC_Carrier-PcbDoc-rescue-AMC_FMC_Carrier-PcbDoc-rescue U13
+L marble_misc:LP5951-clocks-SchDoc-cache U13
 U 1 1 5C2E75E7
 P 1700 2500
@@
 $EndComp
 $Comp
-L AMC_FMC_Carrier-PcbDoc-rescue:+3V3_CLEAN-powerMG-AMC_FMC_Carrier-PcbDoc-rescue-AMC_FMC_Carrier-PcbDoc-rescue-AMC_FMC_Carrier-PcbDoc-rescue-AMC_FMC_Carrier-PcbDoc-rescue #PWR0169
+L marble_misc:+3V3_CLEAN #PWR0169
 U 1 1 5C2EF25E
 P 700 2500
@@
 $EndComp
 $Comp
-L AMC_FMC_Carrier-PcbDoc-rescue:Oscillator_1VC_2GND_3OUT_4+Vs-clocks-SchDoc-cache-AMC_FMC_Carrier-PcbDoc-rescue-AMC_FMC_Carrier-PcbDoc-rescue-AMC_FMC_Carrier-PcbDoc-rescue-AMC_FMC_Carrier-PcbDoc-rescue Y2
+L marble_misc:Oscillator_1VC_2GND_3OUT_4+Vs-clocks-SchDoc-cache Y2
 U 1 1 5C2F3070
 P 4050 1950
@@
 $EndComp
 $Comp
-L AMC_FMC_Carrier-PcbDoc-rescue:+3V3_CLEAN-powerMG-AMC_FMC_Carrier-PcbDoc-rescue-AMC_FMC_Carrier-PcbDoc-rescue-AMC_FMC_Carrier-PcbDoc-rescue-AMC_FMC_Carrier-PcbDoc-rescue #PWR0206
+L marble_misc:+3V3_CLEAN #PWR0206
 U 1 1 5C33B37A
 P 6550 6900
@@
 	6300 6250 6300 6300
 $Comp
-L AMC_FMC_Carrier-PcbDoc-rescue:+3V3_CLEAN-powerMG-AMC_FMC_Carrier-PcbDoc-rescue-AMC_FMC_Carrier-PcbDoc-rescue-AMC_FMC_Carrier-PcbDoc-rescue-AMC_FMC_Carrier-PcbDoc-rescue #PWR0189
+L marble_misc:+3V3_CLEAN #PWR0189
 U 1 1 5C3A12D5
 P 5300 5900
@@
 	5300 5900 5300 5950
 $Comp
-L AMC_FMC_Carrier-PcbDoc-rescue:+3V3_CLEAN-powerMG-AMC_FMC_Carrier-PcbDoc-rescue-AMC_FMC_Carrier-PcbDoc-rescue-AMC_FMC_Carrier-PcbDoc-rescue-AMC_FMC_Carrier-PcbDoc-rescue #PWR0211
+L marble_misc:+3V3_CLEAN #PWR0211
 U 1 1 5C8A0C88
 P 6500 1450
@@
 	10150 3050 10150 3100
 $Comp
-L AMC_FMC_Carrier-PcbDoc-rescue:+3V3_CLEAN-powerMG-AMC_FMC_Carrier-PcbDoc-rescue-AMC_FMC_Carrier-PcbDoc-rescue-AMC_FMC_Carrier-PcbDoc-rescue-AMC_FMC_Carrier-PcbDoc-rescue #PWR0399
+L marble_misc:+3V3_CLEAN #PWR0399
 U 1 1 5D15AFE0
 P 10450 3400
@@
 NoConn ~ 2500 2800
 $Comp
-L AMC_FMC_Carrier-PcbDoc-rescue:+3V3_CLEAN-powerMG-AMC_FMC_Carrier-PcbDoc-rescue-AMC_FMC_Carrier-PcbDoc-rescue-AMC_FMC_Carrier-PcbDoc-rescue-AMC_FMC_Carrier-PcbDoc-rescue #PWR0401
+L marble_misc:+3V3_CLEAN #PWR0401
 U 1 1 5D19EDBE
 P 10850 2700

Commit message: shave ERC report down to 5 issues
  * mostly by adding power inputs / outputs to the symbols (many
    power pins were set to bidirectional, which causes issues)
  * remove some stray power symbols which were not connected to
    anything
  * FMC connector: change all VCC and GND pins to Power input type
    (there's a lot of them!!)
Connections:
- wire segments 183 -> 184
Changed lines of the file:
@@
 	6000 5800 6000 5750
 Wire Wire Line
-	6500 5800 7350 5800
+	6500 5800 6850 5800
 Connection ~ 8950 2850
 Wire Wire Line
@@
 NoConn ~ 8850 1550
 NoConn ~ 8850 1650
+$Comp
+L power:PWR_FLAG #FLG0111
+U 1 1 5FA82370
+P 6850 5800
+F 0 "#FLG0111" H 6850 5875 50  0001 C CNN
+F 1 "PWR_FLAG" H 6850 5973 50  0000 C CNN
+F 2 "" H 6850 5800 50  0001 C CNN
+F 3 "" H 6850 5800 50  0001 C CNN
+	1    6850 5800
+	-1   0    0    1
+$EndComp
+Connection ~ 6850 5800
+Wire Wire Line
+	6850 5800 7350 5800
 $EndSCHEMATC

Commit message: I2C voltage translator added, rotated POE bridges, I2C connected to SODIMM, NMOS for power leds indicator, 3V3P connected to SI570 and SODIMM
Connections:
- net labels added: +3.3P
Changed lines of the file:
@@
 	0    1    1    0
-$EndComp
-$Comp
-L power:+3V3 #PWR?
-U 1 1 5EA72B2F
-P 7650 5200
-AR Path="/5BD32060/5EA72B2F" Ref="#PWR?"  Part="1"
-AR Path="/5BABAC65/5EA72B2F" Ref="#PWR?"  Part="1"
-AR Path="/5CC24E97/5EA72B2F" Ref="#PWR?"  Part="1"
-AR Path="/5CC393D3/5EA72B2F" Ref="#PWR?"  Part="1"
-AR Path="/5CC6DBF7/5EA72B2F" Ref="#PWR?"  Part="1"
-AR Path="/5CC8AFE1/5EA72B2F" Ref="#PWR?"  Part="1"
-AR Path="/5BCEDA59/5EA72B2F" Ref="#PWR?"  Part="1"
-AR Path="/5C16BF13/5EA72B2F" Ref="#PWR033"  Part="1"
-F 0 "#PWR033" H 7650 5050 50  0001 C CNN
-F 1 "+3V3" H 7665 5373 50  0000 C CNN
-F 2 "" H 7650 5200 50  0001 C CNN
-F 3 "" H 7650 5200 50  0001 C CNN
-	1    7650 5200
-	1    0    0    -1
 $EndComp
 Connection ~ 7650 5500
@@
 Wire Wire Line
 	8850 5600 9650 5600
-$Comp
-L power:+3V3 #PWR?
-U 1 1 5FEDB9B9
-P 6000 5750
-AR Path="/5BD32060/5FEDB9B9" Ref="#PWR?"  Part="1"
-AR Path="/5BABAC65/5FEDB9B9" Ref="#PWR?"  Part="1"
-AR Path="/5CC24E97/5FEDB9B9" Ref="#PWR?"  Part="1"
-AR Path="/5CC393D3/5FEDB9B9" Ref="#PWR?"  Part="1"
-AR Path="/5CC6DBF7/5FEDB9B9" Ref="#PWR?"  Part="1"
-AR Path="/5CC8AFE1/5FEDB9B9" Ref="#PWR?"  Part="1"
-AR Path="/5BCEDA59/5FEDB9B9" Ref="#PWR?"  Part="1"
-AR Path="/5C16BF13/5FEDB9B9" Ref="#PWR029"  Part="1"
-F 0 "#PWR029" H 6000 5600 50  0001 C CNN
-F 1 "+3V3" H 6015 5923 50  0000 C CNN
-F 2 "" H 6000 5750 50  0001 C CNN
-F 3 "" H 6000 5750 50  0001 C CNN
-	1    6000 5750
-	1    0    0    -1
-$EndComp
 $Comp
 L Inductors_SMD:IND0603_MURATA_BLM18SG121TN1D L?
@@
 Wire Wire Line
 	6850 5800 7350 5800
+$Comp
+L power:+3.3P #PWR?
+U 1 1 602CC128
+P 6000 5750
+AR Path="/5C16C03C/602CC128" Ref="#PWR?"  Part="1"
+AR Path="/5BCEDA39/602CC128" Ref="#PWR?"  Part="1"
+AR Path="/5D05A99E/602CC128" Ref="#PWR?"  Part="1"
+AR Path="/5C16BF8E/602CC128" Ref="#PWR?"  Part="1"
+AR Path="/602CC128" Ref="#PWR?"  Part="1"
+AR Path="/5C16BF13/602CC128" Ref="#PWR0841"  Part="1"
+F 0 "#PWR0841" H 6000 5600 50  0001 C CNN
+F 1 "+3.3P" H 6015 5923 50  0000 C CNN
+F 2 "" H 6000 5750 50  0001 C CNN
+F 3 "" H 6000 5750 50  0001 C CNN
+	1    6000 5750
+	1    0    0    -1
+$EndComp
+$Comp
+L power:+3.3P #PWR?
+U 1 1 602FC8CD
+P 7650 5200
+AR Path="/5C16C03C/602FC8CD" Ref="#PWR?"  Part="1"
+AR Path="/5BCEDA39/602FC8CD" Ref="#PWR?"  Part="1"
+AR Path="/5D05A99E/602FC8CD" Ref="#PWR?"  Part="1"
+AR Path="/5C16BF8E/602FC8CD" Ref="#PWR?"  Part="1"
+AR Path="/602FC8CD" Ref="#PWR?"  Part="1"
+AR Path="/5C16BF13/602FC8CD" Ref="#PWR0842"  Part="1"
+F 0 "#PWR0842" H 7650 5050 50  0001 C CNN
+F 1 "+3.3P" H 7665 5373 50  0000 C CNN
+F 2 "" H 7650 5200 50  0001 C CNN
+F 3 "" H 7650 5200 50  0001 C CNN
+	1    7650 5200
+	1    0    0    -1
+$EndComp
 $EndSCHEMATC
