File: Power_SW.sch (KiCad schematic (older format))
At the start: 134 parts, among them J9 2057-PH1-04-UA-ND, Q10 FDMS7608S, Q11 FDMS7608S, Q12 FDMS7608S, Q13 FDMS7608S, Q26 BC847BV, Q27 BC847BV, U35 XRP7724ILBTR-F, U36 TPS74401RGWT, U37 TPS74401RGWT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

Commit message: I2C voltage translator added, rotated POE bridges, I2C connected to SODIMM, NMOS for power leds indicator, 3V3P connected to SI570 and SODIMM
Parts:
- removed Q26, Q27: BC847BV, SOTFL50P160X60-6N, symbol Transistors:BC847BV
- added LD18, LD19: LED_KINGBRIGHT_KPH-1608CGCK, ICs And Semiconductors SMD:LED_KINGBRIGHT_KPH-1608CGCK, symbol LEDs_&_Displays:LED_KINGBRIGHT_KPH-1608CGCK
- added Q20, Q3: NX3008NBKV, ICs And Semiconductors SMD:SOTFL50P160X60-6N, symbol Transistors:NX3008NBKV
- added R61, R78: R0402_1K_1%_0.0625W_100PPM, RESC1005X40N, symbol Resistors_SMD:R0402_1K_1%_0.0625W_100PPM
Connections:
- net labels added: +3V3_USB
- wire segments 383 -> 385
Other:
- moved on the sheet: R247, R250, R253, R255

Commit message: More consistent attributes for LEDs and BSS138
Should match Marble-Mini
Fewer complaints from KiBoM
Parts:
- LD10, LD18, LD19, LD4, LD5, LD6, LD7, LD8, LD9: Manufacturer KINGBRIGHT -> WURTH; Part Number 150060VS75000 -> LED_KINGBRIGHT_KPH-1608CGCK
Changed lines of the file:
@@
 F 3 "" H 1450 5890 60  0001 L CNN
 F 4 "Green" H 1450 5800 60  0001 L CNN "Pole4"
-F 5 "150060VS75000" H 1450 5800 60  0001 L CNN "Part Number"
+F 5 "LED_KINGBRIGHT_KPH-1608CGCK" H 1450 5800 60  0001 L CNN "Part Number"
 F 6 "LED Green 1C 2A" H 1450 5710 60  0001 L CNN "Library Ref"
 F 7 "SchLib\\LEDs & Displays.SchLib" H 1450 5620 60  0001 L CNN "Library Path"
@@
 F 14 "~~" H 1450 4900 60  0001 L CNN "Status"
 F 15 "SMD Green LED, Case 1.6mmX0.8mm(0603), 0.65mm Thickness" H 1450 4810 60  0001 L CNN "Part Description"
-F 16 "KINGBRIGHT" H 1450 4720 60  0001 L CNN "Manufacturer"
+F 16 "WURTH" H 1450 4720 60  0001 L CNN "Manufacturer"
 F 17 "150060VS75000" H 1450 4630 60  0001 L CNN "Manufacturer Part Number"
 F 18 "2" H 1450 4540 60  0001 L CNN "Pin Count"
@@
 F 3 "" H 2500 5890 60  0001 L CNN
 F 4 "Green" H 2500 5800 60  0001 L CNN "Pole4"
-F 5 "150060VS75000" H 2500 5800 60  0001 L CNN "Part Number"
+F 5 "LED_KINGBRIGHT_KPH-1608CGCK" H 2500 5800 60  0001 L CNN "Part Number"
 F 6 "LED Green 1C 2A" H 2500 5710 60  0001 L CNN "Library Ref"
 F 7 "SchLib\\LEDs & Displays.SchLib" H 2500 5620 60  0001 L CNN "Library Path"
@@
 F 14 "~~" H 2500 4900 60  0001 L CNN "Status"
 F 15 "SMD Green LED, Case 1.6mmX0.8mm(0603), 0.65mm Thickness" H 2500 4810 60  0001 L CNN "Part Description"
-F 16 "KINGBRIGHT" H 2500 4720 60  0001 L CNN "Manufacturer"
+F 16 "WURTH" H 2500 4720 60  0001 L CNN "Manufacturer"
 F 17 "150060VS75000" H 2500 4630 60  0001 L CNN "Manufacturer Part Number"
 F 18 "2" H 2500 4540 60  0001 L CNN "Pin Count"
@@
 F 3 "" H 3650 5890 60  0001 L CNN
 F 4 "Green" H 3650 5800 60  0001 L CNN "Pole4"
-F 5 "150060VS75000" H 3650 5800 60  0001 L CNN "Part Number"
+F 5 "LED_KINGBRIGHT_KPH-1608CGCK" H 3650 5800 60  0001 L CNN "Part Number"
 F 6 "LED Green 1C 2A" H 3650 5710 60  0001 L CNN "Library Ref"
 F 7 "SchLib\\LEDs & Displays.SchLib" H 3650 5620 60  0001 L CNN "Library Path"
@@
 F 14 "~~" H 3650 4900 60  0001 L CNN "Status"
 F 15 "SMD Green LED, Case 1.6mmX0.8mm(0603), 0.65mm Thickness" H 3650 4810 60  0001 L CNN "Part Description"
-F 16 "KINGBRIGHT" H 3650 4720 60  0001 L CNN "Manufacturer"
+F 16 "WURTH" H 3650 4720 60  0001 L CNN "Manufacturer"
 F 17 "150060VS75000" H 3650 4630 60  0001 L CNN "Manufacturer Part Number"
 F 18 "2" H 3650 4540 60  0001 L CNN "Pin Count"
@@
 F 3 "" H 4700 5890 60  0001 L CNN
 F 4 "Green" H 4700 5800 60  0001 L CNN "Pole4"
-F 5 "150060VS75000" H 4700 5800 60  0001 L CNN "Part Number"
+F 5 "LED_KINGBRIGHT_KPH-1608CGCK" H 4700 5800 60  0001 L CNN "Part Number"
 F 6 "LED Green 1C 2A" H 4700 5710 60  0001 L CNN "Library Ref"
 F 7 "SchLib\\LEDs & Displays.SchLib" H 4700 5620 60  0001 L CNN "Library Path"
@@
 F 14 "~~" H 4700 4900 60  0001 L CNN "Status"
 F 15 "SMD Green LED, Case 1.6mmX0.8mm(0603), 0.65mm Thickness" H 4700 4810 60  0001 L CNN "Part Description"
-F 16 "KINGBRIGHT" H 4700 4720 60  0001 L CNN "Manufacturer"
+F 16 "WURTH" H 4700 4720 60  0001 L CNN "Manufacturer"
 F 17 "150060VS75000" H 4700 4630 60  0001 L CNN "Manufacturer Part Number"
 F 18 "2" H 4700 4540 60  0001 L CNN "Pin Count"
@@
 F 3 "" H 5250 5890 60  0001 L CNN
 F 4 "Green" H 5250 5800 60  0001 L CNN "Pole4"
-F 5 "150060VS75000" H 5250 5800 60  0001 L CNN "Part Number"
+F 5 "LED_KINGBRIGHT_KPH-1608CGCK" H 5250 5800 60  0001 L CNN "Part Number"
 F 6 "LED Green 1C 2A" H 5250 5710 60  0001 L CNN "Library Ref"
 F 7 "SchLib\\LEDs & Displays.SchLib" H 5250 5620 60  0001 L CNN "Library Path"
@@
 F 14 "~~" H 5250 4900 60  0001 L CNN "Status"
 F 15 "SMD Green LED, Case 1.6mmX0.8mm(0603), 0.65mm Thickness" H 5250 4810 60  0001 L CNN "Part Description"
-F 16 "KINGBRIGHT" H 5250 4720 60  0001 L CNN "Manufacturer"
+F 16 "WURTH" H 5250 4720 60  0001 L CNN "Manufacturer"
 F 17 "150060VS75000" H 5250 4630 60  0001 L CNN "Manufacturer Part Number"
 F 18 "2" H 5250 4540 60  0001 L CNN "Pin Count"
@@
 F 3 "" H 1400 7490 60  0001 L CNN
 F 4 "Green" H 1400 7400 60  0001 L CNN "Pole4"
-F 5 "150060VS75000" H 1400 7400 60  0001 L CNN "Part Number"
+F 5 "LED_KINGBRIGHT_KPH-1608CGCK" H 1400 7400 60  0001 L CNN "Part Number"
 F 6 "LED Green 1C 2A" H 1400 7310 60  0001 L CNN "Library Ref"
 F 7 "SchLib\\LEDs & Displays.SchLib" H 1400 7220 60  0001 L CNN "Library Path"
@@
 F 14 "~~" H 1400 6500 60  0001 L CNN "Status"
 F 15 "SMD Green LED, Case 1.6mmX0.8mm(0603), 0.65mm Thickness" H 1400 6410 60  0001 L CNN "Part Description"
-F 16 "KINGBRIGHT" H 1400 6320 60  0001 L CNN "Manufacturer"
+F 16 "WURTH" H 1400 6320 60  0001 L CNN "Manufacturer"
 F 17 "150060VS75000" H 1400 6230 60  0001 L CNN "Manufacturer Part Number"
 F 18 "2" H 1400 6140 60  0001 L CNN "Pin Count"
@@
 F 3 "" H 2050 7490 60  0001 L CNN
 F 4 "Green" H 2050 7400 60  0001 L CNN "Pole4"
-F 5 "150060VS75000" H 2050 7400 60  0001 L CNN "Part Number"
+F 5 "LED_KINGBRIGHT_KPH-1608CGCK" H 2050 7400 60  0001 L CNN "Part Number"
 F 6 "LED Green 1C 2A" H 2050 7310 60  0001 L CNN "Library Ref"
 F 7 "SchLib\\LEDs & Displays.SchLib" H 2050 7220 60  0001 L CNN "Library Path"
@@
 F 14 "~~" H 2050 6500 60  0001 L CNN "Status"
 F 15 "SMD Green LED, Case 1.6mmX0.8mm(0603), 0.65mm Thickness" H 2050 6410 60  0001 L CNN "Part Description"
-F 16 "KINGBRIGHT" H 2050 6320 60  0001 L CNN "Manufacturer"
+F 16 "WURTH" H 2050 6320 60  0001 L CNN "Manufacturer"
 F 17 "150060VS75000" H 2050 6230 60  0001 L CNN "Manufacturer Part Number"
 F 18 "2" H 2050 6140 60  0001 L CNN "Pin Count"
@@
 F 3 "" H 2700 7490 60  0001 L CNN
 F 4 "Green" H 2700 7400 60  0001 L CNN "Pole4"
-F 5 "150060VS75000" H 2700 7400 60  0001 L CNN "Part Number"
+F 5 "LED_KINGBRIGHT_KPH-1608CGCK" H 2700 7400 60  0001 L CNN "Part Number"
 F 6 "LED Green 1C 2A" H 2700 7310 60  0001 L CNN "Library Ref"
 F 7 "SchLib\\LEDs & Displays.SchLib" H 2700 7220 60  0001 L CNN "Library Path"
@@
 F 14 "~~" H 2700 6500 60  0001 L CNN "Status"
 F 15 "SMD Green LED, Case 1.6mmX0.8mm(0603), 0.65mm Thickness" H 2700 6410 60  0001 L CNN "Part Description"
-F 16 "KINGBRIGHT" H 2700 6320 60  0001 L CNN "Manufacturer"
+F 16 "WURTH" H 2700 6320 60  0001 L CNN "Manufacturer"
 F 17 "150060VS75000" H 2700 6230 60  0001 L CNN "Manufacturer Part Number"
 F 18 "2" H 2700 6140 60  0001 L CNN "Pin Count"
@@
 F 3 "" H 3350 7490 60  0001 L CNN
 F 4 "Green" H 3350 7400 60  0001 L CNN "Pole4"
-F 5 "150060VS75000" H 3350 7400 60  0001 L CNN "Part Number"
+F 5 "LED_KINGBRIGHT_KPH-1608CGCK" H 3350 7400 60  0001 L CNN "Part Number"
 F 6 "LED Green 1C 2A" H 3350 7310 60  0001 L CNN "Library Ref"
 F 7 "SchLib\\LEDs & Displays.SchLib" H 3350 7220 60  0001 L CNN "Library Path"
@@
 F 14 "~~" H 3350 6500 60  0001 L CNN "Status"
 F 15 "SMD Green LED, Case 1.6mmX0.8mm(0603), 0.65mm Thickness" H 3350 6410 60  0001 L CNN "Part Description"
-F 16 "KINGBRIGHT" H 3350 6320 60  0001 L CNN "Manufacturer"
+F 16 "WURTH" H 3350 6320 60  0001 L CNN "Manufacturer"
 F 17 "150060VS75000" H 3350 6230 60  0001 L CNN "Manufacturer Part Number"
 F 18 "2" H 3350 6140 60  0001 L CNN "Pin Count"

Commit message: reduced reels with components, DDR 1V5 enable signal connected to MMC, DDR I2C pull-ups powerd from 3.3VP
Parts:
- removed C141: CC1206_47UF_25V_20%_X5R, CAPC3216X180N, symbol Capacitors_SMD:CC1206_47UF_25V_20%_X5R
- removed R189: R0603_4K99_0.1%_0.063W_10PPM, Resistors SMD:RESC1608X55N, symbol Resistors_SMD:R0603_4K99_0.1%_0.063W_10PPM
- removed R71: R0402_10K_0.1%_0.063W_25PPM, RESC1005X35N, symbol Resistors_SMD:R0402_10K_0.1%_0.063W_25PPM
- added C141, C416: CC1206_22UF_25V_20%_X5R, Capacitors SMD:CAPC3216X180N, symbol Capacitors_SMD:CC1206_22UF_25V_20%_X5R
- added R189: R0603_4K99_1%_0.063W_50PPM, Resistors SMD:RESC1608X55N, symbol Resistors_SMD:R0603_4K99_1%_0.063W_50PPM
- added R71: R0402_10K_1%_0.0625W_100PPM, Resistors SMD:RESC1005X40N, symbol Resistors_SMD:R0402_10K_1%_0.0625W_100PPM
- C127, C144, C347, C348, C349, C361: value CC0603_4.7UF_16V_10%_X5R -> CC0603_4.7UF_25V_10%_X5R; footprint CAPC1709X95N -> Capacitors SMD:CAPC1608X90N; symbol Capacitors_SMD:CC0603_4.7UF_16V_10%_X5R -> Capacitors_SMD:CC0603_4.7UF_25V_10%_X5R; Comment =Value -> 4.7uF; ComponentHeight ~~ -> (none); CreateDate 12/16/13 00:00:00 -> 11/10/14 00:00:00; Database Table Name (none) -> Capacitors SMD; Footprint Library (none) -> Capacitors SMD; Footprint Ref CAPC1709X95N -> CAPC1608X90N; LatestRevisionDate 09/16/14 00:00:00 -> 11/10/14 00:00:00; Library Name Capacitors SMD -> Capacitors.DbLib; Manufacturer Part Number CC0603_4.7UF_16V_10%_X5R -> CC0603_4.7UF_25V_10%_X5R; Manufacturer1 Example TAIYO YUDEN -> MURATA; Manufacturer1 Part Number EMK107ABJ475KA-T -> GRM188R61E475KE11D; PackageDescription ~~ -> (none); Part Number CC0603_4.7UF_16V_10%_X5R -> CC0603_4.7UF_25V_10%_X5R; Pin Count 2.0000000000000000e+00 -> 2; PressFit ~~ -> (none); Sense Comment ~~ -> (none); Status Comment ~~ -> (none); Voltage 16V -> 25V
- R72: value R0402_0R_JUMPER -> R0402_100K_1%_0.0625W_100PPM; footprint RESC1005X40N -> Resistors SMD:RESC1005X40N; symbol Resistors_SMD:R0402_0R_JUMPER -> Resistors_SMD:R0402_100K_1%_0.0625W_100PPM; Comment =Value -> 100k; ComponentHeight ~~ -> (none); Database Table Name (none) -> Resistors SMD; Footprint Library (none) -> Resistors SMD; Library Name Resistors SMD -> Resistors.DbLib; Library Ref Resistor -> Resistor - 1%; Manufacturer Part Number R0402_0R_JUMPER -> R0402_100K_1%_0.0625W_100PPM; Manufacturer1 Part Number 232270591001L -> 232270671004L; PackageDescription ~~ -> (none); Part Description 1A (0.05R Max DC Resistance) Zero Ohm Jumper -> General Purpose Thick Film Chip Resistor; Part Number R0402_0R_JUMPER -> R0402_100K_1%_0.0625W_100PPM; Power ~~ -> 0.0625W; Sense Comment ~~ -> (none); Status Comment ~~ -> (none); TC ~~ -> ±100ppm/°C; Tolerance ~~ -> ±1%; Val 0 -> 100k; Voltage ~~ -> (none); ~ 0 -> 100k
Connections:
- net labels added: 1V5_EN, DDR_1V5_EN
- wire segments 385 -> 389
Other:
- moved on the sheet: C411, C413, C414, L42

Commit message: Unify CC0402_100NF part numbers
CC0402_100NF_16V_10%_X5R and CC0402_100NF_25V_10%_X7R_YUDEN_TMK105B7104KVHF
become CC0402_100NF_25V_10%_X5R, matching Marble-Mini
generic_subst converts this to Samsung CL05A104KA5NNNC
15 refids: C5 C61 C128 C130 C131 C134 C135 C137 C140 C147 C148 C149 C150 C362 C363
Parts:
- C137, C140, C147, C148, C149, C150, C362: value CC0402_100NF_25V_10%_X7R_YUDEN_TMK105B7104KVHF -> CC0402_100NF_25V_10%_X5R; footprint Capacitors SMD:CAPC1005X55N -> Marble:CAPC1005X55N; symbol Capacitors_SMD:CC0402_100NF_25V_10%_X7R_YUDEN_TMK105B7104KVHF -> Capacitors_SMD:CC0402_100NF_25V_10%_X5R; ComponentHeight 0.55mm -> (none); CreateDate 05/10/17 00:00:00 -> 12/10/13 00:00:00; LatestRevisionDate 05/10/17 00:00:00 -> 05/25/20 00:00:00; Library Name Capacitors.DbLib -> Capacitors SMD; Manufacturer TAIYO YUDEN -> GENERIC; Manufacturer Part Number TMK105B7104KVHF -> CC0402_100NF_25V_10%_X5R; Manufacturer1 ComponentHeight (none) -> 0.55mm; Manufacturer1 Example (none) -> Samsung; Manufacturer1 Part Number (none) -> CL05A104KA5NNNC; Part Description SMD Multilayer Chip Ceramic Capacitor (High Dielectric Type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 -> SMD Multilayer Chip Ceramic Capacitor; Part Number CC0402_100NF_25V_10%_X7R_YUDEN_TMK105B7104KVHF -> CC0402_100NF_25V_10%_X5R; Status Not Recommended -> None; TC X7R -> X5R
- C363: value CC0402_100NF_16V_10%_X5R -> CC0402_100NF_25V_10%_X5R; footprint CAPC1005X55N -> Marble:CAPC1005X55N; symbol Capacitors_SMD:CC0402_100NF_25V_10%_X7R_YUDEN_TMK105B7104KVHF -> Capacitors_SMD:CC0402_100NF_25V_10%_X5R; Comment =Value -> 100nF; ComponentHeight ~~ -> (none); LatestRevisionDate 12/10/13 00:00:00 -> 05/25/20 00:00:00; Manufacturer Part Number CC0402_100NF_16V_10%_X5R -> CC0402_100NF_25V_10%_X5R; Manufacturer1 Example MURATA -> Samsung; Manufacturer1 Part Number GRM155R61C104KA88D -> CL05A104KA5NNNC; PackageDescription ~~ -> (none); Part Number CC0402_100NF_16V_10%_X5R -> CC0402_100NF_25V_10%_X5R; Pin Count 2.0000000000000000e+00 -> 2; PressFit ~~ -> (none); Sense Comment ~~ -> (none); Status Comment ~~ -> (none); Voltage 16V -> 25V

Commit message: all test points have THT pads, a new test point for GND
Parts:
- added TP12: TestPoint, TestPoint:TestPoint_THTPad_D1.5mm_Drill0.7mm, symbol Connector_Generic:TestPoint
- TP10, TP11, TP4, TP5, TP6, TP7, TP8, TP9: footprint TestPoint:TestPoint_Pad_D1.0mm -> TestPoint:TestPoint_THTPad_D1.5mm_Drill0.7mm
Connections:
- wire segments 389 -> 390
Changed lines of the file:
@@
 F 0 "TP10" H 14758 2618 50  0000 L CNN
 F 1 "TestPoint" H 14758 2527 50  0000 L CNN
-F 2 "TestPoint:TestPoint_Pad_D1.0mm" H 14900 2500 50  0001 C CNN
+F 2 "TestPoint:TestPoint_THTPad_D1.5mm_Drill0.7mm" H 14900 2500 50  0001 C CNN
 F 3 "~" H 14900 2500 50  0001 C CNN
 	1    14700 2500
@@
 F 0 "TP11" H 14758 4418 50  0000 L CNN
 F 1 "TestPoint" H 14758 4327 50  0000 L CNN
-F 2 "TestPoint:TestPoint_Pad_D1.0mm" H 14900 4300 50  0001 C CNN
+F 2 "TestPoint:TestPoint_THTPad_D1.5mm_Drill0.7mm" H 14900 4300 50  0001 C CNN
 F 3 "~" H 14900 4300 50  0001 C CNN
 	1    14700 4300
@@
 F 0 "TP9" H 14608 6218 50  0000 L CNN
 F 1 "TestPoint" H 14608 6127 50  0000 L CNN
-F 2 "TestPoint:TestPoint_Pad_D1.0mm" H 14750 6100 50  0001 C CNN
+F 2 "TestPoint:TestPoint_THTPad_D1.5mm_Drill0.7mm" H 14750 6100 50  0001 C CNN
 F 3 "~" H 14750 6100 50  0001 C CNN
 	1    14550 6100
@@
 F 0 "TP8" H 14458 8518 50  0000 L CNN
 F 1 "TestPoint" H 14458 8427 50  0000 L CNN
-F 2 "TestPoint:TestPoint_Pad_D1.0mm" H 14600 8400 50  0001 C CNN
+F 2 "TestPoint:TestPoint_THTPad_D1.5mm_Drill0.7mm" H 14600 8400 50  0001 C CNN
 F 3 "~" H 14600 8400 50  0001 C CNN
 	1    14400 8400
@@
 F 0 "TP7" H 9508 7618 50  0000 L CNN
 F 1 "TestPoint" H 9508 7527 50  0000 L CNN
-F 2 "TestPoint:TestPoint_Pad_D1.0mm" H 9650 7500 50  0001 C CNN
+F 2 "TestPoint:TestPoint_THTPad_D1.5mm_Drill0.7mm" H 9650 7500 50  0001 C CNN
 F 3 "~" H 9650 7500 50  0001 C CNN
 	1    9450 7500
@@
 F 0 "TP5" H 8058 9768 50  0000 L CNN
 F 1 "TestPoint" H 8058 9677 50  0000 L CNN
-F 2 "TestPoint:TestPoint_Pad_D1.0mm" H 8200 9650 50  0001 C CNN
+F 2 "TestPoint:TestPoint_THTPad_D1.5mm_Drill0.7mm" H 8200 9650 50  0001 C CNN
 F 3 "~" H 8200 9650 50  0001 C CNN
 	1    8000 9650
@@
 F 0 "TP4" H 3308 9268 50  0000 L CNN
 F 1 "TestPoint" H 3308 9177 50  0000 L CNN
-F 2 "TestPoint:TestPoint_Pad_D1.0mm" H 3450 9150 50  0001 C CNN
+F 2 "TestPoint:TestPoint_THTPad_D1.5mm_Drill0.7mm" H 3450 9150 50  0001 C CNN
 F 3 "~" H 3450 9150 50  0001 C CNN
 	1    3250 9150
@@
 F 0 "TP6" V 9708 6768 50  0000 L CNN
 F 1 "TestPoint" V 9800 6650 50  0000 L CNN
-F 2 "TestPoint:TestPoint_Pad_D1.0mm" H 9850 6650 50  0001 C CNN
+F 2 "TestPoint:TestPoint_THTPad_D1.5mm_Drill0.7mm" H 9850 6650 50  0001 C CNN
 F 3 "~" H 9850 6650 50  0001 C CNN
 	1    9650 6650
@@
 Wire Wire Line
 	6450 7100 6450 7050
+$Comp
+L Connector_Generic:TestPoint TP?
+U 1 1 5FC62BFE
+P 8000 10150
+AR Path="/5C16BF8E/5FC62BFE" Ref="TP?"  Part="1"
+AR Path="/5C16BF8E/5DB9B7E6/5FC62BFE" Ref="TP12"  Part="1"
+F 0 "TP12" H 8058 10268 50  0000 L CNN
+F 1 "TestPoint" H 8058 10177 50  0000 L CNN
+F 2 "TestPoint:TestPoint_THTPad_D1.5mm_Drill0.7mm" H 8200 10150 50  0001 C CNN
+F 3 "~" H 8200 10150 50  0001 C CNN
+	1    8000 10150
+	0    1    1    0
+$EndComp
+$Comp
+L power:GND #PWR?
+U 1 1 5FC94969
+P 7850 10150
+AR Path="/5C16C03C/5FC94969" Ref="#PWR?"  Part="1"
+AR Path="/5BCEDA59/5FC94969" Ref="#PWR?"  Part="1"
+AR Path="/5C16BF8E/5FC94969" Ref="#PWR?"  Part="1"
+AR Path="/5C16BF8E/5DB9B7E6/5FC94969" Ref="#PWR029"  Part="1"
+F 0 "#PWR029" H 7850 9900 50  0001 C CNN
+F 1 "GND" H 7855 9977 50  0000 C CNN
+F 2 "" H 7850 10150 50  0001 C CNN
+F 3 "" H 7850 10150 50  0001 C CNN
+	1    7850 10150
+	1    0    0    -1
+$EndComp
+Wire Wire Line
+	7850 10150 8000 10150
 $EndSCHEMATC

Commit message: no 0.1% resistors, added R79 (40R4), C114 -> 2.2nF
Parts:
- removed R168: R0603_2K49_0.1%_0.063W_10PPM, Resistors SMD:RESC1608X55N, symbol Resistors_SMD:R0603_2K49_0.1%_0.063W_10PPM
- removed R189: R0603_4K99_1%_0.063W_50PPM, Resistors SMD:RESC1608X55N, symbol Resistors_SMD:R0603_4K99_1%_0.063W_50PPM
- removed R195: R0603_1K37_0.1%_0.063W_10PPM, Resistors SMD:RESC1608X55N, symbol Resistors_SMD:R0603_1K37_0.1%_0.063W_10PPM
- removed R196: R0603_4K42_0.1%_0.063W_10PPM, Resistors SMD:RESC1608X55N, symbol Resistors_SMD:R0603_4K42_0.1%_0.063W_10PPM
- removed R68: R0603_10K7_0.1%_0.063W_10PPM, Resistors SMD:RESC1608X55N, symbol Resistors_SMD:R0603_10K7_0.1%_0.063W_10PPM
- removed R69: R0603_9K31_0.1%_0.063W_10PPM, Resistors SMD:RESC1608X55N, symbol Resistors_SMD:R0603_9K31_0.1%_0.063W_10PPM
- removed R70: R0603_15K_0.1%_0.063W_10PPM, RESC1608X55N, symbol Resistors_SMD:R0603_15K_0.1%_0.063W_10PPM
- added R168: R0402_1K8_1%_0.0625W_100PPM, Resistors SMD:RESC1005X40N, symbol Resistors_SMD2:R0402_1K8_1%_0.0625W_100PPM
- added R189: R0402_3K6_1%_0.0625W_100PPM, Resistors SMD:RESC1005X40N, symbol Resistors_SMD2:R0402_3K6_1%_0.0625W_100PPM
- added R195: R0402_7K5_1%_0.0625W_100PPM, Resistors SMD:RESC1005X40N, symbol Resistors_SMD2:R0402_7K5_1%_0.0625W_100PPM
- added R196: R0402_24K_1%_0.0625W_100PPM, Resistors SMD:RESC1005X40N, symbol Resistors_SMD2:R0402_24K_1%_0.0625W_100PPM
- added R68, R70: R0402_15K_1%_0.0625W_100PPM, Resistors SMD:RESC1005X40N, symbol Resistors_SMD2:R0402_15K_1%_0.0625W_100PPM
- added R69: R0402_13K_1%_0.0625W_100PPM, Resistors SMD:RESC1005X40N, symbol Resistors_SMD2:R0402_13K_1%_0.0625W_100PPM

Commit message: fixed a corrupted schematic
Parts:
- removed R168: R0402_1K8_1%_0.0625W_100PPM, Resistors SMD:RESC1005X40N, symbol Resistors_SMD2:R0402_1K8_1%_0.0625W_100PPM
- removed R189: R0402_3K6_1%_0.0625W_100PPM, Resistors SMD:RESC1005X40N, symbol Resistors_SMD2:R0402_3K6_1%_0.0625W_100PPM
- removed R195: R0402_7K5_1%_0.0625W_100PPM, Resistors SMD:RESC1005X40N, symbol Resistors_SMD2:R0402_7K5_1%_0.0625W_100PPM
- removed R196: R0402_24K_1%_0.0625W_100PPM, Resistors SMD:RESC1005X40N, symbol Resistors_SMD2:R0402_24K_1%_0.0625W_100PPM
- removed R68, R70: R0402_15K_1%_0.0625W_100PPM, Resistors SMD:RESC1005X40N, symbol Resistors_SMD2:R0402_15K_1%_0.0625W_100PPM
- removed R69: R0402_13K_1%_0.0625W_100PPM, Resistors SMD:RESC1005X40N, symbol Resistors_SMD2:R0402_13K_1%_0.0625W_100PPM
- added R168: R0402_1K8_1%_0.0625W_100PPM, Resistors SMD:RESC1005X40N, symbol Resistors_SMD:R0402_1K8_1%_0.0625W_100PPM
- added R189: R0402_3K6_1%_0.0625W_100PPM, Resistors SMD:RESC1005X40N, symbol Resistors_SMD:R0402_3K6_1%_0.0625W_100PPM
- added R195: R0402_7K5_1%_0.0625W_100PPM, Resistors SMD:RESC1005X40N, symbol Resistors_SMD:R0402_7K5_1%_0.0625W_100PPM
- added R196: R0402_24K_1%_0.0625W_100PPM, Resistors SMD:RESC1005X40N, symbol Resistors_SMD:R0402_24K_1%_0.0625W_100PPM
- added R68, R70: R0402_15K_1%_0.0625W_100PPM, Resistors SMD:RESC1005X40N, symbol Resistors_SMD:R0402_15K_1%_0.0625W_100PPM
- added R69: R0402_13K_1%_0.0625W_100PPM, Resistors SMD:RESC1005X40N, symbol Resistors_SMD:R0402_13K_1%_0.0625W_100PPM

Commit message: Flag duplicate generic parts in BOM, and refresh a few cap instances from library to reduce such dups
Parts:
- C138: footprint CAPC1005X55N -> Capacitors SMD:CAPC1005X55N; Comment =Value -> 2.2nF; ComponentHeight ~~ -> (none); Database Table Name (none) -> Capacitors SMD; Footprint Library (none) -> Capacitors SMD; Library Name Capacitors SMD -> Capacitors.DbLib; PackageDescription ~~ -> (none); Pin Count 2.0000000000000000e+00 -> 2; PressFit ~~ -> (none); Sense Comment ~~ -> (none); Status Comment ~~ -> (none)
Changed lines of the file:
@@
 F 0 "C138" H 5850 3450 50  0000 C CNN
 F 1 "CC0402_2.2NF_50V_10%_X7R" H 5700 3040 60  0001 L CNN
-F 2 "CAPC1005X55N" H 5700 2230 60  0001 L CNN
+F 2 "Capacitors SMD:CAPC1005X55N" H 5700 2230 60  0001 L CNN
 F 3 "\\\\cern.ch\\dfs\\Applications\\Altium\\Datasheets\\CC0402_X7R_PHYCOMP.pdf" H 5700 2860 60  0001 L CNN
 F 4 "2.2nF" H 5850 3150 50  0000 C CNN "~"
@@
 F 6 "Capacitor - non polarized" H 5700 2680 60  0001 L CNN "Library Ref"
 F 7 "SchLib\\Capacitors.SchLib" H 5700 2590 60  0001 L CNN "Library Path"
-F 8 "=Value" H 5700 2500 60  0001 L CNN "Comment"
+F 8 "2.2nF" H 5700 2500 60  0001 L CNN "Comment"
 F 9 "Standard" H 5700 2410 60  0001 L CNN "Component Kind"
 F 10 "Standard" H 5700 2320 60  0001 L CNN "Component Type"
-F 11 "2.0000000000000000e+00" H 5700 2140 60  0001 L CNN "Pin Count"
+F 11 "2" H 5700 2140 60  0001 L CNN "Pin Count"
 F 12 "PcbLib\\Capacitors SMD.PcbLib" H 5700 2050 60  0001 L CNN "Footprint Path"
 F 13 "CAPC1005X55N" H 5700 1960 60  0001 L CNN "Footprint Ref"
-F 14 "~~" H 5700 1870 60  0001 L CNN "PackageDescription"
+F 14 " " H 5700 1870 60  0001 L CNN "PackageDescription"
 F 15 "2.2nF" H 5700 1780 60  0001 L CNN "Val"
 F 16 "Not Recommended" H 5700 1690 60  0001 L CNN "Status"
-F 17 "~~" H 5700 1600 60  0001 L CNN "Status Comment"
+F 17 " " H 5700 1600 60  0001 L CNN "Status Comment"
 F 18 "50V" H 5700 1510 60  0001 L CNN "Voltage"
 F 19 "X7R" H 5700 1420 60  0001 L CNN "TC"
@@
 F 26 "No" H 5700 790 60  0001 L CNN "Socket"
 F 27 "Yes" H 5700 700 60  0001 L CNN "SMD"
-F 28 "~~" H 5700 610 60  0001 L CNN "PressFit"
+F 28 " " H 5700 610 60  0001 L CNN "PressFit"
 F 29 "No" H 5700 520 60  0001 L CNN "Sense"
-F 30 "~~" H 5700 430 60  0001 L CNN "Sense Comment"
-F 31 "~~" H 5700 340 60  0001 L CNN "ComponentHeight"
+F 30 " " H 5700 430 60  0001 L CNN "Sense Comment"
+F 31 " " H 5700 340 60  0001 L CNN "ComponentHeight"
 F 32 "PHYCOMP" H 5700 250 60  0001 L CNN "Manufacturer1 Example"
 F 33 "223858715627" H 5700 160 60  0001 L CNN "Manufacturer1 Part Number"
@@
 F 37 "12/03/07 00:00:00" H 5700 -200 60  0001 L CNN "CreateDate"
 F 38 "12/03/07 00:00:00" H 5700 -290 60  0001 L CNN "LatestRevisionDate"
-F 39 "Capacitors SMD" H 5700 -380 60  0001 L CNN "Library Name"
+F 39 "Capacitors.DbLib" H 5700 -380 60  0001 L CNN "Library Name"
 F 40 "This work is licensed under the Creative Commons CC-BY-SA 4.0 License. To the extent that circuit schematics that use Licensed Material can be considered to be ‘Adapted Material’, then the copyright holder waives article 3.b of the license with respect to these schematics." H 5700 -470 60  0001 L CNN "License"
+F 41 "Capacitors SMD" H 5700 3300 50  0001 C CNN "Database Table Name"
+F 42 "Capacitors SMD" H 5700 3300 50  0001 C CNN "Footprint Library"
 	1    5700 3300
 	1    0    0    -1
