File: ETH_PHY.sch (KiCad schematic (older format))
At the start: 44 parts, among them J4 BELFUSE_0826-1X1T-GH-F, U4 88E1512-A0-NNP2I000, U6 TXS0102DCUR

Commit message: new PN for LEDs
Parts:
- J4: symbol AMC_FMC_Carrier-PcbDoc-rescue:BELFUSE_0826-1X1T-HS-F-Miscellaneous-AMC_FMC_Carrier-PcbDoc-rescue -> AMC_FMC_Carrier-PcbDoc-rescue:BELFUSE_0826-1X1T-HS-F-Miscellaneous-AMC_FMC_Carrier-PcbDoc-rescue-AMC_FMC_Carrier-PcbDoc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
- OSC1: symbol AMC_FMC_Carrier-PcbDoc-rescue:Oscillator-powerMG-AMC_FMC_Carrier-PcbDoc-rescue-AMC_FMC_Carrier-PcbDoc-rescue -> AMC_FMC_Carrier-PcbDoc-rescue:Oscillator-powerMG-AMC_FMC_Carrier-PcbDoc-rescue-AMC_FMC_Carrier-PcbDoc-rescue-AMC_FMC_Ca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
Changed lines of the file:
@@
 RGMII_RX_CLK
 $Comp
-L AMC_FMC_Carrier-PcbDoc-rescue:Oscillator-powerMG-AMC_FMC_Carrier-PcbDoc-rescue-AMC_FMC_Carrier-PcbDoc-rescue OSC1
+L AMC_FMC_Carrier-PcbDoc-rescue:Oscillator-powerMG-AMC_FMC_Carrier-PcbDoc-rescue-AMC_FMC_Carrier-PcbDoc-rescue-AMC_FMC_Carrier-PcbDoc-rescue OSC1
 U 1 1 5C76AE78
 P 4600 3400
@@
 	3050 1500 3250 1500
 $Comp
-L AMC_FMC_Carrier-PcbDoc-rescue:BELFUSE_0826-1X1T-HS-F-Miscellaneous-AMC_FMC_Carrier-PcbDoc-rescue J4
+L AMC_FMC_Carrier-PcbDoc-rescue:BELFUSE_0826-1X1T-HS-F-Miscellaneous-AMC_FMC_Carrier-PcbDoc-rescue-AMC_FMC_Carrier-PcbDoc-rescue J4
 U 1 1 5DB81DF6
 P 12500 1900
@@
 Connection ~ 14500 4500
 $Comp
-L AMC_FMC_Carrier-PcbDoc-rescue:power_PWR_FLAG-AMC_FMC_Carrier-PcbDoc-cache-AMC_FMC_Carrier-PcbDoc-rescue #FLG0103
+L AMC_FMC_Carrier-PcbDoc-rescue:power_PWR_FLAG-AMC_FMC_Carrier-PcbDoc-cache-AMC_FMC_Carrier-PcbDoc-rescue-AMC_FMC_Carrier-PcbDoc-rescue #FLG0103
 U 1 1 5D15ABC3
 P 5250 6650
@@
 $EndComp
 $Comp
-L AMC_FMC_Carrier-PcbDoc-rescue:power_PWR_FLAG-AMC_FMC_Carrier-PcbDoc-cache-AMC_FMC_Carrier-PcbDoc-rescue #FLG0104
+L AMC_FMC_Carrier-PcbDoc-rescue:power_PWR_FLAG-AMC_FMC_Carrier-PcbDoc-cache-AMC_FMC_Carrier-PcbDoc-rescue-AMC_FMC_Carrier-PcbDoc-rescue #FLG0104
 U 1 1 5D15B1F6
 P 5250 7600
@@
 $EndComp
 $Comp
-L AMC_FMC_Carrier-PcbDoc-rescue:power_PWR_FLAG-AMC_FMC_Carrier-PcbDoc-cache-AMC_FMC_Carrier-PcbDoc-rescue #FLG0105
+L AMC_FMC_Carrier-PcbDoc-rescue:power_PWR_FLAG-AMC_FMC_Carrier-PcbDoc-cache-AMC_FMC_Carrier-PcbDoc-rescue-AMC_FMC_Carrier-PcbDoc-rescue #FLG0105
 U 1 1 5D15B45E
 P 14500 2000

Commit message: fixed bugs
Parts:
- J4: symbol AMC_FMC_Carrier-PcbDoc-rescue:BELFUSE_0826-1X1T-HS-F-Miscellaneous-AMC_FMC_Carrier-PcbDoc-rescue-AMC_FMC_Carrier-PcbDoc-rescue -> AMC_FMC_Carrier-PcbDoc-rescue:BELFUSE_0826-1X1T-HS-F-Miscellaneous-AMC_FMC_Carrier-PcbDoc-rescue-AMC_FMC_Carrier-PcbDoc-rescue-AMC_FMC_Carrier-PcbDoc-rescue
- OSC1: symbol AMC_FMC_Carrier-PcbDoc-rescue:Oscillator-powerMG-AMC_FMC_Carrier-PcbDoc-rescue-AMC_FMC_Carrier-PcbDoc-rescue-AMC_FMC_Carrier-PcbDoc-rescue -> AMC_FMC_Carrier-PcbDoc-rescue:Oscillator-powerMG-AMC_FMC_Carrier-PcbDoc-rescue-AMC_FMC_Carrier-PcbDoc-rescue-AMC_FMC_Carrier-PcbDoc-rescue-AMC_FMC_Carrier-PcbDoc-rescue
Changed lines of the file:
@@
 RGMII_RX_CLK
 $Comp
-L AMC_FMC_Carrier-PcbDoc-rescue:Oscillator-powerMG-AMC_FMC_Carrier-PcbDoc-rescue-AMC_FMC_Carrier-PcbDoc-rescue-AMC_FMC_Carrier-PcbDoc-rescue OSC1
+L AMC_FMC_Carrier-PcbDoc-rescue:Oscillator-powerMG-AMC_FMC_Carrier-PcbDoc-rescue-AMC_FMC_Carrier-PcbDoc-rescue-AMC_FMC_Carrier-PcbDoc-rescue-AMC_FMC_Carrier-PcbDoc-rescue OSC1
 U 1 1 5C76AE78
 P 4600 3400
@@
 	3050 1500 3250 1500
 $Comp
-L AMC_FMC_Carrier-PcbDoc-rescue:BELFUSE_0826-1X1T-HS-F-Miscellaneous-AMC_FMC_Carrier-PcbDoc-rescue-AMC_FMC_Carrier-PcbDoc-rescue J4
+L AMC_FMC_Carrier-PcbDoc-rescue:BELFUSE_0826-1X1T-HS-F-Miscellaneous-AMC_FMC_Carrier-PcbDoc-rescue-AMC_FMC_Carrier-PcbDoc-rescue-AMC_FMC_Carrier-PcbDoc-rescue J4
 U 1 1 5DB81DF6
 P 12500 1900
@@
 Connection ~ 14500 4500
 $Comp
-L AMC_FMC_Carrier-PcbDoc-rescue:power_PWR_FLAG-AMC_FMC_Carrier-PcbDoc-cache-AMC_FMC_Carrier-PcbDoc-rescue-AMC_FMC_Carrier-PcbDoc-rescue #FLG0103
+L AMC_FMC_Carrier-PcbDoc-rescue:power_PWR_FLAG-AMC_FMC_Carrier-PcbDoc-cache-AMC_FMC_Carrier-PcbDoc-rescue-AMC_FMC_Carrier-PcbDoc-rescue-AMC_FMC_Carrier-PcbDoc-rescue #FLG0103
 U 1 1 5D15ABC3
 P 5250 6650
@@
 $EndComp
 $Comp
-L AMC_FMC_Carrier-PcbDoc-rescue:power_PWR_FLAG-AMC_FMC_Carrier-PcbDoc-cache-AMC_FMC_Carrier-PcbDoc-rescue-AMC_FMC_Carrier-PcbDoc-rescue #FLG0104
+L AMC_FMC_Carrier-PcbDoc-rescue:power_PWR_FLAG-AMC_FMC_Carrier-PcbDoc-cache-AMC_FMC_Carrier-PcbDoc-rescue-AMC_FMC_Carrier-PcbDoc-rescue-AMC_FMC_Carrier-PcbDoc-rescue #FLG0104
 U 1 1 5D15B1F6
 P 5250 7600
@@
 $EndComp
 $Comp
-L AMC_FMC_Carrier-PcbDoc-rescue:power_PWR_FLAG-AMC_FMC_Carrier-PcbDoc-cache-AMC_FMC_Carrier-PcbDoc-rescue-AMC_FMC_Carrier-PcbDoc-rescue #FLG0105
+L AMC_FMC_Carrier-PcbDoc-rescue:power_PWR_FLAG-AMC_FMC_Carrier-PcbDoc-cache-AMC_FMC_Carrier-PcbDoc-rescue-AMC_FMC_Carrier-PcbDoc-rescue-AMC_FMC_Carrier-PcbDoc-rescue #FLG0105
 U 1 1 5D15B45E
 P 14500 2000

Commit message: added J9 connector compatibile with STM-NUCLEO programming header, added testpoints at MDIO
Parts:
- added TP24, TP25, TP26, TP27: TestPoint, TestPoint:TestPoint_Pad_D1.0mm, symbol Connector:TestPoint
Connections:
- net MII_MDC: now also TP25.1
- net MII_MDIO: now also TP24.1
- net at U4.7 (MDC), U6.1 (B2): now also TP27.1
- net at R64.1, U4.8 (MDIO), U6.8 (B1): now also TP26.1
Changed lines of the file:
@@
 	1    0    0    -1
 $EndComp
-Text Label 2050 1750 0    50   ~ 10
+Text Label 2150 1750 0    50   ~ 10
 MII_MDIO
-Text Label 2050 1950 0    50   ~ 10
+Text Label 2150 1950 0    50   ~ 10
 MII_MDC
 $Comp
@@
 $EndComp
 Wire Wire Line
-	1750 1750 2700 1750
+	1750 1750 1800 1750
 Wire Wire Line
 	2800 1750 2800 1700
@@
 	2700 1750 2800 1750
 Wire Wire Line
-	1750 1950 2900 1950
+	1750 1950 2050 1950
 Wire Wire Line
 	2900 1950 2900 1800
@@
 	2900 1800 3250 1800
 Wire Wire Line
-	4250 1800 5300 1800
-Wire Wire Line
 	5300 1800 5300 2400
 Wire Wire Line
-	4250 1700 5400 1700
+	4250 1700 4550 1700
 Wire Wire Line
 	5400 1700 5400 2300
@@
 	8100 7400 8600 7400
 Connection ~ 8100 7400
+$Comp
+L Connector:TestPoint TP?
+U 1 1 5FA94591
+P 4550 1600
+AR Path="/5C16BF8E/5FA94591" Ref="TP?"  Part="1"
+AR Path="/5C16BF8E/5DB9B7E6/5FA94591" Ref="TP?"  Part="1"
+AR Path="/5BCEDA59/5FA94591" Ref="TP26"  Part="1"
+F 0 "TP26" H 4608 1718 50  0000 L CNN
+F 1 "TestPoint" H 4600 1650 50  0001 L CNN
+F 2 "TestPoint:TestPoint_Pad_D1.0mm" H 4750 1600 50  0001 C CNN
+F 3 "~" H 4750 1600 50  0001 C CNN
+	1    4550 1600
+	1    0    0    -1
+$EndComp
+$Comp
+L Connector:TestPoint TP?
+U 1 1 5FAA8F84
+P 4800 1600
+AR Path="/5C16BF8E/5FAA8F84" Ref="TP?"  Part="1"
+AR Path="/5C16BF8E/5DB9B7E6/5FAA8F84" Ref="TP?"  Part="1"
+AR Path="/5BCEDA59/5FAA8F84" Ref="TP27"  Part="1"
+F 0 "TP27" H 4858 1718 50  0000 L CNN
+F 1 "TestPoint" H 4850 1650 50  0001 L CNN
+F 2 "TestPoint:TestPoint_Pad_D1.0mm" H 5000 1600 50  0001 C CNN
+F 3 "~" H 5000 1600 50  0001 C CNN
+	1    4800 1600
+	1    0    0    -1
+$EndComp
+Wire Wire Line
+	4550 1600 4550 1700
+Connection ~ 4550 1700
+Wire Wire Line
+	4550 1700 5400 1700
+Wire Wire Line
+	4800 1600 4800 1800
+Wire Wire Line
+	4250 1800 4800 1800
+Connection ~ 4800 1800
+Wire Wire Line
+	4800 1800 5300 1800
+$Comp
+L Connector:TestPoint TP?
+U 1 1 5FAC8015
+P 1800 1600
+AR Path="/5C16BF8E/5FAC8015" Ref="TP?"  Part="1"
+AR Path="/5C16BF8E/5DB9B7E6/5FAC8015" Ref="TP?"  Part="1"
+AR Path="/5BCEDA59/5FAC8015" Ref="TP24"  Part="1"
+F 0 "TP24" H 1858 1718 50  0000 L CNN
+F 1 "TestPoint" H 1850 1650 50  0001 L CNN
+F 2 "TestPoint:TestPoint_Pad_D1.0mm" H 2000 1600 50  0001 C CNN
+F 3 "~" H 2000 1600 50  0001 C CNN
+	1    1800 1600
+	1    0    0    -1
+$EndComp
+$Comp
+L Connector:TestPoint TP?
+U 1 1 5FAC801B
+P 2050 1600
+AR Path="/5C16BF8E/5FAC801B" Ref="TP?"  Part="1"
+AR Path="/5C16BF8E/5DB9B7E6/5FAC801B" Ref="TP?"  Part="1"
+AR Path="/5BCEDA59/5FAC801B" Ref="TP25"  Part="1"
+F 0 "TP25" H 2108 1718 50  0000 L CNN
+F 1 "TestPoint" H 2100 1650 50  0001 L CNN
+F 2 "TestPoint:TestPoint_Pad_D1.0mm" H 2250 1600 50  0001 C CNN
+F 3 "~" H 2250 1600 50  0001 C CNN
+	1    2050 1600
+	1    0    0    -1
+$EndComp
+Wire Wire Line
+	1800 1600 1800 1750
+Connection ~ 1800 1750
+Wire Wire Line
+	1800 1750 2700 1750
+Wire Wire Line
+	2050 1600 2050 1950
 Wire Bus Line
 	8900 4500 8900 4800
@@
 Wire Bus Line
 	9300 3800 9300 4100
+Connection ~ 2050 1950
+Wire Wire Line
+	2050 1950 2900 1950
 $EndSCHEMATC

Commit message: Automated edit to move cache / rescue symbols to actual eeschem library
Results of running dissect_lib3.py, not posted here
Parts:
- J4: symbol AMC_FMC_Carrier-PcbDoc-rescue:BELFUSE_0826-1X1T-HS-F-Miscellaneous-AMC_FMC_Carrier-PcbDoc-rescue-AMC_FMC_Carrier-PcbDoc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 -> marble_misc:BELFUSE_0826-1X1T-HS-F-Miscellaneous
- OSC1: symbol AMC_FMC_Carrier-PcbDoc-rescue:Oscillator-powerMG-AMC_FMC_Carrier-PcbDoc-rescue-AMC_FMC_Carrier-PcbDoc-rescue-AMC_FMC_Ca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 -> marble_misc:Oscillator
- TP24, TP25, TP26, TP27: symbol Connector:TestPoint -> Connector_Generic:TestPoint
Changed lines of the file:
@@
 RGMII_RX_CLK
 $Comp
-L AMC_FMC_Carrier-PcbDoc-rescue:Oscillator-powerMG-AMC_FMC_Carrier-PcbDoc-rescue-AMC_FMC_Carrier-PcbDoc-rescue-AMC_FMC_Carrier-PcbDoc-rescue-AMC_FMC_Carrier-PcbDoc-rescue OSC1
+L marble_misc:Oscillator OSC1
 U 1 1 5C76AE78
 P 4600 3400
@@
 	3050 1500 3250 1500
 $Comp
-L AMC_FMC_Carrier-PcbDoc-rescue:BELFUSE_0826-1X1T-HS-F-Miscellaneous-AMC_FMC_Carrier-PcbDoc-rescue-AMC_FMC_Carrier-PcbDoc-rescue-AMC_FMC_Carrier-PcbDoc-rescue J4
+L marble_misc:BELFUSE_0826-1X1T-HS-F-Miscellaneous J4
 U 1 1 5DB81DF6
 P 12500 1900
@@
 Connection ~ 14500 4500
 $Comp
-L AMC_FMC_Carrier-PcbDoc-rescue:power_PWR_FLAG-AMC_FMC_Carrier-PcbDoc-cache-AMC_FMC_Carrier-PcbDoc-rescue-AMC_FMC_Carrier-PcbDoc-rescue-AMC_FMC_Carrier-PcbDoc-rescue #FLG0103
+L marble_misc:power_PWR_FLAG-AMC_FMC_Carrier-PcbDoc-cache #FLG0103
 U 1 1 5D15ABC3
 P 5250 6650
@@
 $EndComp
 $Comp
-L AMC_FMC_Carrier-PcbDoc-rescue:power_PWR_FLAG-AMC_FMC_Carrier-PcbDoc-cache-AMC_FMC_Carrier-PcbDoc-rescue-AMC_FMC_Carrier-PcbDoc-rescue-AMC_FMC_Carrier-PcbDoc-rescue #FLG0104
+L marble_misc:power_PWR_FLAG-AMC_FMC_Carrier-PcbDoc-cache #FLG0104
 U 1 1 5D15B1F6
 P 5250 7600
@@
 $EndComp
 $Comp
-L AMC_FMC_Carrier-PcbDoc-rescue:power_PWR_FLAG-AMC_FMC_Carrier-PcbDoc-cache-AMC_FMC_Carrier-PcbDoc-rescue-AMC_FMC_Carrier-PcbDoc-rescue-AMC_FMC_Carrier-PcbDoc-rescue #FLG0105
+L marble_misc:power_PWR_FLAG-AMC_FMC_Carrier-PcbDoc-cache #FLG0105
 U 1 1 5D15B45E
 P 14500 2000
@@
 Connection ~ 8100 7400
 $Comp
-L Connector:TestPoint TP?
+L Connector_Generic:TestPoint TP?
 U 1 1 5FA94591
 P 4550 1600
@@
 $EndComp
 $Comp
-L Connector:TestPoint TP?
+L Connector_Generic:TestPoint TP?
 U 1 1 5FAA8F84
 P 4800 1600
@@
 	4800 1800 5300 1800
 $Comp
-L Connector:TestPoint TP?
+L Connector_Generic:TestPoint TP?
 U 1 1 5FAC8015
 P 1800 1600
@@
 $EndComp
 $Comp
-L Connector:TestPoint TP?
+L Connector_Generic:TestPoint TP?
 U 1 1 5FAC801B
 P 2050 1600

Commit message: 16 warnings, 16 errors
Connections:
- net SD_IN_N: no longer names the net of U4.2 (S_INN)
- net SD_IN_P: no longer names the net of U4.1 (S_INP)
- net SD_OUT_N: no longer names the net of U4.5 (S_OUTN)
- net SD_OUT_P: no longer names the net of U4.4 (S_OUTP)
- no-connect marks 11 -> 15
Changed lines of the file:
@@
 Text Label 5950 4200 0    50   ~ 10
 PHY_RSTn
-Text Label 5350 2600 0    50   ~ 10
-SD_IN_P
-Text Label 5350 2700 0    50   ~ 10
-SD_IN_N
-Text Label 5350 2900 0    50   ~ 10
-SD_OUT_P
-Text Label 5350 3000 0    50   ~ 10
-SD_OUT_N
 Wire Wire Line
 	6000 2150 6000 2300
@@
 Wire Wire Line
 	8450 4000 9200 4000
-Wire Wire Line
-	5350 2600 6500 2600
-Wire Wire Line
-	5350 2700 6500 2700
-Wire Wire Line
-	5350 2900 6500 2900
-Wire Wire Line
-	5350 3000 6500 3000
 $Comp
 L power:GND #PWR?
@@
 Wire Wire Line
 	2050 1600 2050 1950
+Connection ~ 2050 1950
+Wire Wire Line
+	2050 1950 2900 1950
+NoConn ~ 6500 2600
+NoConn ~ 6500 2700
+NoConn ~ 6500 2900
+NoConn ~ 6500 3000
 Wire Bus Line
 	8900 4500 8900 4800
@@
 Wire Bus Line
 	9300 3800 9300 4100
-Connection ~ 2050 1950
-Wire Wire Line
-	2050 1950 2900 1950
 $EndSCHEMATC

Commit message: reduced reels with components, DDR 1V5 enable signal connected to MMC, DDR I2C pull-ups powerd from 3.3VP
Parts:
- C57: value CC0603_4.7UF_16V_10%_X5R -> CC0603_4.7UF_25V_10%_X5R; footprint CAPC1709X95N -> Capacitors SMD:CAPC1608X90N; symbol Capacitors_SMD:CC0603_4.7UF_16V_10%_X5R -> Capacitors_SMD:CC0603_4.7UF_25V_10%_X5R; Comment =Value -> 4.7uF; ComponentHeight ~~ -> (none); CreateDate 12/16/13 00:00:00 -> 11/10/14 00:00:00; Database Table Name (none) -> Capacitors SMD; Footprint Library (none) -> Capacitors SMD; Footprint Ref CAPC1709X95N -> CAPC1608X90N; LatestRevisionDate 09/16/14 00:00:00 -> 11/10/14 00:00:00; Library Name Capacitors SMD -> Capacitors.DbLib; Manufacturer Part Number CC0603_4.7UF_16V_10%_X5R -> CC0603_4.7UF_25V_10%_X5R; Manufacturer1 Example TAIYO YUDEN -> MURATA; Manufacturer1 Part Number EMK107ABJ475KA-T -> GRM188R61E475KE11D; PackageDescription ~~ -> (none); Part Number CC0603_4.7UF_16V_10%_X5R -> CC0603_4.7UF_25V_10%_X5R; Pin Count 2.0000000000000000e+00 -> 2; PressFit ~~ -> (none); Sense Comment ~~ -> (none); Status Comment ~~ -> (none); Voltage 16V -> 25V
Changed lines of the file:
@@
 $EndComp
 $Comp
-L Capacitors_SMD:CC0603_4.7UF_16V_10%_X5R C?
+L Capacitors_SMD:CC0603_4.7UF_25V_10%_X5R C?
 U 1 1 5C8E158D
 P 9550 7400
@@
 AR Path="/5BCEDA59/5C8E158D" Ref="C57"  Part="1"
 F 0 "C57" V 9600 7400 50  0000 L CNN
-F 1 "CC0603_4.7UF_16V_10%_X5R" H 9550 7140 60  0001 L CNN
-F 2 "CAPC1709X95N" H 9550 6330 60  0001 L CNN
+F 1 "CC0603_4.7UF_25V_10%_X5R" H 9550 7140 60  0001 L CNN
+F 2 "Capacitors SMD:CAPC1608X90N" H 9550 6330 60  0001 L CNN
 F 3 "\\\\cern.ch\\dfs\\Applications\\Altium\\Datasheets\\CC0603_X7R_TAIYO-YUDEN_HIGH-VALUE.pdf" H 9550 6960 60  0001 L CNN
 F 4 "4.7uF" V 9800 7400 50  0000 L CNN "~"
-F 5 "CC0603_4.7UF_16V_10%_X5R" H 9550 6870 60  0001 L CNN "Part Number"
+F 5 "CC0603_4.7UF_25V_10%_X5R" H 9550 6870 60  0001 L CNN "Part Number"
 F 6 "Capacitor - non polarized" H 9550 6780 60  0001 L CNN "Library Ref"
 F 7 "SchLib\\Capacitors.SchLib" H 9550 6690 60  0001 L CNN "Library Path"
-F 8 "=Value" H 9550 6600 60  0001 L CNN "Comment"
+F 8 "4.7uF" H 9550 6600 60  0001 L CNN "Comment"
 F 9 "Standard" H 9550 6510 60  0001 L CNN "Component Kind"
 F 10 "Standard" H 9550 6420 60  0001 L CNN "Component Type"
-F 11 "2.0000000000000000e+00" H 9550 6240 60  0001 L CNN "Pin Count"
+F 11 "2" H 9550 6240 60  0001 L CNN "Pin Count"
 F 12 "PcbLib\\Capacitors SMD.PcbLib" H 9550 6150 60  0001 L CNN "Footprint Path"
-F 13 "CAPC1709X95N" H 9550 6060 60  0001 L CNN "Footprint Ref"
-F 14 "~~" H 9550 5970 60  0001 L CNN "PackageDescription"
+F 13 "CAPC1608X90N" H 9550 6060 60  0001 L CNN "Footprint Ref"
+F 14 " " H 9550 5970 60  0001 L CNN "PackageDescription"
 F 15 "4.7uF" H 9550 5880 60  0001 L CNN "Val"
 F 16 "None" H 9550 5790 60  0001 L CNN "Status"
-F 17 "~~" H 9550 5700 60  0001 L CNN "Status Comment"
-F 18 "16V" H 9550 5610 60  0001 L CNN "Voltage"
+F 17 " " H 9550 5700 60  0001 L CNN "Status Comment"
+F 18 "25V" H 9550 5610 60  0001 L CNN "Voltage"
 F 19 "X5R" H 9550 5520 60  0001 L CNN "TC"
 F 20 "±10%" H 9550 5430 60  0001 L CNN "Tolerance"
 F 21 "SMD Multilayer Chip Ceramic Capacitor" H 9550 5340 60  0001 L CNN "Part Description"
 F 22 "GENERIC" H 9550 5250 60  0001 L CNN "Manufacturer"
-F 23 "CC0603_4.7UF_16V_10%_X5R" H 9550 5160 60  0001 L CNN "Manufacturer Part Number"
+F 23 "CC0603_4.7UF_25V_10%_X5R" H 9550 5160 60  0001 L CNN "Manufacturer Part Number"
 F 24 "0603" H 9550 5070 60  0001 L CNN "Case"
 F 25 "Yes" H 9550 4980 60  0001 L CNN "Mounted"
 F 26 "No" H 9550 4890 60  0001 L CNN "Socket"
 F 27 "Yes" H 9550 4800 60  0001 L CNN "SMD"
-F 28 "~~" H 9550 4710 60  0001 L CNN "PressFit"
+F 28 " " H 9550 4710 60  0001 L CNN "PressFit"
 F 29 "No" H 9550 4620 60  0001 L CNN "Sense"
-F 30 "~~" H 9550 4530 60  0001 L CNN "Sense Comment"
-F 31 "~~" H 9550 4440 60  0001 L CNN "ComponentHeight"
-F 32 "TAIYO YUDEN" H 9550 4350 60  0001 L CNN "Manufacturer1 Example"
-F 33 "EMK107ABJ475KA-T" H 9550 4260 60  0001 L CNN "Manufacturer1 Part Number"
+F 30 " " H 9550 4530 60  0001 L CNN "Sense Comment"
+F 31 " " H 9550 4440 60  0001 L CNN "ComponentHeight"
+F 32 "MURATA" H 9550 4350 60  0001 L CNN "Manufacturer1 Example"
+F 33 "GRM188R61E475KE11D" H 9550 4260 60  0001 L CNN "Manufacturer1 Part Number"
 F 34 "0.95mm" H 9550 4170 60  0001 L CNN "Manufacturer1 ComponentHeight"
 F 35 "\\\\cern.ch\\dfs\\Applications\\Altium\\Datasheets\\CC0603_X7R_TAIYO-YUDEN_HIGH-VALUE.pdf" H 9550 4080 60  0001 L CNN "HelpURL"
 F 36 "CERN DEM JLC" H 9550 3990 60  0001 L CNN "Author"
-F 37 "12/16/13 00:00:00" H 9550 3900 60  0001 L CNN "CreateDate"
-F 38 "09/16/14 00:00:00" H 9550 3810 60  0001 L CNN "LatestRevisionDate"
-F 39 "Capacitors SMD" H 9550 3720 60  0001 L CNN "Library Name"
+F 37 "11/10/14 00:00:00" H 9550 3900 60  0001 L CNN "CreateDate"
+F 38 "11/10/14 00:00:00" H 9550 3810 60  0001 L CNN "LatestRevisionDate"
+F 39 "Capacitors.DbLib" H 9550 3720 60  0001 L CNN "Library Name"
 F 40 "This work is licensed under the Creative Commons CC-BY-SA 4.0 License. To the extent that circuit schematics that use Licensed Material can be considered to be ‘Adapted Material’, then the copyright holder waives article 3.b of the license with respect to these schematics." H 9550 3630 60  0001 L CNN "License"
+F 41 "Capacitors SMD" H 9550 7400 50  0001 C CNN "Database Table Name"
+F 42 "Capacitors SMD" H 9550 7400 50  0001 C CNN "Footprint Library"
 	1    9550 7400
 	0    1    1    0
