File: ETH_PHY.sch (KiCad schematic (older format))
At the start: 48 parts, among them J4 BELFUSE_0826-1X1T-GH-F, U4 88E1512-A0-NNP2I000, U6 TXS0102DCUR

Commit message: Flag duplicate generic parts in BOM, and refresh a few cap instances from library to reduce such dups
Parts:
- C374, C375: footprint CAPC1005X55N -> Capacitors SMD:CAPC1005X55N; Comment =Value -> 100pF; ComponentHeight ~~ -> (none); Database Table Name (none) -> Capacitors SMD; Footprint Library (none) -> Capacitors SMD; HelpURL \\\\cern.ch\\dfs\\Applications\\Altium\\Datasheets\\CC0805_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 -> (none); Library Name Capacitors SMD -> Capacitors.DbLib; PackageDescription ~~ -> (none); Pin Count 2.0000000000000000e+00 -> 2; PressFit ~~ -> (none); Sense Comment ~~ -> (none); Status Comment ~~ -> (none)
Changed lines of the file:
@@
 F 0 "C375" V 3704 3460 50  0000 L CNN
 F 1 "CC0402_100PF_50V_5%_C0G" H 3600 3090 60  0001 L CNN
-F 2 "CAPC1005X55N" H 3600 2280 60  0001 L CNN
-F 3 "\\\\cern.ch\\dfs\\Applications\\Altium\\Datasheets\\CC0805_C0G_KEMET_(Commercial Grade).pdf" H 3600 2910 60  0001 L CNN
+F 2 "Capacitors SMD:CAPC1005X55N" H 3600 2280 60  0001 L CNN
+F 3 " " H 3600 2910 60  0001 L CNN
 F 4 "100pF" V 3795 3460 50  0000 L CNN "~"
 F 5 "CC0402_100PF_50V_5%_C0G" H 3600 2820 60  0001 L CNN "Part Number"
 F 6 "Capacitor - non polarized" H 3600 2730 60  0001 L CNN "Library Ref"
 F 7 "SchLib\\Capacitors.SchLib" H 3600 2640 60  0001 L CNN "Library Path"
-F 8 "=Value" H 3600 2550 60  0001 L CNN "Comment"
+F 8 "100pF" H 3600 2550 60  0001 L CNN "Comment"
 F 9 "Standard" H 3600 2460 60  0001 L CNN "Component Kind"
 F 10 "Standard" H 3600 2370 60  0001 L CNN "Component Type"
-F 11 "2.0000000000000000e+00" H 3600 2190 60  0001 L CNN "Pin Count"
+F 11 "2" H 3600 2190 60  0001 L CNN "Pin Count"
 F 12 "PcbLib\\Capacitors SMD.PcbLib" H 3600 2100 60  0001 L CNN "Footprint Path"
 F 13 "CAPC1005X55N" H 3600 2010 60  0001 L CNN "Footprint Ref"
-F 14 "~~" H 3600 1920 60  0001 L CNN "PackageDescription"
+F 14 " " H 3600 1920 60  0001 L CNN "PackageDescription"
 F 15 "100pF" H 3600 1830 60  0001 L CNN "Val"
 F 16 "Preferred" H 3600 1740 60  0001 L CNN "Status"
-F 17 "~~" H 3600 1650 60  0001 L CNN "Status Comment"
+F 17 " " H 3600 1650 60  0001 L CNN "Status Comment"
 F 18 "50V" H 3600 1560 60  0001 L CNN "Voltage"
 F 19 "C0G/NP0" H 3600 1470 60  0001 L CNN "TC"
@@
 F 26 "No" H 3600 840 60  0001 L CNN "Socket"
 F 27 "Yes" H 3600 750 60  0001 L CNN "SMD"
-F 28 "~~" H 3600 660 60  0001 L CNN "PressFit"
+F 28 " " H 3600 660 60  0001 L CNN "PressFit"
 F 29 "No" H 3600 570 60  0001 L CNN "Sense"
-F 30 "~~" H 3600 480 60  0001 L CNN "Sense Comment"
-F 31 "~~" H 3600 390 60  0001 L CNN "ComponentHeight"
+F 30 " " H 3600 480 60  0001 L CNN "Sense Comment"
+F 31 " " H 3600 390 60  0001 L CNN "ComponentHeight"
 F 32 "KEMET" H 3600 300 60  0001 L CNN "Manufacturer1 Example"
 F 33 "C0402C101J5GACTU" H 3600 210 60  0001 L CNN "Manufacturer1 Part Number"
 F 34 "0.55mm" H 3600 120 60  0001 L CNN "Manufacturer1 ComponentHeight"
-F 35 "\\\\cern.ch\\dfs\\Applications\\Altium\\Datasheets\\CC0805_C0G_KEMET_(Commercial Grade).pdf" H 3600 30  60  0001 L CNN "HelpURL"
-F 36 "CERN DEM JLC" H 3600 -60 60  0001 L CNN "Author"
-F 37 "12/03/07 00:00:00" H 3600 -150 60  0001 L CNN "CreateDate"
-F 38 "04/22/15 00:00:00" H 3600 -240 60  0001 L CNN "LatestRevisionDate"
-F 39 "Capacitors SMD" H 3600 -330 60  0001 L CNN "Library Name"
-F 40 "This work is licensed under the Creative Commons CC-BY-SA 4.0 License. To the extent that circuit schematics that use Licensed Material can be considered to be ‘Adapted Material’, then the copyright holder waives article 3.b of the license with respect to these schematics." H 3600 -420 60  0001 L CNN "License"
+F 35 "CERN DEM JLC" H 3600 -60 60  0001 L CNN "Author"
+F 36 "12/03/07 00:00:00" H 3600 -150 60  0001 L CNN "CreateDate"
+F 37 "04/22/15 00:00:00" H 3600 -240 60  0001 L CNN "LatestRevisionDate"
+F 38 "Capacitors SMD" H 7100 3180 50  0001 L CNN "Database Table Name"
+F 39 "Capacitors.DbLib" H 7100 3105 50  0001 L CNN "Library Name"
+F 40 "Capacitors SMD" H 7100 3030 50  0001 L CNN "Footprint Library"
+F 41 "This work is licensed under the Creative Commons CC-BY-SA 4.0 License. To the extent that circuit schematics that use Licensed Material can be considered to be ‘Adapted Material’, then the copyright holder waives article 3.b of the license with respect to these schematics." H 3600 -420 60  0001 L CNN "License"
 	1    3600 3350
 	0    1    1    0
@@
 F 0 "C374" H 3700 3100 50  0000 L CNN
 F 1 "CC0402_100PF_50V_5%_C0G" H 3600 2990 60  0001 L CNN
-F 2 "CAPC1005X55N" H 3600 2180 60  0001 L CNN
-F 3 "\\\\cern.ch\\dfs\\Applications\\Altium\\Datasheets\\CC0805_C0G_KEMET_(Commercial Grade).pdf" H 3600 2810 60  0001 L CNN
+F 2 "Capacitors SMD:CAPC1005X55N" H 3600 2180 60  0001 L CNN
+F 3 " " H 3600 2810 60  0001 L CNN
 F 4 "100pF" H 3650 3400 50  0000 L CNN "~"
 F 5 "CC0402_100PF_50V_5%_C0G" H 3600 2720 60  0001 L CNN "Part Number"
 F 6 "Capacitor - non polarized" H 3600 2630 60  0001 L CNN "Library Ref"
 F 7 "SchLib\\Capacitors.SchLib" H 3600 2540 60  0001 L CNN "Library Path"
-F 8 "=Value" H 3600 2450 60  0001 L CNN "Comment"
+F 8 "100pF" H 3600 2450 60  0001 L CNN "Comment"
 F 9 "Standard" H 3600 2360 60  0001 L CNN "Component Kind"
 F 10 "Standard" H 3600 2270 60  0001 L CNN "Component Type"
-F 11 "2.0000000000000000e+00" H 3600 2090 60  0001 L CNN "Pin Count"
+F 11 "2" H 3600 2090 60  0001 L CNN "Pin Count"
 F 12 "PcbLib\\Capacitors SMD.PcbLib" H 3600 2000 60  0001 L CNN "Footprint Path"
 F 13 "CAPC1005X55N" H 3600 1910 60  0001 L CNN "Footprint Ref"
-F 14 "~~" H 3600 1820 60  0001 L CNN "PackageDescription"
+F 14 " " H 3600 1820 60  0001 L CNN "PackageDescription"
 F 15 "100pF" H 3600 1730 60  0001 L CNN "Val"
 F 16 "Preferred" H 3600 1640 60  0001 L CNN "Status"
-F 17 "~~" H 3600 1550 60  0001 L CNN "Status Comment"
+F 17 " " H 3600 1550 60  0001 L CNN "Status Comment"
 F 18 "50V" H 3600 1460 60  0001 L CNN "Voltage"
 F 19 "C0G/NP0" H 3600 1370 60  0001 L CNN "TC"
@@
 F 26 "No" H 3600 740 60  0001 L CNN "Socket"
 F 27 "Yes" H 3600 650 60  0001 L CNN "SMD"
-F 28 "~~" H 3600 560 60  0001 L CNN "PressFit"
+F 28 " " H 3600 560 60  0001 L CNN "PressFit"
 F 29 "No" H 3600 470 60  0001 L CNN "Sense"
-F 30 "~~" H 3600 380 60  0001 L CNN "Sense Comment"
-F 31 "~~" H 3600 290 60  0001 L CNN "ComponentHeight"
+F 30 " " H 3600 380 60  0001 L CNN "Sense Comment"
+F 31 " " H 3600 290 60  0001 L CNN "ComponentHeight"
 F 32 "KEMET" H 3600 200 60  0001 L CNN "Manufacturer1 Example"
 F 33 "C0402C101J5GACTU" H 3600 110 60  0001 L CNN "Manufacturer1 Part Number"
 F 34 "0.55mm" H 3600 20  60  0001 L CNN "Manufacturer1 ComponentHeight"
-F 35 "\\\\cern.ch\\dfs\\Applications\\Altium\\Datasheets\\CC0805_C0G_KEMET_(Commercial Grade).pdf" H 3600 -70 60  0001 L CNN "HelpURL"
-F 36 "CERN DEM JLC" H 3600 -160 60  0001 L CNN "Author"
-F 37 "12/03/07 00:00:00" H 3600 -250 60  0001 L CNN "CreateDate"
-F 38 "04/22/15 00:00:00" H 3600 -340 60  0001 L CNN "LatestRevisionDate"
-F 39 "Capacitors SMD" H 3600 -430 60  0001 L CNN "Library Name"
-F 40 "This work is licensed under the Creative Commons CC-BY-SA 4.0 License. To the extent that circuit schematics that use Licensed Material can be considered to be ‘Adapted Material’, then the copyright holder waives article 3.b of the license with respect to these schematics." H 3600 -520 60  0001 L CNN "License"
+F 35 "CERN DEM JLC" H 3600 -160 60  0001 L CNN "Author"
+F 36 "12/03/07 00:00:00" H 3600 -250 60  0001 L CNN "CreateDate"
+F 37 "04/22/15 00:00:00" H 3600 -340 60  0001 L CNN "LatestRevisionDate"
+F 38 "Capacitors.DbLib" H 3600 -430 60  0001 L CNN "Library Name"
+F 39 "This work is licensed under the Creative Commons CC-BY-SA 4.0 License. To the extent that circuit schematics that use Licensed Material can be considered to be ‘Adapted Material’, then the copyright holder waives article 3.b of the license with respect to these schematics." H 3600 -520 60  0001 L CNN "License"
+F 40 "Capacitors SMD" H 3600 3250 50  0001 C CNN "Database Table Name"
+F 41 "Capacitors SMD" H 3600 3250 50  0001 C CNN "Footprint Library"
 	1    3600 3250
 	-1   0    0    1

Commit message: Tweak Resistor attributes to improve BOM output
Clean according to KiBoM and non_generic.py
Still a metric ton of buried inconsistencies
Parts:
- R156, R67: footprint RESC1005X40N -> Resistors SMD:RESC1005X40N; Comment =Value -> 240
Changed lines of the file:
@@
 F 0 "R67" H 9000 4950 50  0000 C CNN
 F 1 "R0402_240R_1%_0.0625W_100PPM" H 8650 4690 60  0001 L CNN
-F 2 "RESC1005X40N" H 8650 3880 60  0001 L CNN
+F 2 "Resistors SMD:RESC1005X40N" H 8650 3880 60  0001 L CNN
 F 3 "\\\\cern.ch\\dfs\\Applications\\Altium\\Datasheets\\R0402_Phycomp_RC0402.pdf" H 8650 4510 60  0001 L CNN
 F 4 "240" H 8600 4950 50  0000 C CNN "~"
@@
 F 6 "Resistor - 1%" H 8650 4330 60  0001 L CNN "Library Ref"
 F 7 "SchLib\\Resistors.SchLib" H 8650 4240 60  0001 L CNN "Library Path"
-F 8 "=Value" H 8650 4150 60  0001 L CNN "Comment"
+F 8 "240" H 8650 4150 60  0001 L CNN "Comment"
 F 9 "Standard" H 8650 4060 60  0001 L CNN "Component Kind"
 F 10 "Standard" H 8650 3970 60  0001 L CNN "Component Type"
@@
 F 0 "R156" H 9000 5050 50  0000 C CNN
 F 1 "R0402_240R_1%_0.0625W_100PPM" H 8650 4790 60  0001 L CNN
-F 2 "RESC1005X40N" H 8650 3980 60  0001 L CNN
+F 2 "Resistors SMD:RESC1005X40N" H 8650 3980 60  0001 L CNN
 F 3 "\\\\cern.ch\\dfs\\Applications\\Altium\\Datasheets\\R0402_Phycomp_RC0402.pdf" H 8650 4610 60  0001 L CNN
 F 4 "240" H 8600 5050 50  0000 C CNN "~"
@@
 F 6 "Resistor - 1%" H 8650 4430 60  0001 L CNN "Library Ref"
 F 7 "SchLib\\Resistors.SchLib" H 8650 4340 60  0001 L CNN "Library Path"
-F 8 "=Value" H 8650 4250 60  0001 L CNN "Comment"
+F 8 "240" H 8650 4250 60  0001 L CNN "Comment"
 F 9 "Standard" H 8650 4160 60  0001 L CNN "Component Kind"
 F 10 "Standard" H 8650 4070 60  0001 L CNN "Component Type"
