File: FPGA_14_15.sch (KiCad schematic (older format))
At the start: 24 parts, among them SW1 SW_DIP_x01, U1 XC7K160T-2FFG676C, U11 SN74LVC1G125DCKT, U30 S25FL128SAGMFIR01, U52 TCA9517DGKR, U53 TXB0108PW

Commit message: Automated edit to move cache / rescue symbols to actual eeschem library
Results of running dissect_lib3.py, not posted here
Parts:
- SW1: symbol AMC_FMC_Carrier-PcbDoc-rescue:SW_DIP_x01-Switch-AMC_FMC_Carrier-PcbDoc-rescue-AMC_FMC_Carrier-PcbDoc-rescue-AMC_FMC_Car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 -> marble_misc:SW_DIP_x01-Switch
- U1: symbol FPGA_Xilinx_Kintex7:XC7K160T-FFG676 -> marble_misc:XC7K160T-FFG676
- U11: symbol AMC_FMC_Carrier-PcbDoc-rescue:SN74LVC1G125DCKT-Standard_Logic-AMC_FMC_Carrier-PcbDoc-rescue-AMC_FMC_Carrier-PcbDoc-resc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 -> marble_misc:SN74LVC1G125DCKT-Standard_Logic
- U30: symbol AMC_FMC_Carrier-PcbDoc-rescue:S25FL128SAGMFIR01-powerMG-AMC_FMC_Carrier-PcbDoc-rescue-AMC_FMC_Carrier-PcbDoc-rescue-AMC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 -> marble_misc:S25FL128SAGMFIR01
Changed lines of the file:
@@
 	6900 2300 6900 2200
 $Comp
-L AMC_FMC_Carrier-PcbDoc-rescue:S25FL128SAGMFIR01-powerMG-AMC_FMC_Carrier-PcbDoc-rescue-AMC_FMC_Carrier-PcbDoc-rescue-AMC_FMC_Carrier-PcbDoc-rescue-AMC_FMC_Carrier-PcbDoc-rescue U30
+L marble_misc:S25FL128SAGMFIR01 U30
 U 1 1 5C40DA57
 P 13400 850
@@
 $EndComp
 $Comp
-L AMC_FMC_Carrier-PcbDoc-rescue:S25FL128SAGMFIR01-powerMG-AMC_FMC_Carrier-PcbDoc-rescue-AMC_FMC_Carrier-PcbDoc-rescue-AMC_FMC_Carrier-PcbDoc-rescue-AMC_FMC_Carrier-PcbDoc-rescue U30
+L marble_misc:S25FL128SAGMFIR01 U30
 U 2 1 5C40DA9C
 P 14700 850
@@
 	12650 1650 13200 1650
 $Comp
-L AMC_FMC_Carrier-PcbDoc-rescue:SW_DIP_x01-Switch-AMC_FMC_Carrier-PcbDoc-rescue-AMC_FMC_Carrier-PcbDoc-rescue-AMC_FMC_Carrier-PcbDoc-rescue-AMC_FMC_Carrier-PcbDoc-rescue SW1
+L marble_misc:SW_DIP_x01-Switch SW1
 U 1 1 5C881CE2
 P 13300 3000
@@
 $EndComp
 $Comp
-L AMC_FMC_Carrier-PcbDoc-rescue:SN74LVC1G125DCKT-Standard_Logic-AMC_FMC_Carrier-PcbDoc-rescue-AMC_FMC_Carrier-PcbDoc-rescue-AMC_FMC_Carrier-PcbDoc-rescue-AMC_FMC_Carrier-PcbDoc-rescue U11
+L marble_misc:SN74LVC1G125DCKT-Standard_Logic U11
 U 1 1 5C4235B4
 P 14150 2800
@@
 Connection ~ 12200 3600
 $Comp
-L FPGA_Xilinx_Kintex7:XC7K160T-FFG676 U?
+L marble_misc:XC7K160T-FFG676 U?
 U 2 1 5EE5BCB0
 P 8500 5200
@@
 $EndComp
 $Comp
-L power2:+3.3P #PWR?
+L power:+3.3P #PWR?
 U 1 1 6343FC7E
 P 2550 3600

Commit message: 16 warnings, 16 errors
Connections:
- no-connect marks 7 -> 19
Changed lines of the file:
@@
 $EndComp
 Connection ~ 3900 3700
+NoConn ~ 3400 6250
+NoConn ~ 3400 6450
+NoConn ~ 3400 6650
+NoConn ~ 3400 6850
+NoConn ~ 2400 6250
+NoConn ~ 2400 6450
+NoConn ~ 2400 6650
+NoConn ~ 2400 6850
+NoConn ~ 3900 3500
+NoConn ~ 10500 3700
+NoConn ~ 10500 3800
+NoConn ~ 10500 3900
 Wire Bus Line
 	14750 7100 14750 7850

Commit message: Tweak Resistor attributes to improve BOM output
Clean according to KiBoM and non_generic.py
Still a metric ton of buried inconsistencies
Parts:
- R7: footprint Resistors SMD:RESC1005X40N -> RESC1005X40N; Comment 0 -> =Value; Library Name Resistors.DbLib -> Resistors SMD
Changed lines of the file:
@@
 F 0 "R7" H 2250 5447 50  0000 C CNN
 F 1 "R0402_0R_JUMPER" H 2100 5055 50  0001 L CNN
-F 2 "Resistors SMD:RESC1005X40N" H 2100 4980 50  0001 L CNN
+F 2 "RESC1005X40N" H 2100 4980 50  0001 L CNN
 F 3 " " H 2100 4905 50  0001 L CNN
 F 4 "0" H 2250 5356 50  0000 C CNN "Val"
@@
 F 6 "Resistor" H 2100 4755 50  0001 L CNN "Library Ref"
 F 7 "SchLib\\Resistors.SchLib" H 2100 4680 50  0001 L CNN "Library Path"
-F 8 "0" H 2100 4605 50  0001 L CNN "Comment"
+F 8 "=Value" H 2100 4605 50  0001 L CNN "Comment"
 F 9 "Standard" H 2100 4530 50  0001 L CNN "Component Kind"
 F 10 "Standard" H 2100 4455 50  0001 L CNN "Component Type"
@@
 F 37 "10/17/12 00:00:00" H 2100 2430 50  0001 L CNN "LatestRevisionDate"
 F 38 "Resistors SMD" H 2100 2355 50  0001 L CNN "Database Table Name"
-F 39 "Resistors.DbLib" H 2100 2280 50  0001 L CNN "Library Name"
+F 39 "Resistors SMD" H 2100 2280 50  0001 L CNN "Library Name"
 F 40 "Resistors SMD" H 2100 2205 50  0001 L CNN "Footprint Library"
 F 41 "This work is licensed under the Creative Commons CC-BY-SA 4.0 License. To the extent that circuit schematics that use Licensed Material can be considered to be ‘Adapted Material’, then the copyright holder waives article 3.b of the license with respect to these schematics." H 2100 2130 50  0001 L CNN "License"

Commit message: Progress on the BOM
Fill in many Manufacturer fields
Move dnf flag from Y1 to Y2
Manufacturer Part Number changes for Y1 D8 J6 J9
Parts:
- SW1: Manufacturer (none) -> OMRON
- U30: Manufacturer (none) -> INFINEON
Changed lines of the file:
@@
 F 2 "ICs And Semiconductors SMD:SOIC127P1030X265-16N" H 13400 850 50  0001 C CNN
 F 3 "" H 13400 850 50  0001 C CNN
-F 4 "S25FL128SAGMFIR01" H 13400 850 50  0001 C CNN "Manufacturer Part Number"
+F 4 "INFINEON" H 13400 850 50  0001 C CNN "Manufacturer"
+F 5 "S25FL128SAGMFIR01" H 13400 850 50  0001 C CNN "Manufacturer Part Number"
 	1    13400 850
 	1    0    0    -1
@@
 F 3 "" H 14700 850 50  0001 C CNN
 F 4 "S25FL128SAGMFIR01" H 14700 850 50  0001 C CNN "Manufacturer Part Number"
+F 5 "INFINEON" H 14700 850 50  0001 C CNN "Manufacturer"
 	2    14700 850
 	1    0    0    -1
@@
 F 3 "" H 13300 3000 50  0001 C CNN
 F 4 "A6SN-1101" H 13300 3000 50  0001 C CNN "Manufacturer Part Number"
+F 5 "OMRON" H 13300 3000 50  0001 C CNN "Manufacturer"
 	1    13300 3000
 	-1   0    0    -1

Commit message: More progress on the BOM
Fill in more Manufacturer and Manufacturer Part Number
Manufacturer Part Number changes for D6 D7
Parts:
- U1: Manufacturer (none) -> XILINX; Manufacturer Part Number (none) -> XC7K160T-2FFG676C
Changed lines of the file:
@@
 F 2 "ICs And Semiconductors SMD_BGA:BGA676C100P26X26_2700X2700X260" H 8500 5200 50  0001 C CNN
 F 3 "" H 8500 5200 50  0000 C CNN
+F 4 "XILINX" H 8500 5200 50  0001 C CNN "Manufacturer"
+F 5 "XC7K160T-2FFG676C" H 8500 5200 50  0001 C CNN "Manufacturer Part Number"
 	2    8500 5200
 	-1   0    0    -1

Commit message: Adjust BOM details
Fix spelling of "config" attribute for SW2
Part number changes:
FC68148 (DC-10A) to FC68148
TXB0108PW to TXB0108PWR
XRP7724ILBTR-F to XRP7724ILB-F
Parts:
- U53: Manufacturer Part Number TXB0108PW -> TXB0108PWR
Changed lines of the file:
@@
 F 13 "8-Bit Bidirectional Voltage-Level Translator with Automatic Direction Sensing and ±15kV ESD Protection" H 2600 1975 50  0001 L CNN "Part Description"
 F 14 "TEXAS INSTRUMENTS" H 2600 1900 50  0001 L CNN "Manufacturer"
-F 15 "TXB0108PW" H 2600 1825 50  0001 L CNN "Manufacturer Part Number"
+F 15 "TXB0108PWR" H 2600 1825 50  0001 L CNN "Manufacturer Part Number"
 F 16 "20" H 2600 1750 50  0001 L CNN "Pin Count"
 F 17 "TSSOP20" H 2600 1675 50  0001 L CNN "Case"

Commit message: Stop saying that 2-pin devices have "2.0000000000000000e+00" pins
Parts:
- C20, C21, C318, C319, C38, C39, C78: Pin Count 2.0000000000000000e+00 -> 2
Changed lines of the file:
@@
 F 9 "Standard" H 15250 2710 60  0001 L CNN "Component Kind"
 F 10 "Standard" H 15250 2620 60  0001 L CNN "Component Type"
-F 11 "2.0000000000000000e+00" H 15250 2440 60  0001 L CNN "Pin Count"
+F 11 "2" H 15250 2440 60  0001 L CNN "Pin Count"
 F 12 "PcbLib\\Capacitors SMD.PcbLib" H 15250 2350 60  0001 L CNN "Footprint Path"
 F 13 "CAPC0603X33N" H 15250 2260 60  0001 L CNN "Footprint Ref"
@@
 F 9 "Standard" H 12750 1110 60  0001 L CNN "Component Kind"
 F 10 "Standard" H 12750 1020 60  0001 L CNN "Component Type"
-F 11 "2.0000000000000000e+00" H 12750 840 60  0001 L CNN "Pin Count"
+F 11 "2" H 12750 840 60  0001 L CNN "Pin Count"
 F 12 "PcbLib\\Capacitors SMD.PcbLib" H 12750 750 60  0001 L CNN "Footprint Path"
 F 13 "CAPC0603X33N" H 12750 660 60  0001 L CNN "Footprint Ref"
@@
 F 9 "Standard" H 13150 1110 60  0001 L CNN "Component Kind"
 F 10 "Standard" H 13150 1020 60  0001 L CNN "Component Type"
-F 11 "2.0000000000000000e+00" H 13150 840 60  0001 L CNN "Pin Count"
+F 11 "2" H 13150 840 60  0001 L CNN "Pin Count"
 F 12 "PcbLib\\Capacitors SMD.PcbLib" H 13150 750 60  0001 L CNN "Footprint Path"
 F 13 "CAPC0603X33N" H 13150 660 60  0001 L CNN "Footprint Ref"
@@
 F 9 "Standard" H 3900 2860 60  0001 L CNN "Component Kind"
 F 10 "Standard" H 3900 2770 60  0001 L CNN "Component Type"
-F 11 "2.0000000000000000e+00" H 3900 2590 60  0001 L CNN "Pin Count"
+F 11 "2" H 3900 2590 60  0001 L CNN "Pin Count"
 F 12 "PcbLib\\Capacitors SMD.PcbLib" H 3900 2500 60  0001 L CNN "Footprint Path"
 F 13 "CAPC0603X33N" H 3900 2410 60  0001 L CNN "Footprint Ref"
@@
 F 9 "Standard" H 2550 2760 60  0001 L CNN "Component Kind"
 F 10 "Standard" H 2550 2670 60  0001 L CNN "Component Type"
-F 11 "2.0000000000000000e+00" H 2550 2490 60  0001 L CNN "Pin Count"
+F 11 "2" H 2550 2490 60  0001 L CNN "Pin Count"
 F 12 "PcbLib\\Capacitors SMD.PcbLib" H 2550 2400 60  0001 L CNN "Footprint Path"
 F 13 "CAPC0603X33N" H 2550 2310 60  0001 L CNN "Footprint Ref"
@@
 F 9 "Standard" H 2050 6210 60  0001 L CNN "Component Kind"
 F 10 "Standard" H 2050 6120 60  0001 L CNN "Component Type"
-F 11 "2.0000000000000000e+00" H 2050 5940 60  0001 L CNN "Pin Count"
+F 11 "2" H 2050 5940 60  0001 L CNN "Pin Count"
 F 12 "PcbLib\\Capacitors SMD.PcbLib" H 2050 5850 60  0001 L CNN "Footprint Path"
 F 13 "CAPC0603X33N" H 2050 5760 60  0001 L CNN "Footprint Ref"
@@
 F 9 "Standard" H 3550 6210 60  0001 L CNN "Component Kind"
 F 10 "Standard" H 3550 6120 60  0001 L CNN "Component Type"
-F 11 "2.0000000000000000e+00" H 3550 5940 60  0001 L CNN "Pin Count"
+F 11 "2" H 3550 5940 60  0001 L CNN "Pin Count"
 F 12 "PcbLib\\Capacitors SMD.PcbLib" H 3550 5850 60  0001 L CNN "Footprint Path"
 F 13 "CAPC0603X33N" H 3550 5760 60  0001 L CNN "Footprint Ref"

Commit message: Convert "~" and "~~" in .sch and .lib files to " "
cf. commit ef029e49 in Marble-Mini, May 21 2020
Parts:
- C20, C21, C318, C319, C38, C39, C78: ComponentHeight ~~ -> (none); PackageDescription ~~ -> (none); PressFit ~~ -> (none); Sense Comment ~~ -> (none); Status Comment ~~ -> (none)
- R1, R2, R221, R222, R223: ComponentHeight ~~ -> (none); PackageDescription ~~ -> (none); Sense Comment ~~ -> (none); Status Comment ~~ -> (none); Voltage ~~ -> (none)
- R209, R210, R224, R225, R227: ComponentHeight ~~ -> (none); PackageDescription ~~ -> (none); Power ~~ -> (none); Sense Comment ~~ -> (none); Status Comment ~~ -> (none); TC ~~ -> (none); Tolerance ~~ -> (none); Voltage ~~ -> (none)
- U11: ComponentLink1Description ~~ -> (none); ComponentLink1URL ~~ -> (none); ComponentLink2Description ~~ -> (none); ComponentLink2URL ~~ -> (none); Sense Comment ~~ -> (none); Status ~~ -> (none); Status Comment ~~ -> (none)
