File: Power.sch (KiCad schematic (older format))
At the start: 76 parts, among them J1 CLIFF_FC68148(DC-10A), J19 TE_641119-2, Q1 BC857BV, Q15 BC857BV, Q16 SI4425DDY-T1-GE3, Q2 SI4425DDY-T1-GE3, Q22 BC857BV, Q23 SI4425DDY-T1-GE3, Q25 Si2315BDS-T1-E3, Q4 SI4425DDY-T1-GE3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

Commit message: Unify CC0402_100NF part numbers
CC0402_100NF_16V_10%_X5R and CC0402_100NF_25V_10%_X7R_YUDEN_TMK105B7104KVHF
become CC0402_100NF_25V_10%_X5R, matching Marble-Mini
generic_subst converts this to Samsung CL05A104KA5NNNC
15 refids: C5 C61 C128 C130 C131 C134 C135 C137 C140 C147 C148 C149 C150 C362 C363
Parts:
- C128, C130, C131, C134, C135: value CC0402_100NF_25V_10%_X7R_YUDEN_TMK105B7104KVHF -> CC0402_100NF_25V_10%_X5R; footprint Capacitors SMD:CAPC1005X55N -> Marble:CAPC1005X55N; symbol Capacitors_SMD:CC0402_100NF_25V_10%_X7R_YUDEN_TMK105B7104KVHF -> Capacitors_SMD:CC0402_100NF_25V_10%_X5R; ComponentHeight 0.55mm -> (none); CreateDate 05/10/17 00:00:00 -> 12/10/13 00:00:00; LatestRevisionDate 05/10/17 00:00:00 -> 05/25/20 00:00:00; Library Name Capacitors.DbLib -> Capacitors SMD; Manufacturer TAIYO YUDEN -> GENERIC; Manufacturer Part Number TMK105B7104KVHF -> CC0402_100NF_25V_10%_X5R; Manufacturer1 ComponentHeight (none) -> 0.55mm; Manufacturer1 Example (none) -> Samsung; Manufacturer1 Part Number (none) -> CL05A104KA5NNNC; Part Description SMD Multilayer Chip Ceramic Capacitor (High Dielectric Type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 -> SMD Multilayer Chip Ceramic Capacitor; Part Number CC0402_100NF_25V_10%_X7R_YUDEN_TMK105B7104KVHF -> CC0402_100NF_25V_10%_X5R; Status Not Recommended -> None; TC X7R -> X5R

Commit message: fixed drc errors, removed Q25, more test points
Parts:
- removed Q15: BC857BV, SOTFL50P160X60-6N, symbol Transistors:BC857BV
- removed Q25: Si2315BDS-T1-E3, ICs And Semiconductors SMD:SOT95P237X112-3N, symbol Transistors:Si2315BDS-T1-E3
- removed R171: R0402_10K_1%_0.0625W_100PPM, RESC1005X40N, symbol Resistors_SMD:R0402_10K_1%_0.0625W_100PPM
- removed R180: R0402_47K_1%_0.0625W_100PPM, RESC1005X40N, symbol Resistors_SMD:R0402_47K_1%_0.0625W_100PPM
- added TP14: TestPoint, TestPoint:TestPoint_THTPad_D1.5mm_Drill0.7mm, symbol Connector_Generic:TestPoint
Connections:
- wire segments 247 -> 237

Commit message: Progress on the BOM
Fill in many Manufacturer fields
Move dnf flag from Y1 to Y2
Manufacturer Part Number changes for Y1 D8 J6 J9
Parts:
- D8: Manufacturer (none) -> DIODES INC; Manufacturer Part Number SMAJ58A -> SMAJ58A-13-F
- L35, L36, L37, L38, L39, L40: Manufacturer (none) -> TDK
- U40: Manufacturer (none) -> Silvertel; Manufacturer_Name Silvertel -> (none)
Changed lines of the file:
@@
 F 4 "Power-over-Ethernet Plus Module" H 6700 8200 50  0001 L CNN "Description"
 F 5 "14" H 6700 8100 50  0001 L CNN "Height"
-F 6 "Silvertel" H 6700 7900 50  0001 L CNN "Manufacturer_Name"
+F 6 "Silvertel" H 6700 7900 50  0001 L CNN "Manufacturer"
 F 7 "AG5300" H 6700 7800 50  0001 L CNN "Manufacturer Part Number"
 	1    5550 8300
@@
 F 3 "~" H 4250 8650 50  0001 C CNN
 F 4 "MPZ2012S102A" V 4250 8650 50  0001 C CNN "Manufacturer Part Number"
+F 5 "TDK" H 4250 8650 50  0001 C CNN "Manufacturer"
 	1    4250 8650
 	0    -1   -1   0
@@
 F 3 "~" H 4750 8650 50  0001 C CNN
 F 4 "MPZ2012S102A" V 4750 8650 50  0001 C CNN "Manufacturer Part Number"
+F 5 "TDK" H 4750 8650 50  0001 C CNN "Manufacturer"
 	1    4750 8650
 	0    -1   -1   0
@@
 F 3 "~" H 5250 8650 50  0001 C CNN
 F 4 "MPZ2012S102A" V 5250 8650 50  0001 C CNN "Manufacturer Part Number"
+F 5 "TDK" H 5250 8650 50  0001 C CNN "Manufacturer"
 	1    5250 8650
 	0    -1   -1   0
@@
 F 3 "~" H 4250 9050 50  0001 C CNN
 F 4 "MPZ2012S102A" V 4250 9050 50  0001 C CNN "Manufacturer Part Number"
+F 5 "TDK" H 4250 9050 50  0001 C CNN "Manufacturer"
 	1    4250 9050
 	0    -1   -1   0
@@
 F 3 "~" H 4750 9050 50  0001 C CNN
 F 4 "MPZ2012S102A" V 4750 9050 50  0001 C CNN "Manufacturer Part Number"
+F 5 "TDK" H 4750 9050 50  0001 C CNN "Manufacturer"
 	1    4750 9050
 	0    -1   -1   0
@@
 F 3 "~" H 5250 9050 50  0001 C CNN
 F 4 "MPZ2012S102A" V 5250 9050 50  0001 C CNN "Manufacturer Part Number"
+F 5 "TDK" H 5250 9050 50  0001 C CNN "Manufacturer"
 	1    5250 9050
 	0    -1   -1   0
@@
 F 2 "ICs And Semiconductors SMD:DIOM5226X262N" H 3600 8650 50  0001 C CNN
 F 3 "https://www.vishay.com/docs/88301/15ke.pdf" H 3550 8850 50  0001 C CNN
-F 4 "SMAJ58A" H 3600 8850 50  0001 C CNN "Manufacturer Part Number"
+F 4 "SMAJ58A-13-F" H 3600 8850 50  0001 C CNN "Manufacturer Part Number"
+F 5 "DIODES INC" H 3600 8850 50  0001 C CNN "Manufacturer"
 	1    3600 8850
 	0    1    1    0

Commit message: More progress on the BOM
Fill in more Manufacturer and Manufacturer Part Number
Manufacturer Part Number changes for D6 D7
Parts:
- D6, D7: Manufacturer (none) -> SMC; Manufacturer Part Number MB210S-TP -> KMB210STR
- J19: Manufacturer (none) -> AMP; Manufacturer Part Number (none) -> 641119-2
Changed lines of the file:
@@
 F 2 "ICs And Semiconductors SMD:SOIC254P665X290-4N" H 3400 8775 50  0001 L CNN
 F 3 "http://www.vishay.com/docs/88573/dfs.pdf" H 3250 8650 50  0001 C CNN
-F 4 "MB210S-TP" H 3250 8650 50  0001 C CNN "Manufacturer Part Number"
+F 4 "KMB210STR" H 3250 8650 50  0001 C CNN "Manufacturer Part Number"
+F 5 "SMC" H 3250 8650 50  0001 C CNN "Manufacturer"
 	1    3250 8650
 	1    0    0    -1
@@
 F 2 "ICs And Semiconductors SMD:SOIC254P665X290-4N" H 3400 9775 50  0001 L CNN
 F 3 "http://www.vishay.com/docs/88573/dfs.pdf" H 3250 9650 50  0001 C CNN
-F 4 "MB210S-TP" H 3250 9650 50  0001 C CNN "Manufacturer Part Number"
+F 4 "KMB210STR" H 3250 9650 50  0001 C CNN "Manufacturer Part Number"
+F 5 "SMC" H 3250 9650 50  0001 C CNN "Manufacturer"
 	1    3250 9650
 	1    0    0    -1
@@
 F 2 "Marble:641119-2" H 1100 1000 50  0001 C CNN
 F 3 "" H 1100 1300 50  0001 C CNN
+F 4 "AMP" H 1100 1300 50  0001 C CNN "Manufacturer"
+F 5 "641119-2" H 1100 1300 50  0001 C CNN "Manufacturer Part Number"
 	1    1100 1300
 	1    0    0    1

Commit message: Adjust BOM details
Fix spelling of "config" attribute for SW2
Part number changes:
FC68148 (DC-10A) to FC68148
TXB0108PW to TXB0108PWR
XRP7724ILBTR-F to XRP7724ILB-F
Parts:
- J1: Manufacturer Part Number FC68148 (DC-10A) -> FC68148
Changed lines of the file:
@@
 F 27 "12V/5A, 2.1mm Diameter Pin, DC Power Socket With  Switch (DC10A Type)" H 1250 -1080 60  0001 L CNN "Part Description"
 F 28 "CLIFF ELECTRONIC COMPONENTS" H 1250 -1170 60  0001 L CNN "Manufacturer"
-F 29 "FC68148 (DC-10A)" H 1250 -1260 60  0001 L CNN "Manufacturer Part Number"
+F 29 "FC68148" H 1250 -1260 60  0001 L CNN "Manufacturer Part Number"
 F 30 "11mm" H 1250 -1350 60  0001 L CNN "ComponentHeight"
 F 31 "\\\\cern.ch\\dfs\\Applications\\Altium\\Datasheets\\CLIFF_FC68148(DC-10A).pdf" H 1250 -1440 60  0001 L CNN "HelpURL"

Commit message: Stop saying that 2-pin devices have "2.0000000000000000e+00" pins
Parts:
- C132, C133, C136, C350, C351, C353, C354, C378, L13: Pin Count 2.0000000000000000e+00 -> 2
Changed lines of the file:
@@
 F 9 "Standard" H 7900 7760 60  0001 L CNN "Component Kind"
 F 10 "Standard" H 7900 7670 60  0001 L CNN "Component Type"
-F 11 "2.0000000000000000e+00" H 7900 7490 60  0001 L CNN "Pin Count"
+F 11 "2" H 7900 7490 60  0001 L CNN "Pin Count"
 F 12 "PcbLib\\Capacitors SMD.PcbLib" H 7900 7400 60  0001 L CNN "Footprint Path"
 F 13 "CAPAE830X1020N" H 7900 7310 60  0001 L CNN "Footprint Ref"
@@
 F 9 "Standard" H 5950 3160 60  0001 L CNN "Component Kind"
 F 10 "Standard" H 5950 3070 60  0001 L CNN "Component Type"
-F 11 "2.0000000000000000e+00" H 5950 2890 60  0001 L CNN "Pin Count"
+F 11 "2" H 5950 2890 60  0001 L CNN "Pin Count"
 F 12 "PcbLib\\Capacitors SMD.PcbLib" H 5950 2800 60  0001 L CNN "Footprint Path"
 F 13 "CAPC0603X33N" H 5950 2710 60  0001 L CNN "Footprint Ref"
@@
 F 9 "Standard" H 5450 3160 60  0001 L CNN "Component Kind"
 F 10 "Standard" H 5450 3070 60  0001 L CNN "Component Type"
-F 11 "2.0000000000000000e+00" H 5450 2890 60  0001 L CNN "Pin Count"
+F 11 "2" H 5450 2890 60  0001 L CNN "Pin Count"
 F 12 "PcbLib\\Capacitors SMD.PcbLib" H 5450 2800 60  0001 L CNN "Footprint Path"
 F 13 "CAPC1709X100N" H 5450 2710 60  0001 L CNN "Footprint Ref"
@@
 F 9 "Standard" H 12050 5510 60  0001 L CNN "Component Kind"
 F 10 "Standard" H 12050 5420 60  0001 L CNN "Component Type"
-F 11 "2.0000000000000000e+00" H 12050 5240 60  0001 L CNN "Pin Count"
+F 11 "2" H 12050 5240 60  0001 L CNN "Pin Count"
 F 12 "PcbLib\\Capacitors SMD.PcbLib" H 12050 5150 60  0001 L CNN "Footprint Path"
 F 13 "CAPC0603X33N" H 12050 5060 60  0001 L CNN "Footprint Ref"
@@
 F 9 "Standard" H 12050 2110 60  0001 L CNN "Component Kind"
 F 10 "Standard" H 12050 2020 60  0001 L CNN "Component Type"
-F 11 "2.0000000000000000e+00" H 12050 1840 60  0001 L CNN "Pin Count"
+F 11 "2" H 12050 1840 60  0001 L CNN "Pin Count"
 F 12 "PcbLib\\Capacitors SMD.PcbLib" H 12050 1750 60  0001 L CNN "Footprint Path"
 F 13 "CAPC0603X33N" H 12050 1660 60  0001 L CNN "Footprint Ref"
@@
 F 10 "Standard" H 6200 7220 60  0001 L CNN "Component Type"
 F 11 "~~" H 6200 7040 60  0001 L CNN "PackageDescription"
-F 12 "2.0000000000000000e+00" H 6200 6950 60  0001 L CNN "Pin Count"
+F 12 "2" H 6200 6950 60  0001 L CNN "Pin Count"
 F 13 "PcbLib\\Capacitors THD.PcbLib" H 6200 6860 60  0001 L CNN "Footprint Path"
 F 14 "CAPR500-250X720X650" H 6200 6770 60  0001 L CNN "Footprint Ref"
@@
 F 10 "Standard" H 6200 8470 60  0001 L CNN "Component Type"
 F 11 "~~" H 6200 8290 60  0001 L CNN "PackageDescription"
-F 12 "2.0000000000000000e+00" H 6200 8200 60  0001 L CNN "Pin Count"
+F 12 "2" H 6200 8200 60  0001 L CNN "Pin Count"
 F 13 "PcbLib\\Capacitors THD.PcbLib" H 6200 8110 60  0001 L CNN "Footprint Path"
 F 14 "CAPR500-250X720X650" H 6200 8020 60  0001 L CNN "Footprint Ref"
@@
 F 10 "Standard" H 4350 3140 60  0001 L CNN "Component Type"
 F 11 "~~" H 4350 2960 60  0001 L CNN "PackageDescription"
-F 12 "2.0000000000000000e+00" H 4350 2870 60  0001 L CNN "Pin Count"
+F 12 "2" H 4350 2870 60  0001 L CNN "Pin Count"
 F 13 "PcbLib\\Inductors SMD.PcbLib" H 4350 2780 60  0001 L CNN "Footprint Path"
 F 14 "IND_TDK_VLCF5020-1" H 4350 2690 60  0001 L CNN "Footprint Ref"
@@
 F 9 "Standard" H 5000 1860 60  0001 L CNN "Component Kind"
 F 10 "Standard" H 5000 1770 60  0001 L CNN "Component Type"
-F 11 "2.0000000000000000e+00" H 5000 1590 60  0001 L CNN "Pin Count"
+F 11 "2" H 5000 1590 60  0001 L CNN "Pin Count"
 F 12 "PcbLib\\Capacitors SMD.PcbLib" H 5000 1500 60  0001 L CNN "Footprint Path"
 F 13 "CAPC0603X33N" H 5000 1410 60  0001 L CNN "Footprint Ref"

Commit message: new hole for mounting holes, new PN for D6 and D7
Parts:
- D6, D7: value MB210S-TP -> KMB215STR; Manufacturer Part Number KMB210STR -> KMB215STR
Changed lines of the file:
@@
 Text Label 2250 8950 0    50   ~ 10
 POE_VC3
-Text Label 2250 9950 0    50   ~ 10
+Text Label 2300 9950 0    50   ~ 10
 POE_VC4
 Wire Bus Line
@@
 P 3250 8650
 F 0 "D6" H 3450 8800 50  0000 L CNN
-F 1 "MB210S-TP" H 2650 8800 50  0000 L CNN
+F 1 "KMB215STR" H 2650 8800 50  0000 L CNN
 F 2 "ICs And Semiconductors SMD:SOIC254P665X290-4N" H 3400 8775 50  0001 L CNN
 F 3 "http://www.vishay.com/docs/88573/dfs.pdf" H 3250 8650 50  0001 C CNN
-F 4 "KMB210STR" H 3250 8650 50  0001 C CNN "Manufacturer Part Number"
+F 4 "KMB215STR" H 3250 8650 50  0001 C CNN "Manufacturer Part Number"
 F 5 "SMC" H 3250 8650 50  0001 C CNN "Manufacturer"
 	1    3250 8650
@@
 P 3250 9650
 F 0 "D7" H 3500 9750 50  0000 L CNN
-F 1 "MB210S-TP" H 2700 9850 50  0000 L CNN
+F 1 "KMB215STR" H 2700 9850 50  0000 L CNN
 F 2 "ICs And Semiconductors SMD:SOIC254P665X290-4N" H 3400 9775 50  0001 L CNN
 F 3 "http://www.vishay.com/docs/88573/dfs.pdf" H 3250 9650 50  0001 C CNN
-F 4 "KMB210STR" H 3250 9650 50  0001 C CNN "Manufacturer Part Number"
+F 4 "KMB215STR" H 3250 9650 50  0001 C CNN "Manufacturer Part Number"
 F 5 "SMC" H 3250 9650 50  0001 C CNN "Manufacturer"
 	1    3250 9650

Commit message: Convert "~" and "~~" in .sch and .lib files to " "
cf. commit ef029e49 in Marble-Mini, May 21 2020
Parts:
- C132, C133, C136, C351, C378: ComponentHeight ~~ -> (none); PackageDescription ~~ -> (none); PressFit ~~ -> (none); Sense Comment ~~ -> (none); Status Comment ~~ -> (none)
- C350, C353, C354: Manufacturer1 ComponentHeight ~~ -> (none); Manufacturer1 Example ~~ -> (none); Manufacturer1 Part Number ~~ -> (none); PackageDescription ~~ -> (none); PressFit ~~ -> (none); Sense Comment ~~ -> (none); Status Comment ~~ -> (none); TC ~~ -> (none)
- D12, D4, Q1, Q16, Q2, Q22, Q23, Q4, Q8, Q9, U17, U32, U41, U57: ComponentLink1Description ~~ -> (none); ComponentLink1URL ~~ -> (none); ComponentLink2Description ~~ -> (none); ComponentLink2URL ~~ -> (none); Sense Comment ~~ -> (none); Status ~~ -> (none); Status Comment ~~ -> (none)
- J1: Case ~~ -> (none); Comment ~~ -> (none); ComponentLink1Description ~~ -> (none); ComponentLink1URL ~~ -> (none); ComponentLink2Description ~~ -> (none); ComponentLink2URL ~~ -> (none); Device ~~ -> (none); PackageDescription ~~ -> (none); SCEM ~~ -> (none); Sense Comment ~~ -> (none); Status Comment ~~ -> (none)
- L13: Case ~~ -> (none); PackageDescription ~~ -> (none); Sense Comment ~~ -> (none); Status Comment ~~ -> (none)
- LD1, LD2: Case ~~ -> (none); Comment ~~ -> (none); ComponentLink1Description ~~ -> (none); ComponentLink1URL ~~ -> (none); ComponentLink2Description ~~ -> (none); ComponentLink2URL ~~ -> (none); Device ~~ -> (none); Sense Comment ~~ -> (none); Status ~~ -> (none); Status Comment ~~ -> (none)
- R104, R107, R108, R109, R110, R179, R181, R184, R188, R201, R202, R203, R212, R213, R214, R235, R236: ComponentHeight ~~ -> (none); PackageDescription ~~ -> (none); Sense Comment ~~ -> (none); Status Comment ~~ -> (none); Voltage ~~ -> (none)
- R182, R183: Manufacturer1 ComponentHeight ~~ -> (none); Manufacturer1 Example ~~ -> (none); Manufacturer1 Part Number ~~ -> (none); PackageDescription ~~ -> (none); Sense Comment ~~ -> (none); Status Comment ~~ -> (none); Voltage ~~ -> (none)
- R197, R198, R281: ComponentHeight ~~ -> (none); PackageDescription ~~ -> (none); Power ~~ -> (none); Sense Comment ~~ -> (none); Status Comment ~~ -> (none); TC ~~ -> (none); Tolerance ~~ -> (none); Voltage ~~ -> (none)
- U18: ComponentLink1Description ~~ -> (none); ComponentLink1URL ~~ -> (none); ComponentLink2Description ~~ -> (none); ComponentLink2URL ~~ -> (none); SCEM ~~ -> (none); Sense Comment ~~ -> (none); Status ~~ -> (none); Status Comment ~~ -> (none)
