File: Thermometers.sch (KiCad schematic (older format))
At the start: 22 parts, among them M1 Fan_Tacho_PC, M2 Fan_Tacho_PC, Q7 STS8DN6LF6AG, U27 MAX6639AEE+, U28 LM75AIMM/NOPB, U29 LM75AIMM/NOPB

Commit message: Automated edit to move cache / rescue symbols to actual eeschem library
Results of running dissect_lib3.py, not posted here
Parts:
- Q7: symbol AMC_FMC_Carrier-PcbDoc-rescue:STS2DNE60-Transistor_FET-AMC_FMC_Carrier-PcbDoc-rescue-AMC_FMC_Carrier-PcbDoc-rescue-AMC_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 -> marble_misc:STS2DNE60-Transistor_FET
- U28, U29: symbol AMC_FMC_Carrier-PcbDoc-rescue:LM75B-Sensor_Temperature-AMC_FMC_Carrier-PcbDoc-rescue-AMC_FMC_Carrier-PcbDoc-rescue-AMC_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 -> marble_misc:LM75B-Sensor_Temperature
Changed lines of the file:
@@
 $EndDescr
 $Comp
-L AMC_FMC_Carrier-PcbDoc-rescue:LM75B-Sensor_Temperature-AMC_FMC_Carrier-PcbDoc-rescue-AMC_FMC_Carrier-PcbDoc-rescue-AMC_FMC_Carrier-PcbDoc-rescue-AMC_FMC_Carrier-PcbDoc-rescue U28
+L marble_misc:LM75B-Sensor_Temperature U28
 U 1 1 5D05AA1A
 P 6900 1850
@@
 $EndComp
 $Comp
-L power2:+3.3P #PWR?
+L power:+3.3P #PWR?
 U 1 1 5D05AEC2
 P 6900 1100
@@
 $EndComp
 $Comp
-L power2:+3.3P #PWR?
+L power:+3.3P #PWR?
 U 1 1 5D05B18E
 P 7500 1750
@@
 $EndComp
 $Comp
-L power2:+3.3P #PWR?
+L power:+3.3P #PWR?
 U 1 1 5D05B203
 P 7500 1850
@@
 	7500 1950 7300 1950
 $Comp
-L AMC_FMC_Carrier-PcbDoc-rescue:LM75B-Sensor_Temperature-AMC_FMC_Carrier-PcbDoc-rescue-AMC_FMC_Carrier-PcbDoc-rescue-AMC_FMC_Carrier-PcbDoc-rescue-AMC_FMC_Carrier-PcbDoc-rescue U29
+L marble_misc:LM75B-Sensor_Temperature U29
 U 1 1 5D05B2F7
 P 6900 3750
@@
 $EndComp
 $Comp
-L power2:+3.3P #PWR?
+L power:+3.3P #PWR?
 U 1 1 5D05B306
 P 6900 3000
@@
 $EndComp
 $Comp
-L power2:+3.3P #PWR?
+L power:+3.3P #PWR?
 U 1 1 5D05B324
 P 7500 3650
@@
 Connection ~ 6300 1950
 $Comp
-L power2:+3.3P #PWR?
+L power:+3.3P #PWR?
 U 1 1 5D05D39D
 P 6300 1100
@@
 	6300 1100 6300 1200
 $Comp
-L power2:+3.3P #PWR?
+L power:+3.3P #PWR?
 U 1 1 5D0665E3
 P 2300 6000
@@
 	2750 5200 2850 5200
 $Comp
-L AMC_FMC_Carrier-PcbDoc-rescue:STS2DNE60-Transistor_FET-AMC_FMC_Carrier-PcbDoc-rescue-AMC_FMC_Carrier-PcbDoc-rescue-AMC_FMC_Carrier-PcbDoc-rescue-AMC_FMC_Carrier-PcbDoc-rescue Q7
+L marble_misc:STS2DNE60-Transistor_FET Q7
 U 1 1 5D559F89
 P 6700 5750
@@
 $EndComp
 $Comp
-L AMC_FMC_Carrier-PcbDoc-rescue:STS2DNE60-Transistor_FET-AMC_FMC_Carrier-PcbDoc-rescue-AMC_FMC_Carrier-PcbDoc-rescue-AMC_FMC_Carrier-PcbDoc-rescue-AMC_FMC_Carrier-PcbDoc-rescue Q7
+L marble_misc:STS2DNE60-Transistor_FET Q7
 U 2 1 5D559FE8
 P 8300 5750
@@
 	4800 5100 4800 5200
 $Comp
-L power2:+3.3P #PWR?
+L power:+3.3P #PWR?
 U 1 1 5D57B1C9
 P 4800 4750
@@
 $EndComp
 $Comp
-L power2:+3.3P #PWR?
+L power:+3.3P #PWR?
 U 1 1 5D581F39
 P 5350 4750
@@
 Connection ~ 4600 6000
 $Comp
-L power2:+3.3P #PWR?
+L power:+3.3P #PWR?
 U 1 1 5D5D3DE2
 P 4200 4750

Commit message: reduced reels with components, DDR 1V5 enable signal connected to MMC, DDR I2C pull-ups powerd from 3.3VP
Parts:
- C343, C344: value CC0603_4.7UF_16V_10%_X5R -> CC0603_4.7UF_25V_10%_X5R; footprint CAPC1709X95N -> Capacitors SMD:CAPC1608X90N; symbol Capacitors_SMD:CC0603_4.7UF_16V_10%_X5R -> Capacitors_SMD:CC0603_4.7UF_25V_10%_X5R; Comment =Value -> 4.7uF; ComponentHeight ~~ -> (none); CreateDate 12/16/13 00:00:00 -> 11/10/14 00:00:00; Database Table Name (none) -> Capacitors SMD; Footprint Library (none) -> Capacitors SMD; Footprint Ref CAPC1709X95N -> CAPC1608X90N; LatestRevisionDate 09/16/14 00:00:00 -> 11/10/14 00:00:00; Library Name Capacitors SMD -> Capacitors.DbLib; Manufacturer Part Number CC0603_4.7UF_16V_10%_X5R -> CC0603_4.7UF_25V_10%_X5R; Manufacturer1 Example TAIYO YUDEN -> MURATA; Manufacturer1 Part Number EMK107ABJ475KA-T -> GRM188R61E475KE11D; PackageDescription ~~ -> (none); Part Number CC0603_4.7UF_16V_10%_X5R -> CC0603_4.7UF_25V_10%_X5R; Pin Count 2.0000000000000000e+00 -> 2; PressFit ~~ -> (none); Sense Comment ~~ -> (none); Status Comment ~~ -> (none); Voltage 16V -> 25V
Changed lines of the file:
@@
 	6300 3850 6300 6100
 $Comp
-L Capacitors_SMD:CC0603_4.7UF_16V_10%_X5R C?
+L Capacitors_SMD:CC0603_4.7UF_25V_10%_X5R C?
 U 1 1 5D041D3E
 P 9550 4900
@@
 AR Path="/5D05A99E/5D041D3E" Ref="C343"  Part="1"
 F 0 "C343" V 9600 4900 50  0000 L CNN
-F 1 "CC0603_4.7UF_16V_10%_X5R" H 9550 4640 60  0001 L CNN
-F 2 "CAPC1709X95N" H 9550 3830 60  0001 L CNN
+F 1 "CC0603_4.7UF_25V_10%_X5R" H 9550 4640 60  0001 L CNN
+F 2 "Capacitors SMD:CAPC1608X90N" H 9550 3830 60  0001 L CNN
 F 3 "\\\\cern.ch\\dfs\\Applications\\Altium\\Datasheets\\CC0603_X7R_TAIYO-YUDEN_HIGH-VALUE.pdf" H 9550 4460 60  0001 L CNN
 F 4 "4.7uF" V 9800 4900 50  0000 L CNN "~"
-F 5 "CC0603_4.7UF_16V_10%_X5R" H 9550 4370 60  0001 L CNN "Part Number"
+F 5 "CC0603_4.7UF_25V_10%_X5R" H 9550 4370 60  0001 L CNN "Part Number"
 F 6 "Capacitor - non polarized" H 9550 4280 60  0001 L CNN "Library Ref"
 F 7 "SchLib\\Capacitors.SchLib" H 9550 4190 60  0001 L CNN "Library Path"
-F 8 "=Value" H 9550 4100 60  0001 L CNN "Comment"
+F 8 "4.7uF" H 9550 4100 60  0001 L CNN "Comment"
 F 9 "Standard" H 9550 4010 60  0001 L CNN "Component Kind"
 F 10 "Standard" H 9550 3920 60  0001 L CNN "Component Type"
-F 11 "2.0000000000000000e+00" H 9550 3740 60  0001 L CNN "Pin Count"
+F 11 "2" H 9550 3740 60  0001 L CNN "Pin Count"
 F 12 "PcbLib\\Capacitors SMD.PcbLib" H 9550 3650 60  0001 L CNN "Footprint Path"
-F 13 "CAPC1709X95N" H 9550 3560 60  0001 L CNN "Footprint Ref"
-F 14 "~~" H 9550 3470 60  0001 L CNN "PackageDescription"
+F 13 "CAPC1608X90N" H 9550 3560 60  0001 L CNN "Footprint Ref"
+F 14 " " H 9550 3470 60  0001 L CNN "PackageDescription"
 F 15 "4.7uF" H 9550 3380 60  0001 L CNN "Val"
 F 16 "None" H 9550 3290 60  0001 L CNN "Status"
-F 17 "~~" H 9550 3200 60  0001 L CNN "Status Comment"
-F 18 "16V" H 9550 3110 60  0001 L CNN "Voltage"
+F 17 " " H 9550 3200 60  0001 L CNN "Status Comment"
+F 18 "25V" H 9550 3110 60  0001 L CNN "Voltage"
 F 19 "X5R" H 9550 3020 60  0001 L CNN "TC"
 F 20 "±10%" H 9550 2930 60  0001 L CNN "Tolerance"
 F 21 "SMD Multilayer Chip Ceramic Capacitor" H 9550 2840 60  0001 L CNN "Part Description"
 F 22 "GENERIC" H 9550 2750 60  0001 L CNN "Manufacturer"
-F 23 "CC0603_4.7UF_16V_10%_X5R" H 9550 2660 60  0001 L CNN "Manufacturer Part Number"
+F 23 "CC0603_4.7UF_25V_10%_X5R" H 9550 2660 60  0001 L CNN "Manufacturer Part Number"
 F 24 "0603" H 9550 2570 60  0001 L CNN "Case"
 F 25 "Yes" H 9550 2480 60  0001 L CNN "Mounted"
 F 26 "No" H 9550 2390 60  0001 L CNN "Socket"
 F 27 "Yes" H 9550 2300 60  0001 L CNN "SMD"
-F 28 "~~" H 9550 2210 60  0001 L CNN "PressFit"
+F 28 " " H 9550 2210 60  0001 L CNN "PressFit"
 F 29 "No" H 9550 2120 60  0001 L CNN "Sense"
-F 30 "~~" H 9550 2030 60  0001 L CNN "Sense Comment"
-F 31 "~~" H 9550 1940 60  0001 L CNN "ComponentHeight"
-F 32 "TAIYO YUDEN" H 9550 1850 60  0001 L CNN "Manufacturer1 Example"
-F 33 "EMK107ABJ475KA-T" H 9550 1760 60  0001 L CNN "Manufacturer1 Part Number"
+F 30 " " H 9550 2030 60  0001 L CNN "Sense Comment"
+F 31 " " H 9550 1940 60  0001 L CNN "ComponentHeight"
+F 32 "MURATA" H 9550 1850 60  0001 L CNN "Manufacturer1 Example"
+F 33 "GRM188R61E475KE11D" H 9550 1760 60  0001 L CNN "Manufacturer1 Part Number"
 F 34 "0.95mm" H 9550 1670 60  0001 L CNN "Manufacturer1 ComponentHeight"
 F 35 "\\\\cern.ch\\dfs\\Applications\\Altium\\Datasheets\\CC0603_X7R_TAIYO-YUDEN_HIGH-VALUE.pdf" H 9550 1580 60  0001 L CNN "HelpURL"
 F 36 "CERN DEM JLC" H 9550 1490 60  0001 L CNN "Author"
-F 37 "12/16/13 00:00:00" H 9550 1400 60  0001 L CNN "CreateDate"
-F 38 "09/16/14 00:00:00" H 9550 1310 60  0001 L CNN "LatestRevisionDate"
-F 39 "Capacitors SMD" H 9550 1220 60  0001 L CNN "Library Name"
+F 37 "11/10/14 00:00:00" H 9550 1400 60  0001 L CNN "CreateDate"
+F 38 "11/10/14 00:00:00" H 9550 1310 60  0001 L CNN "LatestRevisionDate"
+F 39 "Capacitors.DbLib" H 9550 1220 60  0001 L CNN "Library Name"
 F 40 "This work is licensed under the Creative Commons CC-BY-SA 4.0 License. To the extent that circuit schematics that use Licensed Material can be considered to be ‘Adapted Material’, then the copyright holder waives article 3.b of the license with respect to these schematics." H 9550 1130 60  0001 L CNN "License"
+F 41 "Capacitors SMD" H 9550 4900 50  0001 C CNN "Database Table Name"
+F 42 "Capacitors SMD" H 9550 4900 50  0001 C CNN "Footprint Library"
 	1    9550 4900
 	0    1    1    0
 $EndComp
 $Comp
-L Capacitors_SMD:CC0603_4.7UF_16V_10%_X5R C?
+L Capacitors_SMD:CC0603_4.7UF_25V_10%_X5R C?
 U 1 1 5D044AE9
 P 10000 4900
@@
 AR Path="/5D05A99E/5D044AE9" Ref="C344"  Part="1"
 F 0 "C344" V 10050 4900 50  0000 L CNN
-F 1 "CC0603_4.7UF_16V_10%_X5R" H 10000 4640 60  0001 L CNN
-F 2 "CAPC1709X95N" H 10000 3830 60  0001 L CNN
+F 1 "CC0603_4.7UF_25V_10%_X5R" H 10000 4640 60  0001 L CNN
+F 2 "Capacitors SMD:CAPC1608X90N" H 10000 3830 60  0001 L CNN
 F 3 "\\\\cern.ch\\dfs\\Applications\\Altium\\Datasheets\\CC0603_X7R_TAIYO-YUDEN_HIGH-VALUE.pdf" H 10000 4460 60  0001 L CNN
 F 4 "4.7uF" V 10250 4900 50  0000 L CNN "~"
-F 5 "CC0603_4.7UF_16V_10%_X5R" H 10000 4370 60  0001 L CNN "Part Number"
+F 5 "CC0603_4.7UF_25V_10%_X5R" H 10000 4370 60  0001 L CNN "Part Number"
 F 6 "Capacitor - non polarized" H 10000 4280 60  0001 L CNN "Library Ref"
 F 7 "SchLib\\Capacitors.SchLib" H 10000 4190 60  0001 L CNN "Library Path"
-F 8 "=Value" H 10000 4100 60  0001 L CNN "Comment"
+F 8 "4.7uF" H 10000 4100 60  0001 L CNN "Comment"
 F 9 "Standard" H 10000 4010 60  0001 L CNN "Component Kind"
 F 10 "Standard" H 10000 3920 60  0001 L CNN "Component Type"
-F 11 "2.0000000000000000e+00" H 10000 3740 60  0001 L CNN "Pin Count"
+F 11 "2" H 10000 3740 60  0001 L CNN "Pin Count"
 F 12 "PcbLib\\Capacitors SMD.PcbLib" H 10000 3650 60  0001 L CNN "Footprint Path"
-F 13 "CAPC1709X95N" H 10000 3560 60  0001 L CNN "Footprint Ref"
-F 14 "~~" H 10000 3470 60  0001 L CNN "PackageDescription"
+F 13 "CAPC1608X90N" H 10000 3560 60  0001 L CNN "Footprint Ref"
+F 14 " " H 10000 3470 60  0001 L CNN "PackageDescription"
 F 15 "4.7uF" H 10000 3380 60  0001 L CNN "Val"
 F 16 "None" H 10000 3290 60  0001 L CNN "Status"
-F 17 "~~" H 10000 3200 60  0001 L CNN "Status Comment"
-F 18 "16V" H 10000 3110 60  0001 L CNN "Voltage"
+F 17 " " H 10000 3200 60  0001 L CNN "Status Comment"
+F 18 "25V" H 10000 3110 60  0001 L CNN "Voltage"
 F 19 "X5R" H 10000 3020 60  0001 L CNN "TC"
 F 20 "±10%" H 10000 2930 60  0001 L CNN "Tolerance"
 F 21 "SMD Multilayer Chip Ceramic Capacitor" H 10000 2840 60  0001 L CNN "Part Description"
 F 22 "GENERIC" H 10000 2750 60  0001 L CNN "Manufacturer"
-F 23 "CC0603_4.7UF_16V_10%_X5R" H 10000 2660 60  0001 L CNN "Manufacturer Part Number"
+F 23 "CC0603_4.7UF_25V_10%_X5R" H 10000 2660 60  0001 L CNN "Manufacturer Part Number"
 F 24 "0603" H 10000 2570 60  0001 L CNN "Case"
 F 25 "Yes" H 10000 2480 60  0001 L CNN "Mounted"
 F 26 "No" H 10000 2390 60  0001 L CNN "Socket"
 F 27 "Yes" H 10000 2300 60  0001 L CNN "SMD"
-F 28 "~~" H 10000 2210 60  0001 L CNN "PressFit"
+F 28 " " H 10000 2210 60  0001 L CNN "PressFit"
 F 29 "No" H 10000 2120 60  0001 L CNN "Sense"
-F 30 "~~" H 10000 2030 60  0001 L CNN "Sense Comment"
-F 31 "~~" H 10000 1940 60  0001 L CNN "ComponentHeight"
-F 32 "TAIYO YUDEN" H 10000 1850 60  0001 L CNN "Manufacturer1 Example"
-F 33 "EMK107ABJ475KA-T" H 10000 1760 60  0001 L CNN "Manufacturer1 Part Number"
+F 30 " " H 10000 2030 60  0001 L CNN "Sense Comment"
+F 31 " " H 10000 1940 60  0001 L CNN "ComponentHeight"
+F 32 "MURATA" H 10000 1850 60  0001 L CNN "Manufacturer1 Example"
+F 33 "GRM188R61E475KE11D" H 10000 1760 60  0001 L CNN "Manufacturer1 Part Number"
 F 34 "0.95mm" H 10000 1670 60  0001 L CNN "Manufacturer1 ComponentHeight"
 F 35 "\\\\cern.ch\\dfs\\Applications\\Altium\\Datasheets\\CC0603_X7R_TAIYO-YUDEN_HIGH-VALUE.pdf" H 10000 1580 60  0001 L CNN "HelpURL"
 F 36 "CERN DEM JLC" H 10000 1490 60  0001 L CNN "Author"
-F 37 "12/16/13 00:00:00" H 10000 1400 60  0001 L CNN "CreateDate"
-F 38 "09/16/14 00:00:00" H 10000 1310 60  0001 L CNN "LatestRevisionDate"
-F 39 "Capacitors SMD" H 10000 1220 60  0001 L CNN "Library Name"
+F 37 "11/10/14 00:00:00" H 10000 1400 60  0001 L CNN "CreateDate"
+F 38 "11/10/14 00:00:00" H 10000 1310 60  0001 L CNN "LatestRevisionDate"
+F 39 "Capacitors.DbLib" H 10000 1220 60  0001 L CNN "Library Name"
 F 40 "This work is licensed under the Creative Commons CC-BY-SA 4.0 License. To the extent that circuit schematics that use Licensed Material can be considered to be ‘Adapted Material’, then the copyright holder waives article 3.b of the license with respect to these schematics." H 10000 1130 60  0001 L CNN "License"
+F 41 "Capacitors SMD" H 10000 4900 50  0001 C CNN "Database Table Name"
+F 42 "Capacitors SMD" H 10000 4900 50  0001 C CNN "Footprint Library"
 	1    10000 4900
 	0    1    1    0

Commit message: Flag duplicate generic parts in BOM, and refresh a few cap instances from library to reduce such dups
Parts:
- C188, C189: footprint CAPC1005X55N -> Capacitors SMD:CAPC1005X55N; Comment =Value -> 1nF; ComponentHeight ~~ -> (none); Database Table Name (none) -> Capacitors SMD; Footprint Library (none) -> Capacitors SMD; Library Name Capacitors SMD -> Capacitors.DbLib; PackageDescription ~~ -> (none); Pin Count 2.0000000000000000e+00 -> 2; PressFit ~~ -> (none); Sense Comment ~~ -> (none); Status Comment ~~ -> (none)
Changed lines of the file:
@@
 F 0 "C188" V 2054 5110 50  0000 L CNN
 F 1 "CC0402_1NF_50V_10%_X7R" H 1950 4740 60  0001 L CNN
-F 2 "CAPC1005X55N" H 1950 3930 60  0001 L CNN
+F 2 "Capacitors SMD:CAPC1005X55N" H 1950 3930 60  0001 L CNN
 F 3 "\\\\cern.ch\\dfs\\Applications\\Altium\\Datasheets\\CC0402_X7R_PHYCOMP.pdf" H 1950 4560 60  0001 L CNN
 F 4 "1nF" V 2145 5110 50  0000 L CNN "~"
@@
 F 6 "Capacitor - non polarized" H 1950 4380 60  0001 L CNN "Library Ref"
 F 7 "SchLib\\Capacitors.SchLib" H 1950 4290 60  0001 L CNN "Library Path"
-F 8 "=Value" H 1950 4200 60  0001 L CNN "Comment"
+F 8 "1nF" H 1950 4200 60  0001 L CNN "Comment"
 F 9 "Standard" H 1950 4110 60  0001 L CNN "Component Kind"
 F 10 "Standard" H 1950 4020 60  0001 L CNN "Component Type"
-F 11 "2.0000000000000000e+00" H 1950 3840 60  0001 L CNN "Pin Count"
+F 11 "2" H 1950 3840 60  0001 L CNN "Pin Count"
 F 12 "PcbLib\\Capacitors SMD.PcbLib" H 1950 3750 60  0001 L CNN "Footprint Path"
 F 13 "CAPC1005X55N" H 1950 3660 60  0001 L CNN "Footprint Ref"
-F 14 "~~" H 1950 3570 60  0001 L CNN "PackageDescription"
+F 14 " " H 1950 3570 60  0001 L CNN "PackageDescription"
 F 15 "1nF" H 1950 3480 60  0001 L CNN "Val"
 F 16 "Not Recommended" H 1950 3390 60  0001 L CNN "Status"
-F 17 "~~" H 1950 3300 60  0001 L CNN "Status Comment"
+F 17 " " H 1950 3300 60  0001 L CNN "Status Comment"
 F 18 "50V" H 1950 3210 60  0001 L CNN "Voltage"
 F 19 "X7R" H 1950 3120 60  0001 L CNN "TC"
@@
 F 26 "No" H 1950 2490 60  0001 L CNN "Socket"
 F 27 "Yes" H 1950 2400 60  0001 L CNN "SMD"
-F 28 "~~" H 1950 2310 60  0001 L CNN "PressFit"
+F 28 " " H 1950 2310 60  0001 L CNN "PressFit"
 F 29 "No" H 1950 2220 60  0001 L CNN "Sense"
-F 30 "~~" H 1950 2130 60  0001 L CNN "Sense Comment"
-F 31 "~~" H 1950 2040 60  0001 L CNN "ComponentHeight"
+F 30 " " H 1950 2130 60  0001 L CNN "Sense Comment"
+F 31 " " H 1950 2040 60  0001 L CNN "ComponentHeight"
 F 32 "PHYCOMP" H 1950 1950 60  0001 L CNN "Manufacturer1 Example"
 F 33 "223858715623" H 1950 1860 60  0001 L CNN "Manufacturer1 Part Number"
@@
 F 37 "12/03/07 00:00:00" H 1950 1500 60  0001 L CNN "CreateDate"
 F 38 "12/03/07 00:00:00" H 1950 1410 60  0001 L CNN "LatestRevisionDate"
-F 39 "Capacitors SMD" H 1950 1320 60  0001 L CNN "Library Name"
+F 39 "Capacitors.DbLib" H 1950 1320 60  0001 L CNN "Library Name"
 F 40 "This work is licensed under the Creative Commons CC-BY-SA 4.0 License. To the extent that circuit schematics that use Licensed Material can be considered to be ‘Adapted Material’, then the copyright holder waives article 3.b of the license with respect to these schematics." H 1950 1230 60  0001 L CNN "License"
+F 41 "Capacitors SMD" H 1950 5000 50  0001 C CNN "Database Table Name"
+F 42 "Capacitors SMD" H 1950 5000 50  0001 C CNN "Footprint Library"
 	1    1950 5000
 	0    1    1    0
@@
 F 0 "C189" V 2504 5110 50  0000 L CNN
 F 1 "CC0402_1NF_50V_10%_X7R" H 2400 4740 60  0001 L CNN
-F 2 "CAPC1005X55N" H 2400 3930 60  0001 L CNN
+F 2 "Capacitors SMD:CAPC1005X55N" H 2400 3930 60  0001 L CNN
 F 3 "\\\\cern.ch\\dfs\\Applications\\Altium\\Datasheets\\CC0402_X7R_PHYCOMP.pdf" H 2400 4560 60  0001 L CNN
 F 4 "1nF" V 2595 5110 50  0000 L CNN "~"
@@
 F 6 "Capacitor - non polarized" H 2400 4380 60  0001 L CNN "Library Ref"
 F 7 "SchLib\\Capacitors.SchLib" H 2400 4290 60  0001 L CNN "Library Path"
-F 8 "=Value" H 2400 4200 60  0001 L CNN "Comment"
+F 8 "1nF" H 2400 4200 60  0001 L CNN "Comment"
 F 9 "Standard" H 2400 4110 60  0001 L CNN "Component Kind"
 F 10 "Standard" H 2400 4020 60  0001 L CNN "Component Type"
-F 11 "2.0000000000000000e+00" H 2400 3840 60  0001 L CNN "Pin Count"
+F 11 "2" H 2400 3840 60  0001 L CNN "Pin Count"
 F 12 "PcbLib\\Capacitors SMD.PcbLib" H 2400 3750 60  0001 L CNN "Footprint Path"
 F 13 "CAPC1005X55N" H 2400 3660 60  0001 L CNN "Footprint Ref"
-F 14 "~~" H 2400 3570 60  0001 L CNN "PackageDescription"
+F 14 " " H 2400 3570 60  0001 L CNN "PackageDescription"
 F 15 "1nF" H 2400 3480 60  0001 L CNN "Val"
 F 16 "Not Recommended" H 2400 3390 60  0001 L CNN "Status"
-F 17 "~~" H 2400 3300 60  0001 L CNN "Status Comment"
+F 17 " " H 2400 3300 60  0001 L CNN "Status Comment"
 F 18 "50V" H 2400 3210 60  0001 L CNN "Voltage"
 F 19 "X7R" H 2400 3120 60  0001 L CNN "TC"
@@
 F 26 "No" H 2400 2490 60  0001 L CNN "Socket"
 F 27 "Yes" H 2400 2400 60  0001 L CNN "SMD"
-F 28 "~~" H 2400 2310 60  0001 L CNN "PressFit"
+F 28 " " H 2400 2310 60  0001 L CNN "PressFit"
 F 29 "No" H 2400 2220 60  0001 L CNN "Sense"
-F 30 "~~" H 2400 2130 60  0001 L CNN "Sense Comment"
-F 31 "~~" H 2400 2040 60  0001 L CNN "ComponentHeight"
+F 30 " " H 2400 2130 60  0001 L CNN "Sense Comment"
+F 31 " " H 2400 2040 60  0001 L CNN "ComponentHeight"
 F 32 "PHYCOMP" H 2400 1950 60  0001 L CNN "Manufacturer1 Example"
 F 33 "223858715623" H 2400 1860 60  0001 L CNN "Manufacturer1 Part Number"
@@
 F 37 "12/03/07 00:00:00" H 2400 1500 60  0001 L CNN "CreateDate"
 F 38 "12/03/07 00:00:00" H 2400 1410 60  0001 L CNN "LatestRevisionDate"
-F 39 "Capacitors SMD" H 2400 1320 60  0001 L CNN "Library Name"
+F 39 "Capacitors.DbLib" H 2400 1320 60  0001 L CNN "Library Name"
 F 40 "This work is licensed under the Creative Commons CC-BY-SA 4.0 License. To the extent that circuit schematics that use Licensed Material can be considered to be ‘Adapted Material’, then the copyright holder waives article 3.b of the license with respect to these schematics." H 2400 1230 60  0001 L CNN "License"
+F 41 "Capacitors SMD" H 2400 5000 50  0001 C CNN "Database Table Name"
+F 42 "Capacitors SMD" H 2400 5000 50  0001 C CNN "Footprint Library"
 	1    2400 5000
 	0    1    1    0

Commit message: Progress on the BOM
Fill in many Manufacturer fields
Move dnf flag from Y1 to Y2
Manufacturer Part Number changes for Y1 D8 J6 J9
Parts:
- Q7: Manufacturer (none) -> ST MICROELECTRONICS
- U28, U29: Manufacturer (none) -> TEXAS INSTRUMENTS
Changed lines of the file:
@@
 F 3 "http://www.ti.com/lit/ds/symlink/lm75b.pdf" H 6900 1850 50  0001 C CNN
 F 4 "LM75AIMM/NOPB" H 6900 1850 50  0001 C CNN "Manufacturer Part Number"
+F 5 "TEXAS INSTRUMENTS" H 6900 1850 50  0001 C CNN "Manufacturer"
 	1    6900 1850
 	1    0    0    -1
@@
 F 3 "http://www.ti.com/lit/ds/symlink/lm75b.pdf" H 6900 3750 50  0001 C CNN
 F 4 "LM75AIMM/NOPB" H 6900 3750 50  0001 C CNN "Manufacturer Part Number"
+F 5 "TEXAS INSTRUMENTS" H 6900 3750 50  0001 C CNN "Manufacturer"
 	1    6900 3750
 	1    0    0    -1
@@
 F 3 "www.st.com/resource/en/datasheet/CD00001537.pdf" H 6700 5750 50  0001 L CNN
 F 4 "STS8DN6LF6AG" H 6700 5750 50  0001 C CNN "Manufacturer Part Number"
+F 5 "ST MICROELECTRONICS" H 6700 5750 50  0001 C CNN "Manufacturer"
 	1    6700 5750
 	1    0    0    -1
@@
 F 3 "www.st.com/resource/en/datasheet/CD00001537.pdf" H 8300 5750 50  0001 L CNN
 F 4 "STS8DN6LF6AG" H 8300 5750 50  0001 C CNN "Manufacturer Part Number"
+F 5 "ST MICROELECTRONICS" H 8300 5750 50  0001 C CNN "Manufacturer"
 	2    8300 5750
 	1    0    0    -1

Commit message: More progress on the BOM
Fill in more Manufacturer and Manufacturer Part Number
Manufacturer Part Number changes for D6 D7
Parts:
- M1, M2: Manufacturer (none) -> SULLINS; Manufacturer Part Number (none) -> SWR25X-NRTC-S03-ST-BA
Changed lines of the file:
@@
 F 2 "Connector:FanPinHeader_1x03_P2.54mm_Vertical" H 8400 5060 50  0001 C CNN
 F 3 "http://www.hardwarecanucks.com/forum/attachments/new-builds/16287d1330775095-help-chassis-power-fan-connectors-motherboard-asus_p8z68.jpg" H 8400 5060 50  0001 C CNN
+F 4 "SULLINS" H 8400 5150 50  0001 C CNN "Manufacturer"
+F 5 "SWR25X-NRTC-S03-ST-BA" H 8400 5150 50  0001 C CNN "Manufacturer Part Number"
 	1    8400 5150
 	1    0    0    -1
@@
 F 2 "Connector:FanPinHeader_1x03_P2.54mm_Vertical" H 6800 5060 50  0001 C CNN
 F 3 "http://www.hardwarecanucks.com/forum/attachments/new-builds/16287d1330775095-help-chassis-power-fan-connectors-motherboard-asus_p8z68.jpg" H 6800 5060 50  0001 C CNN
+F 4 "SULLINS" H 6800 5150 50  0001 C CNN "Manufacturer"
+F 5 "SWR25X-NRTC-S03-ST-BA" H 6800 5150 50  0001 C CNN "Manufacturer Part Number"
 	1    6800 5150
 	1    0    0    -1

Commit message: Stop saying that 2-pin devices have "2.0000000000000000e+00" pins
Parts:
- C190, C191, C192: Pin Count 2.0000000000000000e+00 -> 2
Changed lines of the file:
@@
 F 9 "Standard" H 2400 5160 60  0001 L CNN "Component Kind"
 F 10 "Standard" H 2400 5070 60  0001 L CNN "Component Type"
-F 11 "2.0000000000000000e+00" H 2400 4890 60  0001 L CNN "Pin Count"
+F 11 "2" H 2400 4890 60  0001 L CNN "Pin Count"
 F 12 "PcbLib\\Capacitors SMD.PcbLib" H 2400 4800 60  0001 L CNN "Footprint Path"
 F 13 "CAPC0603X33N" H 2400 4710 60  0001 L CNN "Footprint Ref"
@@
 F 9 "Standard" H 7300 2260 60  0001 L CNN "Component Kind"
 F 10 "Standard" H 7300 2170 60  0001 L CNN "Component Type"
-F 11 "2.0000000000000000e+00" H 7300 1990 60  0001 L CNN "Pin Count"
+F 11 "2" H 7300 1990 60  0001 L CNN "Pin Count"
 F 12 "PcbLib\\Capacitors SMD.PcbLib" H 7300 1900 60  0001 L CNN "Footprint Path"
 F 13 "CAPC0603X33N" H 7300 1810 60  0001 L CNN "Footprint Ref"
@@
 F 9 "Standard" H 7300 360 60  0001 L CNN "Component Kind"
 F 10 "Standard" H 7300 270 60  0001 L CNN "Component Type"
-F 11 "2.0000000000000000e+00" H 7300 90  60  0001 L CNN "Pin Count"
+F 11 "2" H 7300 90  60  0001 L CNN "Pin Count"
 F 12 "PcbLib\\Capacitors SMD.PcbLib" H 7300 0   60  0001 L CNN "Footprint Path"
 F 13 "CAPC0603X33N" H 7300 -90 60  0001 L CNN "Footprint Ref"
