File: Thermometers.sch (KiCad schematic (older format))
At the start: 22 parts, among them M1 Fan_Tacho_PC, M2 Fan_Tacho_PC, Q7 STS8DN6LF6AG, U27 MAX6639AEE+, U28 LM75AIMM/NOPB, U29 LM75AIMM/NOPB

Commit message: Convert "~" and "~~" in .sch and .lib files to " "
cf. commit ef029e49 in Marble-Mini, May 21 2020
Parts:
- C190, C191, C192: ComponentHeight ~~ -> (none); PackageDescription ~~ -> (none); PressFit ~~ -> (none); Sense Comment ~~ -> (none); Status Comment ~~ -> (none)
- R129: ComponentHeight ~~ -> (none); PackageDescription ~~ -> (none); Power ~~ -> (none); Sense Comment ~~ -> (none); Status Comment ~~ -> (none); TC ~~ -> (none); Tolerance ~~ -> (none); Voltage ~~ -> (none)
- R130, R172, R173, R174, R175, R176, R177, R178: ComponentHeight ~~ -> (none); PackageDescription ~~ -> (none); Sense Comment ~~ -> (none); Status Comment ~~ -> (none); Voltage ~~ -> (none)
- U27: ComponentLink1Description ~~ -> (none); ComponentLink1URL ~~ -> (none); ComponentLink2Description ~~ -> (none); ComponentLink2URL ~~ -> (none); Sense Comment ~~ -> (none); Status ~~ -> (none); Status Comment ~~ -> (none)

Commit message: Remove some un-helpful attributes
Pole4
SCEM
Footprint Library
Database Table Name
HelpURL
ComponentLink1URL
ComponentLink2URL
CreateDate1
LatestRevisionDate1

cf. commits 8f7a3695 c705ea46 d128e165 ffe4a47d in Marble-Mini, May 21 2020
Cuts number of attrib_lint complaints in half, to 2334.
Parts:
- C188, C189: Database Table Name Capacitors SMD -> (none); Footprint Library Capacitors SMD -> (none); HelpURL \\\\cern.ch\\dfs\\Applications\\Altium\\Datasheets\\CC0402_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 -> (none)
- C190, C191, C192: HelpURL \\\\cern.ch\\dfs\\Applications\\Altium\\Datasheets\\CC0201_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 -> (none)
- C343, C344: Database Table Name Capacitors SMD -> (none); Footprint Library Capacitors SMD -> (none); HelpURL \\\\cern.ch\\dfs\\Applications\\Altium\\Datasheets\\CC0603_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 -> (none)
- R129, R130, R172, R173, R174, R175, R176, R177, R178: HelpURL \\\\cern.ch\\dfs\\Applications\\Altium\\Datasheets\\R0402_P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 -> (none)
- U27: ComponentLink1URL (none) -> (none); ComponentLink2URL (none) -> (none); HelpURL \\\\cern.ch\\dfs\\Applications\\Altium\\Datasheets\\MAX6639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 -> (none)
Changed lines of the file:
@@
 F 28 "SOP63P600X175-16N" H 3050 1290 60  0001 L CNN "Footprint Ref"
 F 29 "CERN DEM JLC" H 3050 1200 60  0001 L CNN "Author"
-F 30 "\\\\cern.ch\\dfs\\Applications\\Altium\\Datasheets\\MAX6639AEE+.pdf" H 3050 1110 60  0001 L CNN "HelpURL"
-F 31 " " H 3050 1020 60  0001 L CNN "ComponentLink1URL"
-F 32 " " H 3050 930 60  0001 L CNN "ComponentLink2URL"
 F 33 " " H 3050 840 60  0001 L CNN "ComponentLink2Description"
 F 34 " " H 3050 750 60  0001 L CNN "ComponentLink1Description"
@@
 F 33 "GRM188R61E475KE11D" H 9550 1760 60  0001 L CNN "Manufacturer1 Part Number"
 F 34 "0.95mm" H 9550 1670 60  0001 L CNN "Manufacturer1 ComponentHeight"
-F 35 "\\\\cern.ch\\dfs\\Applications\\Altium\\Datasheets\\CC0603_X7R_TAIYO-YUDEN_HIGH-VALUE.pdf" H 9550 1580 60  0001 L CNN "HelpURL"
 F 36 "CERN DEM JLC" H 9550 1490 60  0001 L CNN "Author"
 F 37 "11/10/14 00:00:00" H 9550 1400 60  0001 L CNN "CreateDate"
@@
 F 39 "Capacitors.DbLib" H 9550 1220 60  0001 L CNN "Library Name"
 F 40 "This work is licensed under the Creative Commons CC-BY-SA 4.0 License. To the extent that circuit schematics that use Licensed Material can be considered to be ‘Adapted Material’, then the copyright holder waives article 3.b of the license with respect to these schematics." H 9550 1130 60  0001 L CNN "License"
-F 41 "Capacitors SMD" H 9550 4900 50  0001 C CNN "Database Table Name"
-F 42 "Capacitors SMD" H 9550 4900 50  0001 C CNN "Footprint Library"
 	1    9550 4900
 	0    1    1    0
@@
 F 33 "GRM188R61E475KE11D" H 10000 1760 60  0001 L CNN "Manufacturer1 Part Number"
 F 34 "0.95mm" H 10000 1670 60  0001 L CNN "Manufacturer1 ComponentHeight"
-F 35 "\\\\cern.ch\\dfs\\Applications\\Altium\\Datasheets\\CC0603_X7R_TAIYO-YUDEN_HIGH-VALUE.pdf" H 10000 1580 60  0001 L CNN "HelpURL"
 F 36 "CERN DEM JLC" H 10000 1490 60  0001 L CNN "Author"
 F 37 "11/10/14 00:00:00" H 10000 1400 60  0001 L CNN "CreateDate"
@@
 F 39 "Capacitors.DbLib" H 10000 1220 60  0001 L CNN "Library Name"
 F 40 "This work is licensed under the Creative Commons CC-BY-SA 4.0 License. To the extent that circuit schematics that use Licensed Material can be considered to be ‘Adapted Material’, then the copyright holder waives article 3.b of the license with respect to these schematics." H 10000 1130 60  0001 L CNN "License"
-F 41 "Capacitors SMD" H 10000 4900 50  0001 C CNN "Database Table Name"
-F 42 "Capacitors SMD" H 10000 4900 50  0001 C CNN "Footprint Library"
 	1    10000 4900
 	0    1    1    0
@@
 F 33 "223858715623" H 1950 1860 60  0001 L CNN "Manufacturer1 Part Number"
 F 34 "0.55mm" H 1950 1770 60  0001 L CNN "Manufacturer1 ComponentHeight"
-F 35 "\\\\cern.ch\\dfs\\Applications\\Altium\\Datasheets\\CC0402_X7R_PHYCOMP.pdf" H 1950 1680 60  0001 L CNN "HelpURL"
 F 36 "CERN DEM JLC" H 1950 1590 60  0001 L CNN "Author"
 F 37 "12/03/07 00:00:00" H 1950 1500 60  0001 L CNN "CreateDate"
@@
 F 39 "Capacitors.DbLib" H 1950 1320 60  0001 L CNN "Library Name"
 F 40 "This work is licensed under the Creative Commons CC-BY-SA 4.0 License. To the extent that circuit schematics that use Licensed Material can be considered to be ‘Adapted Material’, then the copyright holder waives article 3.b of the license with respect to these schematics." H 1950 1230 60  0001 L CNN "License"
-F 41 "Capacitors SMD" H 1950 5000 50  0001 C CNN "Database Table Name"
-F 42 "Capacitors SMD" H 1950 5000 50  0001 C CNN "Footprint Library"
 	1    1950 5000
 	0    1    1    0
@@
 F 33 "223858715623" H 2400 1860 60  0001 L CNN "Manufacturer1 Part Number"
 F 34 "0.55mm" H 2400 1770 60  0001 L CNN "Manufacturer1 ComponentHeight"
-F 35 "\\\\cern.ch\\dfs\\Applications\\Altium\\Datasheets\\CC0402_X7R_PHYCOMP.pdf" H 2400 1680 60  0001 L CNN "HelpURL"
 F 36 "CERN DEM JLC" H 2400 1590 60  0001 L CNN "Author"
 F 37 "12/03/07 00:00:00" H 2400 1500 60  0001 L CNN "CreateDate"
@@
 F 39 "Capacitors.DbLib" H 2400 1320 60  0001 L CNN "Library Name"
 F 40 "This work is licensed under the Creative Commons CC-BY-SA 4.0 License. To the extent that circuit schematics that use Licensed Material can be considered to be ‘Adapted Material’, then the copyright holder waives article 3.b of the license with respect to these schematics." H 2400 1230 60  0001 L CNN "License"
-F 41 "Capacitors SMD" H 2400 5000 50  0001 C CNN "Database Table Name"
-F 42 "Capacitors SMD" H 2400 5000 50  0001 C CNN "Footprint Library"
 	1    2400 5000
 	0    1    1    0
@@
 F 33 "02016D104KAT2A" H 2400 2910 60  0001 L CNN "Manufacturer1 Part Number"
 F 34 "0.33mm" H 2400 2820 60  0001 L CNN "Manufacturer1 ComponentHeight"
-F 35 "\\\\cern.ch\\dfs\\Applications\\Altium\\Datasheets\\CC0201_X5R_AVX.pdf" H 2400 2730 60  0001 L CNN "HelpURL"
 F 36 "CERN DEM JLC" H 2400 2640 60  0001 L CNN "Author"
 F 37 "12/03/07 00:00:00" H 2400 2550 60  0001 L CNN "CreateDate"
@@
 F 33 "02016D104KAT2A" H 7300 10  60  0001 L CNN "Manufacturer1 Part Number"
 F 34 "0.33mm" H 7300 -80 60  0001 L CNN "Manufacturer1 ComponentHeight"
-F 35 "\\\\cern.ch\\dfs\\Applications\\Altium\\Datasheets\\CC0201_X5R_AVX.pdf" H 7300 -170 60  0001 L CNN "HelpURL"
 F 36 "CERN DEM JLC" H 7300 -260 60  0001 L CNN "Author"
 F 37 "12/03/07 00:00:00" H 7300 -350 60  0001 L CNN "CreateDate"
@@
 F 33 "02016D104KAT2A" H 7300 -1890 60  0001 L CNN "Manufacturer1 Part Number"
 F 34 "0.33mm" H 7300 -1980 60  0001 L CNN "Manufacturer1 ComponentHeight"
-F 35 "\\\\cern.ch\\dfs\\Applications\\Altium\\Datasheets\\CC0201_X5R_AVX.pdf" H 7300 -2070 60  0001 L CNN "HelpURL"
 F 36 "CERN DEM JLC" H 7300 -2160 60  0001 L CNN "Author"
 F 37 "12/03/07 00:00:00" H 7300 -2250 60  0001 L CNN "CreateDate"
@@
 F 34 "232270671003L" H 4200 1620 60  0001 L CNN "Manufacturer1 Part Number"
 F 35 "0.4mm" H 4200 1530 60  0001 L CNN "Manufacturer1 ComponentHeight"
-F 36 "\\\\cern.ch\\dfs\\Applications\\Altium\\Datasheets\\R0402_Phycomp_RC0402.pdf" H 4200 1440 60  0001 L CNN "HelpURL"
 F 37 "CERN DEM JLC" H 4200 1350 60  0001 L CNN "Author"
 F 38 "12/03/07 00:00:00" H 4200 1260 60  0001 L CNN "CreateDate"
@@
 F 34 "232270671003L" H 4400 1620 60  0001 L CNN "Manufacturer1 Part Number"
 F 35 "0.4mm" H 4400 1530 60  0001 L CNN "Manufacturer1 ComponentHeight"
-F 36 "\\\\cern.ch\\dfs\\Applications\\Altium\\Datasheets\\R0402_Phycomp_RC0402.pdf" H 4400 1440 60  0001 L CNN "HelpURL"
 F 37 "CERN DEM JLC" H 4400 1350 60  0001 L CNN "Author"
 F 38 "12/03/07 00:00:00" H 4400 1260 60  0001 L CNN "CreateDate"
@@
 F 34 "232270671003L" H 4600 1620 60  0001 L CNN "Manufacturer1 Part Number"
 F 35 "0.4mm" H 4600 1530 60  0001 L CNN "Manufacturer1 ComponentHeight"
-F 36 "\\\\cern.ch\\dfs\\Applications\\Altium\\Datasheets\\R0402_Phycomp_RC0402.pdf" H 4600 1440 60  0001 L CNN "HelpURL"
 F 37 "CERN DEM JLC" H 4600 1350 60  0001 L CNN "Author"
 F 38 "12/03/07 00:00:00" H 4600 1260 60  0001 L CNN "CreateDate"
@@
 F 34 "232270671003L" H 4800 1620 60  0001 L CNN "Manufacturer1 Part Number"
 F 35 "0.4mm" H 4800 1530 60  0001 L CNN "Manufacturer1 ComponentHeight"
-F 36 "\\\\cern.ch\\dfs\\Applications\\Altium\\Datasheets\\R0402_Phycomp_RC0402.pdf" H 4800 1440 60  0001 L CNN "HelpURL"
 F 37 "CERN DEM JLC" H 4800 1350 60  0001 L CNN "Author"
 F 38 "12/03/07 00:00:00" H 4800 1260 60  0001 L CNN "CreateDate"
@@
 F 34 "232270671003L" H 5000 1620 60  0001 L CNN "Manufacturer1 Part Number"
 F 35 "0.4mm" H 5000 1530 60  0001 L CNN "Manufacturer1 ComponentHeight"
-F 36 "\\\\cern.ch\\dfs\\Applications\\Altium\\Datasheets\\R0402_Phycomp_RC0402.pdf" H 5000 1440 60  0001 L CNN "HelpURL"
 F 37 "CERN DEM JLC" H 5000 1350 60  0001 L CNN "Author"
 F 38 "12/03/07 00:00:00" H 5000 1260 60  0001 L CNN "CreateDate"
@@
 F 34 "232270671003L" H 5350 1620 60  0001 L CNN "Manufacturer1 Part Number"
 F 35 "0.4mm" H 5350 1530 60  0001 L CNN "Manufacturer1 ComponentHeight"
-F 36 "\\\\cern.ch\\dfs\\Applications\\Altium\\Datasheets\\R0402_Phycomp_RC0402.pdf" H 5350 1440 60  0001 L CNN "HelpURL"
 F 37 "CERN DEM JLC" H 5350 1350 60  0001 L CNN "Author"
 F 38 "12/03/07 00:00:00" H 5350 1260 60  0001 L CNN "CreateDate"
@@
 F 34 "232270671003L" H 5650 1620 60  0001 L CNN "Manufacturer1 Part Number"
 F 35 "0.4mm" H 5650 1530 60  0001 L CNN "Manufacturer1 ComponentHeight"
-F 36 "\\\\cern.ch\\dfs\\Applications\\Altium\\Datasheets\\R0402_Phycomp_RC0402.pdf" H 5650 1440 60  0001 L CNN "HelpURL"
 F 37 "CERN DEM JLC" H 5650 1350 60  0001 L CNN "Author"
 F 38 "12/03/07 00:00:00" H 5650 1260 60  0001 L CNN "CreateDate"
@@
 F 34 "232270671003L" H 6300 -1980 60  0001 L CNN "Manufacturer1 Part Number"
 F 35 "0.4mm" H 6300 -2070 60  0001 L CNN "Manufacturer1 ComponentHeight"
-F 36 "\\\\cern.ch\\dfs\\Applications\\Altium\\Datasheets\\R0402_Phycomp_RC0402.pdf" H 6300 -2160 60  0001 L CNN "HelpURL"
 F 37 "CERN DEM JLC" H 6300 -2250 60  0001 L CNN "Author"
 F 38 "12/03/07 00:00:00" H 6300 -2340 60  0001 L CNN "CreateDate"
@@
 F 34 "232270591001L" H 1400 2120 60  0001 L CNN "Manufacturer1 Part Number"
 F 35 "0.4mm" H 1400 2030 60  0001 L CNN "Manufacturer1 ComponentHeight"
-F 36 "\\\\cern.ch\\dfs\\Applications\\Altium\\Datasheets\\R0402_Phycomp_RC0402.pdf" H 1400 1940 60  0001 L CNN "HelpURL"
 F 37 "CERN DEM JLC" H 1400 1850 60  0001 L CNN "Author"
 F 38 "12/03/07 00:00:00" H 1400 1760 60  0001 L CNN "CreateDate"
