File: design/FPGA_12_13.sch (KiCad schematic (older format))
At the start: 5 parts, among them U1 XC7K160T-2FFG676C, U51 TXB0104D

Commit message: alternative part numbers, two footprints for INA219
Parts:
- U1: Manufacturer Part Number XC7K160T-2FFG676C -> XC7K160T-2FFG676C or XC7K160T-3FFG676E
Changed lines of the file:
@@
 F 3 "" H 8600 5150 50  0000 C CNN
 F 4 "XILINX" H 8600 5150 50  0001 C CNN "Manufacturer"
-F 5 "XC7K160T-2FFG676C" H 8600 5150 50  0001 C CNN "Manufacturer Part Number"
+F 5 "XC7K160T-2FFG676C or XC7K160T-3FFG676E" H 8600 5150 50  0001 C CNN "Manufacturer Part Number"
 	1    8600 5150
 	1    0    0    -1
