File: design/FPGA_32_16.sch (KiCad schematic (older format))
At the start: 3 parts, among them U1 XC7K160T-2FFG676C

Commit message: alternative part numbers, two footprints for INA219
Parts:
- U1: Manufacturer Part Number XC7K160T-2FFG676C -> XC7K160T-2FFG676C or XC7K160T-3FFG676E
Changed lines of the file:
@@
 F 3 "" H 7250 3900 50  0000 C CNN
 F 4 "XILINX" H 7250 3900 50  0001 C CNN "Manufacturer"
-F 5 "XC7K160T-2FFG676C" H 7250 3900 50  0001 C CNN "Manufacturer Part Number"
+F 5 "XC7K160T-2FFG676C or XC7K160T-3FFG676E" H 7250 3900 50  0001 C CNN "Manufacturer Part Number"
 	3    7250 3900
 	-1   0    0    -1
