File: design/SDRAM.sch (KiCad schematic (older format))
At the start: 12 parts, among them IC1 MT8JTF12864HZ-1G6G1 or VR7PU2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, U31 TPS51200DRC

Commit message: alternative part numbers, two footprints for INA219
Parts:
- IC1: Manufacturer Part Number MT8JTF12864HZ-1G6G1 -> MT8JTF12864HZ-1G6G1 or VR7PU286458FBAMJT
Changed lines of the file:
@@
 F 13 "1Gb (128Mx64) SODIMM 204-Pin DDR3 SDRAM Module" H 2700 -5375 50  0001 L CNN "Part Description"
 F 14 "MICRON TECHNOLOGY" H 2700 -5450 50  0001 L CNN "Manufacturer"
-F 15 "MT8JTF12864HZ-1G6G1" H 2700 -5525 50  0001 L CNN "Manufacturer Part Number"
+F 15 "MT8JTF12864HZ-1G6G1 or VR7PU286458FBAMJT" H 2700 -5525 50  0001 L CNN "Manufacturer Part Number"
 F 16 "0" H 2700 -5600 50  0001 L CNN "Pin Count"
 F 17 "SODIMM" H 2700 -5675 50  0001 L CNN "Case"

Commit message: Fuss with schematic attributes
Add Manufacturer field for MYRGC075050R31RA NA219AIDR ADM7155ACPZ-02-R7
Mark IC1 (DDR3 module) dnf
Make Part Number attribute for DDR3 visible on schematic
Parts:
- IC1: config (none) -> dnf
Changed lines of the file:
@@
 F 2 "ICs And Semiconductors SMD:SODIMM60P6760X3000X380-204" H 7700 -4550 50  0001 L CNN
 F 3 " " H 7700 -4625 50  0001 L CNN
-F 4 "MT8JTF12864HZ-1G6G1 or VR7PU286458FBAMJT" H 7700 -4700 50  0001 L CNN "Part Number"
+F 4 "MT8JTF12864HZ-1G6G1 or VR7PU286458FBAMJT" H 7350 -4550 50  0000 L CNN "Part Number"
 F 5 "MT8JTF12864HZ" H 7700 -4775 50  0001 L CNN "Library Ref"
 F 6 "SchLib\\Logic.SchLib" H 7700 -4850 50  0001 L CNN "Library Path"
@@
 F 34 "ICs And Semiconductors.DbLib" H 7700 -7100 50  0001 L CNN "Library Name"
 F 35 "This work is licensed under the Creative Commons CC-BY-SA 4.0 License. To the extent that circuit schematics that use Licensed Material can be considered to be ‘Adapted Material’, then the copyright holder waives article 3.b of the license with respect to these schematics." H 7700 -7250 50  0001 L CNN "License"
+F 36 "dnf" H 8250 -4650 50  0000 C CNN "config"
 	2    7700 900
 	1    0    0    -1
