File: design/FMC_1.sch (KiCad schematic (older format))
At the start: 16 parts, among them P1 SAMTEC_ASP-134486-01, U43 MIC2090-1YM5TR

Commit message: alternative part numbers, two footprints for INA219
Parts:
- U43: Manufacturer Part Number MIC2090-1YM5 -> MIC2090-1YM5 or FPF2116
Changed lines of the file:
@@
 F 5 "SOT-23-5" H 13800 3800 50  0001 L BNN "Case"
 F 6 "MICREL SEMICONDUCTOR" H 13800 4100 50  0001 L BNN "Manufacturer"
-F 7 "MIC2090-1YM5" H 13800 4600 50  0001 C CNN "Manufacturer Part Number"
+F 7 "MIC2090-1YM5 or FPF2116" H 13800 4600 50  0001 C CNN "Manufacturer Part Number"
 	1    13800 4600
 	-1   0    0    -1

Commit message: fixed issues with: 1V5 rail, FMC pins, I2C pull-up resistors
Connections:
- no-connect marks 133 -> 135
Changed lines of the file:
@@
-$Comp
-L power:+2V5 #PWR?
-U 1 1 5F088825
-P 12850 9400
-AR Path="/5BD31F9F/5F088825" Ref="#PWR?"  Part="1"
-AR Path="/5BD31F9A/5F088825" Ref="#PWR0121"  Part="1"
-F 0 "#PWR0121" H 12850 9250 50  0001 C CNN
-F 1 "+2V5" V 12865 9528 50  0000 L CNN
-F 2 "" H 12850 9400 50  0001 C CNN
-F 3 "" H 12850 9400 50  0001 C CNN
-	1    12850 9400
-	0    -1   -1   0
-$EndComp
-$Comp
-L power:+2V5 #PWR?
-U 1 1 5F08882B
-P 10200 10250
-AR Path="/5BD31F9F/5F08882B" Ref="#PWR?"  Part="1"
-AR Path="/5BD31F9A/5F08882B" Ref="#PWR0124"  Part="1"
-F 0 "#PWR0124" H 10200 10100 50  0001 C CNN
-F 1 "+2V5" V 10215 10378 50  0000 L CNN
-F 2 "" H 10200 10250 50  0001 C CNN
-F 3 "" H 10200 10250 50  0001 C CNN
-	1    10200 10250
-	0    -1   -1   0
-$EndComp
 $Comp
 L power:+2V5 #PWR?
@@
 NoConn ~ 8700 6450
 NoConn ~ 13600 5500
+NoConn ~ 12850 9400
+NoConn ~ 10200 10250
 $EndSCHEMATC

Commit message: VIO_B_M2Cs connected to MMC's adc inputs
Connections:
- net labels added: VIO_B_M2C
- no-connect marks 135 -> 133
Changed lines of the file:
@@
 NoConn ~ 8700 6450
 NoConn ~ 13600 5500
-NoConn ~ 12850 9400
-NoConn ~ 10200 10250
+Text HLabel 10200 10250 0    50   Output ~ 0
+VIO_B_M2C
+Text Label 10300 10250 0    50   ~ 0
+VIO_B_M2C
+Text Label 12850 9400 0    50   ~ 0
+VIO_B_M2C
 $EndSCHEMATC
