File: design/FMC_2.sch (KiCad schematic (older format))
At the start: 16 parts, among them P2 SAMTEC_ASP-134486-01, U55 MIC2090-1YM5TR

Commit message: alternative part numbers, two footprints for INA219
Parts:
- U55: Manufacturer Part Number MIC2090-1YM5 -> MIC2090-1YM5 or FPF2116
Changed lines of the file:
@@
 F 5 "SOT-23-5" H 13850 4000 50  0001 L BNN "Case"
 F 6 "MICREL SEMICONDUCTOR" H 13850 4300 50  0001 L BNN "Manufacturer"
-F 7 "MIC2090-1YM5" H 13850 4800 50  0001 C CNN "Manufacturer Part Number"
+F 7 "MIC2090-1YM5 or FPF2116" H 13850 4800 50  0001 C CNN "Manufacturer Part Number"
 	1    13850 4800
 	-1   0    0    -1

Commit message: fixed issues with: 1V5 rail, FMC pins, I2C pull-up resistors
Changed lines of the file:
@@
 FMC2_HA23_N
-$Comp
-L power:+2V5 #PWR0678
-U 1 1 5D9281BB
-P 12400 9550
-F 0 "#PWR0678" H 12400 9400 50  0001 C CNN
-F 1 "+2V5" V 12415 9678 50  0000 L CNN
-F 2 "" H 12400 9550 50  0001 C CNN
-F 3 "" H 12400 9550 50  0001 C CNN
-	1    12400 9550
-	0    -1   -1   0
-$EndComp
-$Comp
-L power:+2V5 #PWR0679
-U 1 1 5D931FAD
-P 9750 10400
-F 0 "#PWR0679" H 9750 10250 50  0001 C CNN
-F 1 "+2V5" V 9765 10528 50  0000 L CNN
-F 2 "" H 9750 10400 50  0001 C CNN
-F 3 "" H 9750 10400 50  0001 C CNN
-	1    9750 10400
-	0    -1   -1   0
-$EndComp
 $Comp
 L power:+2V5 #PWR0685

Commit message: VIO_B_M2Cs connected to MMC's adc inputs
Connections:
- net labels added: VIO_B_M2C
Changed lines of the file:
@@
 NoConn ~ 13150 6050
 NoConn ~ 8250 6600
+Text HLabel 9750 10400 0    50   Output ~ 0
+VIO_B_M2C
+Text Label 9750 10400 0    50   ~ 0
+VIO_B_M2C
+Text Label 12400 9550 0    50   ~ 0
+VIO_B_M2C
+Text HLabel 12400 9550 0    50   Output ~ 0
+VIO_B_M2C
 $EndSCHEMATC
