File: design/MGT_CLK_Crosspoint.sch (KiCad schematic (older format))
At the start: 54 parts, among them J2 HIROSE_U.FL-R-SMT-1(10), J3 HIROSE_U.FL-R-SMT-1(10), J5 HIROSE_U.FL-R-SMT-1(10), J7 HIROSE_U.FL-R-SMT-1(10), U2 ADN4600ACPZ

Commit message: Get rid of unicode in output BOM CSV
Strip them out with the non_generic.py program
Mostly no-value-added characters like trademark
Descriptions are still readable without degree and +/- symbols
Adjust the ADN4600 description to use x instead of a fancy unicode times
Parts:
- U2: Part Description 4.25Gbps, 8 × 8, Asynchronous Crosspoint Switch -> 4.25Gbps, 8 x 8, Asynchronous Crosspoint Switch
Changed lines of the file:
@@
 F 11 "QFN, 0.50mm Pitch, Square; 64 Pin, 9.00mm L X 9.00mm W X 1.00mm H body (6.15mm X 6.15mm Thermal Tab), IPC Medium Density" H 5100 -2925 50  0001 L CNN "PackageDescription"
 F 12 " " H 5100 -3000 50  0001 L CNN "Status"
-F 13 "4.25Gbps, 8 × 8, Asynchronous Crosspoint Switch" H 5100 -3075 50  0001 L CNN "Part Description"
+F 13 "4.25Gbps, 8 x 8, Asynchronous Crosspoint Switch" H 5100 -3075 50  0001 L CNN "Part Description"
 F 14 "ANALOG DEVICES" H 5100 -3150 50  0001 L CNN "Manufacturer"
 F 15 "ADN4600ACPZ" H 5100 -3225 50  0001 L CNN "Manufacturer Part Number"
@@
 F 11 "QFN, 0.50mm Pitch, Square; 64 Pin, 9.00mm L X 9.00mm W X 1.00mm H body (6.15mm X 6.15mm Thermal Tab), IPC Medium Density" H 5100 525 50  0001 L CNN "PackageDescription"
 F 12 " " H 5100 450 50  0001 L CNN "Status"
-F 13 "4.25Gbps, 8 × 8, Asynchronous Crosspoint Switch" H 5100 375 50  0001 L CNN "Part Description"
+F 13 "4.25Gbps, 8 x 8, Asynchronous Crosspoint Switch" H 5100 375 50  0001 L CNN "Part Description"
 F 14 "ANALOG DEVICES" H 5100 300 50  0001 L CNN "Manufacturer"
 F 15 "ADN4600ACPZ" H 5100 225 50  0001 L CNN "Manufacturer Part Number"
