File: design/FPGA_33_34.sch (KiCad schematic (older format))
At the start: 21 parts, among them Q15 NX3008NBKV, U1 XC7K160T-2FFG676C, U42 TXB0108PW

Commit message: Update part numbers to be closer to as-manufactured
new (at least in form) listings:
Murata  GRM188R61A106KA73D
Samsung  CL32A107MQVNNWE
Yageo  AC0402FR-0722R
Yageo  RT0402BRD0710KL
Stackpole  RMCF0402FT82K0
NXP SEMICONDUCTORS  PRTR5V0U2X,215
FTDI  FT4232H-56Q-REEL
TEXAS INSTRUMENTS  CDCM61004RHB
TEXAS INSTRUMENTS  TLV62565DBVR
TEXAS INSTRUMENTS  TPS3703A7330DSER
XILINX  XC7K160T-2FFG676I
SILICON LABS  570NCB000933DG
IQD FREQUENCY PRODUCTS  ECS-VXO-73-20.00-TR
Parts:
- U1: Manufacturer Part Number XC7K160T-2FFG676C or XC7K160T-3FFG676E -> XC7K160T-2FFG676I
Changed lines of the file:
@@
 F 3 "" H 8350 4650 50  0000 C CNN
 F 4 "XILINX" H 8350 4650 50  0001 C CNN "Manufacturer"
-F 5 "XC7K160T-2FFG676C or XC7K160T-3FFG676E" H 8350 4650 50  0001 C CNN "Manufacturer Part Number"
+F 5 "XC7K160T-2FFG676I" H 8350 4650 50  0001 C CNN "Manufacturer Part Number"
 	4    8350 4650
 	1    0    0    -1

Commit message: Update more "Manufacturer Part Number"
Corresponding to specific parts that are actually usable and available.

PANASONIC EEEFK1C471AP or 16SEV470M8X10.5 becomes NICHICON UCD1C471MNL1GS
  (described as 470 uF on schematic)
INFINEON BAT165AX or BAT165E6327HTSA1 becomes BAT165E6327HTSA1
  (described as BAT165 on schematic)
VISHAY GENERAL SEMICONDUCTOR SS16 or SS16FP becomes ONSEMI SS16FP
  (schematic simply shows Schottky diode)
NXP SEMICONDUCTORS BC857BV or BCM857BV,115 becomes MICRO COMMERCIAL BC857BV-TP
  (described as BC857BV on schematic)
NXP NX3008NBKV or SI1036X-T1-GE3 becomes VISHAY SILICONIX SI1036X-T1-GE3
  (changed marking on schematic to SI1036X)
ST MICROELECTRONICS STS8DN6LF6AG or SQ4920EY-T1_BE3 becomes VISHAY SILICONIX SQ4920EY-T1_GE3
  (changed marking on schematic to SQ4920EY)
NXP SEMICONDUCTORS 74AHC1G04GW becomes NEXPERIA 74AHC1G04GW-Q100H
  (schematic simply shows generic logic inverter)
Monolithic Power Systems (MPS) MPM3830GQV-P becomes Monolithic Power Systems (MPS) MPM3830GQVP
  (changed marking on schematic to MPM3830GQV)
TEXAS INSTRUMENTS SN74LVC1G125DCKT or SN74AUC1G17DCKR becomes TEXAS INSTRUMENTS SN74LVC1G125DCK3
  (schematic simply shows generic logic buffer)
Parts:
- Q15: value NX3008NBKV -> SI1036X; symbol Transistors:NX3008NBKV -> Transistors:SI1036X; Manufacturer NXP -> VISHAY SILICONIX; Manufacturer Part Number NX3008NBKV or SI1036X-T1-GE3 -> SI1036X-T1-GE3
Changed lines of the file:
@@
 	4200 9650 3850 9650
 $Comp
-L Transistors:NX3008NBKV Q?
+L Transistors:SI1036X Q?
 U 1 1 60B13CE1
 P 3350 9650
@@
 AR Path="/5C907554/5C721515/60B13CE1" Ref="Q15"  Part="1"
 F 0 "Q15" H 3350 9450 50  0000 L CNN
-F 1 "NX3008NBKV" H 3150 9300 50  0000 L CNN
+F 1 "SI1036X" H 3150 9300 50  0000 L CNN
 F 2 "ICs And Semiconductors SMD:SOTFL50P160X60-6N" H 3350 9650 50  0001 C CNN
 F 3 "" H 3350 9650 50  0001 C CNN
-F 4 "NXP" H 3350 9650 50  0001 C CNN "Manufacturer"
-F 5 "NX3008NBKV or SI1036X-T1-GE3" H 3350 9650 50  0001 C CNN "Manufacturer Part Number"
+F 4 "VISHAY SILICONIX" H 3350 9650 50  0001 C CNN "Manufacturer"
+F 5 "SI1036X-T1-GE3" H 3350 9650 50  0001 C CNN "Manufacturer Part Number"
 	1    3350 9650
 	-1   0    0    -1
 $EndComp
 $Comp
-L Transistors:NX3008NBKV Q?
+L Transistors:SI1036X Q?
 U 2 1 60B13CE9
 P 3950 9350
@@
 AR Path="/5C907554/5C721515/60B13CE9" Ref="Q15"  Part="2"
 F 0 "Q15" H 3950 9100 50  0000 L CNN
-F 1 "NX3008NBKV" H 3750 8950 50  0000 L CNN
+F 1 "SI1036X" H 3750 8950 50  0000 L CNN
 F 2 "ICs And Semiconductors SMD:SOTFL50P160X60-6N" H 3950 9350 50  0001 C CNN
 F 3 "" H 3950 9350 50  0001 C CNN
-F 4 "NXP" H 3950 9350 50  0001 C CNN "Manufacturer"
-F 5 "NX3008NBKV or SI1036X-T1-GE3" H 3950 9350 50  0001 C CNN "Manufacturer Part Number"
+F 4 "VISHAY SILICONIX" H 3950 9350 50  0001 C CNN "Manufacturer"
+F 5 "SI1036X-T1-GE3" H 3950 9350 50  0001 C CNN "Manufacturer Part Number"
 	2    3950 9350
 	-1   0    0    -1
