File: design/Power.sch (KiCad schematic (older format))
At the start: 76 parts, among them J1 CLIFF_FC68148(DC-10A), J19 TE_641119-2, Q1 BC857BV, Q16 SI4425DDY-T1-GE3, Q2 SI4425DDY-T1-GE3, Q22 BC857BV, Q23 SI4425DDY-T1-GE3, Q4 SI4425DDY-T1-GE3, Q8 BSS138LT1G, Q9 BSS138LT1G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

Commit message: BOM: switch P-MOSFET from SI4425DDY-T1-GE3 to SI4459BDY-T1-GE3
more modern part with half the on-resistance, and actually available in 2022
Parts:
- Q16, Q2, Q23, Q4: value SI4425DDY-T1-GE3 -> SI4459BDY-T1-GE3; symbol Transistors:SI4425DDY-T1-GE3 -> Transistors:SI4459BDY-T1-GE3; Device SI4425DDY-T1-GE3 -> SI4459BDY-T1-GE3; Library Ref SI4425DDY -> SI4459BDY; Manufacturer Part Number SI4425DDY-T1-GE3 or SI4459BDY-T1-GE3 -> SI4459BDY-T1-GE3; Part Description -30V -19.7A P-Channel MOSFET -> -30V -20A P-Channel MOSFET; Part Number SI4425DDY-T1-GE3 -> SI4459BDY-T1-GE3
Changed lines of the file:
@@
 	12550 5300 12550 6000
 $Comp
-L Transistors:SI4425DDY-T1-GE3 Q16
+L Transistors:SI4459BDY-T1-GE3 Q16
 U 1 1 5D111201
 P 11450 1700
 F 0 "Q16" H 11978 1496 50  0000 L CNN
-F 1 "SI4425DDY-T1-GE3" H 11978 1405 50  0000 L CNN
+F 1 "SI4459BDY-T1-GE3" H 11978 1405 50  0000 L CNN
 F 2 "ICs And Semiconductors SMD:SOIC127P600X175-8N" H 11450 -60 60  0001 L CNN
 F 3 "" H 11450 660 60  0001 L CNN
-F 4 "SI4425DDY-T1-GE3" H 11450 570 60  0001 L CNN "Part Number"
-F 5 "SI4425DDY" H 11450 480 60  0001 L CNN "Library Ref"
+F 4 "SI4459BDY-T1-GE3" H 11450 570 60  0001 L CNN "Part Number"
+F 5 "SI4459BDY" H 11450 480 60  0001 L CNN "Library Ref"
 F 6 "SchLib\\Transistors.SchLib" H 11450 390 60  0001 L CNN "Library Path"
 F 7 "=Device" H 11450 300 60  0001 L CNN "Comment"
 F 8 "Standard" H 11450 210 60  0001 L CNN "Component Kind"
 F 9 "Standard" H 11450 120 60  0001 L CNN "Component Type"
-F 10 "SI4425DDY-T1-GE3" H 11450 30  60  0001 L CNN "Device"
+F 10 "SI4459BDY-T1-GE3" H 11450 30  60  0001 L CNN "Device"
 F 11 "SOIC 8, Pitch 1.27mm - Body 4x5mm, IPC Medium Density" H 11450 -150 60  0001 L CNN "PackageDescription"
 F 12 " " H 11450 -240 60  0001 L CNN "Status"
-F 13 "-30V -19.7A P-Channel MOSFET" H 11450 -330 60  0001 L CNN "Part Description"
+F 13 "-30V -20A P-Channel MOSFET" H 11450 -330 60  0001 L CNN "Part Description"
 F 14 "VISHAY SILICONIX" H 11450 -420 60  0001 L CNN "Manufacturer"
-F 15 "SI4425DDY-T1-GE3 or SI4459BDY-T1-GE3" H 11450 -510 60  0001 L CNN "Manufacturer Part Number"
+F 15 "SI4459BDY-T1-GE3" H 11450 -510 60  0001 L CNN "Manufacturer Part Number"
 F 16 "8" H 11450 -600 60  0001 L CNN "Pin Count"
 F 17 "SOIC8" H 11450 -690 60  0001 L CNN "Case"
@@
 	11650 1000 11750 1000
 $Comp
-L Transistors:SI4425DDY-T1-GE3 Q23
+L Transistors:SI4459BDY-T1-GE3 Q23
 U 1 1 5D1DA1B3
 P 11450 5100
 F 0 "Q23" H 11978 4896 50  0000 L CNN
-F 1 "SI4425DDY-T1-GE3" H 11978 4805 50  0000 L CNN
+F 1 "SI4459BDY-T1-GE3" H 11978 4805 50  0000 L CNN
 F 2 "ICs And Semiconductors SMD:SOIC127P600X175-8N" H 11450 3340 60  0001 L CNN
-F 3 "\\\\cern.ch\\dfs\\Applications\\Altium\\Datasheets\\SI4425DDY-T1-GE3.pdf" H 11450 4060 60  0001 L CNN
-F 4 "SI4425DDY-T1-GE3" H 11450 3970 60  0001 L CNN "Part Number"
-F 5 "SI4425DDY" H 11450 3880 60  0001 L CNN "Library Ref"
+F 3 "\\\\cern.ch\\dfs\\Applications\\Altium\\Datasheets\\SI4459BDY-T1-GE3.pdf" H 11450 4060 60  0001 L CNN
+F 4 "SI4459BDY-T1-GE3" H 11450 3970 60  0001 L CNN "Part Number"
+F 5 "SI4459BDY" H 11450 3880 60  0001 L CNN "Library Ref"
 F 6 "SchLib\\Transistors.SchLib" H 11450 3790 60  0001 L CNN "Library Path"
 F 7 "=Device" H 11450 3700 60  0001 L CNN "Comment"
 F 8 "Standard" H 11450 3610 60  0001 L CNN "Component Kind"
 F 9 "Standard" H 11450 3520 60  0001 L CNN "Component Type"
-F 10 "SI4425DDY-T1-GE3" H 11450 3430 60  0001 L CNN "Device"
+F 10 "SI4459BDY-T1-GE3" H 11450 3430 60  0001 L CNN "Device"
 F 11 "SOIC 8, Pitch 1.27mm - Body 4x5mm, IPC Medium Density" H 11450 3250 60  0001 L CNN "PackageDescription"
 F 12 " " H 11450 3160 60  0001 L CNN "Status"
-F 13 "-30V -19.7A P-Channel MOSFET" H 11450 3070 60  0001 L CNN "Part Description"
+F 13 "-30V -20A P-Channel MOSFET" H 11450 3070 60  0001 L CNN "Part Description"
 F 14 "VISHAY SILICONIX" H 11450 2980 60  0001 L CNN "Manufacturer"
-F 15 "SI4425DDY-T1-GE3 or SI4459BDY-T1-GE3" H 11450 2890 60  0001 L CNN "Manufacturer Part Number"
+F 15 "SI4459BDY-T1-GE3" H 11450 2890 60  0001 L CNN "Manufacturer Part Number"
 F 16 "8" H 11450 2800 60  0001 L CNN "Pin Count"
 F 17 "SOIC8" H 11450 2710 60  0001 L CNN "Case"
@@
 Connection ~ 11550 1000
 $Comp
-L Transistors:SI4425DDY-T1-GE3 Q2
+L Transistors:SI4459BDY-T1-GE3 Q2
 U 1 1 5D2D0F80
 P 2750 2250
 F 0 "Q2" V 3400 1950 50  0000 C CNN
-F 1 "SI4425DDY-T1-GE3" V 3300 2000 50  0000 C CNN
+F 1 "SI4459BDY-T1-GE3" V 3300 2000 50  0000 C CNN
 F 2 "ICs And Semiconductors SMD:SOIC127P600X175-8N" H 2750 490 60  0001 L CNN
-F 3 "\\\\cern.ch\\dfs\\Applications\\Altium\\Datasheets\\SI4425DDY-T1-GE3.pdf" H 2750 1210 60  0001 L CNN
-F 4 "SI4425DDY-T1-GE3" H 2750 1120 60  0001 L CNN "Part Number"
-F 5 "SI4425DDY" H 2750 1030 60  0001 L CNN "Library Ref"
+F 3 "\\\\cern.ch\\dfs\\Applications\\Altium\\Datasheets\\SI4459BDY-T1-GE3.pdf" H 2750 1210 60  0001 L CNN
+F 4 "SI4459BDY-T1-GE3" H 2750 1120 60  0001 L CNN "Part Number"
+F 5 "SI4459BDY" H 2750 1030 60  0001 L CNN "Library Ref"
 F 6 "SchLib\\Transistors.SchLib" H 2750 940 60  0001 L CNN "Library Path"
 F 7 "=Device" H 2750 850 60  0001 L CNN "Comment"
 F 8 "Standard" H 2750 760 60  0001 L CNN "Component Kind"
 F 9 "Standard" H 2750 670 60  0001 L CNN "Component Type"
-F 10 "SI4425DDY-T1-GE3" H 2750 580 60  0001 L CNN "Device"
+F 10 "SI4459BDY-T1-GE3" H 2750 580 60  0001 L CNN "Device"
 F 11 "SOIC 8, Pitch 1.27mm - Body 4x5mm, IPC Medium Density" H 2750 400 60  0001 L CNN "PackageDescription"
 F 12 " " H 2750 310 60  0001 L CNN "Status"
-F 13 "-30V -19.7A P-Channel MOSFET" H 2750 220 60  0001 L CNN "Part Description"
+F 13 "-30V -20A P-Channel MOSFET" H 2750 220 60  0001 L CNN "Part Description"
 F 14 "VISHAY SILICONIX" H 2750 130 60  0001 L CNN "Manufacturer"
-F 15 "SI4425DDY-T1-GE3 or SI4459BDY-T1-GE3" H 2750 40  60  0001 L CNN "Manufacturer Part Number"
+F 15 "SI4459BDY-T1-GE3" H 2750 40  60  0001 L CNN "Manufacturer Part Number"
 F 16 "8" H 2750 -50 60  0001 L CNN "Pin Count"
 F 17 "SOIC8" H 2750 -140 60  0001 L CNN "Case"
@@
 $EndComp
 $Comp
-L Transistors:SI4425DDY-T1-GE3 Q4
+L Transistors:SI4459BDY-T1-GE3 Q4
 U 1 1 5D30F7F4
 P 8850 8850
 F 0 "Q4" V 9500 8550 50  0000 C CNN
-F 1 "SI4425DDY-T1-GE3" V 9400 8600 50  0000 C CNN
+F 1 "SI4459BDY-T1-GE3" V 9400 8600 50  0000 C CNN
 F 2 "ICs And Semiconductors SMD:SOIC127P600X175-8N" H 8850 7090 60  0001 L CNN
-F 3 "\\\\cern.ch\\dfs\\Applications\\Altium\\Datasheets\\SI4425DDY-T1-GE3.pdf" H 8850 7810 60  0001 L CNN
-F 4 "SI4425DDY-T1-GE3" H 8850 7720 60  0001 L CNN "Part Number"
-F 5 "SI4425DDY" H 8850 7630 60  0001 L CNN "Library Ref"
+F 3 "\\\\cern.ch\\dfs\\Applications\\Altium\\Datasheets\\SI4459BDY-T1-GE3.pdf" H 8850 7810 60  0001 L CNN
+F 4 "SI4459BDY-T1-GE3" H 8850 7720 60  0001 L CNN "Part Number"
+F 5 "SI4459BDY" H 8850 7630 60  0001 L CNN "Library Ref"
 F 6 "SchLib\\Transistors.SchLib" H 8850 7540 60  0001 L CNN "Library Path"
 F 7 "=Device" H 8850 7450 60  0001 L CNN "Comment"
 F 8 "Standard" H 8850 7360 60  0001 L CNN "Component Kind"
 F 9 "Standard" H 8850 7270 60  0001 L CNN "Component Type"
-F 10 "SI4425DDY-T1-GE3" H 8850 7180 60  0001 L CNN "Device"
+F 10 "SI4459BDY-T1-GE3" H 8850 7180 60  0001 L CNN "Device"
 F 11 "SOIC 8, Pitch 1.27mm - Body 4x5mm, IPC Medium Density" H 8850 7000 60  0001 L CNN "PackageDescription"
 F 12 " " H 8850 6910 60  0001 L CNN "Status"
-F 13 "-30V -19.7A P-Channel MOSFET" H 8850 6820 60  0001 L CNN "Part Description"
+F 13 "-30V -20A P-Channel MOSFET" H 8850 6820 60  0001 L CNN "Part Description"
 F 14 "VISHAY SILICONIX" H 8850 6730 60  0001 L CNN "Manufacturer"
-F 15 "SI4425DDY-T1-GE3 or SI4459BDY-T1-GE3" H 8850 6640 60  0001 L CNN "Manufacturer Part Number"
+F 15 "SI4459BDY-T1-GE3" H 8850 6640 60  0001 L CNN "Manufacturer Part Number"
 F 16 "8" H 8850 6550 60  0001 L CNN "Pin Count"
 F 17 "SOIC8" H 8850 6460 60  0001 L CNN "Case"

Commit message: Update more "Manufacturer Part Number"
Corresponding to specific parts that are actually usable and available.

PANASONIC EEEFK1C471AP or 16SEV470M8X10.5 becomes NICHICON UCD1C471MNL1GS
  (described as 470 uF on schematic)
INFINEON BAT165AX or BAT165E6327HTSA1 becomes BAT165E6327HTSA1
  (described as BAT165 on schematic)
VISHAY GENERAL SEMICONDUCTOR SS16 or SS16FP becomes ONSEMI SS16FP
  (schematic simply shows Schottky diode)
NXP SEMICONDUCTORS BC857BV or BCM857BV,115 becomes MICRO COMMERCIAL BC857BV-TP
  (described as BC857BV on schematic)
NXP NX3008NBKV or SI1036X-T1-GE3 becomes VISHAY SILICONIX SI1036X-T1-GE3
  (changed marking on schematic to SI1036X)
ST MICROELECTRONICS STS8DN6LF6AG or SQ4920EY-T1_BE3 becomes VISHAY SILICONIX SQ4920EY-T1_GE3
  (changed marking on schematic to SQ4920EY)
NXP SEMICONDUCTORS 74AHC1G04GW becomes NEXPERIA 74AHC1G04GW-Q100H
  (schematic simply shows generic logic inverter)
Monolithic Power Systems (MPS) MPM3830GQV-P becomes Monolithic Power Systems (MPS) MPM3830GQVP
  (changed marking on schematic to MPM3830GQV)
TEXAS INSTRUMENTS SN74LVC1G125DCKT or SN74AUC1G17DCKR becomes TEXAS INSTRUMENTS SN74LVC1G125DCK3
  (schematic simply shows generic logic buffer)
Parts:
- C350: Manufacturer PANASONIC -> NICHICON; Manufacturer Part Number EEEFK1C471AP or 16SEV470M8X10.5 -> UCD1C471MNL1GS
- D12, D4: Manufacturer VISHAY GENERAL SEMICONDUCTOR -> ONSEMI; Manufacturer Part Number SS16 or SS16FP -> SS16FP
- Q1, Q22: Manufacturer NXP SEMICONDUCTORS -> MICRO COMMERCIAL; Manufacturer Part Number BC857BV or BCM857BV,115 -> BC857BV-TP
Changed lines of the file:
@@
 F 14 " " H 1900 1400 60  0001 L CNN "Status"
 F 15 "Surface Mount Schottky Barrier Rectifier" H 1900 1310 60  0001 L CNN "Part Description"
-F 16 "VISHAY GENERAL SEMICONDUCTOR" H 1900 1220 60  0001 L CNN "Manufacturer"
-F 17 "SS16 or SS16FP" H 1900 1130 60  0001 L CNN "Manufacturer Part Number"
+F 16 "ONSEMI" H 1900 1220 60  0001 L CNN "Manufacturer"
+F 17 "SS16FP" H 1900 1130 60  0001 L CNN "Manufacturer Part Number"
 F 18 "2" H 1900 1040 60  0001 L CNN "Pin Count"
 F 19 "DO-214AC" H 1900 950 60  0001 L CNN "Case"
@@
 F 14 " " H 7900 6950 60  0001 L CNN "Status"
 F 15 "Surface Mount Schottky Barrier Rectifier" H 7900 6860 60  0001 L CNN "Part Description"
-F 16 "VISHAY GENERAL SEMICONDUCTOR" H 7900 6770 60  0001 L CNN "Manufacturer"
-F 17 "SS16 or SS16FP" H 7900 6680 60  0001 L CNN "Manufacturer Part Number"
+F 16 "ONSEMI" H 7900 6770 60  0001 L CNN "Manufacturer"
+F 17 "SS16FP" H 7900 6680 60  0001 L CNN "Manufacturer Part Number"
 F 18 "2" H 7900 6590 60  0001 L CNN "Pin Count"
 F 19 "DO-214AC" H 7900 6500 60  0001 L CNN "Case"
@@
 F 20 "±20%" H 7900 6680 60  0001 L CNN "Tolerance"
 F 21 "Aluminum Electrolytic SMT Capacitor" H 7900 6590 60  0001 L CNN "Part Description"
-F 22 "PANASONIC" H 7900 6500 60  0001 L CNN "Manufacturer"
-F 23 "EEEFK1C471AP or 16SEV470M8X10.5" H 7900 6410 60  0001 L CNN "Manufacturer Part Number"
+F 22 "NICHICON" H 7900 6500 60  0001 L CNN "Manufacturer"
+F 23 "UCD1C471MNL1GS" H 7900 6410 60  0001 L CNN "Manufacturer Part Number"
 F 24 "F" H 7900 6320 60  0001 L CNN "Case"
 F 25 "Yes" H 7900 6230 60  0001 L CNN "Mounted"
@@
 F 12 " " H 8900 7760 60  0001 L CNN "Status"
 F 13 "-45V -100mA PNP General Purpose Double Transistor" H 8900 7670 60  0001 L CNN "Part Description"
-F 14 "NXP SEMICONDUCTORS" H 8900 7580 60  0001 L CNN "Manufacturer"
-F 15 "BC857BV or BCM857BV,115" H 8900 7490 60  0001 L CNN "Manufacturer Part Number"
+F 14 "MICRO COMMERCIAL" H 8900 7580 60  0001 L CNN "Manufacturer"
+F 15 "BC857BV-TP" H 8900 7490 60  0001 L CNN "Manufacturer Part Number"
 F 16 "6" H 8900 7400 60  0001 L CNN "Pin Count"
 F 17 "SOT666" H 8900 7310 60  0001 L CNN "Case"
@@
 F 12 " " H 9450 7760 60  0001 L CNN "Status"
 F 13 "-45V -100mA PNP General Purpose Double Transistor" H 9450 7670 60  0001 L CNN "Part Description"
-F 14 "NXP SEMICONDUCTORS" H 9450 7580 60  0001 L CNN "Manufacturer"
-F 15 "BC857BV or BCM857BV,115" H 9450 7490 60  0001 L CNN "Manufacturer Part Number"
+F 14 "MICRO COMMERCIAL" H 9450 7580 60  0001 L CNN "Manufacturer"
+F 15 "BC857BV-TP" H 9450 7490 60  0001 L CNN "Manufacturer Part Number"
 F 16 "6" H 9450 7400 60  0001 L CNN "Pin Count"
 F 17 "SOT666" H 9450 7310 60  0001 L CNN "Case"
@@
 F 12 " " H 2800 1160 60  0001 L CNN "Status"
 F 13 "-45V -100mA PNP General Purpose Double Transistor" H 2800 1070 60  0001 L CNN "Part Description"
-F 14 "NXP SEMICONDUCTORS" H 2800 980 60  0001 L CNN "Manufacturer"
-F 15 "BC857BV or BCM857BV,115" H 2800 890 60  0001 L CNN "Manufacturer Part Number"
+F 14 "MICRO COMMERCIAL" H 2800 980 60  0001 L CNN "Manufacturer"
+F 15 "BC857BV-TP" H 2800 890 60  0001 L CNN "Manufacturer Part Number"
 F 16 "6" H 2800 800 60  0001 L CNN "Pin Count"
 F 17 "SOT666" H 2800 710 60  0001 L CNN "Case"
@@
 F 12 " " H 3350 1160 60  0001 L CNN "Status"
 F 13 "-45V -100mA PNP General Purpose Double Transistor" H 3350 1070 60  0001 L CNN "Part Description"
-F 14 "NXP SEMICONDUCTORS" H 3350 980 60  0001 L CNN "Manufacturer"
-F 15 "BC857BV or BCM857BV,115" H 3350 890 60  0001 L CNN "Manufacturer Part Number"
+F 14 "MICRO COMMERCIAL" H 3350 980 60  0001 L CNN "Manufacturer"
+F 15 "BC857BV-TP" H 3350 890 60  0001 L CNN "Manufacturer Part Number"
 F 16 "6" H 3350 800 60  0001 L CNN "Pin Count"
 F 17 "SOT666" H 3350 710 60  0001 L CNN "Case"

Commit message: More BOM updates for manufacturability
Use TDK MPZ2012S102JTD25 for 0805 ferrite bead.

Rename BSS138LT1G as BSS138L, ONSEMI BSS138L, now that onsemi bought Fairchild.
The T1G suffix is all about the tape&reel factory-orderable,
nothing to do with the transistor itself.

Take FPF2116 away as an MIC2090-1 alternate.  Its trip threshold
(200-400 mA) is too high for the MYRGC075050RA regulator powering
the two of them (U43 U55).

Use DAC8550 for the WR DAC (2x).  Electrically compatible with AD5662,
but uses twos-complement instead of unipolar encoding for its 16-bit
data word.  Make a note of that on the schematic.
TEXAS INSTRUMENTS DAC8550IDGK is the full name.
Parts:
- L35, L36, L37, L38, L39, L40: Manufacturer Part Number MPZ2012S102A or ACML-0805H-102-T -> MPZ2012S102JTD25
- Q8, Q9: value BSS138LT1G -> BSS138L; symbol Transistors:BSS138LT1G -> Transistors:BSS138L; Comment BSS138LT1G -> BSS138L; Device BSS138LT1G -> BSS138L; Manufacturer ON SEMICONDUCTOR -> ONSEMI; Manufacturer Part Number BSS138LT1G -> BSS138L; Part Number BSS138LT1G -> BSS138L
Changed lines of the file:
@@
 F 2 "Inductors SMD:INDC2012X145N" H 4250 8650 50  0001 C CNN
 F 3 " " H 4250 8650 50  0001 C CNN
-F 4 "MPZ2012S102A or ACML-0805H-102-T" V 4250 8650 50  0001 C CNN "Manufacturer Part Number"
+F 4 "MPZ2012S102JTD25" V 4250 8650 50  0001 C CNN "Manufacturer Part Number"
 F 5 "TDK" H 4250 8650 50  0001 C CNN "Manufacturer"
 	1    4250 8650
@@
 F 2 "Inductors SMD:INDC2012X145N" H 4750 8650 50  0001 C CNN
 F 3 " " H 4750 8650 50  0001 C CNN
-F 4 "MPZ2012S102A or ACML-0805H-102-T" V 4750 8650 50  0001 C CNN "Manufacturer Part Number"
+F 4 "MPZ2012S102JTD25" V 4750 8650 50  0001 C CNN "Manufacturer Part Number"
 F 5 "TDK" H 4750 8650 50  0001 C CNN "Manufacturer"
 	1    4750 8650
@@
 F 2 "Inductors SMD:INDC2012X145N" H 5250 8650 50  0001 C CNN
 F 3 " " H 5250 8650 50  0001 C CNN
-F 4 "MPZ2012S102A or ACML-0805H-102-T" V 5250 8650 50  0001 C CNN "Manufacturer Part Number"
+F 4 "MPZ2012S102JTD25" V 5250 8650 50  0001 C CNN "Manufacturer Part Number"
 F 5 "TDK" H 5250 8650 50  0001 C CNN "Manufacturer"
 	1    5250 8650
@@
 F 2 "Inductors SMD:INDC2012X145N" H 4250 9050 50  0001 C CNN
 F 3 " " H 4250 9050 50  0001 C CNN
-F 4 "MPZ2012S102A or ACML-0805H-102-T" V 4250 9050 50  0001 C CNN "Manufacturer Part Number"
+F 4 "MPZ2012S102JTD25" V 4250 9050 50  0001 C CNN "Manufacturer Part Number"
 F 5 "TDK" H 4250 9050 50  0001 C CNN "Manufacturer"
 	1    4250 9050
@@
 F 2 "Inductors SMD:INDC2012X145N" H 4750 9050 50  0001 C CNN
 F 3 " " H 4750 9050 50  0001 C CNN
-F 4 "MPZ2012S102A or ACML-0805H-102-T" V 4750 9050 50  0001 C CNN "Manufacturer Part Number"
+F 4 "MPZ2012S102JTD25" V 4750 9050 50  0001 C CNN "Manufacturer Part Number"
 F 5 "TDK" H 4750 9050 50  0001 C CNN "Manufacturer"
 	1    4750 9050
@@
 F 2 "Inductors SMD:INDC2012X145N" H 5250 9050 50  0001 C CNN
 F 3 " " H 5250 9050 50  0001 C CNN
-F 4 "MPZ2012S102A or ACML-0805H-102-T" V 5250 9050 50  0001 C CNN "Manufacturer Part Number"
+F 4 "MPZ2012S102JTD25" V 5250 9050 50  0001 C CNN "Manufacturer Part Number"
 F 5 "TDK" H 5250 9050 50  0001 C CNN "Manufacturer"
 	1    5250 9050
@@
 $EndComp
 $Comp
-L Transistors:BSS138LT1G Q9
+L Transistors:BSS138L Q9
 U 1 1 5CC371BB
 P 10150 5050
 F 0 "Q9" H 10469 5146 50  0000 L CNN
-F 1 "BSS138LT1G" H 10469 5055 50  0000 L CNN
+F 1 "BSS138L" H 10469 5055 50  0000 L CNN
 F 2 "ICs And Semiconductors SMD:SOT95P240X110-3N" H 10150 3840 60  0001 L CNN
 F 3 "" H 10150 4560 60  0001 L CNN
-F 4 "BSS138LT1G" H 10150 4470 60  0001 L CNN "Part Number"
+F 4 "BSS138L" H 10150 4470 60  0001 L CNN "Part Number"
 F 5 "N-MOSFET-D 1G 2S 3D" H 10150 4380 60  0001 L CNN "Library Ref"
 F 6 "SchLib\\Transistors.SchLib" H 10150 4290 60  0001 L CNN "Library Path"
-F 7 "BSS138LT1G" H 10150 4200 60  0001 L CNN "Comment"
+F 7 "BSS138L" H 10150 4200 60  0001 L CNN "Comment"
 F 8 "Standard" H 10150 4110 60  0001 L CNN "Component Kind"
 F 9 "Standard" H 10150 4020 60  0001 L CNN "Component Type"
-F 10 "BSS138LT1G" H 10150 3930 60  0001 L CNN "Device"
+F 10 "BSS138L" H 10150 3930 60  0001 L CNN "Device"
 F 11 "SOT23 3-Leads, Pitch 0.95mm - Body 1.4x3mm, IPC Medium Density" H 10150 3750 60  0001 L CNN "PackageDescription"
 F 12 " " H 10150 3660 60  0001 L CNN "Status"
 F 13 "50V 200mA N-Channel Enhancement Mode Field-Effect Transistor" H 10150 3570 60  0001 L CNN "Part Description"
-F 14 "ON SEMICONDUCTOR" H 10150 3480 60  0001 L CNN "Manufacturer"
-F 15 "BSS138LT1G" H 10150 3390 60  0001 L CNN "Manufacturer Part Number"
+F 14 "ONSEMI" H 10150 3480 60  0001 L CNN "Manufacturer"
+F 15 "BSS138L" H 10150 3390 60  0001 L CNN "Manufacturer Part Number"
 F 16 "3" H 10150 3300 60  0001 L CNN "Pin Count"
 F 17 "SOT23-3" H 10150 3210 60  0001 L CNN "Case"
@@
 Connection ~ 10400 4800
 $Comp
-L Transistors:BSS138LT1G Q8
+L Transistors:BSS138L Q8
 U 1 1 5CC74B8D
 P 10150 1650
 F 0 "Q8" H 10469 1746 50  0000 L CNN
-F 1 "BSS138LT1G" H 10469 1655 50  0000 L CNN
+F 1 "BSS138L" H 10469 1655 50  0000 L CNN
 F 2 "ICs And Semiconductors SMD:SOT95P240X110-3N" H 10150 440 60  0001 L CNN
 F 3 "" H 10150 1160 60  0001 L CNN
-F 4 "BSS138LT1G" H 10150 1070 60  0001 L CNN "Part Number"
+F 4 "BSS138L" H 10150 1070 60  0001 L CNN "Part Number"
 F 5 "N-MOSFET-D 1G 2S 3D" H 10150 980 60  0001 L CNN "Library Ref"
 F 6 "SchLib\\Transistors.SchLib" H 10150 890 60  0001 L CNN "Library Path"
-F 7 "BSS138LT1G" H 10150 800 60  0001 L CNN "Comment"
+F 7 "BSS138L" H 10150 800 60  0001 L CNN "Comment"
 F 8 "Standard" H 10150 710 60  0001 L CNN "Component Kind"
 F 9 "Standard" H 10150 620 60  0001 L CNN "Component Type"
-F 10 "BSS138LT1G" H 10150 530 60  0001 L CNN "Device"
+F 10 "BSS138L" H 10150 530 60  0001 L CNN "Device"
 F 11 "SOT23 3-Leads, Pitch 0.95mm - Body 1.4x3mm, IPC Medium Density" H 10150 350 60  0001 L CNN "PackageDescription"
 F 12 " " H 10150 260 60  0001 L CNN "Status"
 F 13 "50V 200mA N-Channel Enhancement Mode Field-Effect Transistor" H 10150 170 60  0001 L CNN "Part Description"
-F 14 "ON SEMICONDUCTOR" H 10150 80  60  0001 L CNN "Manufacturer"
-F 15 "BSS138LT1G" H 10150 -10 60  0001 L CNN "Manufacturer Part Number"
+F 14 "ONSEMI" H 10150 80  60  0001 L CNN "Manufacturer"
+F 15 "BSS138L" H 10150 -10 60  0001 L CNN "Manufacturer Part Number"
 F 16 "3" H 10150 -100 60  0001 L CNN "Pin Count"
 F 17 "SOT23-3" H 10150 -190 60  0001 L CNN "Case"
