File: design/ETH_PHY.sch (KiCad schematic (older format))
At the start: 45 parts, among them J4 BELFUSE_0826-1X1T-GH-F, U4 88E1512-A0-NNP2I000, U6 TXS0102DCUR

Commit message: Continuing BOM adjustments
drop BLM18SG121TZ1D as an alternate for BLM18SG121TN1D, 0603 ferrite bead

Convert PI3DBS12212AZBSEX to PI3DBS16212ZBBEX, includes part name shown on schematic
(new and improved part tested at high data rates in protoype run)
Parts:
- L3, L4: Manufacturer Part Number BLM18SG121TN1D or BLM18SG121TZ1D -> BLM18SG121TN1D
Changed lines of the file:
@@
 F 20 "SMD EMIFIL Suppression Chip Ferrite Bead" H 4450 5700 60  0001 L CNN "Part Description"
 F 21 "MURATA" H 4450 5610 60  0001 L CNN "Manufacturer"
-F 22 "BLM18SG121TN1D or BLM18SG121TZ1D" H 4450 5520 60  0001 L CNN "Manufacturer Part Number"
+F 22 "BLM18SG121TN1D" H 4450 5520 60  0001 L CNN "Manufacturer Part Number"
 F 23 "0603" H 4450 5430 60  0001 L CNN "Case"
 F 24 "Yes" H 4450 5340 60  0001 L CNN "Mounted"
@@
 F 20 "SMD EMIFIL Suppression Chip Ferrite Bead" H 3550 4750 60  0001 L CNN "Part Description"
 F 21 "MURATA" H 3550 4660 60  0001 L CNN "Manufacturer"
-F 22 "BLM18SG121TN1D or BLM18SG121TZ1D" H 3550 4570 60  0001 L CNN "Manufacturer Part Number"
+F 22 "BLM18SG121TN1D" H 3550 4570 60  0001 L CNN "Manufacturer Part Number"
 F 23 "0603" H 3550 4480 60  0001 L CNN "Case"
 F 24 "Yes" H 3550 4390 60  0001 L CNN "Mounted"
