File: design/FPGA_PWR&MISC.sch (KiCad schematic (older format))
At the start: 121 parts, among them Q19 BSS138LT1G, Q21 BSS138LT1G, SW5 KSS241GLFS, U1 XC7K160T-2FFG676C, U60 TPS3703A7330DSERQ1

Commit message: Update part numbers to be closer to as-manufactured
new (at least in form) listings:
Murata  GRM188R61A106KA73D
Samsung  CL32A107MQVNNWE
Yageo  AC0402FR-0722R
Yageo  RT0402BRD0710KL
Stackpole  RMCF0402FT82K0
NXP SEMICONDUCTORS  PRTR5V0U2X,215
FTDI  FT4232H-56Q-REEL
TEXAS INSTRUMENTS  CDCM61004RHB
TEXAS INSTRUMENTS  TLV62565DBVR
TEXAS INSTRUMENTS  TPS3703A7330DSER
XILINX  XC7K160T-2FFG676I
SILICON LABS  570NCB000933DG
IQD FREQUENCY PRODUCTS  ECS-VXO-73-20.00-TR
Parts:
- U1: Manufacturer Part Number XC7K160T-2FFG676C or XC7K160T-3FFG676E -> XC7K160T-2FFG676I
- U60: value TPS3703A7330DSERQ1 -> TPS3703A7330DSER; symbol Logic:TPS3703A7330DSERQ1 -> Logic:TPS3703A7330DSER; Manufacturer Part Number TPS3703A7330DSERQ1 or TPS3703A7330DSER -> TPS3703A7330DSER
Changed lines of the file:
@@
 F 3 "" H 9250 2050 50  0000 C CNN
 F 4 "XILINX" H 9250 2050 50  0001 C CNN "Manufacturer"
-F 5 "XC7K160T-2FFG676C or XC7K160T-3FFG676E" H 9250 2050 50  0001 C CNN "Manufacturer Part Number"
+F 5 "XC7K160T-2FFG676I" H 9250 2050 50  0001 C CNN "Manufacturer Part Number"
 	6    9250 2050
 	1    0    0    -1
@@
 F 3 "" H 8450 5750 50  0000 C CNN
 F 4 "XILINX" H 8450 5750 50  0001 C CNN "Manufacturer"
-F 5 "XC7K160T-2FFG676C or XC7K160T-3FFG676E" H 8450 5750 50  0001 C CNN "Manufacturer Part Number"
+F 5 "XC7K160T-2FFG676I" H 8450 5750 50  0001 C CNN "Manufacturer Part Number"
 	7    8450 5750
 	1    0    0    -1
@@
 F 3 "" H 5250 4800 50  0000 C CNN
 F 4 "XILINX" H 5250 4800 50  0001 C CNN "Manufacturer"
-F 5 "XC7K160T-2FFG676C or XC7K160T-3FFG676E" H 5250 4800 50  0001 C CNN "Manufacturer Part Number"
+F 5 "XC7K160T-2FFG676I" H 5250 4800 50  0001 C CNN "Manufacturer Part Number"
 	8    5250 4800
 	1    0    0    -1
@@
 	11950 6150 11950 6250
 $Comp
-L Logic:TPS3703A7330DSERQ1 U?
+L Logic:TPS3703A7330DSER U?
 U 1 1 6058579B
 P 14800 7700
@@
 AR Path="/5C907554/5C417BCB/6058579B" Ref="U60"  Part="1"
 F 0 "U60" H 15450 7965 50  0000 C CNN
-F 1 "TPS3703A7330DSERQ1" H 15450 7874 50  0000 C CNN
+F 1 "TPS3703A7330DSER" H 15450 7874 50  0000 C CNN
 F 2 "ICs And Semiconductors SMD:SON50P150X150X80-6N" H 15950 7800 50  0001 L CNN
 F 3 "https://www.ti.com/lit/gpn/TPS3703-Q1" H 15950 7700 50  0001 L CNN
@@
 F 5 "0.8" H 15950 7500 50  0001 L CNN "Height"
 F 6 "TEXAS INSTRUMENTS" H 15950 7200 50  0001 L CNN "Manufacturer"
-F 7 "TPS3703A7330DSERQ1 or TPS3703A7330DSER" H 15950 7100 50  0001 L CNN "Manufacturer Part Number"
+F 7 "TPS3703A7330DSER" H 15950 7100 50  0001 L CNN "Manufacturer Part Number"
 	1    14800 7700
 	-1   0    0    -1

Commit message: Update more "Manufacturer Part Number"
Corresponding to specific parts that are actually usable and available.

PANASONIC EEEFK1C471AP or 16SEV470M8X10.5 becomes NICHICON UCD1C471MNL1GS
  (described as 470 uF on schematic)
INFINEON BAT165AX or BAT165E6327HTSA1 becomes BAT165E6327HTSA1
  (described as BAT165 on schematic)
VISHAY GENERAL SEMICONDUCTOR SS16 or SS16FP becomes ONSEMI SS16FP
  (schematic simply shows Schottky diode)
NXP SEMICONDUCTORS BC857BV or BCM857BV,115 becomes MICRO COMMERCIAL BC857BV-TP
  (described as BC857BV on schematic)
NXP NX3008NBKV or SI1036X-T1-GE3 becomes VISHAY SILICONIX SI1036X-T1-GE3
  (changed marking on schematic to SI1036X)
ST MICROELECTRONICS STS8DN6LF6AG or SQ4920EY-T1_BE3 becomes VISHAY SILICONIX SQ4920EY-T1_GE3
  (changed marking on schematic to SQ4920EY)
NXP SEMICONDUCTORS 74AHC1G04GW becomes NEXPERIA 74AHC1G04GW-Q100H
  (schematic simply shows generic logic inverter)
Monolithic Power Systems (MPS) MPM3830GQV-P becomes Monolithic Power Systems (MPS) MPM3830GQVP
  (changed marking on schematic to MPM3830GQV)
TEXAS INSTRUMENTS SN74LVC1G125DCKT or SN74AUC1G17DCKR becomes TEXAS INSTRUMENTS SN74LVC1G125DCK3
  (schematic simply shows generic logic buffer)
Parts:
- D1, D9: Manufacturer Part Number BAT165AX or BAT165E6327HTSA1 -> BAT165E6327HTSA1
Changed lines of the file:
@@
 F 15 "Medium Power AF Schottky Diode" H 11200 5860 60  0001 L CNN "Part Description"
 F 16 "INFINEON" H 11200 5770 60  0001 L CNN "Manufacturer"
-F 17 "BAT165AX or BAT165E6327HTSA1" H 11200 5680 60  0001 L CNN "Manufacturer Part Number"
+F 17 "BAT165E6327HTSA1" H 11200 5680 60  0001 L CNN "Manufacturer Part Number"
 F 18 "2" H 11200 5590 60  0001 L CNN "Pin Count"
 F 19 "SOD323" H 11200 5500 60  0001 L CNN "Case"
@@
 F 15 "Medium Power AF Schottky Diode" H 11950 5860 60  0001 L CNN "Part Description"
 F 16 "INFINEON" H 11950 5770 60  0001 L CNN "Manufacturer"
-F 17 "BAT165AX or BAT165E6327HTSA1" H 11950 5680 60  0001 L CNN "Manufacturer Part Number"
+F 17 "BAT165E6327HTSA1" H 11950 5680 60  0001 L CNN "Manufacturer Part Number"
 F 18 "2" H 11950 5590 60  0001 L CNN "Pin Count"
 F 19 "SOD323" H 11950 5500 60  0001 L CNN "Case"

Commit message: More BOM updates for manufacturability
Use TDK MPZ2012S102JTD25 for 0805 ferrite bead.

Rename BSS138LT1G as BSS138L, ONSEMI BSS138L, now that onsemi bought Fairchild.
The T1G suffix is all about the tape&reel factory-orderable,
nothing to do with the transistor itself.

Take FPF2116 away as an MIC2090-1 alternate.  Its trip threshold
(200-400 mA) is too high for the MYRGC075050RA regulator powering
the two of them (U43 U55).

Use DAC8550 for the WR DAC (2x).  Electrically compatible with AD5662,
but uses twos-complement instead of unipolar encoding for its 16-bit
data word.  Make a note of that on the schematic.
TEXAS INSTRUMENTS DAC8550IDGK is the full name.
Parts:
- Q19, Q21: value BSS138LT1G -> BSS138L; symbol Transistors:BSS138LT1G -> Transistors:BSS138L; Comment BSS138LT1G -> BSS138L; Device BSS138LT1G -> BSS138L; Manufacturer ON SEMICONDUCTOR -> ONSEMI; Manufacturer Part Number BSS138LT1G -> BSS138L; Part Number BSS138LT1G -> BSS138L
Changed lines of the file:
@@
 $EndComp
 $Comp
-L Transistors:BSS138LT1G Q19
+L Transistors:BSS138L Q19
 U 1 1 5D220E28
 P 15150 5200
 F 0 "Q19" H 15469 5296 50  0000 L CNN
-F 1 "BSS138LT1G" H 15469 5205 50  0000 L CNN
+F 1 "BSS138L" H 15469 5205 50  0000 L CNN
 F 2 "ICs And Semiconductors SMD:SOT95P240X110-3N" H 15150 3990 60  0001 L CNN
 F 3 "\\\\cern.ch\\dfs\\Applications\\Altium\\Datasheets\\BSS138LT1G.pdf" H 15150 4710 60  0001 L CNN
-F 4 "BSS138LT1G" H 15150 4620 60  0001 L CNN "Part Number"
+F 4 "BSS138L" H 15150 4620 60  0001 L CNN "Part Number"
 F 5 "N-MOSFET-D 1G 2S 3D" H 15150 4530 60  0001 L CNN "Library Ref"
 F 6 "SchLib\\Transistors.SchLib" H 15150 4440 60  0001 L CNN "Library Path"
-F 7 "BSS138LT1G" H 15150 4350 60  0001 L CNN "Comment"
+F 7 "BSS138L" H 15150 4350 60  0001 L CNN "Comment"
 F 8 "Standard" H 15150 4260 60  0001 L CNN "Component Kind"
 F 9 "Standard" H 15150 4170 60  0001 L CNN "Component Type"
-F 10 "BSS138LT1G" H 15150 4080 60  0001 L CNN "Device"
+F 10 "BSS138L" H 15150 4080 60  0001 L CNN "Device"
 F 11 "SOT23 3-Leads, Pitch 0.95mm - Body 1.4x3mm, IPC Medium Density" H 15150 3900 60  0001 L CNN "PackageDescription"
 F 12 " " H 15150 3810 60  0001 L CNN "Status"
 F 13 "50V 200mA N-Channel Enhancement Mode Field-Effect Transistor" H 15150 3720 60  0001 L CNN "Part Description"
-F 14 "ON SEMICONDUCTOR" H 15150 3630 60  0001 L CNN "Manufacturer"
-F 15 "BSS138LT1G" H 15150 3540 60  0001 L CNN "Manufacturer Part Number"
+F 14 "ONSEMI" H 15150 3630 60  0001 L CNN "Manufacturer"
+F 15 "BSS138L" H 15150 3540 60  0001 L CNN "Manufacturer Part Number"
 F 16 "3" H 15150 3450 60  0001 L CNN "Pin Count"
 F 17 "SOT23-3" H 15150 3360 60  0001 L CNN "Case"
@@
 $EndComp
 $Comp
-L Transistors:BSS138LT1G Q21
+L Transistors:BSS138L Q21
 U 1 1 605D0D1C
 P 12200 6500
 F 0 "Q21" H 12519 6596 50  0000 L CNN
-F 1 "BSS138LT1G" H 12519 6505 50  0000 L CNN
+F 1 "BSS138L" H 12519 6505 50  0000 L CNN
 F 2 "ICs And Semiconductors SMD:SOT95P240X110-3N" H 12200 5290 60  0001 L CNN
 F 3 "\\\\cern.ch\\dfs\\Applications\\Altium\\Datasheets\\BSS138LT1G.pdf" H 12200 6010 60  0001 L CNN
-F 4 "BSS138LT1G" H 12200 5920 60  0001 L CNN "Part Number"
+F 4 "BSS138L" H 12200 5920 60  0001 L CNN "Part Number"
 F 5 "N-MOSFET-D 1G 2S 3D" H 12200 5830 60  0001 L CNN "Library Ref"
 F 6 "SchLib\\Transistors.SchLib" H 12200 5740 60  0001 L CNN "Library Path"
-F 7 "BSS138LT1G" H 12200 5650 60  0001 L CNN "Comment"
+F 7 "BSS138L" H 12200 5650 60  0001 L CNN "Comment"
 F 8 "Standard" H 12200 5560 60  0001 L CNN "Component Kind"
 F 9 "Standard" H 12200 5470 60  0001 L CNN "Component Type"
-F 10 "BSS138LT1G" H 12200 5380 60  0001 L CNN "Device"
+F 10 "BSS138L" H 12200 5380 60  0001 L CNN "Device"
 F 11 "SOT23 3-Leads, Pitch 0.95mm - Body 1.4x3mm, IPC Medium Density" H 12200 5200 60  0001 L CNN "PackageDescription"
 F 12 " " H 12200 5110 60  0001 L CNN "Status"
 F 13 "50V 200mA N-Channel Enhancement Mode Field-Effect Transistor" H 12200 5020 60  0001 L CNN "Part Description"
-F 14 "ON SEMICONDUCTOR" H 12200 4930 60  0001 L CNN "Manufacturer"
-F 15 "BSS138LT1G" H 12200 4840 60  0001 L CNN "Manufacturer Part Number"
+F 14 "ONSEMI" H 12200 4930 60  0001 L CNN "Manufacturer"
+F 15 "BSS138L" H 12200 4840 60  0001 L CNN "Manufacturer Part Number"
 F 16 "3" H 12200 4750 60  0001 L CNN "Pin Count"
 F 17 "SOT23-3" H 12200 4660 60  0001 L CNN "Case"

Commit message: Continuing BOM adjustments
drop BLM18SG121TZ1D as an alternate for BLM18SG121TN1D, 0603 ferrite bead

Convert PI3DBS12212AZBSEX to PI3DBS16212ZBBEX, includes part name shown on schematic
(new and improved part tested at high data rates in protoype run)
Parts:
- L27, L28: Manufacturer Part Number BLM18SG121TN1D or BLM18SG121TZ1D -> BLM18SG121TN1D
Changed lines of the file:
@@
 F 20 "SMD EMIFIL Suppression Chip Ferrite Bead" H 1800 3600 60  0001 L CNN "Part Description"
 F 21 "MURATA" H 1800 3510 60  0001 L CNN "Manufacturer"
-F 22 "BLM18SG121TN1D or BLM18SG121TZ1D" H 1800 3420 60  0001 L CNN "Manufacturer Part Number"
+F 22 "BLM18SG121TN1D" H 1800 3420 60  0001 L CNN "Manufacturer Part Number"
 F 23 "0603" H 1800 3330 60  0001 L CNN "Case"
 F 24 "Yes" H 1800 3240 60  0001 L CNN "Mounted"
@@
 F 20 "SMD EMIFIL Suppression Chip Ferrite Bead" H 1800 4000 60  0001 L CNN "Part Description"
 F 21 "MURATA" H 1800 3910 60  0001 L CNN "Manufacturer"
-F 22 "BLM18SG121TN1D or BLM18SG121TZ1D" H 1800 3820 60  0001 L CNN "Manufacturer Part Number"
+F 22 "BLM18SG121TN1D" H 1800 3820 60  0001 L CNN "Manufacturer Part Number"
 F 23 "0603" H 1800 3730 60  0001 L CNN "Case"
 F 24 "Yes" H 1800 3640 60  0001 L CNN "Mounted"
