File: design/GBX_MUX.sch (KiCad schematic (older format))
At the start: 24 parts, among them U44 PI3DBS12212AZBSEX, U45 PI3DBS12212AZBSEX, U46 PI3DBS12212AZBSEX, U48 PI3DBS12212AZBSEX, U49 PI3DBS12212AZBSEX, U50 PI3DBS12212AZBSEX, U56 74AHC1G04GW

Commit message: Update more "Manufacturer Part Number"
Corresponding to specific parts that are actually usable and available.

PANASONIC EEEFK1C471AP or 16SEV470M8X10.5 becomes NICHICON UCD1C471MNL1GS
  (described as 470 uF on schematic)
INFINEON BAT165AX or BAT165E6327HTSA1 becomes BAT165E6327HTSA1
  (described as BAT165 on schematic)
VISHAY GENERAL SEMICONDUCTOR SS16 or SS16FP becomes ONSEMI SS16FP
  (schematic simply shows Schottky diode)
NXP SEMICONDUCTORS BC857BV or BCM857BV,115 becomes MICRO COMMERCIAL BC857BV-TP
  (described as BC857BV on schematic)
NXP NX3008NBKV or SI1036X-T1-GE3 becomes VISHAY SILICONIX SI1036X-T1-GE3
  (changed marking on schematic to SI1036X)
ST MICROELECTRONICS STS8DN6LF6AG or SQ4920EY-T1_BE3 becomes VISHAY SILICONIX SQ4920EY-T1_GE3
  (changed marking on schematic to SQ4920EY)
NXP SEMICONDUCTORS 74AHC1G04GW becomes NEXPERIA 74AHC1G04GW-Q100H
  (schematic simply shows generic logic inverter)
Monolithic Power Systems (MPS) MPM3830GQV-P becomes Monolithic Power Systems (MPS) MPM3830GQVP
  (changed marking on schematic to MPM3830GQV)
TEXAS INSTRUMENTS SN74LVC1G125DCKT or SN74AUC1G17DCKR becomes TEXAS INSTRUMENTS SN74LVC1G125DCK3
  (schematic simply shows generic logic buffer)
Parts:
- U56: Manufacturer NXP SEMICONDUCTORS -> NEXPERIA; Manufacturer Part Number 74AHC1G04GW -> 74AHC1G04GW-Q100H
Changed lines of the file:
@@
 F 12 " " H 1600 3340 50  0001 L CNN "Status"
 F 13 "Single Inverter Buffer" H 1600 3265 50  0001 L CNN "Part Description"
-F 14 "NXP SEMICONDUCTORS" H 1600 3190 50  0001 L CNN "Manufacturer"
-F 15 "74AHC1G04GW" H 1600 3115 50  0001 L CNN "Manufacturer Part Number"
+F 14 "NEXPERIA" H 1600 3190 50  0001 L CNN "Manufacturer"
+F 15 "74AHC1G04GW-Q100H" H 1600 3115 50  0001 L CNN "Manufacturer Part Number"
 F 16 "3" H 1600 3040 50  0001 L CNN "Pin Count"
 F 17 "SOT353" H 1600 2965 50  0001 L CNN "Case"

Commit message: Continuing BOM adjustments
drop BLM18SG121TZ1D as an alternate for BLM18SG121TN1D, 0603 ferrite bead

Convert PI3DBS12212AZBSEX to PI3DBS16212ZBBEX, includes part name shown on schematic
(new and improved part tested at high data rates in protoype run)
Parts:
- U44, U45, U46, U48, U49, U50: value PI3DBS12212AZBSEX -> PI3DBS16212ZBBEX; symbol Analog_&_Interface:PI3DBS12212AZBSEX -> Analog_&_Interface:PI3DBS16212ZBBEX; Comment PI3DBS12212AZBSEX -> PI3DBS16212ZBBEX; Device PI3DBS12212AZBSEX -> PI3DBS16212ZBBEX; Library Ref PI3DBS12212AZBSEX -> PI3DBS16212ZBBEX; Manufacturer Part Number PI3DBS12212AZBSEX or PI3DBS16212ZBBEX -> PI3DBS16212ZBBEX; Part Number PI3DBS12212AZBSEX -> PI3DBS16212ZBBEX
