File: design/USB.sch (KiCad schematic (older format))
At the start: 76 parts, among them J10 10103594-0001LF, Q14 BSS138LT1G, Q18 BSS138LT1G, Q24 BSS138LT1G, Q6 BSS138LT1G, U15 SN74AVC2T245RSWR, U21 M93C46-WMN6TP, U22 TLV62565DBVT, U23 FT4232H-56Q, U24 SN74AVC2T245RSWR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

Commit message: Update part numbers to be closer to as-manufactured
new (at least in form) listings:
Murata  GRM188R61A106KA73D
Samsung  CL32A107MQVNNWE
Yageo  AC0402FR-0722R
Yageo  RT0402BRD0710KL
Stackpole  RMCF0402FT82K0
NXP SEMICONDUCTORS  PRTR5V0U2X,215
FTDI  FT4232H-56Q-REEL
TEXAS INSTRUMENTS  CDCM61004RHB
TEXAS INSTRUMENTS  TLV62565DBVR
TEXAS INSTRUMENTS  TPS3703A7330DSER
XILINX  XC7K160T-2FFG676I
SILICON LABS  570NCB000933DG
IQD FREQUENCY PRODUCTS  ECS-VXO-73-20.00-TR
Parts:
- D13: Manufacturer Part Number PRTR5V0U2X -> PRTR5V0U2X,215
- U22: value TLV62565DBVT -> TLV62565DBV; symbol Regulators:TLV62565DBVT -> Regulators:TLV62565DBV; Device TLV62565DBVT -> TLV62565DBV; Manufacturer Part Number TLV62565DBVT or TLV62565DBVR -> TLV62565DBVR; Part Number TLV62565DBVT -> TLV62565DBV
- U23: Manufacturer Part Number FT4232H-56Q -> FT4232H-56Q-REEL
Changed lines of the file:
@@
 F 15 "Ultra Low Capacitance (1pF) Double Rail-to-Rail ESD Protection Diode (8kV)" H 2400 3360 60  0001 L CNN "Part Description"
 F 16 "NXP SEMICONDUCTORS" H 2400 3270 60  0001 L CNN "Manufacturer"
-F 17 "PRTR5V0U2X" H 2400 3180 60  0001 L CNN "Manufacturer Part Number"
+F 17 "PRTR5V0U2X,215" H 2400 3180 60  0001 L CNN "Manufacturer Part Number"
 F 18 "4" H 2400 3090 60  0001 L CNN "Pin Count"
 F 19 "SOT143B" H 2400 3000 60  0001 L CNN "Case"
@@
 F 13 "Quad High Speed USB to Multipurpose UART/MPSSE IC" H 6600 -2960 60  0001 L CNN "Part Description"
 F 14 "FUTURE TECHNOLOGY DEVICES INTERNATIONAL (FTDI)" H 6600 -3050 60  0001 L CNN "Manufacturer"
-F 15 "FT4232H-56Q" H 6600 -3140 60  0001 L CNN "Manufacturer Part Number"
+F 15 "FT4232H-56Q-REEL" H 6600 -3140 60  0001 L CNN "Manufacturer Part Number"
 F 16 "57" H 6600 -3230 60  0001 L CNN "Pin Count"
 F 17 "QFN56" H 6600 -3320 60  0001 L CNN "Case"
@@
 	8000 8100 8000 8300
 $Comp
-L Regulators:TLV62565DBVT U22
+L Regulators:TLV62565DBV U22
 U 1 1 5C6DFD9F
 P 3550 1800
 F 0 "U22" H 3850 1965 50  0000 C CNN
-F 1 "TLV62565DBVT" H 3850 1874 50  0000 C CNN
+F 1 "TLV62565DBV" H 3850 1874 50  0000 C CNN
 F 2 "ICs And Semiconductors SMD:SOT95P280X145-5N" H 3550 310 60  0001 L CNN
 F 3 "" H 3550 1030 60  0001 L CNN
-F 4 "TLV62565DBVT" H 3550 940 60  0001 L CNN "Part Number"
+F 4 "TLV62565DBV" H 3550 940 60  0001 L CNN "Part Number"
 F 5 "TLV62565" H 3550 850 60  0001 L CNN "Library Ref"
 F 6 "SchLib\\Regulators.SchLib" H 3550 760 60  0001 L CNN "Library Path"
@@
 F 8 "Standard" H 3550 580 60  0001 L CNN "Component Kind"
 F 9 "Standard" H 3550 490 60  0001 L CNN "Component Type"
-F 10 "TLV62565DBVT" H 3550 400 60  0001 L CNN "Device"
+F 10 "TLV62565DBV" H 3550 400 60  0001 L CNN "Device"
 F 11 "SOT, 0.95mm Pitch; 5 Pin, 1.60mm W X 2.90mm L X 1.45mm H Body, IPC Medium Density" H 3550 220 60  0001 L CNN "PackageDescription"
 F 12 " " H 3550 130 60  0001 L CNN "Status"
 F 13 "1.5A High Efficiency Step-Down Converter, Adjustable Output Voltage" H 3550 40  60  0001 L CNN "Part Description"
 F 14 "TEXAS INSTRUMENTS" H 3550 -50 60  0001 L CNN "Manufacturer"
-F 15 "TLV62565DBVT or TLV62565DBVR" H 3550 -140 60  0001 L CNN "Manufacturer Part Number"
+F 15 "TLV62565DBVR" H 3550 -140 60  0001 L CNN "Manufacturer Part Number"
 F 16 "5" H 3550 -230 60  0001 L CNN "Pin Count"
 F 17 "SOT23-5" H 3550 -320 60  0001 L CNN "Case"

Commit message: Update more "Manufacturer Part Number"
Corresponding to specific parts that are actually usable and available.

PANASONIC EEEFK1C471AP or 16SEV470M8X10.5 becomes NICHICON UCD1C471MNL1GS
  (described as 470 uF on schematic)
INFINEON BAT165AX or BAT165E6327HTSA1 becomes BAT165E6327HTSA1
  (described as BAT165 on schematic)
VISHAY GENERAL SEMICONDUCTOR SS16 or SS16FP becomes ONSEMI SS16FP
  (schematic simply shows Schottky diode)
NXP SEMICONDUCTORS BC857BV or BCM857BV,115 becomes MICRO COMMERCIAL BC857BV-TP
  (described as BC857BV on schematic)
NXP NX3008NBKV or SI1036X-T1-GE3 becomes VISHAY SILICONIX SI1036X-T1-GE3
  (changed marking on schematic to SI1036X)
ST MICROELECTRONICS STS8DN6LF6AG or SQ4920EY-T1_BE3 becomes VISHAY SILICONIX SQ4920EY-T1_GE3
  (changed marking on schematic to SQ4920EY)
NXP SEMICONDUCTORS 74AHC1G04GW becomes NEXPERIA 74AHC1G04GW-Q100H
  (schematic simply shows generic logic inverter)
Monolithic Power Systems (MPS) MPM3830GQV-P becomes Monolithic Power Systems (MPS) MPM3830GQVP
  (changed marking on schematic to MPM3830GQV)
TEXAS INSTRUMENTS SN74LVC1G125DCKT or SN74AUC1G17DCKR becomes TEXAS INSTRUMENTS SN74LVC1G125DCK3
  (schematic simply shows generic logic buffer)
Parts:
- D16: Manufacturer Part Number BAT165AX or BAT165E6327HTSA1 -> BAT165E6327HTSA1
- U61: value SN74LVC1G125DCKT -> SN74LVC1G125DCK; symbol marble_misc:SN74LVC1G125DCKT-Standard_Logic -> marble_misc:SN74LVC1G125DCK-Standard_Logic; Device SN74LVC1G125DCKT -> SN74LVC1G125DCK; Manufacturer Part Number SN74LVC1G125DCKT or SN74AUC1G17DCKR -> SN74LVC1G125DCK3; Part Number SN74LVC1G125DCKT -> SN74LVC1G125DCK
Changed lines of the file:
@@
 F 15 "Medium Power AF Schottky Diode" H 5150 8960 60  0001 L CNN "Part Description"
 F 16 "INFINEON" H 5150 8870 60  0001 L CNN "Manufacturer"
-F 17 "BAT165AX or BAT165E6327HTSA1" H 5150 8780 60  0001 L CNN "Manufacturer Part Number"
+F 17 "BAT165E6327HTSA1" H 5150 8780 60  0001 L CNN "Manufacturer Part Number"
 F 18 "2" H 5150 8690 60  0001 L CNN "Pin Count"
 F 19 "SOD323" H 5150 8600 60  0001 L CNN "Case"
@@
 Connection ~ 13250 7150
 $Comp
-L marble_misc:SN74LVC1G125DCKT-Standard_Logic U?
+L marble_misc:SN74LVC1G125DCK-Standard_Logic U?
 U 1 1 6245A646
 P 12425 5650
@@
 AR Path="/5C16C03C/6245A646" Ref="U61"  Part="1"
 F 0 "U61" H 12575 5061 50  0000 C CNN
-F 1 "SN74LVC1G125DCKT" H 12575 4970 50  0000 C CNN
+F 1 "SN74LVC1G125DCK" H 12575 4970 50  0000 C CNN
 F 2 "SOT65P210X110-5N" H 12425 4300 60  0001 L CNN
 F 3 "\\\\cern.ch\\dfs\\Applications\\Altium\\Datasheets\\SN74LVC1G125DCKT.pdf" H 12425 5020 60  0001 L CNN
-F 4 "SN74LVC1G125DCKT" H 12425 4930 60  0001 L CNN "Part Number"
+F 4 "SN74LVC1G125DCK" H 12425 4930 60  0001 L CNN "Part Number"
 F 5 "741G125" H 12425 4840 60  0001 L CNN "Library Ref"
 F 6 "SchLib\\Standard Logic.SchLib" H 12425 4750 60  0001 L CNN "Library Path"
@@
 F 8 "Standard" H 12425 4570 60  0001 L CNN "Component Kind"
 F 9 "Standard" H 12425 4480 60  0001 L CNN "Component Type"
-F 10 "SN74LVC1G125DCKT" H 12425 4390 60  0001 L CNN "Device"
+F 10 "SN74LVC1G125DCK" H 12425 4390 60  0001 L CNN "Device"
 F 11 "SOT353, SC70-5, SOT, 0.65mm Pitch, 5 pin, 1.25mm W X 2.00mm L X 1.10mm H, IPC Medium Density" H 12425 4210 60  0001 L CNN "PackageDescription"
 F 12 " " H 12425 4120 60  0001 L CNN "Status"
 F 13 "Single Bus Buffer Gate With 3-State Outputs" H 12425 4030 60  0001 L CNN "Part Description"
 F 14 "TEXAS INSTRUMENTS" H 12425 3940 60  0001 L CNN "Manufacturer"
-F 15 "SN74LVC1G125DCKT or SN74AUC1G17DCKR" H 12425 3850 60  0001 L CNN "Manufacturer Part Number"
+F 15 "SN74LVC1G125DCK3" H 12425 3850 60  0001 L CNN "Manufacturer Part Number"
 F 16 "5" H 12425 3760 60  0001 L CNN "Pin Count"
 F 17 "SOT353" H 12425 3670 60  0001 L CNN "Case"

Commit message: More BOM updates for manufacturability
Use TDK MPZ2012S102JTD25 for 0805 ferrite bead.

Rename BSS138LT1G as BSS138L, ONSEMI BSS138L, now that onsemi bought Fairchild.
The T1G suffix is all about the tape&reel factory-orderable,
nothing to do with the transistor itself.

Take FPF2116 away as an MIC2090-1 alternate.  Its trip threshold
(200-400 mA) is too high for the MYRGC075050RA regulator powering
the two of them (U43 U55).

Use DAC8550 for the WR DAC (2x).  Electrically compatible with AD5662,
but uses twos-complement instead of unipolar encoding for its 16-bit
data word.  Make a note of that on the schematic.
TEXAS INSTRUMENTS DAC8550IDGK is the full name.
Parts:
- Q14, Q18, Q24, Q6: value BSS138LT1G -> BSS138L; symbol Transistors:BSS138LT1G -> Transistors:BSS138L; Comment BSS138LT1G -> BSS138L; Device BSS138LT1G -> BSS138L; Manufacturer ON SEMICONDUCTOR -> ONSEMI; Manufacturer Part Number BSS138LT1G -> BSS138L; Part Number BSS138LT1G -> BSS138L
Changed lines of the file:
@@
 $EndComp
 $Comp
-L Transistors:BSS138LT1G Q?
+L Transistors:BSS138L Q?
 U 1 1 5D45F18B
 P 11050 5600
@@
 AR Path="/5C16C03C/5D45F18B" Ref="Q6"  Part="1"
 F 0 "Q6" H 11369 5696 50  0000 L CNN
-F 1 "BSS138LT1G" H 11369 5605 50  0000 L CNN
+F 1 "BSS138L" H 11369 5605 50  0000 L CNN
 F 2 "ICs And Semiconductors SMD:SOT95P240X110-3N" H 11050 4390 60  0001 L CNN
 F 3 "\\\\cern.ch\\dfs\\Applications\\Altium\\Datasheets\\BSS138LT1G.pdf" H 11050 5110 60  0001 L CNN
-F 4 "BSS138LT1G" H 11050 5020 60  0001 L CNN "Part Number"
+F 4 "BSS138L" H 11050 5020 60  0001 L CNN "Part Number"
 F 5 "N-MOSFET-D 1G 2S 3D" H 11050 4930 60  0001 L CNN "Library Ref"
 F 6 "SchLib\\Transistors.SchLib" H 11050 4840 60  0001 L CNN "Library Path"
-F 7 "BSS138LT1G" H 11050 4750 60  0001 L CNN "Comment"
+F 7 "BSS138L" H 11050 4750 60  0001 L CNN "Comment"
 F 8 "Standard" H 11050 4660 60  0001 L CNN "Component Kind"
 F 9 "Standard" H 11050 4570 60  0001 L CNN "Component Type"
-F 10 "BSS138LT1G" H 11050 4480 60  0001 L CNN "Device"
+F 10 "BSS138L" H 11050 4480 60  0001 L CNN "Device"
 F 11 "SOT23 3-Leads, Pitch 0.95mm - Body 1.4x3mm, IPC Medium Density" H 11050 4300 60  0001 L CNN "PackageDescription"
 F 12 " " H 11050 4210 60  0001 L CNN "Status"
 F 13 "50V 200mA N-Channel Enhancement Mode Field-Effect Transistor" H 11050 4120 60  0001 L CNN "Part Description"
-F 14 "ON SEMICONDUCTOR" H 11050 4030 60  0001 L CNN "Manufacturer"
-F 15 "BSS138LT1G" H 11050 3940 60  0001 L CNN "Manufacturer Part Number"
+F 14 "ONSEMI" H 11050 4030 60  0001 L CNN "Manufacturer"
+F 15 "BSS138L" H 11050 3940 60  0001 L CNN "Manufacturer Part Number"
 F 16 "3" H 11050 3850 60  0001 L CNN "Pin Count"
 F 17 "SOT23-3" H 11050 3760 60  0001 L CNN "Case"
@@
 $EndComp
 $Comp
-L Transistors:BSS138LT1G Q?
+L Transistors:BSS138L Q?
 U 1 1 5CDF0F00
 P 5850 9900
@@
 AR Path="/5C16C03C/5CDF0F00" Ref="Q24"  Part="1"
 F 0 "Q24" H 6169 9996 50  0000 L CNN
-F 1 "BSS138LT1G" H 6169 9905 50  0000 L CNN
+F 1 "BSS138L" H 6169 9905 50  0000 L CNN
 F 2 "ICs And Semiconductors SMD:SOT95P240X110-3N" H 5850 8690 60  0001 L CNN
 F 3 "\\\\cern.ch\\dfs\\Applications\\Altium\\Datasheets\\BSS138LT1G.pdf" H 5850 9410 60  0001 L CNN
-F 4 "BSS138LT1G" H 5850 9320 60  0001 L CNN "Part Number"
+F 4 "BSS138L" H 5850 9320 60  0001 L CNN "Part Number"
 F 5 "N-MOSFET-D 1G 2S 3D" H 5850 9230 60  0001 L CNN "Library Ref"
 F 6 "SchLib\\Transistors.SchLib" H 5850 9140 60  0001 L CNN "Library Path"
-F 7 "BSS138LT1G" H 5850 9050 60  0001 L CNN "Comment"
+F 7 "BSS138L" H 5850 9050 60  0001 L CNN "Comment"
 F 8 "Standard" H 5850 8960 60  0001 L CNN "Component Kind"
 F 9 "Standard" H 5850 8870 60  0001 L CNN "Component Type"
-F 10 "BSS138LT1G" H 5850 8780 60  0001 L CNN "Device"
+F 10 "BSS138L" H 5850 8780 60  0001 L CNN "Device"
 F 11 "SOT23 3-Leads, Pitch 0.95mm - Body 1.4x3mm, IPC Medium Density" H 5850 8600 60  0001 L CNN "PackageDescription"
 F 12 " " H 5850 8510 60  0001 L CNN "Status"
 F 13 "50V 200mA N-Channel Enhancement Mode Field-Effect Transistor" H 5850 8420 60  0001 L CNN "Part Description"
-F 14 "ON SEMICONDUCTOR" H 5850 8330 60  0001 L CNN "Manufacturer"
-F 15 "BSS138LT1G" H 5850 8240 60  0001 L CNN "Manufacturer Part Number"
+F 14 "ONSEMI" H 5850 8330 60  0001 L CNN "Manufacturer"
+F 15 "BSS138L" H 5850 8240 60  0001 L CNN "Manufacturer Part Number"
 F 16 "3" H 5850 8150 60  0001 L CNN "Pin Count"
 F 17 "SOT23-3" H 5850 8060 60  0001 L CNN "Case"
@@
 $EndComp
 $Comp
-L Transistors:BSS138LT1G Q?
+L Transistors:BSS138L Q?
 U 1 1 5CEEEA7F
 P 4700 10150
@@
 AR Path="/5C16C03C/5CEEEA7F" Ref="Q14"  Part="1"
 F 0 "Q14" H 5019 10246 50  0000 L CNN
-F 1 "BSS138LT1G" H 5019 10155 50  0000 L CNN
+F 1 "BSS138L" H 5019 10155 50  0000 L CNN
 F 2 "ICs And Semiconductors SMD:SOT95P240X110-3N" H 4700 8940 60  0001 L CNN
 F 3 "\\\\cern.ch\\dfs\\Applications\\Altium\\Datasheets\\BSS138LT1G.pdf" H 4700 9660 60  0001 L CNN
-F 4 "BSS138LT1G" H 4700 9570 60  0001 L CNN "Part Number"
+F 4 "BSS138L" H 4700 9570 60  0001 L CNN "Part Number"
 F 5 "N-MOSFET-D 1G 2S 3D" H 4700 9480 60  0001 L CNN "Library Ref"
 F 6 "SchLib\\Transistors.SchLib" H 4700 9390 60  0001 L CNN "Library Path"
-F 7 "BSS138LT1G" H 4700 9300 60  0001 L CNN "Comment"
+F 7 "BSS138L" H 4700 9300 60  0001 L CNN "Comment"
 F 8 "Standard" H 4700 9210 60  0001 L CNN "Component Kind"
 F 9 "Standard" H 4700 9120 60  0001 L CNN "Component Type"
-F 10 "BSS138LT1G" H 4700 9030 60  0001 L CNN "Device"
+F 10 "BSS138L" H 4700 9030 60  0001 L CNN "Device"
 F 11 "SOT23 3-Leads, Pitch 0.95mm - Body 1.4x3mm, IPC Medium Density" H 4700 8850 60  0001 L CNN "PackageDescription"
 F 12 " " H 4700 8760 60  0001 L CNN "Status"
 F 13 "50V 200mA N-Channel Enhancement Mode Field-Effect Transistor" H 4700 8670 60  0001 L CNN "Part Description"
-F 14 "ON SEMICONDUCTOR" H 4700 8580 60  0001 L CNN "Manufacturer"
-F 15 "BSS138LT1G" H 4700 8490 60  0001 L CNN "Manufacturer Part Number"
+F 14 "ONSEMI" H 4700 8580 60  0001 L CNN "Manufacturer"
+F 15 "BSS138L" H 4700 8490 60  0001 L CNN "Manufacturer Part Number"
 F 16 "3" H 4700 8400 60  0001 L CNN "Pin Count"
 F 17 "SOT23-3" H 4700 8310 60  0001 L CNN "Case"
@@
 $EndComp
 $Comp
-L Transistors:BSS138LT1G Q?
+L Transistors:BSS138L Q?
 U 1 1 5CF10858
 P 4700 10550
@@
 AR Path="/5C16C03C/5CF10858" Ref="Q18"  Part="1"
 F 0 "Q18" H 5019 10646 50  0000 L CNN
-F 1 "BSS138LT1G" H 5019 10555 50  0000 L CNN
+F 1 "BSS138L" H 5019 10555 50  0000 L CNN
 F 2 "ICs And Semiconductors SMD:SOT95P240X110-3N" H 4700 9340 60  0001 L CNN
 F 3 "\\\\cern.ch\\dfs\\Applications\\Altium\\Datasheets\\BSS138LT1G.pdf" H 4700 10060 60  0001 L CNN
-F 4 "BSS138LT1G" H 4700 9970 60  0001 L CNN "Part Number"
+F 4 "BSS138L" H 4700 9970 60  0001 L CNN "Part Number"
 F 5 "N-MOSFET-D 1G 2S 3D" H 4700 9880 60  0001 L CNN "Library Ref"
 F 6 "SchLib\\Transistors.SchLib" H 4700 9790 60  0001 L CNN "Library Path"
-F 7 "BSS138LT1G" H 4700 9700 60  0001 L CNN "Comment"
+F 7 "BSS138L" H 4700 9700 60  0001 L CNN "Comment"
 F 8 "Standard" H 4700 9610 60  0001 L CNN "Component Kind"
 F 9 "Standard" H 4700 9520 60  0001 L CNN "Component Type"
-F 10 "BSS138LT1G" H 4700 9430 60  0001 L CNN "Device"
+F 10 "BSS138L" H 4700 9430 60  0001 L CNN "Device"
 F 11 "SOT23 3-Leads, Pitch 0.95mm - Body 1.4x3mm, IPC Medium Density" H 4700 9250 60  0001 L CNN "PackageDescription"
 F 12 " " H 4700 9160 60  0001 L CNN "Status"
 F 13 "50V 200mA N-Channel Enhancement Mode Field-Effect Transistor" H 4700 9070 60  0001 L CNN "Part Description"
-F 14 "ON SEMICONDUCTOR" H 4700 8980 60  0001 L CNN "Manufacturer"
-F 15 "BSS138LT1G" H 4700 8890 60  0001 L CNN "Manufacturer Part Number"
+F 14 "ONSEMI" H 4700 8980 60  0001 L CNN "Manufacturer"
+F 15 "BSS138L" H 4700 8890 60  0001 L CNN "Manufacturer Part Number"
 F 16 "3" H 4700 8800 60  0001 L CNN "Pin Count"
 F 17 "SOT23-3" H 4700 8710 60  0001 L CNN "Case"

Commit message: Continuing BOM adjustments
drop BLM18SG121TZ1D as an alternate for BLM18SG121TN1D, 0603 ferrite bead

Convert PI3DBS12212AZBSEX to PI3DBS16212ZBBEX, includes part name shown on schematic
(new and improved part tested at high data rates in protoype run)
Parts:
- L10, L24, L25: Manufacturer Part Number BLM18SG121TN1D or BLM18SG121TZ1D -> BLM18SG121TN1D
Changed lines of the file:
@@
 F 20 "SMD EMIFIL Suppression Chip Ferrite Bead" H 5200 3900 60  0001 L CNN "Part Description"
 F 21 "MURATA" H 5200 3810 60  0001 L CNN "Manufacturer"
-F 22 "BLM18SG121TN1D or BLM18SG121TZ1D" H 5200 3720 60  0001 L CNN "Manufacturer Part Number"
+F 22 "BLM18SG121TN1D" H 5200 3720 60  0001 L CNN "Manufacturer Part Number"
 F 23 "0603" H 5200 3630 60  0001 L CNN "Case"
 F 24 "Yes" H 5200 3540 60  0001 L CNN "Mounted"
@@
 F 20 "SMD EMIFIL Suppression Chip Ferrite Bead" H 5200 4600 60  0001 L CNN "Part Description"
 F 21 "MURATA" H 5200 4510 60  0001 L CNN "Manufacturer"
-F 22 "BLM18SG121TN1D or BLM18SG121TZ1D" H 5200 4420 60  0001 L CNN "Manufacturer Part Number"
+F 22 "BLM18SG121TN1D" H 5200 4420 60  0001 L CNN "Manufacturer Part Number"
 F 23 "0603" H 5200 4330 60  0001 L CNN "Case"
 F 24 "Yes" H 5200 4240 60  0001 L CNN "Mounted"
@@
 F 20 "SMD EMIFIL Suppression Chip Ferrite Bead" H 2500 0   60  0001 L CNN "Part Description"
 F 21 "MURATA" H 2500 -90 60  0001 L CNN "Manufacturer"
-F 22 "BLM18SG121TN1D or BLM18SG121TZ1D" H 2500 -180 60  0001 L CNN "Manufacturer Part Number"
+F 22 "BLM18SG121TN1D" H 2500 -180 60  0001 L CNN "Manufacturer Part Number"
 F 23 "0603" H 2500 -270 60  0001 L CNN "Case"
 F 24 "Yes" H 2500 -360 60  0001 L CNN "Mounted"
