File: design/WhiteRabbit.sch (KiCad schematic (older format))
At the start: 59 parts, among them U13 LP5951MF-3.0/NOPB, U14 LM336M-2.5, U16 AD5662BRMZ-1, U19 AD5662BRMZ-1, U20 CDCM61004RHBT, Y1 OSC_25MHZ_RAKON_IVT3205CR, Y2 VM53S3-25.000-2.5/-30+75, Y3 OSC_20MHZ_IQD_LFVCXO026156, Y6 OSC_10-280MHZ_SILICON-LAB_Si5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

Commit message: Update part numbers to be closer to as-manufactured
new (at least in form) listings:
Murata  GRM188R61A106KA73D
Samsung  CL32A107MQVNNWE
Yageo  AC0402FR-0722R
Yageo  RT0402BRD0710KL
Stackpole  RMCF0402FT82K0
NXP SEMICONDUCTORS  PRTR5V0U2X,215
FTDI  FT4232H-56Q-REEL
TEXAS INSTRUMENTS  CDCM61004RHB
TEXAS INSTRUMENTS  TLV62565DBVR
TEXAS INSTRUMENTS  TPS3703A7330DSER
XILINX  XC7K160T-2FFG676I
SILICON LABS  570NCB000933DG
IQD FREQUENCY PRODUCTS  ECS-VXO-73-20.00-TR
Parts:
- U20: value CDCM61004RHBT -> CDCM61004RHB; symbol Logic:CDCM61004RHBT -> Logic:CDCM61004RHB; Device CDCM61004RHBT -> CDCM61004RHB; Manufacturer Part Number CDCM61004RHBT or CDCM61004RHBR -> CDCM61004RHBT; Part Number CDCM61004RHBT -> CDCM61004RHB
- Y3: Manufacturer Part Number LFVCXO026156 or KV7050B20.0000C3GD00 or ECS-VXO-73-20.00-TR -> ECS-VXO-73-20.00-TR
- Y6: Manufacturer Part Number 570BBC000121DG or 571BJA000107DG -> 570NCB000933DG
Changed lines of the file:
@@
 $EndComp
 $Comp
-L Logic:CDCM61004RHBT U20
+L Logic:CDCM61004RHB U20
 U 1 1 5C5B8FC6
 P 7650 1150
 F 0 "U20" H 8150 1315 50  0000 C CNN
-F 1 "CDCM61004RHBT" H 8150 1224 50  0000 C CNN
+F 1 "CDCM61004RHB" H 8150 1224 50  0000 C CNN
 F 2 "ICs And Semiconductors SMD:QFN50P500X500X100-33N-S355" H 7650 -2340 60  0001 L CNN
 F 3 "" H 7650 -1620 60  0001 L CNN
-F 4 "CDCM61004RHBT" H 7650 -1710 60  0001 L CNN "Part Number"
+F 4 "CDCM61004RHB" H 7650 -1710 60  0001 L CNN "Part Number"
 F 5 "CDCM61004RHB" H 7650 -1800 60  0001 L CNN "Library Ref"
 F 6 "SchLib\\Logic.SchLib" H 7650 -1890 60  0001 L CNN "Library Path"
@@
 F 8 "Standard" H 7650 -2070 60  0001 L CNN "Component Kind"
 F 9 "Standard" H 7650 -2160 60  0001 L CNN "Component Type"
-F 10 "CDCM61004RHBT" H 7650 -2250 60  0001 L CNN "Device"
+F 10 "CDCM61004RHB" H 7650 -2250 60  0001 L CNN "Device"
 F 11 "QFN, (MO-220-VHHD-4) 0.50mm pitch,square; 8 pin X 8 pin, 5mm X 5mm X 1.00mm H body (w/thermal tab 3.5 X 3.5mm),  IPC Medium Density" H 7650 -2430 60  0001 L CNN "PackageDescription"
 F 12 " " H 7650 -2520 60  0001 L CNN "Status"
 F 13 "Four Output, Integrated VCO, Low-Jitter Clock Generator" H 7650 -2610 60  0001 L CNN "Part Description"
 F 14 "TEXAS INSTRUMENTS" H 7650 -2700 60  0001 L CNN "Manufacturer"
-F 15 "CDCM61004RHBT or CDCM61004RHBR" H 7650 -2790 60  0001 L CNN "Manufacturer Part Number"
+F 15 "CDCM61004RHBT" H 7650 -2790 60  0001 L CNN "Manufacturer Part Number"
 F 16 "33" H 7650 -2880 60  0001 L CNN "Pin Count"
 F 17 "QFN32" H 7650 -2970 60  0001 L CNN "Case"
@@
 F 15 "3.3V, ±100ppm, 15pF, 0..70°C, HCMOS Tri-State Surface Mount, VCXO Voltage Controlled Oscillator (CFPV-45 Series)" H 7850 2700 60  0001 L CNN "Part Description"
 F 16 "IQD FREQUENCY PRODUCTS" H 7850 2610 60  0001 L CNN "Manufacturer"
-F 17 "LFVCXO026156 or KV7050B20.0000C3GD00 or ECS-VXO-73-20.00-TR" H 7850 2520 60  0001 L CNN "Manufacturer Part Number"
+F 17 "ECS-VXO-73-20.00-TR" H 7850 4075 50  0000 L CNN "Manufacturer Part Number"
 F 18 "6" H 7850 2430 60  0001 L CNN "Pin Count"
 F 19 " " H 7850 2340 60  0001 L CNN "Case"
@@
 F 14 "10-280MHz 3.3V ±20ppm LVDS Any-Rate I2C Programmable XO Oscillator Si570 Series" H 7850 3825 50  0001 L CNN "Part Description"
 F 15 "SILICON LABS" H 7850 3750 50  0001 L CNN "Manufacturer"
-F 16 "570BBC000121DG or 571BJA000107DG" H 7850 3675 50  0001 L CNN "Manufacturer Part Number"
+F 16 "570NCB000933DG" H 7850 4825 50  0000 L CNN "Manufacturer Part Number"
 F 17 "8" H 7850 3600 50  0001 L CNN "Pin Count"
 F 18 " " H 7850 3525 50  0001 L CNN "Case"

Commit message: More BOM updates for manufacturability
Use TDK MPZ2012S102JTD25 for 0805 ferrite bead.

Rename BSS138LT1G as BSS138L, ONSEMI BSS138L, now that onsemi bought Fairchild.
The T1G suffix is all about the tape&reel factory-orderable,
nothing to do with the transistor itself.

Take FPF2116 away as an MIC2090-1 alternate.  Its trip threshold
(200-400 mA) is too high for the MYRGC075050RA regulator powering
the two of them (U43 U55).

Use DAC8550 for the WR DAC (2x).  Electrically compatible with AD5662,
but uses twos-complement instead of unipolar encoding for its 16-bit
data word.  Make a note of that on the schematic.
TEXAS INSTRUMENTS DAC8550IDGK is the full name.
Parts:
- U16: value AD5662BRMZ-1 -> DAC8550IDGK; symbol Analog_&_Interface:AD5662BRMZ-1 -> Analog_&_Interface:DAC8550IDGK; Device AD5662BRMZ-1 -> DAC8550IDGK; Library Ref AD5662 -> DAC8550; Manufacturer Part Number AD5662BRMZ-1 or DAC8550IDGKT -> DAC8550IDGKT; Part Number AD5662BRMZ-1 or DAC8550IDGKT -> DAC8550IDGKT
- U19: value AD5662BRMZ-1 -> DAC8550IDGK; symbol Analog_&_Interface:AD5662BRMZ-1 -> Analog_&_Interface:DAC8550IDGK; Device AD5662BRMZ-1 or DAC8550IDGKT -> DAC8550IDGKT; Library Ref AD5662 -> DAC8550; Manufacturer Part Number AD5662BRMZ-1 or DAC8550IDGKT -> DAC8550IDGKT; Part Number AD5662BRMZ-1 or DAC8550IDGKT -> DAC8550IDGKT
Other:
- note added: "2022-08-23: Change DAC from AD5662 to DAC8550 due to\ncomponent availability. Electrically compatible, but uses\ntwos-complement instead of offset-binary for its 16-bit data word.\nTested in hardware, works."
Changed lines of the file:
@@
 Connection ~ 1500 2600
 $Comp
-L Analog_&_Interface:AD5662BRMZ-1 U16
+L Analog_&_Interface:DAC8550IDGK U16
 U 1 1 5C59700C
 P 2550 4150
 F 0 "U16" H 2900 4315 50  0000 C CNN
-F 1 "AD5662BRMZ-1" H 2900 4224 50  0000 C CNN
+F 1 "DAC8550IDGK" H 2900 4224 50  0000 C CNN
 F 2 "ICs And Semiconductors SMD:SOP65P490X110-8N" H 2550 2460 60  0001 L CNN
 F 3 "" H 2550 3180 60  0001 L CNN
-F 4 "AD5662BRMZ-1 or DAC8550IDGKT " H 2550 3090 60  0001 L CNN "Part Number"
-F 5 "AD5662" H 2550 3000 60  0001 L CNN "Library Ref"
+F 4 "DAC8550IDGKT " H 2550 3090 60  0001 L CNN "Part Number"
+F 5 "DAC8550" H 2550 3000 60  0001 L CNN "Library Ref"
 F 6 "SchLib\\Analog & Interface.SchLib" H 2550 2910 60  0001 L CNN "Library Path"
 F 7 "=Device" H 2550 2820 60  0001 L CNN "Comment"
 F 8 "Standard" H 2550 2730 60  0001 L CNN "Component Kind"
 F 9 "Standard" H 2550 2640 60  0001 L CNN "Component Type"
-F 10 "AD5662BRMZ-1" H 2550 2550 60  0001 L CNN "Device"
+F 10 "DAC8550IDGK" H 2550 2550 60  0001 L CNN "Device"
 F 11 "SOP, 0.65mm, Pitch; 8 Pin, 3.0mm W X 3.0mm L X 1.10mm H Body, IPC Medium Density" H 2550 2370 60  0001 L CNN "PackageDescription"
 F 12 " " H 2550 2280 60  0001 L CNN "Status"
 F 13 "2.7V to 5.5V, 250uA, Rail-to-Rail Output 16-Bit nanoDAC" H 2550 2190 60  0001 L CNN "Part Description"
 F 14 "ANALOG DEVICES" H 2550 2100 60  0001 L CNN "Manufacturer"
-F 15 "AD5662BRMZ-1 or DAC8550IDGKT" H 2550 2010 60  0001 L CNN "Manufacturer Part Number"
+F 15 "DAC8550IDGKT" H 2550 2010 60  0001 L CNN "Manufacturer Part Number"
 F 16 "8" H 2550 1920 60  0001 L CNN "Pin Count"
 F 17 "MSOP8" H 2550 1830 60  0001 L CNN "Case"
@@
 $EndComp
 $Comp
-L Analog_&_Interface:AD5662BRMZ-1 U19
+L Analog_&_Interface:DAC8550IDGK U19
 U 1 1 5D741523
 P 2550 5150
 F 0 "U19" H 2900 5315 50  0000 C CNN
-F 1 "AD5662BRMZ-1" H 2900 5224 50  0000 C CNN
+F 1 "DAC8550IDGK" H 2900 5224 50  0000 C CNN
 F 2 "ICs And Semiconductors SMD:SOP65P490X110-8N" H 2550 3460 60  0001 L CNN
 F 3 "" H 2550 4180 60  0001 L CNN
-F 4 "AD5662BRMZ-1 or DAC8550IDGKT " H 2550 4090 60  0001 L CNN "Part Number"
-F 5 "AD5662" H 2550 4000 60  0001 L CNN "Library Ref"
+F 4 "DAC8550IDGKT " H 2550 4090 60  0001 L CNN "Part Number"
+F 5 "DAC8550" H 2550 4000 60  0001 L CNN "Library Ref"
 F 6 "SchLib\\Analog & Interface.SchLib" H 2550 3910 60  0001 L CNN "Library Path"
 F 7 "=Device" H 2550 3820 60  0001 L CNN "Comment"
 F 8 "Standard" H 2550 3730 60  0001 L CNN "Component Kind"
 F 9 "Standard" H 2550 3640 60  0001 L CNN "Component Type"
-F 10 "AD5662BRMZ-1 or DAC8550IDGKT " H 2550 3550 60  0001 L CNN "Device"
+F 10 "DAC8550IDGKT " H 2550 3550 60  0001 L CNN "Device"
 F 11 "SOP, 0.65mm, Pitch; 8 Pin, 3.0mm W X 3.0mm L X 1.10mm H Body, IPC Medium Density" H 2550 3370 60  0001 L CNN "PackageDescription"
 F 12 " " H 2550 3280 60  0001 L CNN "Status"
 F 13 "2.7V to 5.5V, 250uA, Rail-to-Rail Output 16-Bit nanoDAC" H 2550 3190 60  0001 L CNN "Part Description"
 F 14 "ANALOG DEVICES" H 2550 3100 60  0001 L CNN "Manufacturer"
-F 15 "AD5662BRMZ-1 or DAC8550IDGKT" H 2550 3010 60  0001 L CNN "Manufacturer Part Number"
+F 15 "DAC8550IDGKT" H 2550 3010 60  0001 L CNN "Manufacturer Part Number"
 F 16 "8" H 2550 2920 60  0001 L CNN "Pin Count"
 F 17 "MSOP8" H 2550 2830 60  0001 L CNN "Case"
@@
 Wire Wire Line
 	3550 1450 3550 2400
+Text Notes 1650 3850 0    50   ~ 0
+2022-08-23:  Change DAC from AD5662 to DAC8550 due to\ncomponent availability.  Electrically compatible, but uses\ntwos-complement instead of offset-binary for its 16-bit data word.\nTested in hardware, works.
 $EndSCHEMATC

Commit message: Continuing BOM adjustments
drop BLM18SG121TZ1D as an alternate for BLM18SG121TN1D, 0603 ferrite bead

Convert PI3DBS12212AZBSEX to PI3DBS16212ZBBEX, includes part name shown on schematic
(new and improved part tested at high data rates in protoype run)
Parts:
- L11, L12, L19, L26: Manufacturer Part Number BLM18SG121TN1D or BLM18SG121TZ1D -> BLM18SG121TN1D
Changed lines of the file:
@@
 F 20 "SMD EMIFIL Suppression Chip Ferrite Bead" H 5050 5050 60  0001 L CNN "Part Description"
 F 21 "MURATA" H 5050 4960 60  0001 L CNN "Manufacturer"
-F 22 "BLM18SG121TN1D or BLM18SG121TZ1D" H 5050 4870 60  0001 L CNN "Manufacturer Part Number"
+F 22 "BLM18SG121TN1D" H 5050 4870 60  0001 L CNN "Manufacturer Part Number"
 F 23 "0603" H 5050 4780 60  0001 L CNN "Case"
 F 24 "Yes" H 5050 4690 60  0001 L CNN "Mounted"
@@
 F 20 "SMD EMIFIL Suppression Chip Ferrite Bead" H 5900 5050 60  0001 L CNN "Part Description"
 F 21 "MURATA" H 5900 4960 60  0001 L CNN "Manufacturer"
-F 22 "BLM18SG121TN1D or BLM18SG121TZ1D" H 5900 4870 60  0001 L CNN "Manufacturer Part Number"
+F 22 "BLM18SG121TN1D" H 5900 4870 60  0001 L CNN "Manufacturer Part Number"
 F 23 "0603" H 5900 4780 60  0001 L CNN "Case"
 F 24 "Yes" H 5900 4690 60  0001 L CNN "Mounted"
@@
 F 20 "SMD EMIFIL Suppression Chip Ferrite Bead" H 10300 850 60  0001 L CNN "Part Description"
 F 21 "MURATA" H 10300 760 60  0001 L CNN "Manufacturer"
-F 22 "BLM18SG121TN1D or BLM18SG121TZ1D" H 10300 670 60  0001 L CNN "Manufacturer Part Number"
+F 22 "BLM18SG121TN1D" H 10300 670 60  0001 L CNN "Manufacturer Part Number"
 F 23 "0603" H 10300 580 60  0001 L CNN "Case"
 F 24 "Yes" H 10300 490 60  0001 L CNN "Mounted"
@@
 F 20 "SMD EMIFIL Suppression Chip Ferrite Bead" H 6200 3900 60  0001 L CNN "Part Description"
 F 21 "MURATA" H 6200 3810 60  0001 L CNN "Manufacturer"
-F 22 "BLM18SG121TN1D or BLM18SG121TZ1D" H 6200 3720 60  0001 L CNN "Manufacturer Part Number"
+F 22 "BLM18SG121TN1D" H 6200 3720 60  0001 L CNN "Manufacturer Part Number"
 F 23 "0603" H 6200 3630 60  0001 L CNN "Case"
 F 24 "Yes" H 6200 3540 60  0001 L CNN "Mounted"
