File: design/Power.kicad_sch (KiCad schematic)
At the start: 77 parts, among them J1 CLIFF_FC68148(DC-10A), J19 TE_641119-2, Q1 BC857BV, Q16 SI4459BDY-T1-GE3, Q2 SI4459BDY-T1-GE3, Q22 BC857BV, Q23 SI4459BDY-T1-GE3, Q4 SI4459BDY-T1-GE3, Q8 BSS138L, Q9 BSS138L, U17 INA219BIDCNT, U18 MYRGC075050R31RA, U32 INA219BIDCNT, U40 AG5300, U41 FOD817DSD, U57 INA219BIDCNT, U62 INA219AIDR, U63 INA219AIDR, U64 INA219AIDR

Commit message: Restore some consistency in schematic metadata
Still 13 problematic footprint names in LTM4673.kicad_sch:

BAD Dup: "Footprint" "CAPC1608X87N" "Capacitors SMD:CAPC1005X55N" in LTM4673-altium-import:0_Capacitor - non polarized
BAD Dup: "Footprint" "CAPC2012X135N" "CAPC1608X87N" in LTM4673-altium-import:1_Capacitor - non polarized
BAD Dup: "Footprint" "CAPC1608X87N" "Capacitors SMD:CAPC1005X55N" in LTM4673-altium-import:1_Capacitor - non polarized
BAD Dup: "Footprint" "CAPC3216X180N" "CAPC3225X270N" in LTM4673-altium-import:1_Capacitor - non polarized
BAD Dup: "Footprint" "CAPC1608X87N" "Capacitors SMD:CAPC1005X55N" in LTM4673-altium-import:0_Capacitor - non polarized
BAD Dup: "Footprint" "CAPC1608X87N" "Capacitors SMD:CAPC1005X55N" in LTM4673-altium-import:0_Capacitor - non polarized
BAD Dup: "Footprint" "CAPC3216X180N" "CAPC3225X270N" in LTM4673-altium-import:1_Capacitor - non polarized
BAD Dup: "Footprint" "CAPC2012X135N" "CAPC1608X87N" in LTM4673-altium-import:1_Capacitor - non polarized
BAD Dup: "Footprint" "CAPC3216X180N" "CAPC3225X270N" in LTM4673-altium-import:1_Capacitor - non polarized
BAD Dup: "Footprint" "CAPC1608X87N" "Capacitors SMD:CAPC1005X55N" in LTM4673-altium-import:0_Capacitor - non polarized
BAD Dup: "Footprint" "CAPC1608X87N" "Capacitors SMD:CAPC1005X55N" in LTM4673-altium-import:1_Capacitor - non polarized
BAD Dup: "Footprint" "CAPC3216X180N" "CAPC3225X270N" in LTM4673-altium-import:1_Capacitor - non polarized
BAD Dup: "Footprint" "CAPMP7343X310N" "Capacitor_Tantalum_SMD:CP_EIA-7343-30_AVX-N" in LTM4673-altium-import:3_Capacitor - polarized

But the Symbol Field editor in eeschema should be more useful now.
Parts:
- C128, C130, C131, C134, C135: ALTIUM_VALUE 100nF -> (none); MANUFACTURER GENERIC -> (none)
- R197, R198, R281: MANUFACTURER GENERIC -> (none)
Changed lines of the file:
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@@
       (effects (font (size 1.524 1.524)) (justify left) hide)
     )
-    (property "ALTIUM_VALUE" "100nF" (id 40) (at 281.94 26.67 0)
-      (effects (font (size 1.27 1.27)) hide)
-    )
-    (property "MANUFACTURER" "GENERIC" (id 41) (at 281.94 26.67 0)
-      (effects (font (size 1.27 1.27)) hide)
-    )
     (pin "1")
     (pin "2")
@@
       (effects (font (size 1.524 1.524)) (justify left) hide)
     )
-    (property "ALTIUM_VALUE" "100nF" (id 40) (at 281.94 113.03 0)
-      (effects (font (size 1.27 1.27)) hide)
-    )
-    (property "MANUFACTURER" "GENERIC" (id 41) (at 281.94 113.03 0)
-      (effects (font (size 1.27 1.27)) hide)
-    )
     (pin "1")
     (pin "2")
@@
       (effects (font (size 1.524 1.524)) (justify left) hide)
     )
-    (property "MANUFACTURER" "GENERIC" (id 41) (at 165.1 257.81 0)
-      (effects (font (size 1.27 1.27)) hide)
-    )
     (pin "1")
     (pin "2")
@@
       (effects (font (size 1.27 1.27)) hide)
     )
-    (property "MANUFACTURER" "GENERIC" (id 42) (at 189.23 214.63 0)
-      (effects (font (size 1.27 1.27)) hide)
-    )
     (pin "1")
     (pin "2")
@@
       (effects (font (size 1.27 1.27)) hide)
     )
-    (property "MANUFACTURER" "GENERIC" (id 42) (at 189.23 222.25 0)
-      (effects (font (size 1.27 1.27)) hide)
-    )
     (pin "1")
     (pin "2")
@@
       (effects (font (size 1.27 1.27)) (justify left) hide)
     )
-    (property "ALTIUM_VALUE" "100nF" (id 39) (at 55.88 46.99 0)
-      (effects (font (size 1.27 1.27)) hide)
-    )
-    (property "MANUFACTURER" "GENERIC" (id 40) (at 55.88 46.99 0)
-      (effects (font (size 1.27 1.27)) hide)
-    )
     (pin "1")
     (pin "2")
@@
       (effects (font (size 1.27 1.27)) (justify left) hide)
     )
-    (property "ALTIUM_VALUE" "100nF" (id 39) (at 101.6 46.99 0)
-      (effects (font (size 1.27 1.27)) hide)
-    )
-    (property "MANUFACTURER" "GENERIC" (id 40) (at 101.6 46.99 0)
-      (effects (font (size 1.27 1.27)) hide)
-    )
     (pin "1")
     (pin "2")
@@
       (effects (font (size 1.27 1.27)) (justify left) hide)
     )
-    (property "ALTIUM_VALUE" "100nF" (id 39) (at 80.01 109.22 0)
-      (effects (font (size 1.27 1.27)) hide)
-    )
-    (property "MANUFACTURER" "GENERIC" (id 40) (at 80.01 109.22 0)
-      (effects (font (size 1.27 1.27)) hide)
-    )
     (pin "1")
