File: design/MMC.kicad_sch (KiCad schematic)
At the start: 58 parts, among them J21 Test connector, J22 Test connector, SW2 SKHHLQA010, SW3 KSS241GLFS, U54 STM32F207VCTx, Y5 XTAL_8MHZ_TXC_7A-8.000MAAE-T

Commit message: Restore some consistency in schematic metadata
Still 13 problematic footprint names in LTM4673.kicad_sch:

BAD Dup: "Footprint" "CAPC1608X87N" "Capacitors SMD:CAPC1005X55N" in LTM4673-altium-import:0_Capacitor - non polarized
BAD Dup: "Footprint" "CAPC2012X135N" "CAPC1608X87N" in LTM4673-altium-import:1_Capacitor - non polarized
BAD Dup: "Footprint" "CAPC1608X87N" "Capacitors SMD:CAPC1005X55N" in LTM4673-altium-import:1_Capacitor - non polarized
BAD Dup: "Footprint" "CAPC3216X180N" "CAPC3225X270N" in LTM4673-altium-import:1_Capacitor - non polarized
BAD Dup: "Footprint" "CAPC1608X87N" "Capacitors SMD:CAPC1005X55N" in LTM4673-altium-import:0_Capacitor - non polarized
BAD Dup: "Footprint" "CAPC1608X87N" "Capacitors SMD:CAPC1005X55N" in LTM4673-altium-import:0_Capacitor - non polarized
BAD Dup: "Footprint" "CAPC3216X180N" "CAPC3225X270N" in LTM4673-altium-import:1_Capacitor - non polarized
BAD Dup: "Footprint" "CAPC2012X135N" "CAPC1608X87N" in LTM4673-altium-import:1_Capacitor - non polarized
BAD Dup: "Footprint" "CAPC3216X180N" "CAPC3225X270N" in LTM4673-altium-import:1_Capacitor - non polarized
BAD Dup: "Footprint" "CAPC1608X87N" "Capacitors SMD:CAPC1005X55N" in LTM4673-altium-import:0_Capacitor - non polarized
BAD Dup: "Footprint" "CAPC1608X87N" "Capacitors SMD:CAPC1005X55N" in LTM4673-altium-import:1_Capacitor - non polarized
BAD Dup: "Footprint" "CAPC3216X180N" "CAPC3225X270N" in LTM4673-altium-import:1_Capacitor - non polarized
BAD Dup: "Footprint" "CAPMP7343X310N" "Capacitor_Tantalum_SMD:CP_EIA-7343-30_AVX-N" in LTM4673-altium-import:3_Capacitor - polarized

But the Symbol Field editor in eeschema should be more useful now.
Parts:
- C307, C308, C309, C311, C92, C93, R132, R135, R136, R151, R152, R153, R154: MANUFACTURER GENERIC -> (none)
Changed lines of the file:
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@@
     )
     (property "config" "dnf" (id 40) (at 55.88 92.71 90))
-    (property "MANUFACTURER" "GENERIC" (id 41) (at 50.8 85.09 0)
-      (effects (font (size 1.27 1.27)) hide)
-    )
     (pin "1")
     (pin "2")
@@
       (effects (font (size 1.524 1.524)) (justify left) hide)
     )
-    (property "MANUFACTURER" "GENERIC" (id 41) (at 227.33 109.22 0)
-      (effects (font (size 1.27 1.27)) hide)
-    )
     (pin "1")
     (pin "2")
@@
       (effects (font (size 1.524 1.524)) (justify left) hide)
     )
-    (property "MANUFACTURER" "GENERIC" (id 41) (at 227.33 106.68 0)
-      (effects (font (size 1.27 1.27)) hide)
-    )
     (pin "1")
     (pin "2")
@@
     )
     (property "config" "dnf" (id 41) (at 78.74 88.9 90))
-    (property "MANUFACTURER" "GENERIC" (id 42) (at 74.93 81.28 0)
-      (effects (font (size 1.27 1.27)) hide)
-    )
     (pin "1")
     (pin "2")
@@
       (effects (font (size 1.524 1.524)) (justify left) hide)
     )
-    (property "MANUFACTURER" "GENERIC" (id 41) (at 162.56 137.16 0)
-      (effects (font (size 1.27 1.27)) hide)
-    )
     (pin "1")
     (pin "2")
@@
       (effects (font (size 1.524 1.524)) (justify left) hide)
     )
-    (property "MANUFACTURER" "GENERIC" (id 41) (at 162.56 139.7 0)
-      (effects (font (size 1.27 1.27)) hide)
-    )
     (pin "1")
     (pin "2")
@@
       (effects (font (size 1.524 1.524)) (justify left) hide)
     )
-    (property "MANUFACTURER" "GENERIC" (id 41) (at 162.56 142.24 0)
-      (effects (font (size 1.27 1.27)) hide)
-    )
     (pin "1")
     (pin "2")
@@
       (effects (font (size 1.524 1.524)) (justify left) hide)
     )
-    (property "MANUFACTURER" "GENERIC" (id 41) (at 162.56 144.78 0)
-      (effects (font (size 1.27 1.27)) hide)
-    )
     (pin "1")
     (pin "2")
@@
       (effects (font (size 1.524 1.524)) (justify left) hide)
     )
-    (property "MANUFACTURER" "GENERIC" (id 40) (at 38.1 85.09 0)
-      (effects (font (size 1.27 1.27)) hide)
-    )
     (pin "1")
     (pin "2")
@@
       (effects (font (size 1.27 1.27)) (justify left) hide)
     )
-    (property "MANUFACTURER" "GENERIC" (id 39) (at 161.29 60.96 0)
-      (effects (font (size 1.27 1.27)) hide)
-    )
     (pin "1")
     (pin "2")
@@
       (effects (font (size 1.27 1.27)) (justify left) hide)
     )
-    (property "MANUFACTURER" "GENERIC" (id 39) (at 154.94 63.5 0)
-      (effects (font (size 1.27 1.27)) hide)
-    )
     (pin "1")
     (pin "2")
@@
       (effects (font (size 1.27 1.27)) (justify left) hide)
     )
-    (property "MANUFACTURER" "GENERIC" (id 39) (at 233.68 31.75 0)
-      (effects (font (size 1.27 1.27)) hide)
-    )
     (pin "1")
     (pin "2")
@@
       (effects (font (size 1.27 1.27)) (justify left) hide)
     )
-    (property "MANUFACTURER" "GENERIC" (id 39) (at 160.02 66.04 0)
-      (effects (font (size 1.27 1.27)) hide)
-    )
     (pin "1")

Commit message: moved some elements into the PCB area
moved some elements into the PCB area
Parts:
- J22: footprint Connector_PinSocket_2.54mm:PinSocket_1x14_P2.54mm_Vertical_SMD_Pin1Left -> Connector_PinHeader_2.54mm:PinHeader_1x14_P2.54mm_Vertical
Changed lines of the file:
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@@
-    (pin "9")
-  )
-  (symbol (lib_id "Connector:Conn_01x14_Male") (at 262.89 223.52 0) (mirror y) (unit 1)
-    (in_bom yes) (on_board yes)
-    (property "Reference" "J22" (id 0) (at 263.6012 224.1804 0)
-      (effects (font (size 1.27 1.27)) (justify right))
-    )
-    (property "Value" "Test connector " (id 1) (at 263.6012 226.4918 0)
-      (effects (font (size 1.27 1.27)) (justify right))
-    )
-    (property "Footprint" "Connector_PinSocket_2.54mm:PinSocket_1x14_P2.54mm_Vertical_SMD_Pin1Left" (id 2) (at 262.89 223.52 0)
-      (effects (font (size 1.27 1.27)) hide)
-    )
-    (property "Datasheet" "~" (id 3) (at 262.89 223.52 0)
-      (effects (font (size 1.27 1.27)) hide)
-    )
-    (pin "1")
-    (pin "10")
-    (pin "11")
-    (pin "12")
-    (pin "13")
-    (pin "14")
-    (pin "2")
-    (pin "3")
-    (pin "4")
-    (pin "5")
-    (pin "6")
-    (pin "7")
-    (pin "8")
     (pin "9")
   )
@@
     (pin "1")
   )
+  (symbol (lib_id "Connector:Conn_01x14_Male") (at 262.89 223.52 0) (mirror y) (unit 1)
+    (in_bom yes) (on_board yes)
+    (property "Reference" "J22" (id 0) (at 263.6012 224.1804 0)
+      (effects (font (size 1.27 1.27)) (justify right))
+    )
+    (property "Value" "Test connector " (id 1) (at 263.6012 226.4918 0)
+      (effects (font (size 1.27 1.27)) (justify right))
+    )
+    (property "Footprint" "Connector_PinHeader_2.54mm:PinHeader_1x14_P2.54mm_Vertical" (id 2) (at 262.89 223.52 0)
+      (effects (font (size 1.27 1.27)) hide)
+    )
+    (property "Datasheet" "~" (id 3) (at 262.89 223.52 0)
+      (effects (font (size 1.27 1.27)) hide)
+    )
+    (pin "1")
+    (pin "10")
+    (pin "11")
+    (pin "12")
+    (pin "13")
+    (pin "14")
+    (pin "2")
+    (pin "3")
+    (pin "4")
+    (pin "5")
+    (pin "6")
+    (pin "7")
+    (pin "8")
+    (pin "9")
+  )
 )
