File: design/FPGA_14_15.kicad_sch (KiCad schematic)
At the start: 24 parts

Commit message: new power converter added
Parts:
- C20, C21, C318, C319, C38, C39, C78: renamed from C?; value (none) -> CC0201_100NF_6.3V_10%_X5R; footprint (none) -> CAPC0603X33N
- R1, R2, R221, R222, R223: renamed from R?; value (none) -> R0402_2K2_1%_0.0625W_100PPM; footprint (none) -> RESC1005X40N
- R209, R210, R224, R225, R227: renamed from R?; value (none) -> R0402_0R_JUMPER; footprint (none) -> RESC1005X40N
- R7: value (none) -> R0402_0R_JUMPER; footprint (none) -> RESC1005X40N
- SW1: value (none) -> SW_DIP_x01; footprint (none) -> Switches:SW_OMRON_A6SN-1101
- U1: renamed from U?; value (none) -> XC7K160T-2FFG676C; footprint (none) -> ICs And Semiconductors SMD_BGA:BGA676C100P26X26_2700X2700X260
- U11: value (none) -> SN74LVC1G125DCK; footprint (none) -> SOT65P210X110-5N
- U30: value (none) -> S25FL128S; footprint (none) -> ICs And Semiconductors SMD:SOIC127P1030X265-16N
- U52: renamed from IC?; value (none) -> TCA9517DGKR; footprint (none) -> ICs And Semiconductors SMD:SOP65P490X110-8N
- U53: renamed from U?; value (none) -> TXS0108E; footprint (none) -> ICs And Semiconductors SMD:SOP65P640X120-20N

Commit message: connected signals to the J9 connector
connected signals to the J9 connector
Parts:
- C20, C21, C318, C319, C38, C39, C78, R1, R2, R209, R210, R221, R222, R223, R224, R225, R227, R7: Author CERN DEM JLC -> (none)
- U11, U52: Author CERN DEM JLC -> (none); Bonding No -> (none)
- U53: Author CERN DEM MR -> (none); Bonding No -> (none)
Changed lines of the file:
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@@
       (effects (font (size 1.524 1.524)) (justify left) hide)
     )
-    (property "Bonding" "No" (id 24) (at 359.41 137.414 0)
+    (property "Bonding" "" (id 24) (at 359.41 137.414 0)
       (effects (font (size 1.524 1.524)) (justify left) hide)
     )
@@
       (effects (font (size 1.524 1.524)) (justify left) hide)
     )
-    (property "Author" "CERN DEM JLC" (id 29) (at 359.41 148.844 0)
+    (property "Author" "" (id 29) (at 359.41 148.844 0)
       (effects (font (size 1.524 1.524)) (justify left) hide)
     )
@@
       (effects (font (size 1.524 1.524)) (justify left) hide)
     )
-    (property "Author" "CERN DEM JLC" (id 36) (at 313.69 127 0)
+    (property "Author" "" (id 36) (at 313.69 127 0)
       (effects (font (size 1.524 1.524)) (justify left) hide)
     )
@@
       (effects (font (size 1.524 1.524)) (justify left) hide)
     )
-    (property "Author" "CERN DEM JLC" (id 36) (at 313.69 129.54 0)
+    (property "Author" "" (id 36) (at 313.69 129.54 0)
       (effects (font (size 1.524 1.524)) (justify left) hide)
     )
@@
       (effects (font (size 1.524 1.524)) (justify left) hide)
     )
-    (property "Author" "CERN DEM JLC" (id 35) (at -34.544 180.34 0)
+    (property "Author" "" (id 35) (at -34.544 180.34 0)
       (effects (font (size 1.524 1.524)) (justify left) hide)
     )
@@
       (effects (font (size 1.524 1.524)) (justify left) hide)
     )
-    (property "Author" "CERN DEM JLC" (id 35) (at 3.556 180.34 0)
+    (property "Author" "" (id 35) (at 3.556 180.34 0)
       (effects (font (size 1.524 1.524)) (justify left) hide)
     )
@@
       (effects (font (size 1.27 1.27)) (justify left) hide)
     )
-    (property "Author" "CERN DEM JLC" (id 35) (at 53.34 201.168 0)
+    (property "Author" "" (id 35) (at 53.34 201.168 0)
       (effects (font (size 1.27 1.27)) (justify left) hide)
     )
@@
       (effects (font (size 1.524 1.524)) (justify left) hide)
     )
-    (property "Author" "CERN DEM JLC" (id 35) (at 300.736 91.44 0)
+    (property "Author" "" (id 35) (at 300.736 91.44 0)
       (effects (font (size 1.524 1.524)) (justify left) hide)
     )
@@
       (effects (font (size 1.524 1.524)) (justify left) hide)
     )
-    (property "Author" "CERN DEM JLC" (id 35) (at 237.236 50.8 0)
+    (property "Author" "" (id 35) (at 237.236 50.8 0)
       (effects (font (size 1.524 1.524)) (justify left) hide)
     )
@@
       (effects (font (size 1.524 1.524)) (justify left) hide)
     )
-    (property "Author" "CERN DEM JLC" (id 35) (at 247.396 50.8 0)
+    (property "Author" "" (id 35) (at 247.396 50.8 0)
       (effects (font (size 1.524 1.524)) (justify left) hide)
     )
@@
       (effects (font (size 1.524 1.524)) (justify left) hide)
     )
-    (property "Author" "CERN DEM JLC" (id 36) (at 222.25 83.82 0)
+    (property "Author" "" (id 36) (at 222.25 83.82 0)
       (effects (font (size 1.524 1.524)) (justify left) hide)
     )
@@
       (effects (font (size 1.524 1.524)) (justify left) hide)
     )
-    (property "Author" "CERN DEM JLC" (id 36) (at 222.25 91.44 0)
+    (property "Author" "" (id 36) (at 222.25 91.44 0)
       (effects (font (size 1.524 1.524)) (justify left) hide)
     )
@@
       (effects (font (size 1.524 1.524)) (justify left) hide)
     )
-    (property "Author" "CERN DEM JLC" (id 36) (at 217.17 22.86 0)
+    (property "Author" "" (id 36) (at 217.17 22.86 0)
       (effects (font (size 1.524 1.524)) (justify left) hide)
     )
@@
       (effects (font (size 1.524 1.524)) (justify left) hide)
     )
-    (property "Author" "CERN DEM JLC" (id 36) (at 308.61 134.62 0)
+    (property "Author" "" (id 36) (at 308.61 134.62 0)
       (effects (font (size 1.524 1.524)) (justify left) hide)
     )
@@
       (effects (font (size 1.524 1.524)) (justify left) hide)
     )
-    (property "Author" "CERN DEM JLC" (id 36) (at 308.61 138.43 0)
+    (property "Author" "" (id 36) (at 308.61 138.43 0)
       (effects (font (size 1.524 1.524)) (justify left) hide)
     )
@@
       (effects (font (size 1.524 1.524)) (justify left) hide)
     )
-    (property "Author" "CERN DEM JLC" (id 36) (at 308.61 142.24 0)
+    (property "Author" "" (id 36) (at 308.61 142.24 0)
       (effects (font (size 1.524 1.524)) (justify left) hide)
     )
@@
       (effects (font (size 1.27 1.27)) (justify left) hide)
     )
-    (property "Bonding" "No" (id 24) (at 93.98 144.78 0)
+    (property "Bonding" "" (id 24) (at 93.98 144.78 0)
       (effects (font (size 1.27 1.27)) (justify left) hide)
     )
@@
       (effects (font (size 1.27 1.27)) (justify left) hide)
     )
-    (property "Author" "CERN DEM JLC" (id 29) (at 93.98 154.305 0)
+    (property "Author" "" (id 29) (at 93.98 154.305 0)
       (effects (font (size 1.27 1.27)) (justify left) hide)
     )
@@
       (effects (font (size 1.524 1.524)) (justify left) hide)
     )
-    (property "Author" "CERN DEM JLC" (id 35) (at 185.674 95.25 0)
+    (property "Author" "" (id 35) (at 185.674 95.25 0)
       (effects (font (size 1.524 1.524)) (justify left) hide)
     )
@@
       (effects (font (size 1.524 1.524)) (justify left) hide)
     )
-    (property "Author" "CERN DEM JLC" (id 35) (at 151.384 92.71 0)
+    (property "Author" "" (id 35) (at 151.384 92.71 0)
       (effects (font (size 1.524 1.524)) (justify left) hide)
     )
@@
       (effects (font (size 1.524 1.524)) (justify left) hide)
     )
-    (property "Author" "CERN DEM JLC" (id 36) (at 194.31 71.12 0)
+    (property "Author" "" (id 36) (at 194.31 71.12 0)
       (effects (font (size 1.524 1.524)) (justify left) hide)
     )
@@
       (effects (font (size 1.524 1.524)) (justify left) hide)
     )
-    (property "Author" "CERN DEM JLC" (id 36) (at 189.23 71.12 0)
+    (property "Author" "" (id 36) (at 189.23 71.12 0)
       (effects (font (size 1.524 1.524)) (justify left) hide)
     )
@@
       (effects (font (size 1.27 1.27)) (justify left) hide)
     )
-    (property "Bonding" "No" (id 24) (at 66.04 232.41 0)
+    (property "Bonding" "" (id 24) (at 66.04 232.41 0)
       (effects (font (size 1.27 1.27)) (justify left) hide)
     )
@@
       (effects (font (size 1.27 1.27)) (justify left) hide)
     )
-    (property "Author" "CERN DEM MR" (id 29) (at 66.04 241.935 0)
+    (property "Author" "" (id 29) (at 66.04 241.935 0)
       (effects (font (size 1.27 1.27)) (justify left) hide)
     )

Commit message: Attempt to add and improve BOM. Added new part numbers for some of the passives
Parts:
- R209, R210, R224, R225, R227, R7: MANUFACTURER (none) -> GENERIC
Changed lines of the file:
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@@
     )
     (property "config" "dnf" (id 41) (at 323.85 38.1 0))
+    (property "MANUFACTURER" "GENERIC" (id 42) (at 313.69 39.37 0)
+      (effects (font (size 1.27 1.27)) hide)
+    )
     (pin "1")
     (pin "2")
@@
     )
     (property "config" "dnf" (id 41) (at 323.85 40.64 0))
+    (property "MANUFACTURER" "GENERIC" (id 42) (at 313.69 41.91 0)
+      (effects (font (size 1.27 1.27)) hide)
+    )
     (pin "1")
     (pin "2")
@@
       (effects (font (size 1.27 1.27)) (justify left) hide)
     )
+    (property "MANUFACTURER" "GENERIC" (id 40) (at 53.34 133.35 0)
+      (effects (font (size 1.27 1.27)) hide)
+    )
     (pin "1")
     (pin "2")
@@
       (effects (font (size 1.524 1.524)) (justify left) hide)
     )
+    (property "MANUFACTURER" "GENERIC" (id 41) (at 308.61 46.99 0)
+      (effects (font (size 1.27 1.27)) hide)
+    )
     (pin "1")
     (pin "2")
@@
     )
     (property "config" "dnf" (id 41) (at 307.34 52.07 0))
+    (property "MANUFACTURER" "GENERIC" (id 42) (at 308.61 50.8 0)
+      (effects (font (size 1.27 1.27)) hide)
+    )
     (pin "1")
     (pin "2")
@@
       (effects (font (size 1.524 1.524)) (justify left) hide)
     )
+    (property "MANUFACTURER" "GENERIC" (id 41) (at 308.61 54.61 0)
+      (effects (font (size 1.27 1.27)) hide)
+    )
     (pin "1")

Commit message: no ERC issues
no ERC issues
Changed lines of the file:
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@@
-    (stroke (width 0) (type default) (color 0 0 0 0))
-  )
-  (wire (pts (xy 64.77 41.91) (xy 38.1 41.91))
     (stroke (width 0) (type default) (color 0 0 0 0))
   )
@@
   )
   (wire (pts (xy 288.29 116.84) (xy 266.7 116.84))
-    (stroke (width 0) (type default) (color 0 0 0 0))
-  )
-  (wire (pts (xy 64.77 39.37) (xy 38.1 39.37))
     (stroke (width 0) (type default) (color 0 0 0 0))
   )
@@
     (effects (font (size 1.27 1.27) (thickness 0.254) bold) (justify left bottom))
   )
-  (label "DDR_REF_CLK_P" (at 39.37 39.37 0)
-    (effects (font (size 1.27 1.27) (thickness 0.254) bold) (justify left bottom))
-  )
   (label "I2C_SCL" (at 118.11 83.82 180)
     (effects (font (size 1.27 1.27) (thickness 0.254) bold) (justify right bottom))
@@
     (effects (font (size 1.27 1.27) (thickness 0.254) bold) (justify left bottom))
   )
-  (label "DDR_REF_CLK_N" (at 39.37 41.91 0)
-    (effects (font (size 1.27 1.27) (thickness 0.254) bold) (justify left bottom))
-  )
   (label "FMC2_LA_20_N" (at 283.21 195.58 180)
     (effects (font (size 1.27 1.27) (thickness 0.254) bold) (justify right bottom))
@@
     )
   )
-  (global_label "DDR_REF_CLK_P" (shape input) (at 64.77 39.37 0) (fields_autoplaced)
-    (effects (font (size 1.27 1.27) (thickness 0.254) bold) (justify left))
-    (property "Intersheet References" "${INTERSHEET_REFS}" (id 0) (at 0 0 0)
-      (effects (font (size 1.27 1.27)) hide)
-    )
-  )
   (global_label "FMC2_LA_23_N" (shape bidirectional) (at 288.29 180.34 0) (fields_autoplaced)
     (effects (font (size 1.27 1.27) (thickness 0.254) bold) (justify left))
@@
     (effects (font (size 1.27 1.27) (thickness 0.254) bold) (justify left))
     (property "Intersheet References" "${INTERSHEET_REFS}" (id 0) (at 0 0 0)
-      (effects (font (size 1.27 1.27)) hide)
-    )
-  )
-  (global_label "DDR_REF_CLK_N" (shape input) (at 64.77 41.91 0) (fields_autoplaced)
-    (effects (font (size 1.27 1.27) (thickness 0.254) bold) (justify left))
-    (property "Intersheet References" "${INTERSHEET_REFS}" (id 0) (at 0 0 0)

Commit message: Restore some consistency in schematic metadata
Still 13 problematic footprint names in LTM4673.kicad_sch:

BAD Dup: "Footprint" "CAPC1608X87N" "Capacitors SMD:CAPC1005X55N" in LTM4673-altium-import:0_Capacitor - non polarized
BAD Dup: "Footprint" "CAPC2012X135N" "CAPC1608X87N" in LTM4673-altium-import:1_Capacitor - non polarized
BAD Dup: "Footprint" "CAPC1608X87N" "Capacitors SMD:CAPC1005X55N" in LTM4673-altium-import:1_Capacitor - non polarized
BAD Dup: "Footprint" "CAPC3216X180N" "CAPC3225X270N" in LTM4673-altium-import:1_Capacitor - non polarized
BAD Dup: "Footprint" "CAPC1608X87N" "Capacitors SMD:CAPC1005X55N" in LTM4673-altium-import:0_Capacitor - non polarized
BAD Dup: "Footprint" "CAPC1608X87N" "Capacitors SMD:CAPC1005X55N" in LTM4673-altium-import:0_Capacitor - non polarized
BAD Dup: "Footprint" "CAPC3216X180N" "CAPC3225X270N" in LTM4673-altium-import:1_Capacitor - non polarized
BAD Dup: "Footprint" "CAPC2012X135N" "CAPC1608X87N" in LTM4673-altium-import:1_Capacitor - non polarized
BAD Dup: "Footprint" "CAPC3216X180N" "CAPC3225X270N" in LTM4673-altium-import:1_Capacitor - non polarized
BAD Dup: "Footprint" "CAPC1608X87N" "Capacitors SMD:CAPC1005X55N" in LTM4673-altium-import:0_Capacitor - non polarized
BAD Dup: "Footprint" "CAPC1608X87N" "Capacitors SMD:CAPC1005X55N" in LTM4673-altium-import:1_Capacitor - non polarized
BAD Dup: "Footprint" "CAPC3216X180N" "CAPC3225X270N" in LTM4673-altium-import:1_Capacitor - non polarized
BAD Dup: "Footprint" "CAPMP7343X310N" "Capacitor_Tantalum_SMD:CP_EIA-7343-30_AVX-N" in LTM4673-altium-import:3_Capacitor - polarized

But the Symbol Field editor in eeschema should be more useful now.
Parts:
- R209, R210, R224, R225, R227, R7: MANUFACTURER GENERIC -> (none)
Changed lines of the file:
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@@
     )
     (property "config" "dnf" (id 41) (at 323.85 38.1 0))
-    (property "MANUFACTURER" "GENERIC" (id 42) (at 313.69 39.37 0)
-      (effects (font (size 1.27 1.27)) hide)
-    )
     (pin "1")
     (pin "2")
@@
     )
     (property "config" "dnf" (id 41) (at 323.85 40.64 0))
-    (property "MANUFACTURER" "GENERIC" (id 42) (at 313.69 41.91 0)
-      (effects (font (size 1.27 1.27)) hide)
-    )
     (pin "1")
     (pin "2")
@@
       (effects (font (size 1.27 1.27)) (justify left) hide)
     )
-    (property "MANUFACTURER" "GENERIC" (id 40) (at 53.34 133.35 0)
-      (effects (font (size 1.27 1.27)) hide)
-    )
     (pin "1")
     (pin "2")
@@
       (effects (font (size 1.524 1.524)) (justify left) hide)
     )
-    (property "MANUFACTURER" "GENERIC" (id 41) (at 308.61 46.99 0)
-      (effects (font (size 1.27 1.27)) hide)
-    )
     (pin "1")
     (pin "2")
@@
     )
     (property "config" "dnf" (id 41) (at 307.34 52.07 0))
-    (property "MANUFACTURER" "GENERIC" (id 42) (at 308.61 50.8 0)
-      (effects (font (size 1.27 1.27)) hide)
-    )
     (pin "1")
     (pin "2")
@@
       (effects (font (size 1.524 1.524)) (justify left) hide)
     )
-    (property "MANUFACTURER" "GENERIC" (id 41) (at 308.61 54.61 0)
-      (effects (font (size 1.27 1.27)) hide)
-    )
     (pin "1")

Commit message: external clock connected to power supply IC, PCB routing
external clock connected to power supply IC, PCB routing
Connections:
- net FPGA_XR_GPIO_0: no longer names the net of U53.4 (A3)
- net FPGA_XR_GPIO_0_T: no longer names the net of U1.A19 (IO_L2N_T0_AD8N_15)
- net FPGA_XR_GPIO_0_T: no longer U53.17 (B3)
- no-connect marks 18 -> 21
Changed lines of the file:
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@@
   (no_connect (at 393.7 24.13))
   (no_connect (at 86.36 163.83))
+  (no_connect (at 165.1 88.9))
+  (no_connect (at 86.36 148.59))
+  (no_connect (at 60.96 148.59))
   (no_connect (at 60.96 158.75))
   (no_connect (at 86.36 168.91))
@@
     (stroke (width 0) (type default) (color 0 0 0 0))
   )
-  (wire (pts (xy 106.68 148.59) (xy 86.36 148.59))
-    (stroke (width 0) (type default) (color 0 0 0 0))
-  )
   (bus (pts (xy 374.65 181.61) (xy 374.65 184.15))
     (stroke (width 0) (type default) (color 0 0 0 0))
@@
     (stroke (width 0) (type default) (color 0 0 0 0))
   )
-  (wire (pts (xy 60.96 148.59) (xy 39.37 148.59))
-    (stroke (width 0) (type default) (color 0 0 0 0))
-  )
   (wire (pts (xy 288.29 152.4) (xy 266.7 152.4))
     (stroke (width 0) (type default) (color 0 0 0 0))
@@
   )
   (wire (pts (xy 165.1 165.1) (xy 148.59 165.1))
-    (stroke (width 0) (type default) (color 0 0 0 0))
-  )
-  (wire (pts (xy 144.78 88.9) (xy 165.1 88.9))
     (stroke (width 0) (type default) (color 0 0 0 0))
   )
@@
     (effects (font (size 1.27 1.27) (thickness 0.254) bold) (justify right bottom))
   )
-  (label "FPGA_XR_GPIO_0_T" (at 144.78 88.9 0)
-    (effects (font (size 1.27 1.27) (thickness 0.254) bold) (justify left bottom))
-  )
   (label "FMC2_LA_18_P" (at 283.21 147.32 180)
     (effects (font (size 1.27 1.27) (thickness 0.254) bold) (justify right bottom))
@@
     (effects (font (size 1.27 1.27) (thickness 0.254) bold) (justify right bottom))
   )
-  (label "FPGA_XR_GPIO_0" (at 43.18 148.59 0)
-    (effects (font (size 1.27 1.27) (thickness 0.254) bold) (justify left bottom))
-  )
   (label "Pmod1_7" (at 151.13 101.6 0)
     (effects (font (size 1.27 1.27) (thickness 0.254) bold) (justify left bottom))
@@
     (effects (font (size 1.27 1.27) (thickness 0.254) bold) (justify right bottom))
   )
-  (label "FPGA_XR_GPIO_0_T" (at 87.63 148.59 0)
-    (effects (font (size 1.27 1.27) (thickness 0.254) bold) (justify left bottom))
-  )
   (label "FMC1_LA_5_N" (at 163.83 165.1 180)
     (effects (font (size 1.27 1.27) (thickness 0.254) bold) (justify right bottom))
@@
     (effects (font (size 1.27 1.27) (thickness 0.254) bold) (justify left))
   )
-  (hierarchical_label "FPGA_XR_GPIO_0" (shape output) (at 39.37 148.59 180)
-    (effects (font (size 1.27 1.27) (thickness 0.254) bold) (justify right))
-  )
   (hierarchical_label "I2C_FPGA_SDA" (shape bidirectional) (at 50.8 81.28 180)

Commit message: Parts substitutions
As researched by Michal
MPZ2012S102JTD25 -> MPZ2012S102ATD25
BC857BV-TP -> BCM857BV-7
TPS51200DRC -> TPS51200DRCR
TXS0108E -> TXS0108EPWR
Parts:
- U53: Manufacturer Part Number TXS0108E -> TXS0108EPWR
Changed lines of the file:
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@@
       (effects (font (size 1.27 1.27)) (justify left) hide)
     )
-    (property "Manufacturer Part Number" "TXS0108E" (id 15) (at 66.04 215.265 0)
+    (property "Manufacturer Part Number" "TXS0108EPWR" (id 15) (at 66.04 215.265 0)
       (effects (font (size 1.27 1.27)) (justify left) hide)
     )
