File: design/FPGA_12_13.kicad_sch (KiCad schematic)
At the start: 7 parts

Commit message: new power converter added
Parts:
- C320, C321, C422, C423: renamed from C?; value (none) -> CC0201_100NF_6.3V_10%_X5R; footprint (none) -> CAPC0603X33N
- U1: renamed from U?; value (none) -> XC7K160T-2FFG676C; footprint (none) -> ICs And Semiconductors SMD_BGA:BGA676C100P26X26_2700X2700X260
- U51, U65: renamed from U?; value (none) -> SN74AVC2T245RSWR; footprint (none) -> ICs And Semiconductors SMD:QFN40P140X180X55-10N

Commit message: connected signals to the J9 connector
connected signals to the J9 connector
Parts:
- C320, C321, C422, C423: Author CERN DEM JLC -> (none)
- U51, U65: Author CERN DEM JLC -> (none); Bonding No -> (none)
Changed lines of the file:
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@@
       (effects (font (size 1.524 1.524)) (justify left) hide)
     )
-    (property "Bonding" "No" (id 24) (at 69.85 165.1 0)
+    (property "Bonding" "" (id 24) (at 69.85 165.1 0)
       (effects (font (size 1.524 1.524)) (justify left) hide)
     )
@@
       (effects (font (size 1.524 1.524)) (justify left) hide)
     )
-    (property "Author" "CERN DEM JLC" (id 29) (at 69.85 176.53 0)
+    (property "Author" "" (id 29) (at 69.85 176.53 0)
       (effects (font (size 1.524 1.524)) (justify left) hide)
     )
@@
       (effects (font (size 1.524 1.524)) (justify left) hide)
     )
-    (property "Author" "CERN DEM JLC" (id 35) (at -16.764 111.76 0)
+    (property "Author" "" (id 35) (at -16.764 111.76 0)
       (effects (font (size 1.524 1.524)) (justify left) hide)
     )
@@
       (effects (font (size 1.524 1.524)) (justify left) hide)
     )
-    (property "Author" "CERN DEM JLC" (id 35) (at -5.334 111.76 0)
+    (property "Author" "" (id 35) (at -5.334 111.76 0)
       (effects (font (size 1.524 1.524)) (justify left) hide)
     )
@@
       (effects (font (size 1.524 1.524)) (justify left) hide)
     )
-    (property "Bonding" "No" (id 24) (at 69.85 218.44 0)
+    (property "Bonding" "" (id 24) (at 69.85 218.44 0)
       (effects (font (size 1.524 1.524)) (justify left) hide)
     )
@@
       (effects (font (size 1.524 1.524)) (justify left) hide)
     )
-    (property "Author" "CERN DEM JLC" (id 29) (at 69.85 229.87 0)
+    (property "Author" "" (id 29) (at 69.85 229.87 0)
       (effects (font (size 1.524 1.524)) (justify left) hide)
     )
@@
       (effects (font (size 1.524 1.524)) (justify left) hide)
     )
-    (property "Author" "CERN DEM JLC" (id 35) (at -16.764 165.1 0)
+    (property "Author" "" (id 35) (at -16.764 165.1 0)
       (effects (font (size 1.524 1.524)) (justify left) hide)
     )
@@
       (effects (font (size 1.524 1.524)) (justify left) hide)
     )
-    (property "Author" "CERN DEM JLC" (id 35) (at -5.334 165.1 0)
-      (effects (font (size 1.524 1.524)) (justify left) hide)
-    )
+    (property "Author" "" (id 35) (at -5.334 165.1 0)
+      (effects (font (size 1.524 1.524)) (justify left) hide)
+    )
