File: design/FPGA_32_16.kicad_sch (KiCad schematic)
At the start: 3 parts

Commit message: new power converter added
Parts:
- C18, C19: renamed from C?; value (none) -> CC0201_100NF_6.3V_10%_X5R; footprint (none) -> CAPC0603X33N
- U1: renamed from U?; value (none) -> XC7K160T-2FFG676C; footprint (none) -> ICs And Semiconductors SMD_BGA:BGA676C100P26X26_2700X2700X260
Changed lines of the file:
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@@
   (symbol (lib_id "marble_misc:XC7K160T-FFG676") (at 184.15 99.06 0) (mirror y) (unit 3)
     (in_bom yes) (on_board yes)
-    (property "Reference" "U?" (id 0) (at 184.15 174.625 0))
-    (property "Value" "" (id 1) (at 184.15 176.9364 0))
-    (property "Footprint" "" (id 2) (at 184.15 99.06 0)
+    (property "Reference" "U1" (id 0) (at 184.15 174.625 0))
+    (property "Value" "XC7K160T-2FFG676C" (id 1) (at 184.15 176.9364 0))
+    (property "Footprint" "ICs And Semiconductors SMD_BGA:BGA676C100P26X26_2700X2700X260" (id 2) (at 184.15 99.06 0)
       (effects (font (size 1.27 1.27)) hide)
     )
@@
   (symbol (lib_id "power:+2V5") (at 212.09 22.86 0) (unit 1)
     (in_bom yes) (on_board yes)
-    (property "Reference" "#PWR?" (id 0) (at 212.09 26.67 0)
-      (effects (font (size 1.27 1.27)) hide)
-    )
-    (property "Value" "" (id 1) (at 212.471 18.4658 0))
+    (property "Reference" "#PWR0794" (id 0) (at 212.09 26.67 0)
+      (effects (font (size 1.27 1.27)) hide)
+    )
+    (property "Value" "+2V5" (id 1) (at 212.471 18.4658 0))
     (property "Footprint" "" (id 2) (at 212.09 22.86 0)
       (effects (font (size 1.27 1.27)) hide)
@@
   (symbol (lib_id "Capacitors_SMD:CC0201_100NF_6.3V_10%_X5R") (at 109.22 142.24 270) (unit 1)
     (in_bom yes) (on_board yes)
-    (property "Reference" "C?" (id 0) (at 109.22 143.51 90)
+    (property "Reference" "C19" (id 0) (at 109.22 143.51 90)
       (effects (font (size 1.27 1.27)) (justify left))
     )
-    (property "Value" "" (id 1) (at 102.616 142.24 0)
-      (effects (font (size 1.524 1.524)) (justify left) hide)
-    )
-    (property "Footprint" "" (id 2) (at 82.042 142.24 0)
+    (property "Value" "CC0201_100NF_6.3V_10%_X5R" (id 1) (at 102.616 142.24 0)
+      (effects (font (size 1.524 1.524)) (justify left) hide)
+    )
+    (property "Footprint" "CAPC0603X33N" (id 2) (at 82.042 142.24 0)
       (effects (font (size 1.524 1.524)) (justify left) hide)
     )
@@
   (symbol (lib_id "Capacitors_SMD:CC0201_100NF_6.3V_10%_X5R") (at 109.22 76.2 270) (unit 1)
     (in_bom yes) (on_board yes)
-    (property "Reference" "C?" (id 0) (at 109.22 77.47 90)
+    (property "Reference" "C18" (id 0) (at 109.22 77.47 90)
       (effects (font (size 1.27 1.27)) (justify left))
     )
-    (property "Value" "" (id 1) (at 102.616 76.2 0)
-      (effects (font (size 1.524 1.524)) (justify left) hide)
-    )
-    (property "Footprint" "" (id 2) (at 82.042 76.2 0)
+    (property "Value" "CC0201_100NF_6.3V_10%_X5R" (id 1) (at 102.616 76.2 0)
+      (effects (font (size 1.524 1.524)) (justify left) hide)
+    )
+    (property "Footprint" "CAPC0603X33N" (id 2) (at 82.042 76.2 0)
       (effects (font (size 1.524 1.524)) (justify left) hide)
     )
@@
   (symbol (lib_id "power:GND") (at 109.22 149.86 0) (unit 1)
     (in_bom yes) (on_board yes)
-    (property "Reference" "#PWR?" (id 0) (at 109.22 156.21 0)
-      (effects (font (size 1.27 1.27)) hide)
-    )
-    (property "Value" "" (id 1) (at 109.347 154.2542 0))
+    (property "Reference" "#PWR0773" (id 0) (at 109.22 156.21 0)
+      (effects (font (size 1.27 1.27)) hide)
+    )
+    (property "Value" "GND" (id 1) (at 109.347 154.2542 0))
     (property "Footprint" "" (id 2) (at 109.22 149.86 0)
       (effects (font (size 1.27 1.27)) hide)
@@
   (symbol (lib_id "power:GND") (at 109.22 83.82 0) (unit 1)
     (in_bom yes) (on_board yes)
-    (property "Reference" "#PWR?" (id 0) (at 109.22 90.17 0)
-      (effects (font (size 1.27 1.27)) hide)
-    )
-    (property "Value" "" (id 1) (at 109.347 88.2142 0))
+    (property "Reference" "#PWR0774" (id 0) (at 109.22 90.17 0)
+      (effects (font (size 1.27 1.27)) hide)
+    )
+    (property "Value" "GND" (id 1) (at 109.347 88.2142 0))
     (property "Footprint" "" (id 2) (at 109.22 83.82 0)
       (effects (font (size 1.27 1.27)) hide)
@@
   (symbol (lib_id "power:+1V5") (at 143.51 22.86 0) (unit 1)
     (in_bom yes) (on_board yes)
-    (property "Reference" "#PWR?" (id 0) (at 143.51 26.67 0)
-      (effects (font (size 1.27 1.27)) hide)
-    )
-    (property "Value" "" (id 1) (at 143.891 18.4658 0))
+    (property "Reference" "#PWR0648" (id 0) (at 143.51 26.67 0)
+      (effects (font (size 1.27 1.27)) hide)
+    )
+    (property "Value" "+1V5" (id 1) (at 143.891 18.4658 0))
     (property "Footprint" "" (id 2) (at 143.51 22.86 0)
       (effects (font (size 1.27 1.27)) hide)

Commit message: connected signals to the J9 connector
connected signals to the J9 connector
Parts:
- C18, C19: Author CERN DEM JLC -> (none)
Changed lines of the file:
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@@
       (effects (font (size 1.524 1.524)) (justify left) hide)
     )
-    (property "Author" "CERN DEM JLC" (id 35) (at 22.606 142.24 0)
+    (property "Author" "" (id 35) (at 22.606 142.24 0)
       (effects (font (size 1.524 1.524)) (justify left) hide)
     )
@@
       (effects (font (size 1.524 1.524)) (justify left) hide)
     )
-    (property "Author" "CERN DEM JLC" (id 35) (at 22.606 76.2 0)
+    (property "Author" "" (id 35) (at 22.606 76.2 0)
       (effects (font (size 1.524 1.524)) (justify left) hide)
     )

Commit message: external clock connected to power supply IC, PCB routing
external clock connected to power supply IC, PCB routing
Connections:
- net FPGA_CLKIN12: now reaches U1.D11 (IO_L14N_T2_SRCC_16)
- net FPGA_CLKIN0: now reaches U1.G11 (IO_L11P_T1_SRCC_16)
- net FPGA_CLKIN3: now reaches U1.J14 (IO_25_16)
- no-connect marks 7 -> 4
Changed lines of the file:
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@@
   (junction (at 153.67 25.4) (diameter 0) (color 0 0 0 0)
   )
-  (no_connect (at 234.95 170.18))
   (no_connect (at 133.35 137.16))
-  (no_connect (at 234.95 99.06))
   (no_connect (at 133.35 45.72))
   (no_connect (at 133.35 170.18))
-  (no_connect (at 234.95 116.84))
   (no_connect (at 133.35 106.68))
   (bus_entry (at 46.99 121.92) (size -2.54 -2.54)
@@
     (stroke (width 0) (type default) (color 0 0 0 0))
   )
+  (wire (pts (xy 234.95 170.18) (xy 269.24 170.18))
+    (stroke (width 0) (type default) (color 0 0 0 0))
+  )
   (wire (pts (xy 33.02 147.32) (xy 50.8 147.32))
     (stroke (width 0) (type default) (color 0 0 0 0))
@@
     (stroke (width 0) (type default) (color 0 0 0 0))
   )
+  (wire (pts (xy 234.95 99.06) (xy 270.51 99.06))
+    (stroke (width 0) (type default) (color 0 0 0 0))
+  )
   (wire (pts (xy 119.38 152.4) (xy 133.35 152.4))
     (stroke (width 0) (type default) (color 0 0 0 0))
@@
     (stroke (width 0) (type default) (color 0 0 0 0))
   )
+  (wire (pts (xy 234.95 116.84) (xy 270.51 116.84))
+    (stroke (width 0) (type default) (color 0 0 0 0))
+  )
   (wire (pts (xy 119.38 132.08) (xy 133.35 132.08))
     (stroke (width 0) (type default) (color 0 0 0 0))
@@
     (effects (font (size 1.27 1.27) (thickness 0.254) bold) (justify right bottom))
   )
+  (label "FPGA_CLKIN3" (at 237.49 170.18 0)
+    (effects (font (size 1.27 1.27) (thickness 0.254) bold) (justify left bottom))
+  )
   (label "FMC1_LA_26_P" (at 250.19 134.62 180)
     (effects (font (size 1.27 1.27) (thickness 0.254) bold) (justify right bottom))
@@
     (effects (font (size 1.27 1.27)) (justify left bottom))
   )
+  (label "FPGA_CLKIN0" (at 238.76 99.06 0)
+    (effects (font (size 1.27 1.27) (thickness 0.254) bold) (justify left bottom))
+  )
   (label "DDR3_DQ24" (at 33.02 88.9 0)
     (effects (font (size 1.27 1.27)) (justify left bottom))
+  )
+  (label "FPGA_CLKIN12" (at 238.76 116.84 0)
+    (effects (font (size 1.27 1.27) (thickness 0.254) bold) (justify left bottom))
   )
   (label "DDR3_DQ12" (at 33.02 58.42 0)
@@
     (effects (font (size 1.27 1.27) (thickness 0.254) bold) (justify left))
   )
+  (hierarchical_label "FPGA_CLKIN0" (shape output) (at 270.51 99.06 0)
+    (effects (font (size 1.27 1.27) (thickness 0.254) bold) (justify left))
+  )
   (hierarchical_label "RGMII_TXD[0..3]" (shape input) (at 332.74 167.64 0)
     (effects (font (size 1.27 1.27) (thickness 0.254) bold) (justify left))
@@
     (effects (font (size 1.27 1.27)) (justify left))
   )
+  (hierarchical_label "FPGA_CLKIN12" (shape output) (at 270.51 116.84 0)
+    (effects (font (size 1.27 1.27) (thickness 0.254) bold) (justify left))
+  )
   (hierarchical_label "DDR3_DQS3_N" (shape bidirectional) (at 50.8 160.02 0)
     (effects (font (size 1.27 1.27)) (justify left))
   )
+  (hierarchical_label "FPGA_CLKIN3" (shape output) (at 269.24 170.18 0)
+    (effects (font (size 1.27 1.27) (thickness 0.254) bold) (justify left))
+  )
   (hierarchical_label "VREF_DDR3" (shape input) (at 107.95 76.2 180)
