File: design/GBX_MUX.kicad_sch (KiCad schematic)
At the start: 24 parts

Commit message: new power converter added
Parts:
- C103, C104, C23, C290, C291, C292, C305, C306, C37, C377, C395, C396, C397: renamed from C?; value (none) -> CC0201_100NF_6.3V_10%_X5R; footprint (none) -> CAPC0603X33N
- R297, R298, R299, R300: renamed from R?; value (none) -> R0402_10K_1%_0.0625W_100PPM; footprint (none) -> RESC1005X40N
- U44, U45, U46, U48, U49, U50: value (none) -> PI3DBS16212ZBBEX; footprint (none) -> ICs And Semiconductors SMD:PERICOM_ZBS20
- U56: value (none) -> 74AHC1G04GW; footprint (none) -> ICs And Semiconductors SMD:SOT65P212X110-5N

Commit message: connected signals to the J9 connector
connected signals to the J9 connector
Parts:
- C103, C104, C23, C290, C291, C292, C305, C306, C37, C377, C395, C396, C397, R297, R298, R299, R300: Author CERN DEM JLC -> (none)
- U44, U45, U46, U48, U49, U50, U56: Author CERN DEM JLC -> (none); Bonding No -> (none)
Changed lines of the file:
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@@
       (effects (font (size 1.27 1.27)) (justify left) hide)
     )
-    (property "Bonding" "No" (id 24) (at 210.82 162.56 0)
+    (property "Bonding" "" (id 24) (at 210.82 162.56 0)
       (effects (font (size 1.27 1.27)) (justify left) hide)
     )
@@
       (effects (font (size 1.27 1.27)) (justify left) hide)
     )
-    (property "Author" "CERN DEM JLC" (id 29) (at 210.82 172.085 0)
+    (property "Author" "" (id 29) (at 210.82 172.085 0)
       (effects (font (size 1.27 1.27)) (justify left) hide)
     )
@@
       (effects (font (size 1.27 1.27)) (justify left) hide)
     )
-    (property "Bonding" "No" (id 24) (at 210.82 209.55 0)
+    (property "Bonding" "" (id 24) (at 210.82 209.55 0)
       (effects (font (size 1.27 1.27)) (justify left) hide)
     )
@@
       (effects (font (size 1.27 1.27)) (justify left) hide)
     )
-    (property "Author" "CERN DEM JLC" (id 29) (at 210.82 219.075 0)
+    (property "Author" "" (id 29) (at 210.82 219.075 0)
       (effects (font (size 1.27 1.27)) (justify left) hide)
     )
@@
       (effects (font (size 1.524 1.524)) (justify left) hide)
     )
-    (property "Author" "CERN DEM JLC" (id 36) (at 143.51 50.8 0)
+    (property "Author" "" (id 36) (at 143.51 50.8 0)
       (effects (font (size 1.524 1.524)) (justify left) hide)
     )
@@
       (effects (font (size 1.524 1.524)) (justify left) hide)
     )
-    (property "Author" "CERN DEM JLC" (id 36) (at 149.86 50.8 0)
+    (property "Author" "" (id 36) (at 149.86 50.8 0)
       (effects (font (size 1.524 1.524)) (justify left) hide)
     )
@@
       (effects (font (size 1.524 1.524)) (justify left) hide)
     )
-    (property "Author" "CERN DEM JLC" (id 36) (at 156.21 50.8 0)
+    (property "Author" "" (id 36) (at 156.21 50.8 0)
       (effects (font (size 1.524 1.524)) (justify left) hide)
     )
@@
       (effects (font (size 1.524 1.524)) (justify left) hide)
     )
-    (property "Author" "CERN DEM JLC" (id 36) (at 137.16 50.8 0)
+    (property "Author" "" (id 36) (at 137.16 50.8 0)
       (effects (font (size 1.524 1.524)) (justify left) hide)
     )
@@
       (effects (font (size 1.524 1.524)) (justify left) hide)
     )
-    (property "Author" "CERN DEM JLC" (id 35) (at 32.766 148.59 0)
+    (property "Author" "" (id 35) (at 32.766 148.59 0)
       (effects (font (size 1.524 1.524)) (justify left) hide)
     )
@@
       (effects (font (size 1.524 1.524)) (justify left) hide)
     )
-    (property "Author" "CERN DEM JLC" (id 35) (at 45.466 148.59 0)
+    (property "Author" "" (id 35) (at 45.466 148.59 0)
       (effects (font (size 1.524 1.524)) (justify left) hide)
     )
@@
       (effects (font (size 1.524 1.524)) (justify left) hide)
     )
-    (property "Author" "CERN DEM JLC" (id 35) (at 58.166 148.59 0)
+    (property "Author" "" (id 35) (at 58.166 148.59 0)
       (effects (font (size 1.524 1.524)) (justify left) hide)
     )
@@
       (effects (font (size 1.27 1.27)) (justify left) hide)
     )
-    (property "Bonding" "No" (id 24) (at 38.1 109.22 0)
+    (property "Bonding" "" (id 24) (at 38.1 109.22 0)
       (effects (font (size 1.27 1.27)) (justify left) hide)
     )
@@
       (effects (font (size 1.27 1.27)) (justify left) hide)
     )
-    (property "Author" "CERN DEM JLC" (id 29) (at 38.1 118.745 0)
+    (property "Author" "" (id 29) (at 38.1 118.745 0)
       (effects (font (size 1.27 1.27)) (justify left) hide)
     )
@@
       (effects (font (size 1.27 1.27)) (justify left) hide)
     )
-    (property "Bonding" "No" (id 24) (at 38.1 156.21 0)
+    (property "Bonding" "" (id 24) (at 38.1 156.21 0)
       (effects (font (size 1.27 1.27)) (justify left) hide)
     )
@@
       (effects (font (size 1.27 1.27)) (justify left) hide)
     )
-    (property "Author" "CERN DEM JLC" (id 29) (at 38.1 165.735 0)
+    (property "Author" "" (id 29) (at 38.1 165.735 0)
       (effects (font (size 1.27 1.27)) (justify left) hide)
     )
@@
       (effects (font (size 1.27 1.27)) (justify left) hide)
     )
-    (property "Bonding" "No" (id 24) (at 119.38 109.22 0)
+    (property "Bonding" "" (id 24) (at 119.38 109.22 0)
       (effects (font (size 1.27 1.27)) (justify left) hide)
     )
@@
       (effects (font (size 1.27 1.27)) (justify left) hide)
     )
-    (property "Author" "CERN DEM JLC" (id 29) (at 119.38 118.745 0)
+    (property "Author" "" (id 29) (at 119.38 118.745 0)
       (effects (font (size 1.27 1.27)) (justify left) hide)
     )
@@
       (effects (font (size 1.27 1.27)) (justify left) hide)
     )
-    (property "Bonding" "No" (id 24) (at 119.38 156.21 0)
+    (property "Bonding" "" (id 24) (at 119.38 156.21 0)
       (effects (font (size 1.27 1.27)) (justify left) hide)
     )
@@
       (effects (font (size 1.27 1.27)) (justify left) hide)
     )
-    (property "Author" "CERN DEM JLC" (id 29) (at 119.38 165.735 0)
+    (property "Author" "" (id 29) (at 119.38 165.735 0)
       (effects (font (size 1.27 1.27)) (justify left) hide)
     )
@@
       (effects (font (size 1.524 1.524)) (justify left) hide)
     )
-    (property "Author" "CERN DEM JLC" (id 35) (at -4.064 148.59 0)
+    (property "Author" "" (id 35) (at -4.064 148.59 0)
       (effects (font (size 1.524 1.524)) (justify left) hide)
     )
@@
       (effects (font (size 1.524 1.524)) (justify left) hide)
     )
-    (property "Author" "CERN DEM JLC" (id 35) (at 8.636 148.59 0)
+    (property "Author" "" (id 35) (at 8.636 148.59 0)
       (effects (font (size 1.524 1.524)) (justify left) hide)
     )
@@
       (effects (font (size 1.524 1.524)) (justify left) hide)
     )
-    (property "Author" "CERN DEM JLC" (id 35) (at 21.336 148.59 0)
+    (property "Author" "" (id 35) (at 21.336 148.59 0)
       (effects (font (size 1.524 1.524)) (justify left) hide)
     )
@@
       (effects (font (size 1.27 1.27)) (justify left) hide)
     )
-    (property "Bonding" "No" (id 24) (at 40.64 171.704 0)
+    (property "Bonding" "" (id 24) (at 40.64 171.704 0)
       (effects (font (size 1.27 1.27)) (justify left) hide)
     )
@@
       (effects (font (size 1.27 1.27)) (justify left) hide)
     )
-    (property "Author" "CERN DEM JLC" (id 29) (at 40.64 181.229 0)
+    (property "Author" "" (id 29) (at 40.64 181.229 0)
       (effects (font (size 1.27 1.27)) (justify left) hide)
     )
@@
       (effects (font (size 1.524 1.524)) (justify left) hide)
     )
-    (property "Author" "CERN DEM JLC" (id 35) (at -40.894 127 0)
+    (property "Author" "" (id 35) (at -40.894 127 0)
       (effects (font (size 1.524 1.524)) (justify left) hide)
     )
@@
       (effects (font (size 1.524 1.524)) (justify left) hide)
     )
-    (property "Author" "CERN DEM JLC" (id 35) (at 32.766 172.72 0)
+    (property "Author" "" (id 35) (at 32.766 172.72 0)
       (effects (font (size 1.524 1.524)) (justify left) hide)
     )
@@
       (effects (font (size 1.524 1.524)) (justify left) hide)
     )
-    (property "Author" "CERN DEM JLC" (id 35) (at 45.466 172.72 0)
+    (property "Author" "" (id 35) (at 45.466 172.72 0)
       (effects (font (size 1.524 1.524)) (justify left) hide)
     )
@@
       (effects (font (size 1.524 1.524)) (justify left) hide)
     )
-    (property "Author" "CERN DEM JLC" (id 35) (at 58.166 172.72 0)
+    (property "Author" "" (id 35) (at 58.166 172.72 0)
       (effects (font (size 1.524 1.524)) (justify left) hide)
     )
@@
       (effects (font (size 1.524 1.524)) (justify left) hide)
     )
-    (property "Author" "CERN DEM JLC" (id 35) (at -4.064 172.72 0)
+    (property "Author" "" (id 35) (at -4.064 172.72 0)
       (effects (font (size 1.524 1.524)) (justify left) hide)
     )
@@
       (effects (font (size 1.524 1.524)) (justify left) hide)
     )
-    (property "Author" "CERN DEM JLC" (id 35) (at 8.636 172.72 0)
+    (property "Author" "" (id 35) (at 8.636 172.72 0)
       (effects (font (size 1.524 1.524)) (justify left) hide)
     )
@@
       (effects (font (size 1.524 1.524)) (justify left) hide)
     )
-    (property "Author" "CERN DEM JLC" (id 35) (at 21.336 172.72 0)
+    (property "Author" "" (id 35) (at 21.336 172.72 0)
       (effects (font (size 1.524 1.524)) (justify left) hide)
     )

Commit message: Attempt to add and improve BOM. Added new part numbers for some of the passives
Changed lines of the file:
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@@
   (junction (at 241.3 156.21) (diameter 0) (color 0 0 0 0)
-  )
-  (junction (at 45.72 127) (diameter 0) (color 0 0 0 0)
   )
   (junction (at 68.58 100.33) (diameter 0) (color 0 0 0 0)

Commit message: no ERC issues
no ERC issues
Changed lines of the file:
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@@
   (symbol (lib_id "Standard_Logic:74AHC1G04GW") (at 40.64 116.84 0) (mirror y) (unit 1)
     (in_bom yes) (on_board yes)
-    (property "Reference" "U56" (id 0) (at 36.83 116.205 0))
+    (property "Reference" "U56" (id 0) (at 44.45 116.205 0))
     (property "Value" "74AHC1G04GW" (id 1) (at 40.64 127.889 0)
       (effects (font (size 1.27 1.27)) (justify left) hide)
