File: design/QSFP.kicad_sch (KiCad schematic)
At the start: 22 parts

Commit message: new power converter added
Parts:
- C293, C294, C295, C299, C300, C301: renamed from C?; value (none) -> CC0201_100NF_6.3V_10%_X5R; footprint (none) -> CAPC0603X33N
- C296, C297, C298, C302, C303, C304: renamed from C?; value (none) -> CC0603_22UF_6.3V_20%_X5R; footprint (none) -> CAPC1709X100N
- J18: value (none) -> QSFPk-PF-2; footprint (none) -> QSFPK-PF-02:QSFPK-PF-02
- J8: renamed from J?; value (none) -> SAMTEC_QSFP8-038-01-L-D-RA1; footprint (none) -> SAMTEC SMD:SAMTEC_QSFP8-038-01-L-D-RA1
- L1, L2, L5: renamed from L?; value (none) -> IND0603_MURATA_BLM18SG121TN1D; footprint (none) -> INDC1608X65N
- R35: renamed from R301; value (none) -> R0402_4K7_1%_0.0625W_100PPM; footprint (none) -> Resistors SMD:RESC1005X40N
- R36: renamed from R302; value (none) -> R0402_4K7_1%_0.0625W_100PPM; footprint (none) -> Resistors SMD:RESC1005X40N
- R37: renamed from R303; value (none) -> R0402_4K7_1%_0.0625W_100PPM; footprint (none) -> Resistors SMD:RESC1005X40N
- R38: renamed from R304; value (none) -> R0402_4K7_1%_0.0625W_100PPM; footprint (none) -> Resistors SMD:RESC1005X40N
- R77: renamed from R305; value (none) -> R0402_4K7_1%_0.0625W_100PPM; footprint (none) -> Resistors SMD:RESC1005X40N

Commit message: connected signals to the J9 connector
connected signals to the J9 connector
Parts:
- C293, C294, C295, C296, C297, C298, C299, C300, C301, C302, C303, C304, J8, L1, L2, L5, R35, R36, R37, R38, R77: Author CERN DEM JLC -> (none)
Changed lines of the file:
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@@
       (effects (font (size 1.27 1.27)) (justify left) hide)
     )
-    (property "Author" "CERN DEM JLC" (id 31) (at 180.34 148.59 0)
+    (property "Author" "" (id 31) (at 180.34 148.59 0)
       (effects (font (size 1.27 1.27)) (justify left) hide)
     )
@@
       (effects (font (size 1.524 1.524)) (justify left) hide)
     )
-    (property "Author" "CERN DEM JLC" (id 35) (at -51.054 54.61 0)
+    (property "Author" "" (id 35) (at -51.054 54.61 0)
       (effects (font (size 1.524 1.524)) (justify left) hide)
     )
@@
       (effects (font (size 1.524 1.524)) (justify left) hide)
     )
-    (property "Author" "CERN DEM JLC" (id 35) (at -18.034 54.61 0)
+    (property "Author" "" (id 35) (at -18.034 54.61 0)
       (effects (font (size 1.524 1.524)) (justify left) hide)
     )
@@
       (effects (font (size 1.524 1.524)) (justify left) hide)
     )
-    (property "Author" "CERN DEM JLC" (id 31) (at 55.88 130.302 0)
+    (property "Author" "" (id 31) (at 55.88 130.302 0)
       (effects (font (size 1.524 1.524)) (justify left) hide)
     )
@@
       (effects (font (size 1.27 1.27)) (justify left) hide)
     )
-    (property "Author" "CERN DEM JLC" (id 35) (at 233.68 124.968 0)
+    (property "Author" "" (id 35) (at 233.68 124.968 0)
       (effects (font (size 1.27 1.27)) (justify left) hide)
     )
@@
       (effects (font (size 1.27 1.27)) (justify left) hide)
     )
-    (property "Author" "CERN DEM JLC" (id 35) (at 233.68 127.508 0)
+    (property "Author" "" (id 35) (at 233.68 127.508 0)
       (effects (font (size 1.27 1.27)) (justify left) hide)
     )
@@
       (effects (font (size 1.27 1.27)) (justify left) hide)
     )
-    (property "Author" "CERN DEM JLC" (id 35) (at 233.68 135.128 0)
+    (property "Author" "" (id 35) (at 233.68 135.128 0)
       (effects (font (size 1.27 1.27)) (justify left) hide)
     )
@@
       (effects (font (size 1.27 1.27)) (justify left) hide)
     )
-    (property "Author" "CERN DEM JLC" (id 35) (at 143.51 124.968 0)
+    (property "Author" "" (id 35) (at 143.51 124.968 0)
       (effects (font (size 1.27 1.27)) (justify left) hide)
     )
@@
       (effects (font (size 1.27 1.27)) (justify left) hide)
     )
-    (property "Author" "CERN DEM JLC" (id 35) (at 143.51 127.508 0)
+    (property "Author" "" (id 35) (at 143.51 127.508 0)
       (effects (font (size 1.27 1.27)) (justify left) hide)
     )
@@
       (effects (font (size 1.524 1.524)) (justify left) hide)
     )
-    (property "Author" "CERN DEM JLC" (id 35) (at -6.604 54.61 0)
+    (property "Author" "" (id 35) (at -6.604 54.61 0)
       (effects (font (size 1.524 1.524)) (justify left) hide)
     )
@@
       (effects (font (size 1.524 1.524)) (justify left) hide)
     )
-    (property "Author" "CERN DEM JLC" (id 35) (at -38.354 54.61 0)
+    (property "Author" "" (id 35) (at -38.354 54.61 0)
       (effects (font (size 1.524 1.524)) (justify left) hide)
     )
@@
       (effects (font (size 1.524 1.524)) (justify left) hide)
     )
-    (property "Author" "CERN DEM JLC" (id 35) (at -51.054 86.36 0)
+    (property "Author" "" (id 35) (at -51.054 86.36 0)
       (effects (font (size 1.524 1.524)) (justify left) hide)
     )
@@
       (effects (font (size 1.524 1.524)) (justify left) hide)
     )
-    (property "Author" "CERN DEM JLC" (id 35) (at -18.034 86.36 0)
+    (property "Author" "" (id 35) (at -18.034 86.36 0)
       (effects (font (size 1.524 1.524)) (justify left) hide)
     )
@@
       (effects (font (size 1.524 1.524)) (justify left) hide)
     )
-    (property "Author" "CERN DEM JLC" (id 31) (at 55.88 162.052 0)
+    (property "Author" "" (id 31) (at 55.88 162.052 0)
       (effects (font (size 1.524 1.524)) (justify left) hide)
     )
@@
       (effects (font (size 1.524 1.524)) (justify left) hide)
     )
-    (property "Author" "CERN DEM JLC" (id 35) (at -6.604 86.36 0)
+    (property "Author" "" (id 35) (at -6.604 86.36 0)
       (effects (font (size 1.524 1.524)) (justify left) hide)
     )
@@
       (effects (font (size 1.524 1.524)) (justify left) hide)
     )
-    (property "Author" "CERN DEM JLC" (id 35) (at -38.354 86.36 0)
+    (property "Author" "" (id 35) (at -38.354 86.36 0)
       (effects (font (size 1.524 1.524)) (justify left) hide)
     )
@@
       (effects (font (size 1.524 1.524)) (justify left) hide)
     )
-    (property "Author" "CERN DEM JLC" (id 35) (at -51.054 115.57 0)
+    (property "Author" "" (id 35) (at -51.054 115.57 0)
       (effects (font (size 1.524 1.524)) (justify left) hide)
     )
@@
       (effects (font (size 1.524 1.524)) (justify left) hide)
     )
-    (property "Author" "CERN DEM JLC" (id 35) (at -18.034 115.57 0)
+    (property "Author" "" (id 35) (at -18.034 115.57 0)
       (effects (font (size 1.524 1.524)) (justify left) hide)
     )
@@
       (effects (font (size 1.524 1.524)) (justify left) hide)
     )
-    (property "Author" "CERN DEM JLC" (id 31) (at 55.88 191.262 0)
+    (property "Author" "" (id 31) (at 55.88 191.262 0)
       (effects (font (size 1.524 1.524)) (justify left) hide)
     )
@@
       (effects (font (size 1.524 1.524)) (justify left) hide)
     )
-    (property "Author" "CERN DEM JLC" (id 35) (at -6.604 115.57 0)
+    (property "Author" "" (id 35) (at -6.604 115.57 0)
       (effects (font (size 1.524 1.524)) (justify left) hide)
     )
@@
       (effects (font (size 1.524 1.524)) (justify left) hide)
     )
-    (property "Author" "CERN DEM JLC" (id 35) (at -38.354 115.57 0)
-      (effects (font (size 1.524 1.524)) (justify left) hide)
-    )
+    (property "Author" "" (id 35) (at -38.354 115.57 0)
+      (effects (font (size 1.524 1.524)) (justify left) hide)
+    )
