File: design/SDRAM.kicad_sch (KiCad schematic)
At the start: 14 parts

Commit message: new power converter added
Parts:
- C22, C26, C27: renamed from C?; value (none) -> CC0603_22UF_6.3V_20%_X5R; footprint (none) -> CAPC1709X100N
- C24: renamed from C?; value (none) -> CC0402_1UF_16V_10%_X5R; footprint (none) -> Capacitors SMD:CAPC1005X55N
- C25: renamed from C?; value (none) -> CC0201_100NF_6.3V_10%_X5R; footprint (none) -> CAPC0603X33N
- IC1: renamed from IC?; value (none) -> MT8JTF12864HZ-1G6G1 or VR7PU286458FBAMJT; footprint (none) -> ICs And Semiconductors SMD:SODIMM60P6760X3000X380-204
- R29, R30, R31: value (none) -> R0402_10K_1%_0.0625W_100PPM; footprint (none) -> RESC1005X40N
- SK1: renamed from SK?; value (none) -> TYCO_2-2013022-1; footprint (none) -> Sockets:TYCO_2-2013022-1
- TP13: renamed from TP?; value (none) -> TestPoint; footprint (none) -> TestPoint:TestPoint_THTPad_D1.5mm_Drill0.7mm
- U31: value (none) -> TPS51200DRC; footprint (none) -> ICs_And_Semiconductors_SMD:TEXAS_DRC (S-PVSON-N10)

Commit message: connected signals to the J9 connector
connected signals to the J9 connector
Parts:
- C22, C24, C25, C26, C27, R29, R30, R31, SK1: Author CERN DEM JLC -> (none)
- IC1: Author CERN DEM JLC -> (none); Bonding No -> (none)
Changed lines of the file:
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@@
       (effects (font (size 1.524 1.524)) (justify left) hide)
     )
-    (property "Author" "CERN DEM JLC" (id 36) (at 97.79 180.34 0)
+    (property "Author" "" (id 36) (at 97.79 180.34 0)
       (effects (font (size 1.524 1.524)) (justify left) hide)
     )
@@
       (effects (font (size 1.524 1.524)) (justify left) hide)
     )
-    (property "Author" "CERN DEM JLC" (id 36) (at 110.49 198.12 0)
+    (property "Author" "" (id 36) (at 110.49 198.12 0)
       (effects (font (size 1.524 1.524)) (justify left) hide)
     )
@@
       (effects (font (size 1.524 1.524)) (justify left) hide)
     )
-    (property "Author" "CERN DEM JLC" (id 36) (at 203.2 285.75 0)
+    (property "Author" "" (id 36) (at 203.2 285.75 0)
       (effects (font (size 1.524 1.524)) (justify left) hide)
     )
@@
       (effects (font (size 1.524 1.524)) (justify left) hide)
     )
-    (property "Author" "CERN DEM JLC" (id 35) (at 54.356 182.88 0)
+    (property "Author" "" (id 35) (at 54.356 182.88 0)
       (effects (font (size 1.524 1.524)) (justify left) hide)
     )
@@
       (effects (font (size 1.524 1.524)) (justify left) hide)
     )
-    (property "Author" "CERN DEM JLC" (id 35) (at 138.176 190.5 0)
+    (property "Author" "" (id 35) (at 138.176 190.5 0)
       (effects (font (size 1.524 1.524)) (justify left) hide)
     )
@@
       (effects (font (size 1.524 1.524)) (justify left) hide)
     )
-    (property "Author" "CERN DEM JLC" (id 35) (at 148.336 190.5 0)
+    (property "Author" "" (id 35) (at 148.336 190.5 0)
       (effects (font (size 1.524 1.524)) (justify left) hide)
     )
@@
       (effects (font (size 1.524 1.524)) (justify left) hide)
     )
-    (property "Author" "CERN DEM JLC" (id 35) (at 64.516 200.66 0)
+    (property "Author" "" (id 35) (at 64.516 200.66 0)
       (effects (font (size 1.524 1.524)) (justify left) hide)
     )
@@
       (effects (font (size 1.524 1.524)) (justify left) hide)
     )
-    (property "Author" "CERN DEM JLC" (id 35) (at 94.996 200.66 0)
+    (property "Author" "" (id 35) (at 94.996 200.66 0)
       (effects (font (size 1.524 1.524)) (justify left) hide)
     )
@@
       (effects (font (size 1.27 1.27)) (justify left) hide)
     )
-    (property "Author" "CERN DEM JLC" (id 33) (at 195.58 220.345 0)
+    (property "Author" "" (id 33) (at 195.58 220.345 0)
       (effects (font (size 1.27 1.27)) (justify left) hide)
     )
@@
       (effects (font (size 1.27 1.27)) (justify left) hide)
     )
-    (property "Author" "CERN DEM JLC" (id 33) (at 68.58 220.345 0)
+    (property "Author" "" (id 33) (at 68.58 220.345 0)
       (effects (font (size 1.27 1.27)) (justify left) hide)
     )
@@
       (effects (font (size 1.27 1.27)) (justify left) hide)
     )
-    (property "Bonding" "No" (id 23) (at 68.58 201.295 0)
+    (property "Bonding" "" (id 23) (at 68.58 201.295 0)
       (effects (font (size 1.27 1.27)) (justify left) hide)
     )
@@
       (effects (font (size 1.27 1.27)) (justify left) hide)
     )
-    (property "Author" "CERN DEM JLC" (id 31) (at 68.58 216.535 0)
+    (property "Author" "" (id 31) (at 68.58 216.535 0)
       (effects (font (size 1.27 1.27)) (justify left) hide)
     )
@@
       (effects (font (size 1.27 1.27)) (justify left) hide)
     )
-    (property "Bonding" "No" (id 23) (at 195.58 201.295 0)
+    (property "Bonding" "" (id 23) (at 195.58 201.295 0)
       (effects (font (size 1.27 1.27)) (justify left) hide)
     )
@@
       (effects (font (size 1.27 1.27)) (justify left) hide)
     )
-    (property "Author" "CERN DEM JLC" (id 31) (at 195.58 216.535 0)
-      (effects (font (size 1.27 1.27)) (justify left) hide)
-    )
+    (property "Author" "" (id 31) (at 195.58 216.535 0)
+      (effects (font (size 1.27 1.27)) (justify left) hide)
+    )

Commit message: Attempt to add and improve BOM. Added new part numbers for some of the passives
Parts:
- C24: MANUFACTURER (none) -> GENERIC
Changed lines of the file:
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@@
       (effects (font (size 1.524 1.524)) (justify left) hide)
+    )
+    (property "MANUFACTURER" "GENERIC" (id 40) (at 151.13 200.66 0)
+      (effects (font (size 1.27 1.27)) hide)
     )
     (pin "1")

Commit message: Restore some consistency in schematic metadata
Still 13 problematic footprint names in LTM4673.kicad_sch:

BAD Dup: "Footprint" "CAPC1608X87N" "Capacitors SMD:CAPC1005X55N" in LTM4673-altium-import:0_Capacitor - non polarized
BAD Dup: "Footprint" "CAPC2012X135N" "CAPC1608X87N" in LTM4673-altium-import:1_Capacitor - non polarized
BAD Dup: "Footprint" "CAPC1608X87N" "Capacitors SMD:CAPC1005X55N" in LTM4673-altium-import:1_Capacitor - non polarized
BAD Dup: "Footprint" "CAPC3216X180N" "CAPC3225X270N" in LTM4673-altium-import:1_Capacitor - non polarized
BAD Dup: "Footprint" "CAPC1608X87N" "Capacitors SMD:CAPC1005X55N" in LTM4673-altium-import:0_Capacitor - non polarized
BAD Dup: "Footprint" "CAPC1608X87N" "Capacitors SMD:CAPC1005X55N" in LTM4673-altium-import:0_Capacitor - non polarized
BAD Dup: "Footprint" "CAPC3216X180N" "CAPC3225X270N" in LTM4673-altium-import:1_Capacitor - non polarized
BAD Dup: "Footprint" "CAPC2012X135N" "CAPC1608X87N" in LTM4673-altium-import:1_Capacitor - non polarized
BAD Dup: "Footprint" "CAPC3216X180N" "CAPC3225X270N" in LTM4673-altium-import:1_Capacitor - non polarized
BAD Dup: "Footprint" "CAPC1608X87N" "Capacitors SMD:CAPC1005X55N" in LTM4673-altium-import:0_Capacitor - non polarized
BAD Dup: "Footprint" "CAPC1608X87N" "Capacitors SMD:CAPC1005X55N" in LTM4673-altium-import:1_Capacitor - non polarized
BAD Dup: "Footprint" "CAPC3216X180N" "CAPC3225X270N" in LTM4673-altium-import:1_Capacitor - non polarized
BAD Dup: "Footprint" "CAPMP7343X310N" "Capacitor_Tantalum_SMD:CP_EIA-7343-30_AVX-N" in LTM4673-altium-import:3_Capacitor - polarized

But the Symbol Field editor in eeschema should be more useful now.
Parts:
- C24: MANUFACTURER GENERIC -> (none)
Changed lines of the file:
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@@
       (effects (font (size 1.524 1.524)) (justify left) hide)
-    )
-    (property "MANUFACTURER" "GENERIC" (id 40) (at 151.13 200.66 0)
-      (effects (font (size 1.27 1.27)) hide)
     )
     (pin "1")

Commit message: Parts substitutions
As researched by Michal
MPZ2012S102JTD25 -> MPZ2012S102ATD25
BC857BV-TP -> BCM857BV-7
TPS51200DRC -> TPS51200DRCR
TXS0108E -> TXS0108EPWR
Parts:
- U31: Manufacturer Part Number TPS51200DRC -> TPS51200DRCR
Changed lines of the file:
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@@
       (effects (font (size 1.27 1.27)) hide)
     )
-    (property "Manufacturer Part Number" "TPS51200DRC" (id 4) (at 167.64 195.58 0)
+    (property "Manufacturer Part Number" "TPS51200DRCR" (id 4) (at 167.64 195.58 0)
       (effects (font (size 1.27 1.27)) hide)
     )
